Commit message: Update generated wxai URDFs

File: urdf/generated/wxai/wxai_base.urdf (robot description, URDF)
Before this commit: robot wxai, 12 links, 11 joints
Joints:
- joint joint_2: limit lower=-3.141592653589793 upper=2.356194490192345 effort=27.0 velocity=3.141592653589793 -> lower=0.0 upper=2.356194490192345 effort=27.0 velocity=3.141592653589793

File: urdf/generated/wxai/wxai_follower.urdf (robot description, URDF)
Before this commit: robot wxai, 15 links, 14 joints
Joints:
- joint joint_2: limit lower=-3.141592653589793 upper=2.356194490192345 effort=27.0 velocity=3.141592653589793 -> lower=0.0 upper=2.356194490192345 effort=27.0 velocity=3.141592653589793

File: urdf/generated/wxai/wxai_leader_left.urdf (robot description, URDF)
Before this commit: robot wxai, 12 links, 11 joints
Joints:
- joint joint_2: limit lower=-3.141592653589793 upper=2.356194490192345 effort=27.0 velocity=3.141592653589793 -> lower=0.0 upper=2.356194490192345 effort=27.0 velocity=3.141592653589793

File: urdf/generated/wxai/wxai_leader_right.urdf (robot description, URDF)
Before this commit: robot wxai, 12 links, 11 joints
Joints:
- joint joint_2: limit lower=-3.141592653589793 upper=2.356194490192345 effort=27.0 velocity=3.141592653589793 -> lower=0.0 upper=2.356194490192345 effort=27.0 velocity=3.141592653589793

Commit message: Update generated URDFs

File: urdf/generated/wxai/wxai_base.urdf (robot description, URDF)
Before this commit: robot wxai, 12 links, 11 joints
Joints:
- joint joint_0: limit lower=-3.0543261909900767 upper=3.0543261909900767 effort=27.0 velocity=3.141592653589793 -> lower=-3.0543261909900767 upper=3.0543261909900767 effort=27.0 velocity=3.375
- joint joint_1: limit lower=0.0 upper=3.141592653589793 effort=27.0 velocity=3.141592653589793 -> lower=0.0 upper=3.141592653589793 effort=27.0 velocity=3.375
- joint joint_2: limit lower=0.0 upper=2.356194490192345 effort=27.0 velocity=3.141592653589793 -> lower=0.0 upper=2.356194490192345 effort=27.0 velocity=3.375
- joint joint_3: limit lower=-1.5707963267948966 upper=1.5707963267948966 effort=7.0 velocity=3.141592653589793 -> lower=-1.5707963267948966 upper=1.5707963267948966 effort=7.0 velocity=7.0
- joint joint_4: limit lower=-1.5707963267948966 upper=1.5707963267948966 effort=7.0 velocity=3.141592653589793 -> lower=-1.5707963267948966 upper=1.5707963267948966 effort=7.0 velocity=7.0
- joint joint_5: limit lower=-3.141592653589793 upper=3.141592653589793 effort=7.0 velocity=3.141592653589793 -> lower=-3.141592653589793 upper=3.141592653589793 effort=7.0 velocity=7.0

File: urdf/generated/wxai/wxai_follower.urdf (robot description, URDF)
Before this commit: robot wxai, 15 links, 14 joints
Joints:
- joint joint_0: limit lower=-3.0543261909900767 upper=3.0543261909900767 effort=27.0 velocity=3.141592653589793 -> lower=-3.0543261909900767 upper=3.0543261909900767 effort=27.0 velocity=3.375
- joint joint_1: limit lower=0.0 upper=3.141592653589793 effort=27.0 velocity=3.141592653589793 -> lower=0.0 upper=3.141592653589793 effort=27.0 velocity=3.375
- joint joint_2: limit lower=0.0 upper=2.356194490192345 effort=27.0 velocity=3.141592653589793 -> lower=0.0 upper=2.356194490192345 effort=27.0 velocity=3.375
- joint joint_3: limit lower=-1.5707963267948966 upper=1.5707963267948966 effort=7.0 velocity=3.141592653589793 -> lower=-1.5707963267948966 upper=1.5707963267948966 effort=7.0 velocity=7.0
- joint joint_4: limit lower=-1.5707963267948966 upper=1.5707963267948966 effort=7.0 velocity=3.141592653589793 -> lower=-1.5707963267948966 upper=1.5707963267948966 effort=7.0 velocity=7.0
- joint joint_5: limit lower=-3.141592653589793 upper=3.141592653589793 effort=7.0 velocity=3.141592653589793 -> lower=-3.141592653589793 upper=3.141592653589793 effort=7.0 velocity=7.0

File: urdf/generated/wxai/wxai_leader_left.urdf (robot description, URDF)
Before this commit: robot wxai, 12 links, 11 joints
Joints:
- joint joint_0: limit lower=-3.0543261909900767 upper=3.0543261909900767 effort=27.0 velocity=3.141592653589793 -> lower=-3.0543261909900767 upper=3.0543261909900767 effort=27.0 velocity=3.375
- joint joint_1: limit lower=0.0 upper=3.141592653589793 effort=27.0 velocity=3.141592653589793 -> lower=0.0 upper=3.141592653589793 effort=27.0 velocity=3.375
- joint joint_2: limit lower=0.0 upper=2.356194490192345 effort=27.0 velocity=3.141592653589793 -> lower=0.0 upper=2.356194490192345 effort=27.0 velocity=3.375
- joint joint_3: limit lower=-1.5707963267948966 upper=1.5707963267948966 effort=7.0 velocity=3.141592653589793 -> lower=-1.5707963267948966 upper=1.5707963267948966 effort=7.0 velocity=7.0
- joint joint_4: limit lower=-1.5707963267948966 upper=1.5707963267948966 effort=7.0 velocity=3.141592653589793 -> lower=-1.5707963267948966 upper=1.5707963267948966 effort=7.0 velocity=7.0
- joint joint_5: limit lower=-3.141592653589793 upper=3.141592653589793 effort=7.0 velocity=3.141592653589793 -> lower=-3.141592653589793 upper=3.141592653589793 effort=7.0 velocity=7.0

File: urdf/generated/wxai/wxai_leader_right.urdf (robot description, URDF)
Before this commit: robot wxai, 12 links, 11 joints
Joints:
- joint joint_0: limit lower=-3.0543261909900767 upper=3.0543261909900767 effort=27.0 velocity=3.141592653589793 -> lower=-3.0543261909900767 upper=3.0543261909900767 effort=27.0 velocity=3.375
- joint joint_1: limit lower=0.0 upper=3.141592653589793 effort=27.0 velocity=3.141592653589793 -> lower=0.0 upper=3.141592653589793 effort=27.0 velocity=3.375
- joint joint_2: limit lower=0.0 upper=2.356194490192345 effort=27.0 velocity=3.141592653589793 -> lower=0.0 upper=2.356194490192345 effort=27.0 velocity=3.375
- joint joint_3: limit lower=-1.5707963267948966 upper=1.5707963267948966 effort=7.0 velocity=3.141592653589793 -> lower=-1.5707963267948966 upper=1.5707963267948966 effort=7.0 velocity=7.0
- joint joint_4: limit lower=-1.5707963267948966 upper=1.5707963267948966 effort=7.0 velocity=3.141592653589793 -> lower=-1.5707963267948966 upper=1.5707963267948966 effort=7.0 velocity=7.0
- joint joint_5: limit lower=-3.141592653589793 upper=3.141592653589793 effort=7.0 velocity=3.141592653589793 -> lower=-3.141592653589793 upper=3.141592653589793 effort=7.0 velocity=7.0

Commit message: Update generated URDFs

File: urdf/generated/wxai/wxai_base.urdf (robot description, URDF)
Before this commit: robot wxai, 12 links, 11 joints
Joints:
- joint ee_gripper: origin xyz=0.142 0 0 rpy=0 0 0 -> xyz=0.154 0 0 rpy=0 0 0
- joint left_carriage_joint: origin xyz=0.0745 0.023 0 rpy=0 0 0 -> xyz=0.0865 0.023 0 rpy=0 0 0
- joint right_carriage_joint: origin xyz=0.0745 -0.023 0 rpy=0 0 0 -> xyz=0.0865 -0.023 0 rpy=0 0 0

File: urdf/generated/wxai/wxai_follower.urdf (robot description, URDF)
Before this commit: robot wxai, 23 links, 22 joints
Joints:
- joint camera_mount_joint: origin xyz=0 0 0 rpy=0 0 0 -> xyz=0.012 0 0 rpy=0 0 0
- joint ee_gripper: origin xyz=0.142 0 0 rpy=0 0 0 -> xyz=0.154 0 0 rpy=0 0 0
- joint left_carriage_joint: origin xyz=0.0745 0.023 0 rpy=0 0 0 -> xyz=0.0865 0.023 0 rpy=0 0 0
- joint right_carriage_joint: origin xyz=0.0745 -0.023 0 rpy=0 0 0 -> xyz=0.0865 -0.023 0 rpy=0 0 0

File: urdf/generated/wxai/wxai_leader_left.urdf (robot description, URDF)
Before this commit: robot wxai, 12 links, 11 joints
Joints:
- joint handle_joint: origin xyz=0 0 0 rpy=0 0 0 -> xyz=0.012 0 0 rpy=0 0 0
- joint left_carriage_joint: origin xyz=0.0745 0.023 0 rpy=0 0 0 -> xyz=0.0865 0.023 0 rpy=0 0 0
- joint right_carriage_joint: origin xyz=0.0745 -0.023 0 rpy=0 0 0 -> xyz=0.0865 -0.023 0 rpy=0 0 0

File: urdf/generated/wxai/wxai_leader_right.urdf (robot description, URDF)
Before this commit: robot wxai, 12 links, 11 joints
Joints:
- joint handle_joint: origin xyz=0 0 0 rpy=0 0 0 -> xyz=0.012 0 0 rpy=0 0 0
- joint left_carriage_joint: origin xyz=0.0745 0.023 0 rpy=0 0 0 -> xyz=0.0865 0.023 0 rpy=0 0 0
- joint right_carriage_joint: origin xyz=0.0745 -0.023 0 rpy=0 0 0 -> xyz=0.0865 -0.023 0 rpy=0 0 0

Commit message: update generated urdfs

File: urdf/generated/wxai/wxai_base.urdf (robot description, URDF)
Before this commit: robot wxai, 12 links, 11 joints
Links:
- link ee_gripper_link: mass 0.001 -> None
Joints:
- joint right_carriage_joint: mimic (none) -> joint=left_carriage_joint

File: urdf/generated/wxai/wxai_follower.urdf (robot description, URDF)
Before this commit: robot wxai, 23 links, 22 joints
Links:
- link ee_gripper_link: mass 0.001 -> None
Joints:
- joint right_carriage_joint: mimic (none) -> joint=left_carriage_joint

File: urdf/generated/wxai/wxai_leader_left.urdf (robot description, URDF)
Before this commit: robot wxai, 12 links, 11 joints
Joints:
- joint right_carriage_joint: mimic (none) -> joint=left_carriage_joint

File: urdf/generated/wxai/wxai_leader_right.urdf (robot description, URDF)
Before this commit: robot wxai, 12 links, 11 joints
Joints:
- joint right_carriage_joint: mimic (none) -> joint=left_carriage_joint
