Commit message: Add compliant follower URDF

File: urdf/generated/wxai/wxai_follower_compliant.urdf (robot description, URDF)
Before this commit: robot wxai, 12 links, 11 joints
Links:
- link gripper_left: geometry collision mesh filename=package://trossen_arm_description/meshes/wxai/gripper_left_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; visual mesh filename=package://trossen_arm_description/meshes/wxai/gripper_left_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
Joints:
- joint ee_gripper: origin xyz=0.156062 0 0 rpy=0 0 0 -> xyz=0.161 0 0 rpy=0 0 0
- joint left_carriage_joint: origin xyz=0.0865 0.023 0 rpy=0 0 0 -> xyz=0.0865 0.0182 0 rpy=0 0 0
- joint right_carriage_joint: origin xyz=0.0865 -0.023 0 rpy=0 0 0 -> xyz=0.0865 -0.0182 0 rpy=0 0 0

File: urdf/generated/wxai/wxai_leader_left.urdf (robot description, URDF)
Before this commit: robot wxai, 12 links, 11 joints
Joints:
- joint left_carriage_joint: origin xyz=0.0865 0.023 0 rpy=0 0 0 -> xyz=0.0865 0.0182 0 rpy=0 0 0
- joint right_carriage_joint: origin xyz=0.0865 -0.023 0 rpy=0 0 0 -> xyz=0.0865 -0.0182 0 rpy=0 0 0

File: urdf/generated/wxai/wxai_leader_right.urdf (robot description, URDF)
Before this commit: robot wxai, 12 links, 11 joints
Joints:
- joint left_carriage_joint: origin xyz=0.0865 0.023 0 rpy=0 0 0 -> xyz=0.0865 0.0182 0 rpy=0 0 0
- joint right_carriage_joint: origin xyz=0.0865 -0.023 0 rpy=0 0 0 -> xyz=0.0865 -0.0182 0 rpy=0 0 0

File: urdf/macros/_wxai.urdf.xacro (robot description, xacro)
@@ -10,4 +10,21 @@
     <xacro:property name="mesh_directory" value="package://trossen_arm_description/meshes/${robot_model}"/>
     <xacro:include filename="$(find trossen_arm_description)/urdf/macros/_wxai.ros2_control.xacro"/>
+    <!-- Finger offsets -->
+    <xacro:if value="${variant == 'base'}">
+      <xacro:property name="offset_finger_left" value="0.0"/>
+      <xacro:property name="offset_finger_right" value="0.0"/>
+    </xacro:if>
+    <xacro:if value="${variant == 'leader'}">
+      <xacro:property name="offset_finger_left" value="-0.0048"/>
+      <xacro:property name="offset_finger_right" value="0.0048"/>
+    </xacro:if>
+    <xacro:if value="${variant == 'follower'}">
+      <xacro:property name="offset_finger_left" value="0.0"/>
+      <xacro:property name="offset_finger_right" value="0.0"/>
+    </xacro:if>
+    <xacro:if value="${variant == 'follower_compliant'}">
+      <xacro:property name="offset_finger_left" value="-0.0048"/>
+      <xacro:property name="offset_finger_right" value="0.0048"/>
+    </xacro:if>
     <xacro:wxai_ros2_control
       prefix="${prefix}"
@@ -351,5 +368,5 @@
     <joint name="${prefix}right_carriage_joint" type="prismatic">
       <origin
-        xyz="0.0865 -0.023 0"
+        xyz="0.0865 ${-0.023 + offset_finger_right} 0"
         rpy="0 0 0" />
       <parent link="${prefix}link_6" />
@@ -397,5 +414,5 @@
     <joint name="${prefix}left_carriage_joint" type="prismatic">
       <origin
-        xyz="0.0865 0.023 0"
+        xyz="0.0865 ${0.023 + offset_finger_left} 0"
         rpy="0 0 0" />
       <parent link="${prefix}link_6" />
@@ -786,4 +803,92 @@
       <link name="${prefix}ee_gripper_link" />
     </xacro:if> <!-- variant in ('base', 'follower') -->
+    <xacro:if value="${variant == 'follower_compliant'}">
+      <link name="${prefix}gripper_left">
+        <inertial>
+          <origin
+            xyz="0.01893993 -0.00901223 -0.00215453"
+            rpy="0 0 0" />
+          <mass value="0.03090787" />
+          <inertia
+            ixx="0.00000769"
+            ixy="0.00000321"
+            ixz="0.00000029"
+            iyy="0.00001487"
+            iyz="-0.00000020"
+            izz="0.00001184" />
+        </inertial>
+        <visual>
+          <origin
+            xyz="0 0 0"
+            rpy="0 0 0" />
+          <geometry>
+            <mesh filename="${mesh_directory}/gripper_left_compliant.stl" />
+          </geometry>
+          <material name="trossen_black"/>
+        </visual>
+        <collision>
+          <origin
+            xyz="0 0 0"
+            rpy="0 0 0" />
+          <geometry>
+            <mesh filename="${mesh_directory}/gripper_left_compliant.stl" />
+          </geometry>
+        </collision>
+      </link>
+      <joint name="${prefix}left_gripper_joint" type="fixed">
+        <origin
+          xyz="0 0 0"
+          rpy="0 0 0" />
+        <parent link="${prefix}carriage_left" />
+        <child link="${prefix}gripper_left" />
+      </joint>
+      <link name="${prefix}gripper_right">
+        <inertial>
+          <origin
+            xyz="0.01893989 0.00901216 -0.00215461"
+            rpy="0 0 0" />
+          <mass value="0.03090786" />
+          <inertia
+            ixx="0.00000769"
+            ixy="-0.00000321"
+            ixz="0.00000029"
+            iyy="0.00001487"
+            iyz="0.00000020"
+            izz="0.00001184" />
+        </inertial>
+        <visual>
+          <origin
+            xyz="0 0 0"
+            rpy="0 0 0" />
+          <geometry>
+            <mesh filename="${mesh_directory}/gripper_right_compliant.stl" />
+          </geometry>
+          <material name="trossen_black"/>
+        </visual>
+        <collision>
+          <origin
+            xyz="0 0 0"
+            rpy="0 0 0" />
+          <geometry>
+            <mesh filename="${mesh_directory}/gripper_right_compliant.stl" />
+          </geometry>
+        </collision>
+      </link>
+      <joint name="${prefix}right_gripper_joint" type="fixed">
+        <origin
+          xyz="0 0 0"
+          rpy="0 0 0" />
+        <parent link="${prefix}carriage_right" />
+        <child link="${prefix}gripper_right" />
+      </joint>
+      <joint name="${prefix}ee_gripper" type="fixed">
+        <origin
+          xyz="0.161 0 0"
+          rpy="0 0 0" />
+        <parent link="${prefix}link_6" />
+        <child link="${prefix}ee_gripper_link" />
+      </joint>
+      <link name="${prefix}ee_gripper_link" />
+    </xacro:if> <!-- variant == 'follower_compliant' -->
   </xacro:macro>  <!-- wxai -->
 </robot>

File: urdf/wxai.urdf.xacro (robot description, xacro)
@@ -1,5 +1,5 @@
 <?xml version="1.0" encoding="utf-8"?>
 <robot name="wxai" xmlns:xacro="http://ros.org/wiki/xacro">
-  <xacro:arg name="variant"                         default="base"/>        <!-- 'base', 'leader', 'follower' -->
+  <xacro:arg name="variant"                         default="base"/>        <!-- 'base', 'leader', 'follower', 'follower_compliant' -->
   <xacro:arg name="arm_side"                        default=""/>            <!-- '', 'left', 'right' -->
   <xacro:arg name="prefix"                          default=""/>
