Commit message: Add texture

File: urdf/wxai.urdf.xacro (robot description, xacro)
@@ -14,4 +14,7 @@
   <xacro:property name="variant"                    value="$(arg variant)"/>
   <xacro:property name="arm_side"                   value="$(arg arm_side)"/>
+  <material name="trossen_black">
+    <texture filename="package://trossen_arm_description/meshes/trossen_black.png"/>
+  </material>
   <xacro:if value="$(arg use_world_frame)">
     <link name="world"/>
@@ -44,7 +47,5 @@
         <mesh filename="${mesh_directory}/base_link.stl" />
       </geometry>
-      <material name="">
-        <color rgba="0.752941176470588 0.752941176470588 0.752941176470588 1" />
-      </material>
+      <material name="trossen_black"/>
     </visual>
     <collision>
@@ -78,7 +79,5 @@
         <mesh filename="${mesh_directory}/link_1.stl" />
       </geometry>
-      <material name="">
-        <color rgba="0.752941176470588 0.752941176470588 0.752941176470588 1" />
-      </material>
+      <material name="trossen_black"/>
     </visual>
     <collision>
@@ -125,7 +124,5 @@
         <mesh filename="${mesh_directory}/link_2.stl" />
       </geometry>
-      <material name="">
-        <color rgba="0.752941176470588 0.752941176470588 0.752941176470588 1" />
-      </material>
+      <material name="trossen_black"/>
     </visual>
     <collision>
@@ -172,7 +169,5 @@
         <mesh filename="${mesh_directory}/link_3.stl" />
       </geometry>
-      <material name="">
-        <color rgba="0.752941176470588 0.752941176470588 0.752941176470588 1" />
-      </material>
+      <material name="trossen_black"/>
     </visual>
     <collision>
@@ -219,7 +214,5 @@
         <mesh filename="${mesh_directory}/link_4.stl" />
       </geometry>
-      <material name="">
-        <color rgba="0.752941176470588 0.752941176470588 0.752941176470588 1" />
-      </material>
+      <material name="trossen_black"/>
     </visual>
     <collision>
@@ -266,7 +259,5 @@
         <mesh filename="${mesh_directory}/link_5.stl" />
       </geometry>
-      <material name="">
-        <color rgba="0.752941176470588 0.752941176470588 0.752941176470588 1" />
-      </material>
+      <material name="trossen_black"/>
     </visual>
     <collision>
@@ -313,7 +304,5 @@
         <mesh filename="${mesh_directory}/link_6.stl" />
       </geometry>
-      <material name="">
-        <color rgba="0.752941176470588 0.752941176470588 0.752941176470588 1" />
-      </material>
+      <material name="trossen_black"/>
     </visual>
     <collision>
@@ -360,7 +349,5 @@
         <mesh filename="${mesh_directory}/carriage_right.stl" />
       </geometry>
-      <material name="">
-        <color rgba="0.752941176470588 0.752941176470588 0.752941176470588 1" />
-      </material>
+      <material name="trossen_black"/>
     </visual>
     <collision>
@@ -407,7 +394,5 @@
         <mesh filename="${mesh_directory}/carriage_left.stl" />
       </geometry>
-      <material name="">
-        <color rgba="0.752941176470588 0.752941176470588 0.752941176470588 1" />
-      </material>
+      <material name="trossen_black"/>
     </visual>
     <collision>
@@ -455,7 +440,5 @@
           <mesh filename="${mesh_directory}/camera_mount_d405.stl" />
         </geometry>
-        <material name="">
-          <color rgba="0.752941176470588 0.752941176470588 0.752941176470588 1" />
-        </material>
+        <material name="trossen_black"/>
       </visual>
       <collision>
@@ -506,7 +489,5 @@
             <mesh filename="${mesh_directory}/handle_left.stl" />
           </geometry>
-          <material name="">
-            <color rgba="0.752941176470588 0.752941176470588 0.752941176470588 1" />
-          </material>
+          <material name="trossen_black"/>
         </visual>
         <collision>
@@ -548,7 +529,5 @@
             <mesh filename="${mesh_directory}/leader_finger_left_index.stl" />
           </geometry>
-          <material name="">
-            <color rgba="0.752941176470588 0.752941176470588 0.752941176470588 1" />
-          </material>
+          <material name="trossen_black"/>
         </visual>
         <collision>
@@ -590,7 +569,5 @@
             <mesh filename="${mesh_directory}/leader_finger_left_thumb.stl" />
           </geometry>
-          <material name="">
-            <color rgba="0.752941176470588 0.752941176470588 0.752941176470588 1" />
-          </material>
+          <material name="trossen_black"/>
         </visual>
         <collision>
@@ -634,7 +611,5 @@
             <mesh filename="${mesh_directory}/handle_right.stl" />
           </geometry>
-          <material name="">
-            <color rgba="0.752941176470588 0.752941176470588 0.752941176470588 1" />
-          </material>
+          <material name="trossen_black"/>
         </visual>
         <collision>
@@ -676,7 +651,5 @@
             <mesh filename="${mesh_directory}/leader_finger_right_thumb.stl" />
           </geometry>
-          <material name="">
-            <color rgba="0.752941176470588 0.752941176470588 0.752941176470588 1" />
-          </material>
+          <material name="trossen_black"/>
         </visual>
         <collision>
@@ -718,7 +691,5 @@
             <mesh filename="${mesh_directory}/leader_finger_right_index.stl" />
           </geometry>
-          <material name="">
-            <color rgba="0.752941176470588 0.752941176470588 0.752941176470588 1" />
-          </material>
+          <material name="trossen_black"/>
         </visual>
         <collision>
@@ -763,7 +734,5 @@
           <mesh filename="${mesh_directory}/gripper_left.stl" />
         </geometry>
-        <material name="">
-          <color rgba="0.752941176470588 0.752941176470588 0.752941176470588 1" />
-        </material>
+        <material name="trossen_black"/>
       </visual>
       <collision>
@@ -805,7 +774,5 @@
           <mesh filename="${mesh_directory}/gripper_right.stl" />
         </geometry>
-        <material name="">
-          <color rgba="0.752941176470588 0.752941176470588 0.752941176470588 1" />
-        </material>
+        <material name="trossen_black"/>
       </visual>
       <collision>

Commit message: Make wxai a macro

File: urdf/wxai.urdf.xacro (robot description, xacro)
@@ -1,20 +1,8 @@
 <?xml version="1.0" encoding="utf-8"?>
 <robot name="wxai" xmlns:xacro="http://ros.org/wiki/xacro">
-  <xacro:property name="robot_model"
-    value="wxai"
-    scope="global"/>
-  <xacro:property name="dof"
-    value="6"
-    scope="global"/>
   <xacro:arg name="variant"                         default="base"/>      <!-- 'base', 'leader', 'follower' -->
   <xacro:arg name="arm_side"                        default=""/>          <!-- '', 'left', 'right' -->
   <xacro:arg name="use_world_frame"                 default="false"/>     <!-- 'true', 'false' -->
   <xacro:arg name="base_link_frame"                 default="base_link"/>
-  <xacro:property name="mesh_directory"             value="package://trossen_arm_description/meshes/${robot_model}"/>
-  <xacro:property name="variant"                    value="$(arg variant)"/>
-  <xacro:property name="arm_side"                   value="$(arg arm_side)"/>
-  <material name="trossen_black">
-    <texture filename="package://trossen_arm_description/meshes/trossen_black.png"/>
-  </material>
   <xacro:if value="$(arg use_world_frame)">
     <link name="world"/>
@@ -26,791 +14,9 @@
     </joint>
   </xacro:if> <!-- use_world_frame -->
-  <link name="base_link">
-    <inertial>
-      <origin
-        xyz="-0.00014175 -0.00005228 0.03175177"
-        rpy="0 0 0" />
-      <mass value="0.45969858" />
-      <inertia
-        ixx="0.00041660"
-        ixy="0.00000011"
-        ixz="-0.00000454"
-        iyy="0.00044896"
-        iyz="-0.00000078"
-        izz="0.00021403" />
-    </inertial>
-    <visual>
-      <origin
-        xyz="0 0 0"
-        rpy="0 0 0" />
-      <geometry>
-        <mesh filename="${mesh_directory}/base_link.stl" />
-      </geometry>
-      <material name="trossen_black"/>
-    </visual>
-    <collision>
-      <origin
-        xyz="0 0 0"
-        rpy="0 0 0" />
-      <geometry>
-        <mesh filename="${mesh_directory}/base_link.stl" />
-      </geometry>
-    </collision>
-  </link>
-  <link name="link_1">
-    <inertial>
-      <origin
-        xyz="-0.00011075 0.00171176 0.02044592"
-        rpy="0 0 0" />
-      <mass value="0.15270428" />
-      <inertia
-        ixx="0.00018509"
-        ixy="-0.00000191"
-        ixz="-0.00001436"
-        iyy="0.00008358"
-        iyz="-0.00000130"
-        izz="0.00019219" />
-    </inertial>
-    <visual>
-      <origin
-        xyz="0 0 0"
-        rpy="0 0 0" />
-      <geometry>
-        <mesh filename="${mesh_directory}/link_1.stl" />
-      </geometry>
-      <material name="trossen_black"/>
-    </visual>
-    <collision>
-      <origin
-        xyz="0 0 0"
-        rpy="0 0 0" />
-      <geometry>
-        <mesh filename="${mesh_directory}/link_1.stl" />
-      </geometry>
-    </collision>
-  </link>
-  <joint name="joint_0" type="revolute">
-    <origin
-      xyz="0 0 0.05725"
-      rpy="0 0 0" />
-    <parent link="base_link" />
-    <child link="link_1" />
-    <axis xyz="0 0 1" />
-    <limit
-      lower="${-radians(180 - 5)}"
-      upper="${radians(180 - 5)}"
-      effort="27.0"
-      velocity="3.375" />
-  </joint>
-  <link name="link_2">
-    <inertial>
-      <origin
-        xyz="-0.13121451 -0.00292583 0.00021345"
-        rpy="0 0 0" />
-      <mass value="1.15316319" />
-      <inertia
-        ixx="0.00102632"
-        ixy="-0.00000319"
-        ixz="-0.00002679"
-        iyy="0.01736118"
-        iyz="-0.00000193"
-        izz="0.01794489" />
-    </inertial>
-    <visual>
-      <origin
-        xyz="0 0 0"
-        rpy="0 0 0" />
-      <geometry>
-        <mesh filename="${mesh_directory}/link_2.stl" />
-      </geometry>
-      <material name="trossen_black"/>
-    </visual>
-    <collision>
-      <origin
-        xyz="0 0 0"
-        rpy="0 0 0" />
-      <geometry>
-        <mesh filename="${mesh_directory}/link_2.stl" />
-      </geometry>
-    </collision>
-  </link>
-  <joint name="joint_1" type="revolute">
-    <origin
-      xyz="0.02 0 0.04625"
-      rpy="0 0 0" />
-    <parent link="link_1" />
-    <child link="link_2" />
-    <axis xyz="0 1 0" />
-    <limit
-      lower="0.0"
-      upper="${pi}"
-      effort="27.0"
-      velocity="3.375" />
-  </joint>
-  <link name="link_3">
-    <inertial>
-      <origin
-        xyz="0.18083602 -0.00094090 0.05554937"
-        rpy="0 0 0" />
-      <mass value="0.68666638" />
-      <inertia
-        ixx="0.00064876"
-        ixy="0.00009128"
-        ixz="-0.00052002"
-        iyy="0.00547407"
-        iyz="0.00001159"
-        izz="0.00561509" />
-    </inertial>
-    <visual>
-      <origin
-        xyz="0 0 0"
-        rpy="0 0 0" />
-      <geometry>
-        <mesh filename="${mesh_directory}/link_3.stl" />
-      </geometry>
-      <material name="trossen_black"/>
-    </visual>
-    <collision>
-      <origin
-        xyz="0 0 0"
-        rpy="0 0 0" />
-      <geometry>
-        <mesh filename="${mesh_directory}/link_3.stl" />
-      </geometry>
-    </collision>
-  </link>
-  <joint name="joint_2" type="revolute">
-    <origin
-      xyz="-0.264 0 0"
-      rpy="0 0 0" />
-    <parent link="link_2" />
-    <child link="link_3" />
-    <axis xyz="0 -1 0" />
-    <limit
-      lower="0.0"
-      upper="${3 * pi / 4}"
-      effort="27.0"
-      velocity="3.375" />
-  </joint>
-  <link name="link_4">
-    <inertial>
-      <origin
-        xyz="0.05797842 0.00027145 0.05884447"
-        rpy="0 0 0" />
-      <mass value="0.45789905" />
-      <inertia
-        ixx="0.00053839"
-        ixy="0.00000690"
-        ixz="-0.00018164"
-        iyy="0.00066138"
-        iyz="0.00000724"
-        izz="0.00042116" />
-    </inertial>
-    <visual>
-      <origin
-        xyz="0 0 0"
-        rpy="0 0 0" />
-      <geometry>
-        <mesh filename="${mesh_directory}/link_4.stl" />
-      </geometry>
-      <material name="trossen_black"/>
-    </visual>
-    <collision>
-      <origin
-        xyz="0 0 0"
-        rpy="0 0 0" />
-      <geometry>
-        <mesh filename="${mesh_directory}/link_4.stl" />
-      </geometry>
-    </collision>
-  </link>
-  <joint name="joint_3" type="revolute">
-    <origin
-      xyz="0.245 0 0.06"
-      rpy="0 0 0" />
-    <parent link="link_3" />
-    <child link="link_4" />
-    <axis xyz="0 -1 0" />
-    <limit
-      lower="-${pi / 2.0}"
-      upper="${pi / 2.0}"
-      effort="7.0"
-      velocity="7.0" />
-  </joint>
-  <link name="link_5">
-    <inertial>
-      <origin
-        xyz="0.00412447 -0.00001138 -0.04283184"
-        rpy="0 0 0" />
-      <mass value="0.36693910" />
-      <inertia
-        ixx="0.00018912"
-        ixy="-0.00000045"
-        ixz="0.00000090"
-        iyy="0.00032062"
-        iyz="0.00000003"
-        izz="0.00026750" />
-    </inertial>
-    <visual>
-      <origin
-        xyz="0 0 0"
-        rpy="0 0 0" />
-      <geometry>
-        <mesh filename="${mesh_directory}/link_5.stl" />
-      </geometry>
-      <material name="trossen_black"/>
-    </visual>
-    <collision>
-      <origin
-        xyz="0 0 0"
-        rpy="0 0 0" />
-      <geometry>
-        <mesh filename="${mesh_directory}/link_5.stl" />
-      </geometry>
-    </collision>
-  </link>
-  <joint name="joint_4" type="revolute">
-    <origin
-      xyz="0.06775 0 0.0455"
-      rpy="0 0 0" />
-    <parent link="link_4" />
-    <child link="link_5" />
-    <axis xyz="0 0 -1" />
-    <limit
-      lower="-${pi / 2.0}"
-      upper="${pi / 2.0}"
-      effort="7.0"
-      velocity="7.0" />
-  </joint>
-  <link name="link_6">
-    <inertial>
-      <origin
-        xyz="0.04572768 -0.00000726 0.00001402"
-        rpy="0 0 0" />
-      <mass value="0.55469347" />
-      <inertia
-        ixx="0.00082429"
-        ixy="-0.00000051"
-        ixz="0.00000010"
-        iyy="0.00048759"
-        iyz="0.00000004"
-        izz="0.00108600" />
-    </inertial>
-    <visual>
-      <origin
-        xyz="0 0 0"
-        rpy="0 0 0" />
-      <geometry>
-        <mesh filename="${mesh_directory}/link_6.stl" />
-      </geometry>
-      <material name="trossen_black"/>
-    </visual>
-    <collision>
-      <origin
-        xyz="0 0 0"
-        rpy="0 0 0" />
-      <geometry>
-        <mesh filename="${mesh_directory}/link_6.stl" />
-      </geometry>
-    </collision>
-  </link>
-  <joint name="joint_5" type="revolute">
-    <origin
-      xyz="0.02895 0 -0.0455"
-      rpy="0 0 0" />
-    <parent link="link_5" />
-    <child link="link_6" />
-    <axis xyz="1 0 0" />
-    <limit
-      lower="-${pi}"
-      upper="${pi}"
-      effort="7.0"
-      velocity="7.0" />
-  </joint>
-  <link name="carriage_right">
-    <inertial>
-      <origin
-        xyz="-0.00889602 0.00403514 0.00457901"
-        rpy="0 0 0" />
-      <mass value="0.05036313" />
-      <inertia
-        ixx="0.00001736"
-        ixy="-0.00000165"
-        ixz="-0.00000104"
-        iyy="0.00000591"
-        iyz="-0.00000172"
-        izz="0.00001378" />
-    </inertial>
-    <visual>
-      <origin
-        xyz="0 0 0"
-        rpy="0 0 0" />
-      <geometry>
-        <mesh filename="${mesh_directory}/carriage_right.stl" />
-      </geometry>
-      <material name="trossen_black"/>
-    </visual>
-    <collision>
-      <origin
-        xyz="0 0 0"
-        rpy="0 0 0" />
-      <geometry>
-        <mesh filename="${mesh_directory}/carriage_right.stl" />
-      </geometry>
-    </collision>
-  </link>
-  <joint name="right_carriage_joint" type="prismatic">
-    <origin
-      xyz="0.0865 -0.023 0"
-      rpy="0 0 0" />
-    <parent link="link_6" />
-    <child link="carriage_right" />
-    <axis xyz="0 -1 0" />
-    <limit
-      lower="0.0"
-      upper="0.044"
-      effort="400.0"
-      velocity="0.0875" />
-  </joint>
-  <link name="carriage_left">
-    <inertial>
-      <origin
-        xyz="-0.00889602 -0.00403515 -0.00457908"
-        rpy="0 0 0" />
-      <mass value="0.05036313" />
-      <inertia
-        ixx="0.00001736"
-        ixy="-0.00000165"
-        ixz="-0.00000104"
-        iyy="0.00000591"
-        iyz="-0.00000172"
-        izz="0.00001378" />
-    </inertial>
-    <visual>
-      <origin
-        xyz="0 0 0"
-        rpy="0 0 0" />
-      <geometry>
-        <mesh filename="${mesh_directory}/carriage_left.stl" />
-      </geometry>
-      <material name="trossen_black"/>
-    </visual>
-    <collision>
-      <origin
-        xyz="0 0 0"
-        rpy="0 0 0" />
-      <geometry>
-        <mesh filename="${mesh_directory}/carriage_left.stl" />
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