Commit message: update mass properties

File: urdf/vxai.urdf.xacro (robot description, xacro)
@@ -4,18 +4,18 @@
   <link
     name="base_link">
-    <!-- <inertial>
-      <origin
-        xyz="6.8153E-06 -0.037025 -4.6856E-06"
-        rpy="0 0 0" />
-      <mass
-        value="0.80227" />
-      <inertia
-        ixx="0.00071132"
-        ixy="9.1583E-08"
-        ixz="2.5948E-08"
-        iyy="0.0012086"
-        iyz="-5.7574E-09"
-        izz="0.00070505" />
-    </inertial> -->
+    <inertial>
+      <origin
+        xyz="-0.00002199 -0.03351643 0.00006205"
+        rpy="0 0 0" />
+      <mass
+        value="1.87165014" />
+      <inertia
+        ixx="0.00209272"
+        ixy="0.00000341"
+        ixz="0.00000001"
+        iyy="0.00299206"
+        iyz="0.00000068"
+        izz="0.00207913" />
+    </inertial>
     <visual>
       <origin
@@ -44,18 +44,18 @@
   <link
     name="link_1">
-    <!-- <inertial>
-      <origin
-        xyz="-0.00298082660667482 -0.0518352980909208 -8.44102257208749E-05"
-        rpy="0 0 0" />
-      <mass
-        value="0.688472720387068" />
-      <inertia
-        ixx="0.000677966794077192"
-        ixy="-8.41991034340278E-07"
-        ixz="7.11006614555938E-07"
-        iyy="0.000455009011284614"
-        iyz="-1.10708544513765E-05"
-        izz="0.000387558366540118" />
-    </inertial> -->
+    <inertial>
+      <origin
+        xyz="0.00275058 -0.05744640 -0.00007470"
+        rpy="0 0 0" />
+      <mass
+        value="1.28114157" />
+      <inertia
+        ixx="0.00180008"
+        ixy="-0.00001517"
+        ixz="-0.00000048"
+        iyy="0.00124234"
+        iyz="0.00000523"
+        izz="0.00154695" />
+    </inertial>
     <visual>
       <origin
@@ -102,18 +102,18 @@
   <link
     name="link_2">
-    <!-- <inertial>
-      <origin
-        xyz="2.40360564334271E-05 -1.53102219933032E-05 -0.0848451366922755"
-        rpy="0 0 0" />
-      <mass
-        value="0.903851513892992" />
-      <inertia
-        ixx="0.000631622619177592"
-        ixy="1.48897028152523E-06"
-        ixz="1.35274589065022E-06"
-        iyy="0.000583087686771591"
-        iyz="-1.14911677663667E-08"
-        izz="0.000907827824933206" />
-    </inertial> -->
+    <inertial>
+      <origin
+        xyz="0.00004155 0.00000477 -0.09223936"
+        rpy="0 0 0" />
+      <mass
+        value="1.58168513" />
+      <inertia
+        ixx="0.00303540"
+        ixy="-0.00000094"
+        ixz="-0.00000007"
+        iyy="0.00325708"
+        iyz="-0.00000058"
+        izz="0.00202764" />
+    </inertial>
     <visual>
       <origin
@@ -160,18 +160,18 @@
   <link
     name="link_3">
-    <!-- <inertial>
-      <origin
-        xyz="0.011108693248786 0.00210739274174987 -0.113878326850928"
-        rpy="0 0 0" />
-      <mass
-        value="0.918096018779917" />
-      <inertia
-        ixx="0.000528560957396802"
-        ixy="7.10938145515933E-07"
-        ixz="8.20249015779571E-06"
-        iyy="0.000738721395755985"
-        iyz="8.41758226028433E-07"
-        izz="0.000433289054319293" />
-    </inertial> -->
+    <inertial>
+      <origin
+        xyz="0.01469489 -0.00233198 -0.13174594"
+        rpy="0 0 0" />
+      <mass
+        value="1.51522891" />
+      <inertia
+        ixx="0.00491722"
+        ixy="-0.00001966"
+        ixz="-0.00061652"
+        iyy="0.00521379"
+        iyz="0.00008813"
+        izz="0.00131018" />
+    </inertial>
     <visual>
       <origin
@@ -218,18 +218,18 @@
   <link
     name="link_4">
-    <!-- <inertial>
-      <origin
-        xyz="0.068479929144433 -2.65480860315581E-05 -0.0166516032356703"
-        rpy="0 0 0" />
-      <mass
-        value="0.3735585648571" />
-      <inertia
-        ixx="0.000215082276839995"
-        ixy="-1.95318962951602E-07"
-        ixz="1.22107646815508E-05"
-        iyy="0.000154452692206455"
-        iyz="-5.04992766600264E-09"
-        izz="0.000160387519405929" />
-    </inertial> -->
+    <inertial>
+      <origin
+        xyz="0.07293047 0.00011005 -0.01788634"
+        rpy="0 0 0" />
+      <mass
+        value="0.59839689" />
+      <inertia
+        ixx="0.00052102"
+        ixy="0.00000093"
+        ixz="-0.00008634"
+        iyy="0.00069719"
+        iyz="-0.00000013"
+        izz="0.00082356" />
+    </inertial>
     <visual>
       <origin
@@ -276,18 +276,18 @@
   <link
     name="link_5">
-    <!-- <inertial>
-      <origin
-        xyz="0.0367432124592126 -0.000515242688117895 -2.02943214192564E-05"
-        rpy="0 0 0" />
-      <mass
-        value="0.384628664073614" />
-      <inertia
-        ixx="0.000151093123220633"
-        ixy="1.72740201374654E-06"
-        ixz="-2.16190529841697E-06"
-        iyy="0.000253912748026685"
-        iyz="-1.12891242195047E-06"
-        izz="0.000226681351891984" />
-    </inertial> -->
+    <inertial>
+      <origin
+        xyz="0.04045078 0.00225112 -0.00011067"
+        rpy="0 0 0" />
+      <mass
+        value="0.60644692" />
+      <inertia
+        ixx="0.00066100"
+        ixy="-0.00000214"
+        ixz="-0.00000789"
+        iyy="0.00054664"
+        iyz="-0.00000375"
+        izz="0.00094550" />
+    </inertial>
     <visual>
       <origin
@@ -334,18 +334,18 @@
   <link
     name="link_6">
-    <!-- <inertial>
-      <origin
-        xyz="4.1088816668533E-06 0.00114373173613513 -0.00183128279020633"
-        rpy="0 0 0" />
-      <mass
-        value="0.191977233295993" />
-      <inertia
-        ixx="5.34811117633044E-05"
-        ixy="-2.49985339462649E-08"
-        ixz="1.53141719303637E-08"
-        iyy="4.91612732925248E-05"
-        iyz="7.048095384809E-09"
-        izz="6.65996754030503E-05" />
-    </inertial> -->
+    <inertial>
+      <origin
+        xyz="-0.00001797 0.00058070 -0.00058762"
+        rpy="0 0 0" />
+      <mass
+        value="0.38858221" />
+      <inertia
+        ixx="0.00031658"
+        ixy="0.00000008"
+        ixz="0.00000001"
+        iyy="0.00026787"
+        iyz="0.00000050"
+        izz="0.00018958" />
+    </inertial>
     <visual>
       <origin
@@ -392,18 +392,18 @@
   <link
     name="link_7">
-    <!-- <inertial>
-      <origin
-        xyz="0.0862240124925011 -2.66160351690414E-05 -0.0171698331637707"
-        rpy="0 0 0" />
-      <mass
-        value="0.380132541517835" />
-      <inertia
-        ixx="0.000295431133709899"
-        ixy="1.20149414515802E-08"
-        ixz="1.29074174223948E-05"
-        iyy="0.000130844955298946"
-        iyz="3.90408903927584E-08"
-        izz="0.000287208425881186" />
-    </inertial> -->
+    <inertial>
+      <origin
+        xyz="0.08476049 -0.00000697 -0.01847211"
+        rpy="0 0 0" />
+      <mass
+        value="0.57903811" />
+      <inertia
+        ixx="0.00085992"
+        ixy="0.00000049"
+        ixz="-0.00009912"
+        iyy="0.00077371"
+        iyz="0.00000006"
+        izz="0.00135277" />
+    </inertial>
     <visual>
       <origin
@@ -450,18 +450,18 @@
   <link
     name="right_carriage">
-    <!-- <inertial>
-      <origin
-        xyz="-0.0088960216342942 0.0040351436142739 0.00457900737971167"
-        rpy="0 0 0" />
-      <mass
-        value="0.0503630726101797" />
-      <inertia
-        ixx="1.05737957274845E-05"
-        ixy="1.46136484822471E-12"
-        ixz="3.6094234914747E-07"
-        iyy="3.3903119527156E-06"
-        iyz="3.1422225082193E-07"
-        izz="8.0053923029398E-06" />
-    </inertial> -->
+    <inertial>
+      <origin
+        xyz="-0.00889602 0.00403514 0.00457901"
+        rpy="0 0 0" />
+      <mass
+        value="0.0503631" />
+      <inertia
+        ixx="0.00001736"
+        ixy="-0.00000165"
+        ixz="-0.00000104"
+        iyy="0.00000591"
+        iyz="0.00000172"
+        izz="0.00001378" />
+    </inertial>
     <visual>
       <origin
@@ -508,18 +508,18 @@
   <link
     name="right_follower_finger">
-    <!-- <inertial>
-      <origin
-        xyz="0.0188673150144285 0.00900062850048977 -0.00215899211185627"
-        rpy="0 0 0" />
-      <mass
-        value="0.0316596868793138" />
-      <inertia
-        ixx="6.87278548528857E-06"
-        ixy="-1.8587623080691E-06"
-        ixz="2.10468318645552E-07"
-        iyy="1.15019142302086E-05"
-        iyz="1.42584909758209E-07"
-        izz="7.84949392243546E-06" />
-    </inertial> -->
+    <inertial>
+      <origin
+        xyz="0.01893989 0.00901216 -0.00215461"
+        rpy="0 0 0" />
+      <mass
+        value="0.03090786" />
+      <inertia
+        ixx="0.00000769"
+        ixy="0.00000321"
+        ixz="-0.00000029"
+        iyy="0.00001487"
+        iyz="-0.00000020"
+        izz="0.00001184" />
+    </inertial>
     <visual>
       <origin
@@ -561,18 +561,18 @@
   <link
     name="left_carriage">
-    <!-- <inertial>
-      <origin
-        xyz="-0.00889602163429409 -0.00403515225638464 -0.00457907970794075"
-        rpy="0 0 0" />
-      <mass
-        value="0.0503630726101797" />
-      <inertia
-        ixx="1.05737957274845E-05"
-        ixy="1.46136486515677E-12"
-        ixz="-3.60957599947595E-07"
-        iyy="3.3903119527156E-06"
-        iyz="3.1422225082193E-07"
-        izz="8.00539230293978E-06" />
-    </inertial> -->
+    <inertial>
+      <origin
+        xyz="-0.00889602 -0.00403515 -0.00457908"
+        rpy="0 0 0" />
+      <mass
+        value="0.05036313" />
+      <inertia
+        ixx="0.00001736"
+        ixy="0.00000165"
+        ixz="0.00000104"
+        iyy="0.00000591"
+        iyz="0.00000172"
+        izz="0.00001378" />
+    </inertial>
     <visual>
       <origin
@@ -619,18 +619,18 @@
   <link
     name="left_follower_finger">
-    <!-- <inertial>
-      <origin
-        xyz="0.0188673477497177 -0.00900068989438087 -0.00215891073625007"
-        rpy="0 0 0" />
-      <mass
-        value="0.0316597159641914" />
-      <inertia
-        ixx="6.87277784866959E-06"
-        ixy="1.85875818224369E-06"
-        ixz="2.10469018011302E-07"
-        iyy="1.1501937626138E-05"
-        iyz="-1.42577967225722E-07"
-        izz="7.8495108271819E-06" />
-    </inertial> -->
+    <inertial>
+      <origin
+        xyz="0.01893993 -0.00901223 -0.00215453"
+        rpy="0 0 0" />
+      <mass
+        value="0.03090787" />
+      <inertia
+        ixx="0.00000769"
+        ixy="-0.00000321"
+        ixz="-0.00000029"
+        iyy="0.00001487"
+        iyz="0.00000020"
+        izz="0.00001184" />
+    </inertial>
     <visual>
       <origin

Commit message: negate off-diagonal inertial elements

File: urdf/vxai.urdf.xacro (robot description, xacro)
@@ -12,8 +12,8 @@
       <inertia
         ixx="0.00209272"
-        ixy="0.00000341"
-        ixz="0.00000001"
+        ixy="-0.00000341"
+        ixz="-0.00000001"
         iyy="0.00299206"
-        iyz="0.00000068"
+        iyz="-0.00000068"
         izz="0.00207913" />
     </inertial>
@@ -52,8 +52,8 @@
       <inertia
         ixx="0.00180008"
-        ixy="-0.00001517"
-        ixz="-0.00000048"
+        ixy="0.00001517"
+        ixz="0.00000048"
         iyy="0.00124234"
-        iyz="0.00000523"
+        iyz="-0.00000523"
         izz="0.00154695" />
     </inertial>
@@ -110,8 +110,8 @@
       <inertia
         ixx="0.00303540"
-        ixy="-0.00000094"
-        ixz="-0.00000007"
+        ixy="0.00000094"
+        ixz="0.00000007"
         iyy="0.00325708"
-        iyz="-0.00000058"
+        iyz="0.00000058"
         izz="0.00202764" />
     </inertial>
@@ -168,8 +168,8 @@
       <inertia
         ixx="0.00491722"
-        ixy="-0.00001966"
-        ixz="-0.00061652"
+        ixy="0.00001966"
+        ixz="0.00061652"
         iyy="0.00521379"
-        iyz="0.00008813"
+        iyz="-0.00008813"
         izz="0.00131018" />
     </inertial>
@@ -226,8 +226,8 @@
       <inertia
         ixx="0.00052102"
-        ixy="0.00000093"
-        ixz="-0.00008634"
+        ixy="-0.00000093"
+        ixz="0.00008634"
         iyy="0.00069719"
-        iyz="-0.00000013"
+        iyz="0.00000013"
         izz="0.00082356" />
     </inertial>
@@ -284,8 +284,8 @@
       <inertia
         ixx="0.00066100"
-        ixy="-0.00000214"
-        ixz="-0.00000789"
+        ixy="0.00000214"
+        ixz="0.00000789"
         iyy="0.00054664"
-        iyz="-0.00000375"
+        iyz="0.00000375"
         izz="0.00094550" />
     </inertial>
@@ -342,8 +342,8 @@
       <inertia
         ixx="0.00031658"
-        ixy="0.00000008"
-        ixz="0.00000001"
+        ixy="-0.00000008"
+        ixz="-0.00000001"
         iyy="0.00026787"
-        iyz="0.00000050"
+        iyz="-0.00000050"
         izz="0.00018958" />
     </inertial>
@@ -400,8 +400,8 @@
       <inertia
         ixx="0.00085992"
-        ixy="0.00000049"
-        ixz="-0.00009912"
+        ixy="-0.00000049"
+        ixz="0.00009912"
         iyy="0.00077371"
-        iyz="0.00000006"
+        iyz="-0.00000006"
         izz="0.00135277" />
     </inertial>
@@ -456,4 +456,115 @@
       <mass
         value="0.0503631" />
+      <inertia
+        ixx="0.00001736"
+        ixy="0.00000165"
+        ixz="0.00000104"
+        iyy="0.00000591"
+        iyz="-0.00000172"
+        izz="0.00001378" />
+    </inertial>
+    <visual>
+      <origin
+        xyz="0 0 0"
+        rpy="0 0 0" />
+      <geometry>
+        <mesh
+          filename="package://trossen_arm_description/meshes/vxai/right_carriage.stl" />
+      </geometry>
+      <material
+        name="">
+        <color
+          rgba="0.752941176470588 0.752941176470588 0.752941176470588 1" />
+      </material>
+    </visual>
+    <collision>
+      <origin
+        xyz="0 0 0"
+        rpy="0 0 0" />
+      <geometry>
+        <mesh
+          filename="package://trossen_arm_description/meshes/vxai/right_carriage.stl" />
+      </geometry>
+    </collision>
+  </link>
+  <joint
+    name="right_carriage_joint"
+    type="prismatic">
+    <origin
+      xyz="0.1305 -0.022974 -0.021"
+      rpy="0 0 0" />
+    <parent
+      link="link_7" />
+    <child
+      link="right_carriage" />
+    <axis
+      xyz="0 -1 0" />
+    <limit
+      effort="0"
+      lower="0.0"
+      upper="0.44"
+      velocity="1.0" />
+  </joint>
+  <link
+    name="right_follower_finger">
+    <inertial>
+      <origin
+        xyz="0.01893989 0.00901216 -0.00215461"
+        rpy="0 0 0" />
+      <mass
+        value="0.03090786" />
+      <inertia
+        ixx="0.00000769"
+        ixy="-0.00000321"
+        ixz="0.00000029"
+        iyy="0.00001487"
+        iyz="0.00000020"
+        izz="0.00001184" />
+    </inertial>
+    <visual>
+      <origin
+        xyz="0 0 0"
+        rpy="0 0 0" />
+      <geometry>
+        <mesh
+          filename="package://trossen_arm_description/meshes/vxai/right_follower_finger.stl" />
+      </geometry>
+      <material
+        name="">
+        <color
+          rgba="0.752941176470588 0.752941176470588 0.752941176470588 1" />
+      </material>
+    </visual>
+    <collision>
+      <origin
+        xyz="0 0 0"
+        rpy="0 0 0" />
+      <geometry>
+        <mesh
+          filename="package://trossen_arm_description/meshes/vxai/right_follower_finger.stl" />
+      </geometry>
+    </collision>
+  </link>
+  <joint
+    name="right_follower_finger_joint"
+    type="fixed">
+    <origin
+      xyz="0 0 0"
+      rpy="0 0 0" />
+    <parent
+      link="right_carriage" />
+    <child
+      link="right_follower_finger" />
+    <axis
+      xyz="0 0 0" />
+  </joint>
+  <link
+    name="left_carriage">
+    <inertial>
+      <origin
+        xyz="-0.00889602 -0.00403515 -0.00457908"
+        rpy="0 0 0" />
+      <mass
+        value="0.05036313" />
       <inertia
         ixx="0.00001736"
@@ -461,5 +572,5 @@
         ixz="-0.00000104"
         iyy="0.00000591"
-        iyz="0.00000172"
+        iyz="-0.00000172"
         izz="0.00001378" />
     </inertial>
@@ -470,34 +581,34 @@
       <geometry>
         <mesh
-          filename="package://trossen_arm_description/meshes/vxai/right_carriage.stl" />
-      </geometry>
-      <material
-        name="">
-        <color
-          rgba="0.752941176470588 0.752941176470588 0.752941176470588 1" />
-      </material>
-    </visual>
-    <collision>
-      <origin
-        xyz="0 0 0"
-        rpy="0 0 0" />
-      <geometry>
-        <mesh
-          filename="package://trossen_arm_description/meshes/vxai/right_carriage.stl" />
-      </geometry>
-    </collision>
-  </link>
-  <joint
-    name="right_carriage_joint"
+          filename="package://trossen_arm_description/meshes/vxai/left_carriage.stl" />
+      </geometry>
+      <material
+        name="">
+        <color
+          rgba="0.752941176470588 0.752941176470588 0.752941176470588 1" />
+      </material>
+    </visual>
+    <collision>
+      <origin
+        xyz="0 0 0"
+        rpy="0 0 0" />
+      <geometry>
+        <mesh
+          filename="package://trossen_arm_description/meshes/vxai/left_carriage.stl" />
+      </geometry>
+    </collision>
+  </link>
+  <joint
+    name="left_carriage_joint"
     type="prismatic">
     <origin
-      xyz="0.1305 -0.022974 -0.021"
+      xyz="0.1305 0.022974 -0.021"
       rpy="0 0 0" />
     <parent
       link="link_7" />
     <child
-      link="right_carriage" />
-    <axis
-      xyz="0 -1 0" />
+      link="left_carriage" />
+    <axis
+      xyz="0 1 0" />
     <limit
       effort="0"
@@ -507,15 +618,15 @@
   </joint>
   <link
-    name="right_follower_finger">
-    <inertial>
-      <origin
-        xyz="0.01893989 0.00901216 -0.00215461"
-        rpy="0 0 0" />
-      <mass
-        value="0.03090786" />
+    name="left_follower_finger">
+    <inertial>
+      <origin
+        xyz="0.01893993 -0.00901223 -0.00215453"
+        rpy="0 0 0" />
+      <mass
+        value="0.03090787" />
       <inertia
         ixx="0.00000769"
         ixy="0.00000321"
-        ixz="-0.00000029"
+        ixz="0.00000029"
         iyy="0.00001487"
         iyz="-0.00000020"
@@ -528,115 +639,4 @@
       <geometry>
         <mesh
-          filename="package://trossen_arm_description/meshes/vxai/right_follower_finger.stl" />
-      </geometry>
-      <material
-        name="">
-        <color
-          rgba="0.752941176470588 0.752941176470588 0.752941176470588 1" />
-      </material>
-    </visual>
-    <collision>
-      <origin
-        xyz="0 0 0"
-        rpy="0 0 0" />
-      <geometry>
-        <mesh
-          filename="package://trossen_arm_description/meshes/vxai/right_follower_finger.stl" />
-      </geometry>
-    </collision>
-  </link>
-  <joint
-    name="right_follower_finger_joint"
-    type="fixed">
-    <origin
-      xyz="0 0 0"
-      rpy="0 0 0" />
-    <parent
-      link="right_carriage" />
-    <child
-      link="right_follower_finger" />
-    <axis
-      xyz="0 0 0" />
-  </joint>
-  <link
-    name="left_carriage">
-    <inertial>
-      <origin
-        xyz="-0.00889602 -0.00403515 -0.00457908"
-        rpy="0 0 0" />
-      <mass
-        value="0.05036313" />
-      <inertia
-        ixx="0.00001736"
-        ixy="0.00000165"
-        ixz="0.00000104"
-        iyy="0.00000591"
-        iyz="0.00000172"
-        izz="0.00001378" />
-    </inertial>
-    <visual>
-      <origin
-        xyz="0 0 0"
-        rpy="0 0 0" />
-      <geometry>
-        <mesh
-          filename="package://trossen_arm_description/meshes/vxai/left_carriage.stl" />
-      </geometry>
-      <material
-        name="">
-        <color
-          rgba="0.752941176470588 0.752941176470588 0.752941176470588 1" />
-      </material>
-    </visual>
-    <collision>
-      <origin
-        xyz="0 0 0"
-        rpy="0 0 0" />
-      <geometry>
-        <mesh
-          filename="package://trossen_arm_description/meshes/vxai/left_carriage.stl" />
-      </geometry>
-    </collision>
-  </link>
-  <joint
-    name="left_carriage_joint"
-    type="prismatic">
-    <origin
-      xyz="0.1305 0.022974 -0.021"
-      rpy="0 0 0" />
-    <parent
-      link="link_7" />
-    <child
-      link="left_carriage" />
-    <axis
-      xyz="0 1 0" />
-    <limit
-      effort="0"
-      lower="0.0"
-      upper="0.44"
-      velocity="1.0" />
-  </joint>
-  <link
-    name="left_follower_finger">
-    <inertial>
-      <origin
-        xyz="0.01893993 -0.00901223 -0.00215453"
-        rpy="0 0 0" />
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