Commit message: xacro

File: urdf/vxai.urdf.xacro (robot description, xacro)
@@ -1,672 +1,22 @@
 <?xml version="1.0" encoding="utf-8"?>
-<robot
-  name="vxai">
-  <link
-    name="base_link">
-    <inertial>
-      <origin
-        xyz="-0.00002199 -0.03351643 0.00006205"
-        rpy="0 0 0" />
-      <mass
-        value="1.87165014" />
-      <inertia
-        ixx="0.00209272"
-        ixy="-0.00000341"
-        ixz="-0.00000001"
-        iyy="0.00299206"
-        iyz="-0.00000068"
-        izz="0.00207913" />
-    </inertial>
-    <visual>
-      <origin
-        xyz="0 0 0"
-        rpy="0 0 0" />
-      <geometry>
-        <mesh
-          filename="package://trossen_arm_description/meshes/vxai/base_link.stl" />
-      </geometry>
-      <material
-        name="">
-        <color
-          rgba="0.75294 0.75294 0.75294 1" />
-      </material>
-    </visual>
-    <collision>
-      <origin
-        xyz="0 0 0"
-        rpy="0 0 0" />
-      <geometry>
-        <mesh
-          filename="package://trossen_arm_description/meshes/vxai/base_link.stl" />
-      </geometry>
-    </collision>
-  </link>
-  <link
-    name="link_1">
-    <inertial>
-      <origin
-        xyz="0.00275058 -0.05744640 -0.00007470"
-        rpy="0 0 0" />
-      <mass
-        value="1.28114157" />
-      <inertia
-        ixx="0.00180008"
-        ixy="0.00001517"
-        ixz="0.00000048"
-        iyy="0.00124234"
-        iyz="-0.00000523"
-        izz="0.00154695" />
-    </inertial>
-    <visual>
-      <origin
-        xyz="0 0 0"
-        rpy="0 0 0" />
-      <geometry>
-        <mesh
-          filename="package://trossen_arm_description/meshes/vxai/link_1.stl" />
-      </geometry>
-      <material
-        name="">
-        <color
-          rgba="0.752941176470588 0.752941176470588 0.752941176470588 1" />
-      </material>
-    </visual>
-    <collision>
-      <origin
-        xyz="0 0 0"
-        rpy="0 0 0" />
-      <geometry>
-        <mesh
-          filename="package://trossen_arm_description/meshes/vxai/link_1.stl" />
-      </geometry>
-    </collision>
-  </link>
-  <joint
-    name="joint_0"
-    type="revolute">
-    <origin
-      xyz="0 -0.068 0"
-      rpy="0 0 0" />
-    <parent
-      link="base_link" />
-    <child
-      link="link_1" />
-    <axis
-      xyz="0 -1 0" />
-    <limit
-      effort="0"
-      lower="-3.14159265358979"
-      upper="3.14159265358979"
-      velocity="3.14" />
-  </joint>
-  <link
-    name="link_2">
-    <inertial>
-      <origin
-        xyz="0.00004155 0.00000477 -0.09223936"
-        rpy="0 0 0" />
-      <mass
-        value="1.58168513" />
-      <inertia
-        ixx="0.00303540"
-        ixy="0.00000094"
-        ixz="0.00000007"
-        iyy="0.00325708"
-        iyz="0.00000058"
-        izz="0.00202764" />
-    </inertial>
-    <visual>
-      <origin
-        xyz="0 0 0"
-        rpy="0 0 0" />
-      <geometry>
-        <mesh
-          filename="package://trossen_arm_description/meshes/vxai/link_2.stl" />
-      </geometry>
-      <material
-        name="">
-        <color
-          rgba="0.752941176470588 0.752941176470588 0.752941176470588 1" />
-      </material>
-    </visual>
-    <collision>
-      <origin
-        xyz="0 0 0"
-        rpy="0 0 0" />
-      <geometry>
-        <mesh
-          filename="package://trossen_arm_description/meshes/vxai/link_2.stl" />
-      </geometry>
-    </collision>
-  </link>
-  <joint
-    name="joint_1"
-    type="revolute">
-    <origin
-      xyz="0 -0.064 0"
-      rpy="0 0 0" />
-    <parent
-      link="link_1" />
-    <child
-      link="link_2" />
-    <axis
-      xyz="1 0 0" />
-    <limit
-      effort="0"
-      lower="-3.14159265358979"
-      upper="3.14159265358979"
-      velocity="3.14" />
-  </joint>
-  <link
-    name="link_3">
-    <inertial>
-      <origin
-        xyz="0.01469489 -0.00233198 -0.13174594"
-        rpy="0 0 0" />
-      <mass
-        value="1.51522891" />
-      <inertia
-        ixx="0.00491722"
-        ixy="0.00001966"
-        ixz="0.00061652"
-        iyy="0.00521379"
-        iyz="-0.00008813"
-        izz="0.00131018" />
-    </inertial>
-    <visual>
-      <origin
-        xyz="0 0 0"
-        rpy="0 0 0" />
-      <geometry>
-        <mesh
-          filename="package://trossen_arm_description/meshes/vxai/link_3.stl" />
-      </geometry>
-      <material
-        name="">
-        <color
-          rgba="0.752941176470588 0.752941176470588 0.752941176470588 1" />
-      </material>
-    </visual>
-    <collision>
-      <origin
-        xyz="0 0 0"
-        rpy="0 0 0" />
-      <geometry>
-        <mesh
-          filename="package://trossen_arm_description/meshes/vxai/link_3.stl" />
-      </geometry>
-    </collision>
-  </link>
-  <joint
-    name="joint_2"
-    type="revolute">
-    <origin
-      xyz="0 0 -0.1408"
-      rpy="0 0 0" />
-    <parent
-      link="link_2" />
-    <child
-      link="link_3" />
-    <axis
-      xyz="0 0 -1" />
-    <limit
-      effort="0"
-      lower="-3.14159265358979"
-      upper="3.14159265358979"
-      velocity="3.14" />
-  </joint>
-  <link
-    name="link_4">
-    <inertial>
-      <origin
-        xyz="0.07293047 0.00011005 -0.01788634"
-        rpy="0 0 0" />
-      <mass
-        value="0.59839689" />
-      <inertia
-        ixx="0.00052102"
-        ixy="-0.00000093"
-        ixz="0.00008634"
-        iyy="0.00069719"
-        iyz="0.00000013"
-        izz="0.00082356" />
-    </inertial>
-    <visual>
-      <origin
-        xyz="0 0 0"
-        rpy="0 0 0" />
-      <geometry>
-        <mesh
-          filename="package://trossen_arm_description/meshes/vxai/link_4.stl" />
-      </geometry>
-      <material
-        name="">
-        <color
-          rgba="0.752941176470588 0.752941176470588 0.752941176470588 1" />
-      </material>
-    </visual>
-    <collision>
-      <origin
-        xyz="0 0 0"
-        rpy="0 0 0" />
-      <geometry>
-        <mesh
-          filename="package://trossen_arm_description/meshes/vxai/link_4.stl" />
-      </geometry>
-    </collision>
-  </link>
-  <joint
-    name="joint_3"
-    type="revolute">
-    <origin
-      xyz="0.02 0 -0.159"
-      rpy="0 0 0" />
-    <parent
-      link="link_3" />
-    <child
-      link="link_4" />
-    <axis
-      xyz="0 -1 0" />
-    <limit
-      effort="0"
-      lower="-3.14159265358979"
-      upper="3.14159265358979"
-      velocity="3.14" />
-  </joint>
-  <link
-    name="link_5">
-    <inertial>
-      <origin
-        xyz="0.04045078 0.00225112 -0.00011067"
-        rpy="0 0 0" />
-      <mass
-        value="0.60644692" />
-      <inertia
-        ixx="0.00066100"
-        ixy="0.00000214"
-        ixz="0.00000789"
-        iyy="0.00054664"
-        iyz="0.00000375"
-        izz="0.00094550" />
-    </inertial>
-    <visual>
-      <origin
-        xyz="0 0 0"
-        rpy="0 0 0" />
-      <geometry>
-        <mesh
-          filename="package://trossen_arm_description/meshes/vxai/link_5.stl" />
-      </geometry>
-      <material
-        name="">
-        <color
-          rgba="0.752941176470588 0.752941176470588 0.752941176470588 1" />
-      </material>
-    </visual>
-    <collision>
-      <origin
-        xyz="0 0 0"
-        rpy="0 0 0" />
-      <geometry>
-        <mesh
-          filename="package://trossen_arm_description/meshes/vxai/link_5.stl" />
-      </geometry>
-    </collision>
-  </link>
-  <joint
-    name="joint_4"
-    type="revolute">
-    <origin
-      xyz="0.1065 0 -0.02"
-      rpy="0 0 0" />
-    <parent
-      link="link_4" />
-    <child
-      link="link_5" />
-    <axis
-      xyz="1 0 0" />
-    <limit
-      effort="0"
-      lower="-3.14159265358979"
-      upper="3.14159265358979"
-      velocity="3.14" />
-  </joint>
-  <link
-    name="link_6">
-    <inertial>
-      <origin
-        xyz="-0.00001797 0.00058070 -0.00058762"
-        rpy="0 0 0" />
-      <mass
-        value="0.38858221" />
-      <inertia
-        ixx="0.00031658"
-        ixy="-0.00000008"
-        ixz="-0.00000001"
-        iyy="0.00026787"
-        iyz="-0.00000050"
-        izz="0.00018958" />
-    </inertial>
-    <visual>
-      <origin
-        xyz="0 0 0"
-        rpy="0 0 0" />
-      <geometry>
-        <mesh
-          filename="package://trossen_arm_description/meshes/vxai/link_6.stl" />
-      </geometry>
-      <material
-        name="">
-        <color
-          rgba="0.752941176470588 0.752941176470588 0.752941176470588 1" />
-      </material>
-    </visual>
-    <collision>
-      <origin
-        xyz="0 0 0"
-        rpy="0 0 0" />
-      <geometry>
-        <mesh
-          filename="package://trossen_arm_description/meshes/vxai/link_6.stl" />
-      </geometry>
-    </collision>
-  </link>
-  <joint
-    name="joint_5"
-    type="revolute">
-    <origin
-      xyz="0.113 0 0"
-      rpy="0 0 0" />
-    <parent
-      link="link_5" />
-    <child
-      link="link_6" />
-    <axis
-      xyz="0 1 0" />
-    <limit
-      effort="0"
-      lower="-3.14159265358979"
-      upper="3.14159265358979"
-      velocity="3.14" />
-  </joint>
-  <link
-    name="link_7">
-    <inertial>
-      <origin
-        xyz="0.08476049 -0.00000697 -0.01847211"
-        rpy="0 0 0" />
-      <mass
-        value="0.57903811" />
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