Commit message: Cleanup

File: urdf/mobile_ai.urdf.xacro (robot description, xacro)
@@ -136,9 +136,4 @@
           filename="${mesh_directory}/base_link.dae" />
       </geometry>
-      <!-- <material
-        name="">
-        <color
-          rgba="0.752941176470588 0.752941176470588 0.752941176470588 1" />
-      </material> -->
     </visual>
     <collision>

Commit message: Add camera, fix inertia

File: urdf/mobile_ai.urdf.xacro (robot description, xacro)
@@ -12,8 +12,8 @@
       <inertial>
         <origin
-          xyz="-0.00642926440937244 -0.00999999999999998 -0.0232437647650167"
+          xyz="-0.00642926 0 -0.02324376"
           rpy="0 0 0" />
         <mass
-          value="0.0318006084570262" />
+          value="0.10000000" />
         <inertia
           ixx="3.29304410034736E-05"
@@ -63,8 +63,8 @@
       <inertial>
         <origin
-          xyz="0 -0.01 0"
+          xyz="0 0 0"
           rpy="0 0 0" />
         <mass
-          value="0.0898231658107286" />
+          value="0.53500000" />
         <inertia
           ixx="3.50667612783944E-05"
@@ -116,8 +116,8 @@
     <inertial>
       <origin
-        xyz="0.0169055503524013 0.00164199144474026 0.23651080871802"
+        xyz="0.01556204 0.00159774 0.22495608"
         rpy="1.57079632679 0 0" />
       <mass
-        value="45.1929991042861" />
+        value="80" />
       <inertia
         ixx="0.800607899578097"
@@ -155,4 +155,13 @@
     <child link="base_link"/>
   </joint>
+  <xacro:include filename="$(find trossen_arm_description)/urdf/peripherals/rs_d405.urdf.xacro" />
+  <xacro:sensor_d405
+    name="camera_low"
+    parent="base_link"
+    use_nominal_extrinsics="true">
+    <origin
+      xyz="0.209805 0 1.031778"
+      rpy="0 ${radians(37)} 0" />
+  </xacro:sensor_d405>
   <joint
     name="left_wheel"
@@ -177,5 +186,5 @@
         rpy="0 0 0" />
       <mass
-        value="0.981755254019503" />
+        value="3.00000000" />
       <inertia
         ixx="0.00165792997375718"

Commit message: Add limits, standardize style

File: urdf/mobile_ai.urdf.xacro (robot description, xacro)
@@ -14,6 +14,5 @@
           xyz="-0.00642926 0 -0.02324376"
           rpy="0 0 0" />
-        <mass
-          value="0.10000000" />
+        <mass value="0.10000000" />
         <inertia
           ixx="3.29304410034736E-05"
@@ -29,6 +28,5 @@
           rpy="0 0 0" />
         <geometry>
-          <mesh
-            filename="${mesh_directory}/caster_swivel.stl" />
+          <mesh filename="${mesh_directory}/caster_swivel.stl" />
         </geometry>
         <material
@@ -43,19 +41,16 @@
           rpy="0 0 0" />
         <geometry>
-          <mesh
-            filename="${mesh_directory}/caster_swivel.stl" />
+          <mesh filename="${mesh_directory}/caster_swivel.stl" />
         </geometry>
       </collision>
     </link>
-    <joint
-      name="caster_swivel_joint_${name}"
-      type="continuous">
+    <joint name="caster_swivel_joint_${name}" type="continuous">
       <xacro:insert_block name="origin" />
-      <parent
-        link="${parent}" />
-      <child
-        link="caster_swivel_${name}" />
-      <axis
-        xyz="0 0 1" />
+      <parent link="${parent}" />
+      <child link="caster_swivel_${name}" />
+      <axis xyz="0 0 1" />
+      <limit
+        effort="0"
+        velocity="${pi}" />
     </joint>
     <link
@@ -65,6 +60,5 @@
           xyz="0 0 0"
           rpy="0 0 0" />
-        <mass
-          value="0.53500000" />
+        <mass value="0.53500000" />
         <inertia
           ixx="3.50667612783944E-05"
@@ -80,6 +74,5 @@
           rpy="0 0 0" />
         <geometry>
-          <mesh
-            filename="${mesh_directory}/caster_wheel.stl" />
+          <mesh filename="${mesh_directory}/caster_wheel.stl" />
         </geometry>
         <material
@@ -94,21 +87,18 @@
           rpy="0 0 0" />
         <geometry>
-          <mesh
-            filename="${mesh_directory}/caster_wheel.stl" />
+          <mesh filename="${mesh_directory}/caster_wheel.stl" />
         </geometry>
       </collision>
     </link>
-    <joint
-      name="caster_wheel_joint_${name}"
-      type="continuous">
+    <joint name="caster_wheel_joint_${name}" type="continuous">
       <origin
         xyz="-0.0345 0 -0.066"
         rpy="0 0 0" />
-      <parent
-        link="caster_swivel_${name}" />
-      <child
-        link="caster_wheel_${name}" />
-      <axis
-        xyz="0 1 0" />
+      <parent link="caster_swivel_${name}" />
+      <child link="caster_wheel_${name}" />
+      <axis xyz="0 1 0" />
+      <limit
+        effort="0"
+        velocity="${pi}" />
     </joint>
   </xacro:macro>  <!-- caster_wheel -->
@@ -118,6 +108,5 @@
         xyz="0.01556204 0.00159774 0.22495608"
         rpy="1.57079632679 0 0" />
-      <mass
-        value="80" />
+      <mass value="80" />
       <inertia
         ixx="0.800607899578097"
@@ -133,6 +122,5 @@
         rpy="-1.57079632679 0 0" />
       <geometry>
-        <mesh
-          filename="${mesh_directory}/base_link.dae" />
+        <mesh filename="${mesh_directory}/base_link.dae" />
       </geometry>
     </visual>
@@ -142,6 +130,5 @@
         rpy="-1.57079632679 0 0" />
       <geometry>
-        <mesh
-          filename="${mesh_directory}/base_link.dae" />
+        <mesh filename="${mesh_directory}/base_link.dae" />
       </geometry>
     </collision>
@@ -170,13 +157,10 @@
       xyz="0 0.192 -0.1259 "
       rpy="0 0 0" />
-    <parent
-      link="base_link" />
-    <child
-      link="left_wheel_link" />
-    <axis
-      xyz="0 1 0" />
+    <parent link="base_link" />
+    <child link="left_wheel_link" />
+    <axis xyz="0 1 0" />
     <limit
-      effort="0"
-      velocity="0" />
+      effort="4"
+      velocity="${4 * pi}" />
   </joint>
   <link name="left_wheel_link">
@@ -185,6 +169,5 @@
         xyz="0 0 0"
         rpy="0 0 0" />
-      <mass
-        value="3.00000000" />
+      <mass value="3.00000000" />
       <inertia
         ixx="0.00165792997375718"
@@ -200,6 +183,5 @@
         rpy="0 0 0" />
       <geometry>
-        <mesh
-          filename="${mesh_directory}/wheel.stl" />
+        <mesh filename="${mesh_directory}/wheel.stl" />
       </geometry>
       <material
@@ -214,6 +196,5 @@
         rpy="0 0 0" />
       <geometry>
-        <mesh
-          filename="${mesh_directory}/wheel.stl" />
+        <mesh filename="${mesh_directory}/wheel.stl" />
       </geometry>
     </collision>
@@ -225,13 +206,10 @@
       xyz="0 -0.192 -0.1259"
       rpy="0 0 0" />
-    <parent
-      link="base_link" />
-    <child
-      link="right_wheel_link" />
-    <axis
-      xyz="0 1 0" />
+    <parent link="base_link" />
+    <child link="right_wheel_link" />
+    <axis xyz="0 1 0" />
     <limit
-      effort="0"
-      velocity="0" />
+      effort="4"
+      velocity="${4 * pi}" />
   </joint>
   <link name="right_wheel_link">
@@ -240,6 +218,5 @@
         xyz="0 0 0"
         rpy="0 0 0" />
-      <mass
-        value="0.981755254019503" />
+      <mass value="0.981755254019503" />
       <inertia
         ixx="0.00165792997375718"
@@ -255,6 +232,5 @@
         rpy="0 0 0" />
       <geometry>
-        <mesh
-          filename="${mesh_directory}/wheel.stl" />
+        <mesh filename="${mesh_directory}/wheel.stl" />
       </geometry>
       <material
@@ -269,6 +245,5 @@
         rpy="0 0 0" />
       <geometry>
-        <mesh
-          filename="${mesh_directory}/wheel.stl" />
+        <mesh filename="${mesh_directory}/wheel.stl" />
       </geometry>
     </collision>
@@ -300,8 +275,6 @@
       xyz="0.331 0.3 0.831"
       rpy="0 0 0" />
-    <parent
-      link="base_link" />
-    <child
-      link="follower_left/base_link" />
+    <parent link="base_link" />
+    <child link="follower_left/base_link" />
   </joint>
   <xacro:wxai
@@ -314,8 +287,6 @@
       xyz="0.331 -0.3 0.831"
       rpy="0 0 0" />
-    <parent
-      link="base_link" />
-    <child
-      link="follower_right/base_link" />
+    <parent link="base_link" />
+    <child link="follower_right/base_link" />
   </joint>
   <xacro:wxai
