Commit message: limits, axes

File: urdf/leader_right.urdf.xacro (robot description, xacro)
@@ -83,15 +83,12 @@
       xyz="0 -0.05325 0"
       rpy="0 0 0" />
-    <parent
-      link="base_link" />
-    <child
-      link="link_1" />
-    <axis
-      xyz="0 -1 0" />
-    <limit
-      lower="0"
-      upper="0"
-      effort="0"
-      velocity="0" />
+    <parent link="base_link" />
+    <child link="link_1" />
+    <axis xyz="0 -1 0" />
+    <limit
+      effort="0"
+      lower="${-pi / 2}"
+      upper="${pi}"
+      velocity="${2 * pi}" />
   </joint>
   <link name="link_2">
@@ -138,15 +135,12 @@
       xyz="0 -0.0365 0"
       rpy="0 0 0" />
-    <parent
-      link="link_1" />
-    <child
-      link="link_2" />
-    <axis
-      xyz="1 0 0" />
-    <limit
-      lower="0"
+    <parent link="link_1" />
+    <child link="link_2" />
+    <axis xyz="1 0 0" />
+    <limit
+      effort="0"
+      lower="${-pi}"
       upper="0"
-      effort="0"
-      velocity="0" />
+      velocity="${2 * pi}" />
   </joint>
   <link name="link_3">
@@ -193,15 +187,12 @@
       xyz="0 0 -0.0979"
       rpy="0 0 0" />
-    <parent
-      link="link_2" />
-    <child
-      link="link_3" />
-    <axis
-      xyz="0 0 -1" />
-    <limit
-      lower="0"
-      upper="0"
-      effort="0"
-      velocity="0" />
+    <parent link="link_2" />
+    <child link="link_3" />
+    <axis xyz="0 0 -1" />
+    <limit
+      effort="0"
+      lower="${-pi / 2}"
+      upper="${pi / 2}"
+      velocity="${2 * pi}" />
   </joint>
   <link name="link_4">
@@ -248,15 +239,12 @@
       xyz="0.02 0 -0.2019"
       rpy="0 0 0" />
-    <parent
-      link="link_3" />
-    <child
-      link="link_4" />
-    <axis
-      xyz="0 1 0" />
-    <limit
+    <parent link="link_3" />
+    <child link="link_4" />
+    <axis xyz="0 -1 0" />
+    <limit
+      effort="0"
       lower="0"
-      upper="0"
-      effort="0"
-      velocity="0" />
+      upper="${3 * pi / 4}"
+      velocity="${2 * pi}" />
   </joint>
   <link name="link_5">
@@ -303,15 +291,12 @@
       xyz="-0.02 0 -0.1185"
       rpy="0 0 0" />
-    <parent
-      link="link_4" />
-    <child
-      link="link_5" />
-    <axis
-      xyz="0 0 -1" />
-    <limit
-      lower="0"
-      upper="0"
-      effort="0"
-      velocity="0" />
+    <parent link="link_4" />
+    <child link="link_5" />
+    <axis xyz="0 0 -1" />
+    <limit
+      effort="0"
+      lower="${-pi / 2}"
+      upper="${pi / 2}"
+      velocity="${2 * pi}" />
   </joint>
   <link name="link_6">
@@ -358,15 +343,12 @@
       xyz="0 0 -0.101"
       rpy="0 0 0" />
-    <parent
-      link="link_5" />
-    <child
-      link="link_6" />
-    <axis
-      xyz="0 1 0" />
-    <limit
-      lower="0"
-      upper="0"
-      effort="0"
-      velocity="0" />
+    <parent link="link_5" />
+    <child link="link_6" />
+    <axis xyz="0 1 0" />
+    <limit
+      effort="0"
+      lower="${-pi / 4}"
+      upper="${pi / 4}"
+      velocity="${2 * pi}" />
   </joint>
   <link name="end_link">
@@ -413,15 +395,12 @@
       xyz="-0.034 0 0"
       rpy="0 0 0" />
-    <parent
-      link="link_6" />
-    <child
-      link="end_link" />
-    <axis
-      xyz="-1 0 0" />
-    <limit
-      lower="0"
-      upper="0"
-      effort="0"
-      velocity="0" />
+    <parent link="link_6" />
+    <child link="end_link" />
+    <axis xyz="1 0 0" />
+    <limit
+      effort="0"
+      lower="${-pi / 2}"
+      upper="${pi / 2}"
+      velocity="${2 * pi}" />
   </joint>
 </robot>

Commit message: updated 7dof leader right

File: urdf/leader_right.urdf.xacro (robot description, xacro)
@@ -2,18 +2,18 @@
 <robot name="leader_right" xmlns:xacro="http://ros.org/wiki/xacro">
   <link name="base_link">
-    <!-- <inertial>
-      <origin
-        xyz="-1.39152180017271E-08 -0.0244562601098712 -7.37998766462572E-05"
-        rpy="0 0 0" />
-      <mass
-        value="0.139112019612118" />
-      <inertia
-        ixx="5.49621467928766E-05"
-        ixy="1.28787223237068E-12"
-        ixz="2.72664645438671E-12"
-        iyy="6.23808866762274E-05"
-        iyz="8.1148771029003E-09"
-        izz="4.83929577581152E-05" />
-    </inertial> -->
+    <inertial>
+      <origin
+        xyz="5.199e-05 -0.03429087 5.295e-05"
+        rpy="0 0 0" />
+      <mass
+        value="0.37290125" />
+      <inertia
+        ixx="0.00034804"
+        ixy="-3.9e-07"
+        ixz="-3e-08"
+        iyy="0.00014057"
+        iyz="-8e-07"
+        izz="0.00034074" />
+    </inertial>
     <visual>
       <origin
@@ -41,18 +41,18 @@
   </link>
   <link name="link_1">
-    <!-- <inertial>
-      <origin
-        xyz="0.00167418519111886 -0.0312005018035526 9.78866061475296E-09"
-        rpy="0 0 0" />
-      <mass
-        value="0.191701343253073" />
-      <inertia
-        ixx="7.9463528295035E-05"
-        ixy="-6.77209190934734E-09"
-        ixz="1.04864059984379E-12"
-        iyy="7.05878958859156E-05"
-        iyz="-2.00221325867351E-12"
-        izz="6.45361069136214E-05" />
-    </inertial> -->
+    <inertial>
+      <origin
+        xyz="0.00331378 -0.03460068 -4.285e-05"
+        rpy="0 0 0" />
+      <mass
+        value="0.4523603" />
+      <inertia
+        ixx="0.0001893"
+        ixy="3.6e-06"
+        ixz="-3.3e-07"
+        iyy="0.00043171"
+        iyz="0.0"
+        izz="0.00045089" />
+    </inertial>
     <visual>
       <origin
@@ -81,5 +81,5 @@
   <joint name="joint_0" type="revolute">
     <origin
-      xyz="0 -0.05325 0"
+      xyz="0 -0.05825 0"
       rpy="0 0 0" />
     <parent link="base_link" />
@@ -93,18 +93,18 @@
   </joint>
   <link name="link_2">
-    <!-- <inertial>
-      <origin
-        xyz="-5.367166166162E-07 5.50462505594373E-05 -0.0631252938879995"
-        rpy="0 0 0" />
-      <mass
-        value="0.0968334760009524" />
-      <inertia
-        ixx="2.42097025430152E-05"
-        ixy="3.20685249522413E-10"
-        ixz="-5.50642459434214E-11"
-        iyy="2.77810904550607E-05"
-        iyz="7.97639885086344E-09"
-        izz="2.76652155506527E-05" />
-    </inertial> -->
+    <inertial>
+      <origin
+        xyz="-5.27e-06 1.239e-05 -0.08091014"
+        rpy="0 0 0" />
+      <mass
+        value="0.33783172" />
+      <inertia
+        ixx="0.00031788"
+        ixy="4e-08"
+        ixz="-4.9e-07"
+        iyy="0.00034942"
+        iyz="-4.5e-07"
+        izz="0.00016037" />
+    </inertial>
     <visual>
       <origin
@@ -145,18 +145,18 @@
   </joint>
   <link name="link_3">
-    <!-- <inertial>
-      <origin
-        xyz="0.0139862989497736 0.000307666016540559 -0.143995683795875"
-        rpy="0 0 0" />
-      <mass
-        value="0.260115273199168" />
-      <inertia
-        ixx="0.000427379966791221"
-        ixy="-7.81704710322318E-09"
-        ixz="-3.77410479282022E-05"
-        iyy="0.000462804238444559"
-        iyz="6.71097359310217E-13"
-        izz="7.59010644862872E-05" />
-    </inertial> -->
+    <inertial>
+      <origin
+        xyz="0.01706827 0.00212153 -0.1667902"
+        rpy="0 0 0" />
+      <mass
+        value="0.46940642" />
+      <inertia
+        ixx="0.00182642"
+        ixy="-3.41e-06"
+        ixz="0.00015666"
+        iyy="0.00165644"
+        iyz="2.673e-05"
+        izz="0.00039819" />
+    </inertial>
     <visual>
       <origin
@@ -185,5 +185,5 @@
   <joint name="joint_2" type="revolute">
     <origin
-      xyz="0 0 -0.0979"
+      xyz="0 0 -0.106"
       rpy="0 0 0" />
     <parent link="link_2" />
@@ -197,18 +197,18 @@
   </joint>
   <link name="link_4">
-    <!-- <inertial>
-      <origin
-        xyz="-0.0172302461757262 0.00148708433063532 -0.0737933680183246"
-        rpy="0 0 0" />
-      <mass
-        value="0.108911932357874" />
-      <inertia
-        ixx="3.67350299124525E-05"
-        ixy="-3.2069352659567E-10"
-        ixz="4.67937259825546E-06"
-        iyy="3.79435353491667E-05"
-        iyz="-5.49520144163367E-11"
-        izz="2.79681494421085E-05" />
-    </inertial> -->
+    <inertial>
+      <origin
+        xyz="-0.01912502 2.771e-05 -0.0899419"
+        rpy="0 0 0" />
+      <mass
+        value="0.19153172" />
+      <inertia
+        ixx="0.00019027"
+        ixy="-1e-07"
+        ixz="-1.489e-05"
+        iyy="0.00015938"
+        iyz="-4.7e-07"
+        izz="8.565e-05" />
+    </inertial>
     <visual>
       <origin
@@ -237,8 +237,9 @@
   <joint name="joint_3" type="revolute">
     <origin
-      xyz="0.02 0 -0.2019"
+      xyz="0.02 0 -0.1938"
       rpy="0 0 0" />
     <parent link="link_3" />
     <child link="link_4" />
+    <!-- <axis xyz="0 1 0" /> -->
     <axis xyz="0 -1 0" />
     <limit
@@ -249,18 +250,18 @@
   </joint>
   <link name="link_5">
-    <!-- <inertial>
-      <origin
-        xyz="4.6197874683856E-05 -0.00189060415458123 -0.0327154665241671"
-        rpy="0 0 0" />
-      <mass
-        value="0.17292687898798" />
-      <inertia
-        ixx="8.34725819373986E-05"
-        ixy="-5.90058376569713E-07"
-        ixz="1.67532783119531E-06"
-        iyy="9.21934779612374E-05"
-        iyz="2.65193411794291E-06"
-        izz="4.30963337539513E-05" />
-    </inertial> -->
+    <inertial>
+      <origin
+        xyz="-0.00025767 0.00302328 -0.03375968"
+        rpy="0 0 0" />
+      <mass
+        value="0.24163171" />
+      <inertia
+        ixx="0.00022638"
+        ixy="1e-06"
+        ixz="-4.42e-06"
+        iyy="0.00016124"
+        iyz="7.25e-06"
+        izz="0.00013726" />
+    </inertial>
     <visual>
       <origin
@@ -301,18 +302,18 @@
   </joint>
   <link name="link_6">
-    <!-- <inertial>
-      <origin
-        xyz="-0.00808258410436435 -1.55757918360311E-05 -5.25824547309428E-05"
-        rpy="0 0 0" />
-      <mass
-        value="0.0945457994340799" />
-      <inertia
-        ixx="2.28857807728819E-05"
-        ixy="-4.18411286496346E-09"
-        ixz="-1.4016527558119E-08"
-        iyy="1.66489373164978E-05"
-        iyz="-1.12312618077519E-09"
-        izz="1.71149397185573E-05" />
-    </inertial> -->
+    <inertial>
+      <origin
+        xyz="-0.01044529 9.1e-06 0.00011242"
+        rpy="0 0 0" />
+      <mass
+        value="0.18731697" />
+      <inertia
+        ixx="6.195e-05"
+        ixy="-1e-08"
+        ixz="-3.2e-07"
+        iyy="5.051e-05"
+        iyz="0.0"
+        izz="6.44e-05" />
+    </inertial>
     <visual>
       <origin
@@ -353,18 +354,18 @@
   </joint>
   <link name="end_link">
-    <!-- <inertial>
-      <origin
-        xyz="-0.0532965871728031 8.96532691141427E-09 -0.0694281601388337"
-        rpy="0 0 0" />
-      <mass
-        value="0.0949576109060715" />
-      <inertia
-        ixx="3.84221007642206E-05"
-        ixy="3.20422759899826E-11"
-        ixz="2.68672960859202E-05"
-        iyy="0.00016377648911462"
-        iyz="4.23116882443166E-12"
-        izz="0.000136448375290933" />
-    </inertial> -->
+    <inertial>
+      <origin
+        xyz="-0.01502064 0.00191435 0.00656522"
+        rpy="0 0 0" />
+      <mass
+        value="0.00915397" />
+      <inertia
+        ixx="1.2e-06"
+        ixy="-2.1e-07"
+        ixz="1.02e-06"
+        iyy="3.85e-06"
+        iyz="1.1e-07"
+        izz="2.84e-06" />
+    </inertial>
     <visual>
       <origin
@@ -397,5 +398,6 @@
     <parent link="link_6" />
     <child link="end_link" />
-    <axis xyz="1 0 0" />
+    <axis xyz="-1 0 0" />
+    <!-- <axis xyz="1 0 0" /> -->
     <limit
       effort="0"

Commit message: add link 8

File: urdf/leader_right.urdf.xacro (robot description, xacro)
@@ -21,20 +21,17 @@
         rpy="0 0 0" />
       <geometry>
-        <mesh
-          filename="package://trossen_arm_description/meshes/leader_right/base_link.stl" />
-      </geometry>
-      <material
-        name="">
-        <color
-          rgba="0.752941176470588 0.752941176470588 0.752941176470588 1" />
-      </material>
-    </visual>
-    <collision>
-      <origin
-        xyz="0 0 0"
-        rpy="0 0 0" />
-      <geometry>
-        <mesh
-          filename="package://trossen_arm_description/meshes/leader_right/base_link.stl" />
+        <mesh filename="package://trossen_arm_description/meshes/leader_right/base_link.stl" />
+      </geometry>
+      <material
+        name="">
+        <color rgba="0.752941176470588 0.752941176470588 0.752941176470588 1" />
+      </material>
+    </visual>
+    <collision>
+      <origin
+        xyz="0 0 0"
+        rpy="0 0 0" />
+      <geometry>
+        <mesh filename="package://trossen_arm_description/meshes/leader_right/base_link.stl" />
       </geometry>
     </collision>
@@ -60,20 +57,17 @@
         rpy="0 0 0" />
       <geometry>
-        <mesh
-          filename="package://trossen_arm_description/meshes/leader_right/link_1.stl" />
-      </geometry>
-      <material
-        name="">
-        <color
-          rgba="0.752941176470588 0.752941176470588 0.752941176470588 1" />
-      </material>
-    </visual>
-    <collision>
-      <origin
-        xyz="0 0 0"
-        rpy="0 0 0" />
-      <geometry>
-        <mesh
-          filename="package://trossen_arm_description/meshes/leader_right/link_1.stl" />
+        <mesh filename="package://trossen_arm_description/meshes/leader_right/link_1.stl" />
+      </geometry>
+      <material
+        name="">
+        <color rgba="0.752941176470588 0.752941176470588 0.752941176470588 1" />
+      </material>
+    </visual>
+    <collision>
+      <origin
+        xyz="0 0 0"
+        rpy="0 0 0" />
+      <geometry>
+        <mesh filename="package://trossen_arm_description/meshes/leader_right/link_1.stl" />
       </geometry>
     </collision>
@@ -112,20 +106,17 @@
         rpy="0 0 0" />
       <geometry>
-        <mesh
-          filename="package://trossen_arm_description/meshes/leader_right/link_2.stl" />
-      </geometry>
-      <material
-        name="">
-        <color
-          rgba="0.752941176470588 0.752941176470588 0.752941176470588 1" />
-      </material>
-    </visual>
-    <collision>
-      <origin
-        xyz="0 0 0"
-        rpy="0 0 0" />
-      <geometry>
-        <mesh
-          filename="package://trossen_arm_description/meshes/leader_right/link_2.stl" />
+        <mesh filename="package://trossen_arm_description/meshes/leader_right/link_2.stl" />
+      </geometry>
+      <material
+        name="">
+        <color rgba="0.752941176470588 0.752941176470588 0.752941176470588 1" />
+      </material>
+    </visual>
+    <collision>
+      <origin
+        xyz="0 0 0"
+        rpy="0 0 0" />
+      <geometry>
+        <mesh filename="package://trossen_arm_description/meshes/leader_right/link_2.stl" />
       </geometry>
     </collision>
@@ -164,20 +155,17 @@
         rpy="0 0 0" />
       <geometry>
-        <mesh
-          filename="package://trossen_arm_description/meshes/leader_right/link_3.stl" />
-      </geometry>
-      <material
-        name="">
-        <color
-          rgba="0.752941176470588 0.752941176470588 0.752941176470588 1" />
-      </material>
-    </visual>
-    <collision>
-      <origin
-        xyz="0 0 0"
-        rpy="0 0 0" />
-      <geometry>
-        <mesh
-          filename="package://trossen_arm_description/meshes/leader_right/link_3.stl" />
+        <mesh filename="package://trossen_arm_description/meshes/leader_right/link_3.stl" />
+      </geometry>
+      <material
+        name="">
+        <color rgba="0.752941176470588 0.752941176470588 0.752941176470588 1" />
+      </material>
+    </visual>
+    <collision>
+      <origin
+        xyz="0 0 0"
+        rpy="0 0 0" />
+      <geometry>
+        <mesh filename="package://trossen_arm_description/meshes/leader_right/link_3.stl" />
       </geometry>
     </collision>
@@ -216,20 +204,17 @@
         rpy="0 0 0" />
       <geometry>
-        <mesh
-          filename="package://trossen_arm_description/meshes/leader_right/link_4.stl" />
-      </geometry>
-      <material
-        name="">
-        <color
-          rgba="0.752941176470588 0.752941176470588 0.752941176470588 1" />
-      </material>
-    </visual>
-    <collision>
-      <origin
-        xyz="0 0 0"
-        rpy="0 0 0" />
-      <geometry>
-        <mesh
-          filename="package://trossen_arm_description/meshes/leader_right/link_4.stl" />
+        <mesh filename="package://trossen_arm_description/meshes/leader_right/link_4.stl" />
+      </geometry>
+      <material
+        name="">
+        <color rgba="0.752941176470588 0.752941176470588 0.752941176470588 1" />
+      </material>
+    </visual>
+    <collision>
+      <origin
+        xyz="0 0 0"
+        rpy="0 0 0" />
+      <geometry>
+        <mesh filename="package://trossen_arm_description/meshes/leader_right/link_4.stl" />
       </geometry>
     </collision>
@@ -241,5 +226,4 @@
     <parent link="link_3" />
     <child link="link_4" />
-    <!-- <axis xyz="0 1 0" /> -->
     <axis xyz="0 -1 0" />
     <limit
@@ -269,20 +253,17 @@
         rpy="0 0 0" />
       <geometry>
-        <mesh
-          filename="package://trossen_arm_description/meshes/leader_right/link_5.stl" />
-      </geometry>
-      <material
-        name="">
-        <color
-          rgba="0.752941176470588 0.752941176470588 0.752941176470588 1" />
-      </material>
-    </visual>
-    <collision>
-      <origin
-        xyz="0 0 0"
-        rpy="0 0 0" />
-      <geometry>
-        <mesh
-          filename="package://trossen_arm_description/meshes/leader_right/link_5.stl" />
+        <mesh filename="package://trossen_arm_description/meshes/leader_right/link_5.stl" />
+      </geometry>
+      <material
+        name="">
+        <color rgba="0.752941176470588 0.752941176470588 0.752941176470588 1" />
+      </material>
+    </visual>
+    <collision>
+      <origin
+        xyz="0 0 0"
+        rpy="0 0 0" />
+      <geometry>
+        <mesh filename="package://trossen_arm_description/meshes/leader_right/link_5.stl" />
       </geometry>
     </collision>
@@ -321,20 +302,17 @@
         rpy="0 0 0" />
       <geometry>
-        <mesh
-          filename="package://trossen_arm_description/meshes/leader_right/link_6.stl" />
-      </geometry>
-      <material
-        name="">
-        <color
-          rgba="0.752941176470588 0.752941176470588 0.752941176470588 1" />
-      </material>
-    </visual>
-    <collision>
-      <origin
-        xyz="0 0 0"
-        rpy="0 0 0" />
-      <geometry>
-        <mesh
-          filename="package://trossen_arm_description/meshes/leader_right/link_6.stl" />
+        <mesh filename="package://trossen_arm_description/meshes/leader_right/link_6.stl" />
+      </geometry>
+      <material
+        name="">
+        <color rgba="0.752941176470588 0.752941176470588 0.752941176470588 1" />
+      </material>
+    </visual>
+    <collision>
+      <origin
+        xyz="0 0 0"
+        rpy="0 0 0" />
+      <geometry>
+        <mesh filename="package://trossen_arm_description/meshes/leader_right/link_6.stl" />
       </geometry>
     </collision>
@@ -348,10 +326,59 @@
     <axis xyz="0 1 0" />
     <limit
-      effort="0"
-      lower="${-pi / 4}"
-      upper="${pi / 4}"
-      velocity="${2 * pi}" />
-  </joint>
-  <link name="end_link">
+      lower="0"
+      upper="0"
+      effort="0"
+      velocity="0" />
+  </joint>
+  <link name="link_7">
+    <inertial>
+      <origin
+        xyz="-0.04169427 0.00058029 -0.06323582"
+        rpy="0 0 0" />
+      <mass
+        value="0.23686287" />
+      <inertia
+        ixx="0.00019957"
+        ixy="-2.03e-06"
+        ixz="0.00016948"
+        iyy="0.00053905"
+        iyz="1.92e-06"
+        izz="0.0003876" />
+    </inertial>
+    <visual>
+      <origin
+        xyz="0 0 0"
+        rpy="0 0 0" />
+      <geometry>
+        <mesh filename="package://trossen_arm_description/meshes/leader_right/link_7.stl" />
+      </geometry>
+      <material
+        name="">
+        <color rgba="0.752941176470588 0.752941176470588 0.752941176470588 1" />
+      </material>
+    </visual>
+    <collision>
+      <origin
+        xyz="0 0 0"
+        rpy="0 0 0" />
+      <geometry>
+        <mesh filename="package://trossen_arm_description/meshes/leader_right/link_7.stl" />
+      </geometry>
+    </collision>
+  </link>
+  <joint name="joint_6" type="revolute">
+    <origin
+      xyz="-0.034 0 0"
+      rpy="0 0 0" />
+    <parent link="link_6" />
+    <child link="link_7" />
+    <axis xyz="-1 0 0" />
+    <limit
+      lower="${-pi / 2}"
+      upper="${pi / 2}"
+      effort="0"
+      velocity="0" />
+  </joint>
+  <link name="link_8">
     <inertial>
       <origin
@@ -373,36 +400,32 @@
         rpy="0 0 0" />
       <geometry>
-        <mesh
-          filename="package://trossen_arm_description/meshes/leader_right/end_link.stl" />
-      </geometry>
-      <material
-        name="">
-        <color
-          rgba="0.752941176470588 0.752941176470588 0.752941176470588 1" />
-      </material>
-    </visual>
-    <collision>
-      <origin
-        xyz="0 0 0"
-        rpy="0 0 0" />
-      <geometry>
-        <mesh
-          filename="package://trossen_arm_description/meshes/leader_right/end_link.stl" />
-      </geometry>
-    </collision>
-  </link>
-  <joint name="joint_6" type="revolute">
-    <origin
-      xyz="-0.034 0 0"
-      rpy="0 0 0" />
-    <parent link="link_6" />
-    <child link="end_link" />
-    <axis xyz="-1 0 0" />
-    <!-- <axis xyz="1 0 0" /> -->
-    <limit
-      effort="0"
+        <mesh filename="package://trossen_arm_description/meshes/leader_right/link_8.stl" />
+      </geometry>
+      <material
+        name="">
+        <color rgba="0.752941176470588 0.752941176470588 0.752941176470588 1" />
+      </material>
+    </visual>
+    <collision>
+      <origin
+        xyz="0 0 0"
+        rpy="0 0 0" />
+      <geometry>
+        <mesh filename="package://trossen_arm_description/meshes/leader_right/link_8.stl" />
+      </geometry>
+    </collision>
+  </link>
+  <joint name="joint_7" type="revolute">
+    <origin
+      xyz="-0.02847106 0.01930000 -0.07900135"
+      rpy="0 0 0" />
+    <parent link="link_7" />
+    <child link="link_8" />
+    <axis xyz="0 1 0" />
+    <limit
       lower="${-pi / 2}"
       upper="${pi / 2}"
-      velocity="${2 * pi}" />
+      effort="0"
+      velocity="0" />
   </joint>
 </robot>
