Commit message: Update generated vxai_right

File: urdf/generated/vxai/vxai_right.urdf (robot description, URDF)
Before this commit: robot vxai, 12 links, 11 joints
Links:
- removed link left_carriage
- removed link left_follower_finger
- removed link right_carriage
- removed link right_follower_finger
- added link carriage_left, mass 0.05036313; collision mesh filename=package://trossen_arm_description/meshes/vxai/carriage_left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; visual mesh filename=package://trossen_arm_description/meshes/vxai/carriage_left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
- added link carriage_right, mass 0.05036313; collision mesh filename=package://trossen_arm_description/meshes/vxai/carriage_righ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; visual mesh filename=package://trossen_arm_description/meshes/vxai/carriage_righ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
- added link gripper_left, mass 0.03090787; collision mesh filename=package://trossen_arm_description/meshes/vxai/gripper_left.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; visual mesh filename=package://trossen_arm_description/meshes/vxai/gripper_left.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
- added link gripper_right, mass 0.03090786; collision mesh filename=package://trossen_arm_description/meshes/vxai/gripper_right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; visual mesh filename=package://trossen_arm_description/meshes/vxai/gripper_right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
- link base_link: mass 1.87165014 -> 1.8716501; geometry collision mesh filename=package://trossen_arm_description/meshes/vxai/base_link_rig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; visual mesh filename=package://trossen_arm_description/meshes/vxai/base_link_rig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
- link link_1: mass 1.28114157 -> 1.2811416; geometry collision mesh filename=package://trossen_arm_description/meshes/vxai/link_1_right.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; visual mesh filename=package://trossen_arm_description/meshes/vxai/link_1_right.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
- link link_2: mass 1.58168513 -> 1.5816851
- link link_3: mass 1.51522891 -> 1.5152289; geometry collision mesh filename=package://trossen_arm_description/meshes/vxai/link_3_right.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; visual mesh filename=package://trossen_arm_description/meshes/vxai/link_3_right.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
Joints:
- removed joint left_follower_finger_joint
- removed joint right_follower_finger_joint
- added joint gripper_left_joint: type fixed, parent carriage_left, child gripper_left, origin xyz=0 0 0 rpy=0 0 0, axis 0 0 0
- added joint right_gripper_joint: type fixed, parent carriage_right, child gripper_right, origin xyz=0 0 0 rpy=0 0 0, axis 0 0 0
- joint joint_1: axis 1 0 0 -> -1 0 0
- joint joint_2: origin xyz=0 0 -0.1408 rpy=0 0 0 -> xyz=0 0 -0.1284 rpy=0 0 0
- joint joint_4: axis 1 0 0 -> 0 0 -1; origin xyz=0.1065 0 -0.02 rpy=0 0 0 -> xyz=-0.02 0 -0.1065 rpy=0 0 0
- joint joint_5: origin xyz=0.113 0 0 rpy=0 0 0 -> xyz=0 0 -0.113 rpy=0 0 0
- joint joint_6: axis 0 0 1 -> 1 0 0; origin xyz=0 0 0.021 rpy=0 0 0 -> xyz=0.021 0 0 rpy=0 0 0
- joint left_carriage_joint: child left_carriage -> carriage_left; origin xyz=0.1305 0.022974 -0.021 rpy=0 0 0 -> xyz=-0.021 0.022974 -0.1305 rpy=0 0 0
- joint right_carriage_joint: child right_carriage -> carriage_right; origin xyz=0.1305 -0.022974 -0.021 rpy=0 0 0 -> xyz=-0.021 -0.022974 -0.1305 rpy=0 0 0

Commit message: Fix viper urdf (#9)
* fixed a flipped axis

* used raw values instead of scientific expression for left viper links

* updated left viper inertia and meshes

* updated joints

* used 0 instead of 0.0 and generated urdf

* removed comments from the generated urdf

* nit

---------

Co-authored-by: Luke Schmitt <luke@trossenrobotics.com>

File: urdf/generated/vxai/vxai_right.urdf (robot description, URDF)
Before this commit: robot vxai, 12 links, 11 joints
Links:
- link base_link: mass 1.8716501 -> 1.87165014
- link link_1: mass 1.2811416 -> 1.28114157
- link link_2: mass 1.5816851 -> 1.58168513
- link link_3: mass 1.5152289 -> 1.51522891
Joints:
- joint joint_0: limit lower=-3.14159265358979 upper=3.14159265358979 effort=0 velocity=3.14 -> lower=-1.5707963267948966 upper=3.141592653589793 effort=0 velocity=6.283185307179586
- joint joint_1: axis -1 0 0 -> 1 0 0; limit lower=-3.14159265358979 upper=3.14159265358979 effort=0 velocity=3.14 -> lower=-3.141592653589793 upper=0 effort=0 velocity=6.283185307179586
- joint joint_2: limit lower=-3.14159265358979 upper=3.14159265358979 effort=0 velocity=3.14 -> lower=-1.5707963267948966 upper=1.5707963267948966 effort=0 velocity=6.283185307179586
- joint joint_3: limit lower=-3.14159265358979 upper=3.14159265358979 effort=0 velocity=3.14 -> lower=0 upper=2.356194490192345 effort=0 velocity=6.283185307179586
- joint joint_4: limit lower=-3.14159265358979 upper=3.14159265358979 effort=0 velocity=3.14 -> lower=-1.5707963267948966 upper=1.5707963267948966 effort=0 velocity=6.283185307179586
- joint joint_5: limit lower=-3.14159265358979 upper=3.14159265358979 effort=0 velocity=3.14 -> lower=-0.7853981633974483 upper=0.7853981633974483 effort=0 velocity=6.283185307179586
- joint joint_6: limit lower=-3.14159265358979 upper=3.14159265358979 effort=0 velocity=3.14 -> lower=-1.5707963267948966 upper=1.5707963267948966 effort=0 velocity=6.283185307179586
- joint left_carriage_joint: limit lower=0.0 upper=0.44 effort=0 velocity=1.0 -> lower=0 upper=0.04 effort=0 velocity=0.25
- joint right_carriage_joint: limit lower=0.0 upper=0.44 effort=0 velocity=1.0 -> lower=0 upper=0.04 effort=0 velocity=0.25

File: urdf/macros/_vxai.urdf.xacro (robot description, xacro)
@@ -13,14 +13,14 @@
         <inertial>
           <origin
-            xyz="-2.199e-05 -0.03351643 6.205e-05"
+            xyz="-0.00002199 -0.03351643 0.00006205"
             rpy="0 0 0" />
           <mass
-            value="1.8716501" />
+            value="1.87165014" />
           <inertia
             ixx="0.00209272"
-            ixy="-3.41e-06"
-            ixz="-1e-08"
+            ixy="-0.00000341"
+            ixz="-0.00000001"
             iyy="0.00299206"
-            iyz="-6.8e-07"
+            iyz="-0.00000068"
             izz="0.00207913" />
         </inertial>
@@ -42,76 +42,4 @@
             <mesh
               filename="package://trossen_arm_description/meshes/vxai/base_link_right.stl" />
-          </geometry>
-        </collision>
-      </xacro:if>  <!-- arm_side == right -->
-      <xacro:if value="${arm_side == 'left'}">
-        <!-- <inertial>
-          <origin
-            xyz="-2.199e-05 -0.03351643 6.205e-05"
-            rpy="0 0 0" />
-          <mass
-            value="1.8716501" />
-          <inertia
-            ixx="0.00209272"
-            ixy="-3.41e-06"
-            ixz="-1e-08"
-            iyy="0.00299206"
-            iyz="-6.8e-07"
-            izz="0.00207913" />
-        </inertial>
-        <visual>
-          <origin
-            xyz="0 0 0"
-            rpy="0 0 0" />
-          <geometry>
-            <mesh
-              filename="package://trossen_arm_description/meshes/vxai/base_link_left.stl" />
-          </geometry>
-          <material name="trossen_black"/>
-        </visual>
-        <collision>
-          <origin
-            xyz="0 0 0"
-            rpy="0 0 0" />
-          <geometry>
-            <mesh
-              filename="package://trossen_arm_description/meshes/vxai/base_link_left.stl" />
-          </geometry>
-        </collision> -->
-      </xacro:if>  <!-- arm_side == left -->
-    </link>
-    <link name="${prefix}link_1">
-      <xacro:if value="${arm_side == 'right'}">
-        <inertial>
-          <origin
-            xyz="0.00275058 -0.0574464 -7.47e-05"
-            rpy="0 0 0" />
-          <mass
-            value="1.2811416" />
-          <inertia
-            ixx="0.00180008"
-            ixy="1.517e-05"
-            ixz="4.8e-07"
-            iyy="0.00124234"
-            iyz="-5.23e-06"
-            izz="0.00154695" />
-        </inertial>
-        <visual>
-          <origin
-            xyz="0 0 0"
-            rpy="0 0 0" />
-          <geometry>
-            <mesh
-              filename="package://trossen_arm_description/meshes/vxai/link_1_right.stl" />
-          </geometry>
-          <material name="trossen_black"/>
-        </visual>
-        <collision>
-          <origin
-            xyz="0 0 0"
-            rpy="0 0 0" />
-          <geometry>
-            <mesh
-              filename="package://trossen_arm_description/meshes/vxai/link_1_right.stl" />
           </geometry>
         </collision>
@@ -120,14 +48,51 @@
         <inertial>
           <origin
-            xyz="0.00275058 -0.0574464 -7.47e-05"
+            xyz="-0.00002199 0.03351643 -0.00006205"
             rpy="0 0 0" />
           <mass
-            value="1.2811416" />
+            value="1.87165014" />
+          <inertia
+            ixx="0.00209272"
+            ixy="0.00000341"
+            ixz="0.00000001"
+            iyy="0.00299206"
+            iyz="-0.00000068"
+            izz="0.00207913" />
+        </inertial>
+        <visual>
+          <origin
+            xyz="0 0 0"
+            rpy="0 0 0" />
+          <geometry>
+            <mesh
+              filename="package://trossen_arm_description/meshes/vxai/base_link_left.stl" />
+          </geometry>
+          <material name="trossen_black"/>
+        </visual>
+        <collision>
+          <origin
+            xyz="0 0 0"
+            rpy="0 0 0" />
+          <geometry>
+            <mesh
+              filename="package://trossen_arm_description/meshes/vxai/base_link_left.stl" />
+          </geometry>
+        </collision>
+      </xacro:if>  <!-- arm_side == left -->
+    </link>
+    <link name="${prefix}link_1">
+      <xacro:if value="${arm_side == 'right'}">
+        <inertial>
+          <origin
+            xyz="0.00275058 -0.05744640 -0.00007470"
+            rpy="0 0 0" />
+          <mass
+            value="1.28114157" />
           <inertia
             ixx="0.00180008"
-            ixy="1.517e-05"
-            ixz="4.8e-07"
+            ixy="0.00001517"
+            ixz="0.00000048"
             iyy="0.00124234"
-            iyz="-5.23e-06"
+            iyz="-0.00000523"
             izz="0.00154695" />
         </inertial>
@@ -138,5 +103,5 @@
           <geometry>
             <mesh
-              filename="package://trossen_arm_description/meshes/vxai/link_1_left.stl" />
+              filename="package://trossen_arm_description/meshes/vxai/link_1_right.stl" />
           </geometry>
           <material name="trossen_black"/>
@@ -148,4 +113,39 @@
           <geometry>
             <mesh
+              filename="package://trossen_arm_description/meshes/vxai/link_1_right.stl" />
+          </geometry>
+        </collision>
+      </xacro:if>  <!-- arm_side == right -->
+      <xacro:if value="${arm_side == 'left'}">
+        <inertial>
+          <origin
+            xyz="0.00275057 0.05743620 -0.00006878"
+            rpy="0 0 0" />
+          <mass
+            value="1.28114157" />
+          <inertia
+            ixx="0.00179991"
+            ixy="-0.00001416"
+            ixz="-0.00000010"
+            iyy="0.00124087"
+            iyz="0.00000433"
+            izz="0.00154826" />
+        </inertial>
+        <visual>
+          <origin
+            xyz="0 0 0"
+            rpy="0 0 0" />
+          <geometry>
+            <mesh
+              filename="package://trossen_arm_description/meshes/vxai/link_1_left.stl" />
+          </geometry>
+          <material name="trossen_black"/>
+        </visual>
+        <collision>
+          <origin
+            xyz="0 0 0"
+            rpy="0 0 0" />
+          <geometry>
+            <mesh
               filename="package://trossen_arm_description/meshes/vxai/link_1_left.stl" />
           </geometry>
@@ -154,15 +154,28 @@
     </link>
     <joint name="${prefix}joint_0" type="revolute">
-      <origin
-        xyz="0 -0.068 0"
-        rpy="0 0 0" />
       <parent link="${prefix}base_link" />
       <child link="${prefix}link_1" />
-      <axis xyz="0 -1 0" />
-      <limit
-        effort="0"
-        lower="-3.14159265358979"
-        upper="3.14159265358979"
-        velocity="3.14" />
+      <xacro:if value="${arm_side == 'right'}">
+        <origin
+          xyz="0 -0.068 0"
+          rpy="0 0 0" />
+        <axis xyz="0 -1 0" />
+        <limit
+          effort="0"
+          lower="${-pi / 2}"
+          upper="${pi}"
+          velocity="${2 * pi}" />
+      </xacro:if>  <!-- arm_side == right -->
+      <xacro:if value="${arm_side == 'left'}">
+        <origin
+          xyz="0 0.068 0"
+          rpy="0 0 0" />
+        <axis xyz="0 1 0" />
+        <limit
+          effort="0"
+          lower="${-pi}"
+          upper="${pi / 2}"
+          velocity="${2 * pi}" />
+      </xacro:if>  <!-- arm_side == left -->
     </joint>
     <!-- link 2 universal -->
@@ -170,13 +183,13 @@
       <inertial>
         <origin
-          xyz="4.155e-05 4.77e-06 -0.09223936"
-          rpy="0 0 0" />
-        <mass value="1.5816851" />
-        <inertia
-          ixx="0.0030354"
-          ixy="9.4e-07"
-          ixz="7e-08"
+          xyz="0.00004155 0.00000477 -0.09223936"
+          rpy="0 0 0" />
+        <mass value="1.58168513" />
+        <inertia
+          ixx="0.00303540"
+          ixy="0.00000094"
+          ixz="0.00000007"
           iyy="0.00325708"
-          iyz="5.8e-07"
+          iyz="0.00000058"
           izz="0.00202764" />
       </inertial>
@@ -200,15 +213,27 @@
     </link>
     <joint name="${prefix}joint_1" type="revolute">
-      <origin
-        xyz="0 -0.064 0"
-        rpy="0 0 0" />
       <parent link="${prefix}link_1" />
       <child link="${prefix}link_2" />
-      <axis xyz="-1 0 0" />
-      <limit
-        effort="0"
-        lower="-3.14159265358979"
-        upper="3.14159265358979"
-        velocity="3.14" />
+      <axis xyz="1 0 0" />
+      <xacro:if value="${arm_side == 'right'}">
+        <origin
+          xyz="0 -0.064 0"
+          rpy="0 0 0" />
+        <limit
+          effort="0"
+          lower="${-pi}"
+          upper="0"
+          velocity="${2 * pi}" />
+      </xacro:if>  <!-- arm_side == right -->
+      <xacro:if value="${arm_side == 'left'}">
+        <origin
+          xyz="0 0.064 0"
+          rpy="0 0 0" />
+        <limit
+          effort="0"
+          lower="0"
+          upper="${pi}"
+          velocity="${2 * pi}" />
+      </xacro:if>  <!-- arm_side == left -->
     </joint>
     <!-- link 3 right -->
@@ -220,11 +245,11 @@
             rpy="0 0 0" />
           <mass
-            value="1.5152289" />
+            value="1.51522891" />
           <inertia
             ixx="0.00491722"
-            ixy="1.966e-05"
+            ixy="0.00001966"
             ixz="0.00061652"
             iyy="0.00521379"
-            iyz="-8.813e-05"
+            iyz="-0.00008813"
             izz="0.00131018" />
         </inertial>
@@ -252,15 +277,15 @@
         <inertial>
           <origin
-            xyz="0.01469489 -0.00233198 -0.13174594"
+            xyz="0.01468991 0.00233199 -0.13173731"
             rpy="0 0 0" />
           <mass
-            value="1.5152289" />
+            value="1.51522891" />
           <inertia
-            ixx="0.00491722"
-            ixy="1.966e-05"
-            ixz="0.00061652"
-            iyy="0.00521379"
-            iyz="-8.813e-05"
-            izz="0.00131018" />
+            ixx="0.00491799"
+            ixy="-0.00001908"
+            ixz="0.00061539"
+            iyy="0.00521300"
+            iyz="0.00008711"
+            izz="0.00130863" />
         </inertial>
         <visual>
@@ -294,20 +319,20 @@
       <limit
         effort="0"
-        lower="-3.14159265358979"
-        upper="3.14159265358979"
-        velocity="3.14" />
+        lower="${-pi / 2}"
+        upper="${pi / 2}"
+        velocity="${2 * pi}" />
     </joint>
     <link name="${prefix}link_4">
       <inertial>
         <origin
-          xyz="-0.01788633 0.00011005 -0.0729305"
+          xyz="-0.01788633 0.00011005 -0.07293050"
           rpy="0 0 0" />
         <mass value="0.59839689" />
         <inertia
           ixx="0.00082356"
-          ixy="1.3e-07"
-          ixz="-8.634e-05"
+          ixy="0.00000013"
+          ixz="-0.00008634"
           iyy="0.00069719"
-          iyz="9.3e-07"
+          iyz="0.00000093"
           izz="0.00052102" />
       </inertial>
@@ -336,10 +361,20 @@
       <parent link="${prefix}link_3" />
       <child link="${prefix}link_4" />
-      <axis xyz="0 -1 0" />
-      <limit
-        effort="0"
-        lower="-3.14159265358979"
-        upper="3.14159265358979"
-        velocity="3.14" />
+      <xacro:if value="${arm_side == 'right'}">
+        <axis xyz="0 -1 0" />
+        <limit
+          effort="0"
+          lower="0"
+          upper="${3 * pi / 4}"
+          velocity="${2 * pi}" />
+      </xacro:if>  <!-- arm_side == right -->
+      <xacro:if value="${arm_side == 'left'}">
+        <axis xyz="0 1 0" />
+        <limit
+          effort="0"
+          lower="${-3 * pi / 4}"
+          upper="0"
+          velocity="${2 * pi}" />
+      </xacro:if>  <!-- arm_side == left -->
     </joint>
     <link name="${prefix}link_5">
@@ -350,10 +385,10 @@
         <mass value="0.60644692" />
         <inertia
-          ixx="0.0009455"
-          ixy="3.75e-06"
-          ixz="-7.89e-06"
+          ixx="0.00094550"
+          ixy="0.00000375"
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