Commit message: used 0 instead of 0.0 and generated urdf

File: urdf/generated/vxai/vxai_left.urdf (robot description, URDF)
Before this commit: robot vxai, 12 links, 11 joints
Links:
- link base_link: geometry collision mesh filename=package://trossen_arm_description/meshes/vxai/base_link_lef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; visual mesh filename=package://trossen_arm_description/meshes/vxai/base_link_lef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
- link link_1: geometry collision mesh filename=package://trossen_arm_description/meshes/vxai/link_1_left.s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; visual mesh filename=package://trossen_arm_description/meshes/vxai/link_1_left.s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
- link link_3: geometry collision mesh filename=package://trossen_arm_description/meshes/vxai/link_3_left.s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; visual mesh filename=package://trossen_arm_description/meshes/vxai/link_3_left.s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
Joints:
- joint joint_0: axis 0 -1 0 -> 0 1 0; limit lower=-1.5707963267948966 upper=3.141592653589793 effort=0 velocity=6.283185307179586 -> lower=-3.141592653589793 upper=1.5707963267948966 effort=0 velocity=6.283185307179586; origin xyz=0 -0.068 0 rpy=0 0 0 -> xyz=0 0.068 0 rpy=0 0 0
- joint joint_1: limit lower=-3.141592653589793 upper=0 effort=0 velocity=6.283185307179586 -> lower=0 upper=3.141592653589793 effort=0 velocity=6.283185307179586; origin xyz=0 -0.064 0 rpy=0 0 0 -> xyz=0 0.064 0 rpy=0 0 0
- joint joint_3: axis 0 -1 0 -> 0 1 0; limit lower=0 upper=2.356194490192345 effort=0 velocity=6.283185307179586 -> lower=-2.356194490192345 upper=0 effort=0 velocity=6.283185307179586

File: urdf/macros/_vxai.urdf.xacro (robot description, xacro)
@@ -223,5 +223,5 @@
           effort="0"
           lower="${-pi}"
-          upper="0.0"
+          upper="0"
           velocity="${2 * pi}" />
       </xacro:if>  <!-- arm_side == right -->
@@ -232,5 +232,5 @@
         <limit
           effort="0"
-          lower="0.0"
+          lower="0"
           upper="${pi}"
           velocity="${2 * pi}" />
@@ -365,5 +365,5 @@
         <limit
           effort="0"
-          lower="0.0"
+          lower="0"
           upper="${3 * pi / 4}"
           velocity="${2 * pi}" />
@@ -374,5 +374,5 @@
           effort="0"
           lower="${-3 * pi / 4}"
-          upper="0.0"
+          upper="0"
           velocity="${2 * pi}" />
       </xacro:if>  <!-- arm_side == left -->
@@ -554,5 +554,5 @@
       <limit
         effort="0"
-        lower="0.0"
+        lower="0"
         upper="0.04"
         velocity="0.25" />
@@ -639,5 +639,5 @@
       <limit
         effort="0"
-        lower="0.0"
+        lower="0"
         upper="0.04"
         velocity="0.25" />

Commit message: added ee gripper

File: urdf/generated/vxai/vxai_left.urdf (robot description, URDF)
Before this commit: robot vxai, 12 links, 11 joints
Links:
- added link ee_gripper_link, mass 0.001
Joints:
- added joint ee_gripper: type fixed, parent link_7, child ee_gripper_link, origin xyz=-0.021 0 -0.200062 rpy=0 0 0, axis 1 0 0

File: urdf/generated/vxai/vxai_right.urdf (robot description, URDF)
Before this commit: robot vxai, 12 links, 11 joints
Links:
- added link ee_gripper_link, mass 0.001
Joints:
- added joint ee_gripper: type fixed, parent link_7, child ee_gripper_link, origin xyz=-0.021 0 -0.200062 rpy=0 0 0, axis 1 0 0

File: urdf/macros/_vxai.urdf.xacro (robot description, xacro)
@@ -683,4 +683,24 @@
       <axis xyz="0 0 0" />
     </joint>
+    <joint name="${prefix}ee_gripper" type="fixed">
+      <origin
+        xyz="-0.021 0 -0.200062"
+        rpy="0 0 0" />
+      <parent link="${prefix}link_7" />
+      <child link="${prefix}ee_gripper_link" />
+      <axis xyz="1 0 0" />
+    </joint>
+    <link name="${prefix}ee_gripper_link">
+      <inertial>
+        <mass value="0.001"/>
+        <inertia
+          ixx="0.0001"
+          iyy="0.0001"
+          izz="0.0001"
+          ixy="0"
+          ixz="0"
+          iyz="0"/>
+      </inertial>
+    </link>
   </xacro:macro>  <!-- vxai -->
 </robot>

Commit message: update generated URDFs

File: urdf/generated/vxai/vxai_left.urdf (robot description, URDF)
Before this commit: robot vxai, 13 links, 12 joints
Links:
- link ee_gripper_link: mass 0.001 -> None
Joints:
- joint right_carriage_joint: mimic (none) -> joint=left_carriage_joint

File: urdf/generated/vxai/vxai_right.urdf (robot description, URDF)
Before this commit: robot vxai, 13 links, 12 joints
Links:
- link ee_gripper_link: mass 0.001 -> None
Joints:
- joint right_carriage_joint: mimic (none) -> joint=left_carriage_joint

Commit message: removed axis from fixed joints

File: urdf/generated/vxai/vxai_left.urdf (robot description, URDF)
Before this commit: robot vxai, 13 links, 12 joints
Joints:
- joint ee_gripper: axis 1 0 0 -> (none)
- joint gripper_left_joint: axis 0 0 0 -> (none)
- joint right_gripper_joint: axis 0 0 0 -> (none)

File: urdf/generated/vxai/vxai_right.urdf (robot description, URDF)
Before this commit: robot vxai, 13 links, 12 joints
Joints:
- joint ee_gripper: axis 1 0 0 -> (none)
- joint gripper_left_joint: axis 0 0 0 -> (none)
- joint right_gripper_joint: axis 0 0 0 -> (none)

File: urdf/macros/_vxai.urdf.xacro (robot description, xacro)
@@ -597,5 +597,4 @@
       <parent link="${prefix}carriage_right" />
       <child link="${prefix}gripper_right" />
-      <axis xyz="0 0 0" />
     </joint>
     <link name="${prefix}carriage_left">
@@ -682,5 +681,4 @@
       <parent link="${prefix}carriage_left" />
       <child link="${prefix}gripper_left" />
-      <axis xyz="0 0 0" />
     </joint>
     <joint name="${prefix}ee_gripper" type="fixed">
@@ -690,5 +688,4 @@
       <parent link="${prefix}link_7" />
       <child link="${prefix}ee_gripper_link" />
-      <axis xyz="1 0 0" />
     </joint>
     <link name="${prefix}ee_gripper_link" />

Commit message: updated limits and mesh filename

File: urdf/generated/vxai/vxai_left.urdf (robot description, URDF)
Before this commit: robot vxai, 13 links, 12 joints
Joints:
- joint joint_0: limit lower=-3.141592653589793 upper=1.5707963267948966 effort=0 velocity=6.283185307179586 -> lower=-3.141592653589793 upper=1.5707963267948966 effort=40.0 velocity=6.283185307179586
- joint joint_1: limit lower=0 upper=3.141592653589793 effort=0 velocity=6.283185307179586 -> lower=0 upper=3.141592653589793 effort=20.0 velocity=6.283185307179586
- joint joint_2: limit lower=-1.5707963267948966 upper=1.5707963267948966 effort=0 velocity=6.283185307179586 -> lower=-1.5707963267948966 upper=1.5707963267948966 effort=20.0 velocity=6.283185307179586
- joint joint_3: limit lower=-2.356194490192345 upper=0 effort=0 velocity=6.283185307179586 -> lower=-2.356194490192345 upper=0 effort=20.0 velocity=6.283185307179586
- joint joint_4: limit lower=-1.5707963267948966 upper=1.5707963267948966 effort=0 velocity=6.283185307179586 -> lower=-1.5707963267948966 upper=1.5707963267948966 effort=11.0 velocity=6.283185307179586
- joint joint_5: limit lower=-0.7853981633974483 upper=0.7853981633974483 effort=0 velocity=6.283185307179586 -> lower=-0.7853981633974483 upper=0.7853981633974483 effort=27.0 velocity=6.283185307179586
- joint joint_6: limit lower=-1.5707963267948966 upper=1.5707963267948966 effort=0 velocity=6.283185307179586 -> lower=-1.5707963267948966 upper=1.5707963267948966 effort=7.0 velocity=6.283185307179586
- joint left_carriage_joint: limit lower=0 upper=0.04 effort=0 velocity=0.25 -> lower=0 upper=0.04 effort=100.0 velocity=0.25
- joint right_carriage_joint: limit lower=0 upper=0.04 effort=0 velocity=0.25 -> lower=0 upper=0.04 effort=100.0 velocity=0.25

File: urdf/generated/vxai/vxai_right.urdf (robot description, URDF)
Before this commit: robot vxai, 13 links, 12 joints
Joints:
- joint joint_0: limit lower=-1.5707963267948966 upper=3.141592653589793 effort=0 velocity=6.283185307179586 -> lower=-1.5707963267948966 upper=3.141592653589793 effort=40.0 velocity=6.283185307179586
- joint joint_1: limit lower=-3.141592653589793 upper=0 effort=0 velocity=6.283185307179586 -> lower=-3.141592653589793 upper=0 effort=20.0 velocity=6.283185307179586
- joint joint_2: limit lower=-1.5707963267948966 upper=1.5707963267948966 effort=0 velocity=6.283185307179586 -> lower=-1.5707963267948966 upper=1.5707963267948966 effort=20.0 velocity=6.283185307179586
- joint joint_3: limit lower=0 upper=2.356194490192345 effort=0 velocity=6.283185307179586 -> lower=0 upper=2.356194490192345 effort=20.0 velocity=6.283185307179586
- joint joint_4: limit lower=-1.5707963267948966 upper=1.5707963267948966 effort=0 velocity=6.283185307179586 -> lower=-1.5707963267948966 upper=1.5707963267948966 effort=11.0 velocity=6.283185307179586
- joint joint_5: limit lower=-0.7853981633974483 upper=0.7853981633974483 effort=0 velocity=6.283185307179586 -> lower=-0.7853981633974483 upper=0.7853981633974483 effort=27.0 velocity=6.283185307179586
- joint joint_6: limit lower=-1.5707963267948966 upper=1.5707963267948966 effort=0 velocity=6.283185307179586 -> lower=-1.5707963267948966 upper=1.5707963267948966 effort=7.0 velocity=6.283185307179586
- joint left_carriage_joint: limit lower=0 upper=0.04 effort=0 velocity=0.25 -> lower=0 upper=0.04 effort=100.0 velocity=0.25
- joint right_carriage_joint: limit lower=0 upper=0.04 effort=0 velocity=0.25 -> lower=0 upper=0.04 effort=100.0 velocity=0.25

File: urdf/macros/_vxai.urdf.xacro (robot description, xacro)
@@ -30,6 +30,5 @@
             rpy="0 0 0" />
           <geometry>
-            <mesh
-              filename="package://trossen_arm_description/meshes/vxai/base_link_right.stl" />
+            <mesh filename="${mesh_directory}/base_link_right.stl" />
           </geometry>
           <material name="trossen_black"/>
@@ -40,6 +39,5 @@
             rpy="0 0 0" />
           <geometry>
-            <mesh
-              filename="package://trossen_arm_description/meshes/vxai/base_link_right.stl" />
+            <mesh filename="${mesh_directory}/base_link_right.stl" />
           </geometry>
         </collision>
@@ -65,6 +63,5 @@
             rpy="0 0 0" />
           <geometry>
-            <mesh
-              filename="package://trossen_arm_description/meshes/vxai/base_link_left.stl" />
+            <mesh filename="${mesh_directory}/base_link_left.stl" />
           </geometry>
           <material name="trossen_black"/>
@@ -75,6 +72,5 @@
             rpy="0 0 0" />
           <geometry>
-            <mesh
-              filename="package://trossen_arm_description/meshes/vxai/base_link_left.stl" />
+            <mesh filename="${mesh_directory}/base_link_left.stl" />
           </geometry>
         </collision>
@@ -102,6 +98,5 @@
             rpy="0 0 0" />
           <geometry>
-            <mesh
-              filename="package://trossen_arm_description/meshes/vxai/link_1_right.stl" />
+            <mesh filename="${mesh_directory}/link_1_right.stl" />
           </geometry>
           <material name="trossen_black"/>
@@ -112,6 +107,5 @@
             rpy="0 0 0" />
           <geometry>
-            <mesh
-              filename="package://trossen_arm_description/meshes/vxai/link_1_right.stl" />
+            <mesh filename="${mesh_directory}/link_1_right.stl" />
           </geometry>
         </collision>
@@ -137,6 +131,5 @@
             rpy="0 0 0" />
           <geometry>
-            <mesh
-              filename="package://trossen_arm_description/meshes/vxai/link_1_left.stl" />
+            <mesh filename="${mesh_directory}/link_1_left.stl" />
           </geometry>
           <material name="trossen_black"/>
@@ -147,6 +140,5 @@
             rpy="0 0 0" />
           <geometry>
-            <mesh
-              filename="package://trossen_arm_description/meshes/vxai/link_1_left.stl" />
+            <mesh filename="${mesh_directory}/link_1_left.stl" />
           </geometry>
         </collision>
@@ -162,5 +154,5 @@
         <axis xyz="0 -1 0" />
         <limit
-          effort="0"
+          effort="40.0"
           lower="${-pi / 2}"
           upper="${pi}"
@@ -173,5 +165,5 @@
         <axis xyz="0 1 0" />
         <limit
-          effort="0"
+          effort="40.0"
           lower="${-pi}"
           upper="${pi / 2}"
@@ -199,14 +191,14 @@
           rpy="0 0 0" />
         <geometry>
-          <mesh filename="package://trossen_arm_description/meshes/vxai/link_2.stl" />
-        </geometry>
-        <material name="trossen_black"/>
-      </visual>
-      <collision>
-        <origin
-          xyz="0 0 0"
-          rpy="0 0 0" />
-        <geometry>
-          <mesh filename="package://trossen_arm_description/meshes/vxai/link_2.stl" />
+          <mesh filename="${mesh_directory}/link_2.stl" />
+        </geometry>
+        <material name="trossen_black"/>
+      </visual>
+      <collision>
+        <origin
+          xyz="0 0 0"
+          rpy="0 0 0" />
+        <geometry>
+          <mesh filename="${mesh_directory}/link_2.stl" />
         </geometry>
       </collision>
@@ -221,5 +213,5 @@
           rpy="0 0 0" />
         <limit
-          effort="0"
+          effort="20.0"
           lower="${-pi}"
           upper="0"
@@ -231,5 +223,5 @@
           rpy="0 0 0" />
         <limit
-          effort="0"
+          effort="20.0"
           lower="0"
           upper="${pi}"
@@ -259,6 +251,5 @@
             rpy="0 0 0" />
           <geometry>
-            <mesh
-              filename="package://trossen_arm_description/meshes/vxai/link_3_right.stl" />
+            <mesh filename="${mesh_directory}/link_3_right.stl" />
           </geometry>
           <material name="trossen_black"/>
@@ -269,6 +260,5 @@
             rpy="0 0 0" />
           <geometry>
-            <mesh
-              filename="package://trossen_arm_description/meshes/vxai/link_3_right.stl" />
+            <mesh filename="${mesh_directory}/link_3_right.stl" />
           </geometry>
         </collision>
@@ -294,6 +284,5 @@
             rpy="0 0 0" />
           <geometry>
-            <mesh
-              filename="package://trossen_arm_description/meshes/vxai/link_3_left.stl" />
+            <mesh filename="${mesh_directory}/link_3_left.stl" />
           </geometry>
           <material name="trossen_black"/>
@@ -304,6 +293,5 @@
             rpy="0 0 0" />
           <geometry>
-            <mesh
-              filename="package://trossen_arm_description/meshes/vxai/link_3_left.stl" />
+            <mesh filename="${mesh_directory}/link_3_left.stl" />
           </geometry>
         </collision>
@@ -318,5 +306,5 @@
       <axis xyz="0 0 -1" />
       <limit
-        effort="0"
+        effort="20.0"
         lower="${-pi / 2}"
         upper="${pi / 2}"
@@ -342,14 +330,14 @@
           rpy="0 0 0" />
         <geometry>
-          <mesh filename="package://trossen_arm_description/meshes/vxai/link_4.stl" />
-        </geometry>
-        <material name="trossen_black"/>
-      </visual>
-      <collision>
-        <origin
-          xyz="0 0 0"
-          rpy="0 0 0" />
-        <geometry>
-          <mesh filename="package://trossen_arm_description/meshes/vxai/link_4.stl" />
+          <mesh filename="${mesh_directory}/link_4.stl" />
+        </geometry>
+        <material name="trossen_black"/>
+      </visual>
+      <collision>
+        <origin
+          xyz="0 0 0"
+          rpy="0 0 0" />
+        <geometry>
+          <mesh filename="${mesh_directory}/link_4.stl" />
         </geometry>
       </collision>
@@ -364,5 +352,5 @@
         <axis xyz="0 -1 0" />
         <limit
-          effort="0"
+          effort="20.0"
           lower="0"
           upper="${3 * pi / 4}"
@@ -372,5 +360,5 @@
         <axis xyz="0 1 0" />
         <limit
-          effort="0"
+          effort="20.0"
           lower="${-3 * pi / 4}"
           upper="0"
@@ -397,14 +385,14 @@
           rpy="0 0 0" />
         <geometry>
-          <mesh filename="package://trossen_arm_description/meshes/vxai/link_5.stl" />
-        </geometry>
-        <material name="trossen_black"/>
-      </visual>
-      <collision>
-        <origin
-          xyz="0 0 0"
-          rpy="0 0 0" />
-        <geometry>
-          <mesh filename="package://trossen_arm_description/meshes/vxai/link_5.stl" />
+          <mesh filename="${mesh_directory}/link_5.stl" />
+        </geometry>
+        <material name="trossen_black"/>
+      </visual>
+      <collision>
+        <origin
+          xyz="0 0 0"
+          rpy="0 0 0" />
+        <geometry>
+          <mesh filename="${mesh_directory}/link_5.stl" />
         </geometry>
       </collision>
@@ -418,5 +406,5 @@
       <axis xyz="0 0 -1" />
       <limit
-        effort="0"
+        effort="11.0"
         lower="${-pi / 2}"
         upper="${pi / 2}"
@@ -442,14 +430,14 @@
           rpy="0 0 0" />
         <geometry>
-          <mesh filename="package://trossen_arm_description/meshes/vxai/link_6.stl" />
-        </geometry>
-        <material name="trossen_black"/>
-      </visual>
-      <collision>
-        <origin
-          xyz="0 0 0"
-          rpy="0 0 0" />
-        <geometry>
-          <mesh filename="package://trossen_arm_description/meshes/vxai/link_6.stl" />
+          <mesh filename="${mesh_directory}/link_6.stl" />
+        </geometry>
+        <material name="trossen_black"/>
+      </visual>
+      <collision>
+        <origin
+          xyz="0 0 0"
+          rpy="0 0 0" />
+        <geometry>
+          <mesh filename="${mesh_directory}/link_6.stl" />
         </geometry>
       </collision>
@@ -463,5 +451,5 @@
       <axis xyz="0 1 0" />
       <limit
-        effort="0"
+        effort="27.0"
         lower="${-pi / 4}"
         upper="${pi / 4}"
@@ -487,14 +475,14 @@
           rpy="0 0 0" />
         <geometry>
-          <mesh filename="package://trossen_arm_description/meshes/vxai/link_7.stl" />
-        </geometry>
-        <material name="trossen_black"/>
-      </visual>
-      <collision>
-        <origin
-          xyz="0 0 0"
-          rpy="0 0 0" />
-        <geometry>
-          <mesh filename="package://trossen_arm_description/meshes/vxai/link_7.stl" />
+          <mesh filename="${mesh_directory}/link_7.stl" />
+        </geometry>
+        <material name="trossen_black"/>
+      </visual>
+      <collision>
+        <origin
+          xyz="0 0 0"
+          rpy="0 0 0" />
+        <geometry>
+          <mesh filename="${mesh_directory}/link_7.stl" />
         </geometry>
       </collision>
@@ -508,5 +496,5 @@
       <axis xyz="1 0 0" />
       <limit
-        effort="0"
+        effort="7.0"
         lower="${-pi / 2}"
         upper="${pi / 2}"
@@ -532,14 +520,14 @@
           rpy="0 0 0" />
         <geometry>
-          <mesh filename="package://trossen_arm_description/meshes/vxai/carriage_right.stl" />
-        </geometry>
-        <material name="trossen_black"/>
-      </visual>
-      <collision>
-        <origin
-          xyz="0 0 0"
-          rpy="0 0 0" />
-        <geometry>
-          <mesh filename="package://trossen_arm_description/meshes/vxai/carriage_right.stl" />
+          <mesh filename="${mesh_directory}/carriage_right.stl" />
+        </geometry>
+        <material name="trossen_black"/>
+      </visual>
+      <collision>
+        <origin
+          xyz="0 0 0"
+          rpy="0 0 0" />
+        <geometry>
+          <mesh filename="${mesh_directory}/carriage_right.stl" />
         </geometry>
       </collision>
@@ -554,5 +542,5 @@
       <axis xyz="0 -1 0" />
       <limit
-        effort="0"
+        effort="100.0"
         lower="0"
         upper="0.04"
@@ -578,14 +566,14 @@
           rpy="0 0 0" />
         <geometry>
-          <mesh filename="package://trossen_arm_description/meshes/vxai/gripper_right.stl" />
-        </geometry>
-        <material name="trossen_black"/>
-      </visual>
-      <collision>
-        <origin
-          xyz="0 0 0"
-          rpy="0 0 0" />
-        <geometry>
-          <mesh filename="package://trossen_arm_description/meshes/vxai/gripper_right.stl" />
+          <mesh filename="${mesh_directory}/gripper_right.stl" />
+        </geometry>
+        <material name="trossen_black"/>
+      </visual>
+      <collision>
+        <origin
+          xyz="0 0 0"
+          rpy="0 0 0" />
+        <geometry>
+          <mesh filename="${mesh_directory}/gripper_right.stl" />
         </geometry>
       </collision>
@@ -617,14 +605,14 @@
           rpy="0 0 0" />
         <geometry>
-          <mesh filename="package://trossen_arm_description/meshes/vxai/carriage_left.stl" />
-        </geometry>
-        <material name="trossen_black"/>
-      </visual>
-      <collision>
-        <origin
-          xyz="0 0 0"
-          rpy="0 0 0" />
-        <geometry>
-          <mesh filename="package://trossen_arm_description/meshes/vxai/carriage_left.stl" />
+          <mesh filename="${mesh_directory}/carriage_left.stl" />
+        </geometry>
+        <material name="trossen_black"/>
+      </visual>
+      <collision>
+        <origin
+          xyz="0 0 0"
+          rpy="0 0 0" />
+        <geometry>
+          <mesh filename="${mesh_directory}/carriage_left.stl" />
         </geometry>
       </collision>
@@ -638,5 +626,5 @@
       <axis xyz="0 1 0" />
       <limit
-        effort="0"
+        effort="100.0"
         lower="0"
         upper="0.04"
@@ -662,14 +650,14 @@
           rpy="0 0 0" />
         <geometry>
-          <mesh filename="package://trossen_arm_description/meshes/vxai/gripper_left.stl" />
-        </geometry>
-        <material name="trossen_black"/>
-      </visual>
-      <collision>
-        <origin
-          xyz="0 0 0"
-          rpy="0 0 0" />
-        <geometry>
-          <mesh filename="package://trossen_arm_description/meshes/vxai/gripper_left.stl" />
+          <mesh filename="${mesh_directory}/gripper_left.stl" />
+        </geometry>
+        <material name="trossen_black"/>
+      </visual>
+      <collision>
+        <origin
+          xyz="0 0 0"
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