Commit message: update default pose

File: urdf/macros/_vxai.urdf.xacro (robot description, xacro)
@@ -9,17 +9,18 @@
   <xacro:macro name="vxai" params="variant arm_side:='' prefix:=''">
     <xacro:property name="mesh_directory" value="package://trossen_arm_description/meshes/${robot_model}"/>
+    <!-- base link right -->
     <link name="${prefix}base_link">
       <inertial>
         <origin
-          xyz="-0.00002199 -0.03351643 0.00006205"
-          rpy="0 0 0" />
-        <mass
-          value="1.87165014" />
+          xyz="-2.199e-05 -0.03351643 6.205e-05"
+          rpy="0 0 0" />
+        <mass
+          value="1.8716501" />
         <inertia
           ixx="0.00209272"
-          ixy="-0.00000341"
-          ixz="-0.00000001"
+          ixy="-3.41e-06"
+          ixz="-1e-08"
           iyy="0.00299206"
-          iyz="-0.00000068"
+          iyz="-6.8e-07"
           izz="0.00207913" />
       </inertial>
@@ -30,5 +31,5 @@
         <geometry>
           <mesh
-            filename="package://trossen_arm_description/meshes/vxai/base_link.stl" />
+            filename="package://trossen_arm_description/meshes/vxai/base_link_right.stl" />
         </geometry>
         <material
@@ -44,21 +45,22 @@
         <geometry>
           <mesh
-            filename="package://trossen_arm_description/meshes/vxai/base_link.stl" />
-        </geometry>
-      </collision>
-    </link>
+            filename="package://trossen_arm_description/meshes/vxai/base_link_right.stl" />
+        </geometry>
+      </collision>
+    </link>
+    <!-- link 1 right -->
     <link name="${prefix}link_1">
       <inertial>
         <origin
-          xyz="0.00275058 -0.05744640 -0.00007470"
-          rpy="0 0 0" />
-        <mass
-          value="1.28114157" />
+          xyz="0.00275058 -0.0574464 -7.47e-05"
+          rpy="0 0 0" />
+        <mass
+          value="1.2811416" />
         <inertia
           ixx="0.00180008"
-          ixy="0.00001517"
-          ixz="0.00000048"
+          ixy="1.517e-05"
+          ixz="4.8e-07"
           iyy="0.00124234"
-          iyz="-0.00000523"
+          iyz="-5.23e-06"
           izz="0.00154695" />
       </inertial>
@@ -69,19 +71,19 @@
         <geometry>
           <mesh
-            filename="package://trossen_arm_description/meshes/vxai/link_1.stl" />
-        </geometry>
-        <material
-          name="">
-          <color
-            rgba="0.752941176470588 0.752941176470588 0.752941176470588 1" />
-        </material>
-      </visual>
-      <collision>
-        <origin
-          xyz="0 0 0"
-          rpy="0 0 0" />
-        <geometry>
-          <mesh
-            filename="package://trossen_arm_description/meshes/vxai/link_1.stl" />
+            filename="package://trossen_arm_description/meshes/vxai/link_1_right.stl" />
+        </geometry>
+        <material
+          name="">
+          <color
+            rgba="0.752941176470588 0.752941176470588 0.752941176470588 1" />
+        </material>
+      </visual>
+      <collision>
+        <origin
+          xyz="0 0 0"
+          rpy="0 0 0" />
+        <geometry>
+          <mesh
+            filename="package://trossen_arm_description/meshes/vxai/link_1_right.stl" />
         </geometry>
       </collision>
@@ -105,17 +107,18 @@
         velocity="3.14" />
     </joint>
+    <!-- link 2 universal -->
     <link name="${prefix}link_2">
       <inertial>
         <origin
-          xyz="0.00004155 0.00000477 -0.09223936"
-          rpy="0 0 0" />
-        <mass
-          value="1.58168513" />
-        <inertia
-          ixx="0.00303540"
-          ixy="0.00000094"
-          ixz="0.00000007"
+          xyz="4.155e-05 4.77e-06 -0.09223936"
+          rpy="0 0 0" />
+        <mass
+          value="1.5816851" />
+        <inertia
+          ixx="0.0030354"
+          ixy="9.4e-07"
+          ixz="7e-08"
           iyy="0.00325708"
-          iyz="0.00000058"
+          iyz="5.8e-07"
           izz="0.00202764" />
       </inertial>
@@ -155,5 +158,5 @@
         link="link_2" />
       <axis
-        xyz="1 0 0" />
+        xyz="-1 0 0" />
       <limit
         effort="0"
@@ -162,4 +165,5 @@
         velocity="3.14" />
     </joint>
+    <!-- link 3 right -->
     <link name="${prefix}link_3">
       <inertial>
@@ -168,11 +172,11 @@
           rpy="0 0 0" />
         <mass
-          value="1.51522891" />
+          value="1.5152289" />
         <inertia
           ixx="0.00491722"
-          ixy="0.00001966"
+          ixy="1.966e-05"
           ixz="0.00061652"
           iyy="0.00521379"
-          iyz="-0.00008813"
+          iyz="-8.813e-05"
           izz="0.00131018" />
       </inertial>
@@ -183,19 +187,19 @@
         <geometry>
           <mesh
-            filename="package://trossen_arm_description/meshes/vxai/link_3.stl" />
-        </geometry>
-        <material
-          name="">
-          <color
-            rgba="0.752941176470588 0.752941176470588 0.752941176470588 1" />
-        </material>
-      </visual>
-      <collision>
-        <origin
-          xyz="0 0 0"
-          rpy="0 0 0" />
-        <geometry>
-          <mesh
-            filename="package://trossen_arm_description/meshes/vxai/link_3.stl" />
+            filename="package://trossen_arm_description/meshes/vxai/link_3_right.stl" />
+        </geometry>
+        <material
+          name="">
+          <color
+            rgba="0.752941176470588 0.752941176470588 0.752941176470588 1" />
+        </material>
+      </visual>
+      <collision>
+        <origin
+          xyz="0 0 0"
+          rpy="0 0 0" />
+        <geometry>
+          <mesh
+            filename="package://trossen_arm_description/meshes/vxai/link_3_right.stl" />
         </geometry>
       </collision>
@@ -205,10 +209,10 @@
       type="revolute">
       <origin
-        xyz="0 0 -0.1408"
-        rpy="0 0 0" />
-      <parent
-        link="link_2" />
-      <child
-        link="link_3" />
+        xyz="0 0 -0.1284"
+        rpy="0 0 0" />
+      <parent
+        link="link_2_universal" />
+      <child
+        link="link_3_right" />
       <axis
         xyz="0 0 -1" />
@@ -219,18 +223,19 @@
         velocity="3.14" />
     </joint>
+    <!-- link 4 universal -->
     <link name="${prefix}link_4">
       <inertial>
         <origin
-          xyz="0.07293047 0.00011005 -0.01788634"
+          xyz="-0.01788633 0.00011005 -0.0729305"
           rpy="0 0 0" />
         <mass
           value="0.59839689" />
         <inertia
-          ixx="0.00052102"
-          ixy="-0.00000093"
-          ixz="0.00008634"
+          ixx="0.00082356"
+          ixy="1.3e-07"
+          ixz="-8.634e-05"
           iyy="0.00069719"
-          iyz="0.00000013"
-          izz="0.00082356" />
+          iyz="9.3e-07"
+          izz="0.00052102" />
       </inertial>
       <visual>
@@ -269,5 +274,5 @@
         link="link_4" />
       <axis
-        xyz="0 -1 0" />
+        xyz="0 1 0" />
       <limit
         effort="0"
@@ -276,18 +281,19 @@
         velocity="3.14" />
     </joint>
+    <!-- link 5 universal -->
     <link name="${prefix}link_5">
       <inertial>
         <origin
-          xyz="0.04045078 0.00225112 -0.00011067"
+          xyz="-0.00011067 0.00225112 -0.04045079"
           rpy="0 0 0" />
         <mass
           value="0.60644692" />
         <inertia
-          ixx="0.00066100"
-          ixy="0.00000214"
-          ixz="0.00000789"
+          ixx="0.0009455"
+          ixy="3.75e-06"
+          ixz="-7.89e-06"
           iyy="0.00054664"
-          iyz="0.00000375"
-          izz="0.00094550" />
+          iyz="-2.14e-06"
+          izz="0.000661" />
       </inertial>
       <visual>
@@ -319,5 +325,5 @@
       type="revolute">
       <origin
-        xyz="0.1065 0 -0.02"
+        xyz="-0.02 0 -0.1065"
         rpy="0 0 0" />
       <parent
@@ -326,5 +332,5 @@
         link="link_5" />
       <axis
-        xyz="1 0 0" />
+        xyz="0 0 -1" />
       <limit
         effort="0"
@@ -333,18 +339,19 @@
         velocity="3.14" />
     </joint>
+    <!-- link 6 universal -->
     <link name="${prefix}link_6">
       <inertial>
         <origin
-          xyz="-0.00001797 0.00058070 -0.00058762"
+          xyz="-0.00058762 0.0005807 1.797e-05"
           rpy="0 0 0" />
         <mass
           value="0.38858221" />
         <inertia
-          ixx="0.00031658"
-          ixy="-0.00000008"
-          ixz="-0.00000001"
+          ixx="0.00018958"
+          ixy="-5e-07"
+          ixz="1e-08"
           iyy="0.00026787"
-          iyz="-0.00000050"
-          izz="0.00018958" />
+          iyz="8e-08"
+          izz="0.00031658" />
       </inertial>
       <visual>
@@ -376,5 +383,5 @@
       type="revolute">
       <origin
-        xyz="0.113 0 0"
+        xyz="0 0 -0.113"
         rpy="0 0 0" />
       <parent
@@ -390,18 +397,19 @@
         velocity="3.14" />
     </joint>
+    <!-- link 7 universal -->
     <link name="${prefix}link_7">
       <inertial>
         <origin
-          xyz="0.08476049 -0.00000697 -0.01847211"
+          xyz="-0.01847211 -6.97e-06 -0.08476049"
           rpy="0 0 0" />
         <mass
           value="0.57903811" />
         <inertia
-          ixx="0.00085992"
-          ixy="-0.00000049"
-          ixz="0.00009912"
+          ixx="0.00135277"
+          ixy="-6e-08"
+          ixz="-9.912e-05"
           iyy="0.00077371"
-          iyz="-0.00000006"
-          izz="0.00135277" />
+          iyz="4.9e-07"
+          izz="0.00085992" />
       </inertial>
       <visual>
@@ -433,5 +441,5 @@
       type="revolute">
       <origin
-        xyz="0 0 0.021"
+        xyz="0.021 0 0"
         rpy="0 0 0" />
       <parent
@@ -440,5 +448,5 @@
         link="link_7" />
       <axis
-        xyz="0 0 1" />
+        xyz="1 0 0" />
       <limit
         effort="0"
@@ -450,15 +458,15 @@
       <inertial>
         <origin
-          xyz="-0.00889602 0.00403514 0.00457901"
-          rpy="0 0 0" />
-        <mass
-          value="0.0503631" />
-        <inertia
-          ixx="0.00001736"
-          ixy="0.00000165"
-          ixz="0.00000104"
-          iyy="0.00000591"
-          iyz="-0.00000172"
-          izz="0.00001378" />
+          xyz="0.00457901 0.00403514 0.00889602"
+          rpy="0 0 0" />
+        <mass
+          value="0.05036313" />
+        <inertia
+          ixx="1.378e-05"
+          ixy="-1.72e-06"
+          ixz="-1.04e-06"
+          iyy="5.91e-06"
+          iyz="-1.65e-06"
+          izz="1.736e-05" />
       </inertial>
       <visual>
@@ -490,5 +498,5 @@
       type="prismatic">
       <origin
-        xyz="0.1305 -0.022974 -0.021"
+        xyz="-0.021 -0.022974 -0.1305"
         rpy="0 0 0" />
       <parent
@@ -507,15 +515,15 @@
       <inertial>
         <origin
-          xyz="0.01893989 0.00901216 -0.00215461"
+          xyz="-0.00215452 0.00901223 -0.01893989"
           rpy="0 0 0" />
         <mass
           value="0.03090786" />
         <inertia
-          ixx="0.00000769"
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
Commit message: material

File: urdf/macros/_vxai.urdf.xacro (robot description, xacro)
@@ -33,9 +33,5 @@
             filename="package://trossen_arm_description/meshes/vxai/base_link_right.stl" />
         </geometry>
-        <material
-          name="">
-          <color
-            rgba="0.75294 0.75294 0.75294 1" />
-        </material>
+        <material name="trossen_black"/>
       </visual>
       <collision>
@@ -73,9 +69,5 @@
             filename="package://trossen_arm_description/meshes/vxai/link_1_right.stl" />
         </geometry>
-        <material
-          name="">
-          <color
-            rgba="0.752941176470588 0.752941176470588 0.752941176470588 1" />
-        </material>
+        <material name="trossen_black"/>
       </visual>
       <collision>
@@ -131,9 +123,5 @@
             filename="package://trossen_arm_description/meshes/vxai/link_2.stl" />
         </geometry>
-        <material
-          name="">
-          <color
-            rgba="0.752941176470588 0.752941176470588 0.752941176470588 1" />
-        </material>
+        <material name="trossen_black"/>
       </visual>
       <collision>
@@ -189,9 +177,5 @@
             filename="package://trossen_arm_description/meshes/vxai/link_3_right.stl" />
         </geometry>
-        <material
-          name="">
-          <color
-            rgba="0.752941176470588 0.752941176470588 0.752941176470588 1" />
-        </material>
+        <material name="trossen_black"/>
       </visual>
       <collision>
@@ -247,9 +231,5 @@
             filename="package://trossen_arm_description/meshes/vxai/link_4.stl" />
         </geometry>
-        <material
-          name="">
-          <color
-            rgba="0.752941176470588 0.752941176470588 0.752941176470588 1" />
-        </material>
+        <material name="trossen_black"/>
       </visual>
       <collision>
@@ -305,9 +285,5 @@
             filename="package://trossen_arm_description/meshes/vxai/link_5.stl" />
         </geometry>
-        <material
-          name="">
-          <color
-            rgba="0.752941176470588 0.752941176470588 0.752941176470588 1" />
-        </material>
+        <material name="trossen_black"/>
       </visual>
       <collision>
@@ -363,9 +339,5 @@
             filename="package://trossen_arm_description/meshes/vxai/link_6.stl" />
         </geometry>
-        <material
-          name="">
-          <color
-            rgba="0.752941176470588 0.752941176470588 0.752941176470588 1" />
-        </material>
+        <material name="trossen_black"/>
       </visual>
       <collision>
@@ -421,9 +393,5 @@
             filename="package://trossen_arm_description/meshes/vxai/link_7.stl" />
         </geometry>
-        <material
-          name="">
-          <color
-            rgba="0.752941176470588 0.752941176470588 0.752941176470588 1" />
-        </material>
+        <material name="trossen_black"/>
       </visual>
       <collision>
@@ -478,9 +446,5 @@
             filename="package://trossen_arm_description/meshes/vxai/right_carriage.stl" />
         </geometry>
-        <material
-          name="">
-          <color
-            rgba="0.752941176470588 0.752941176470588 0.752941176470588 1" />
-        </material>
+        <material name="trossen_black"/>
       </visual>
       <collision>
@@ -535,9 +499,5 @@
             filename="package://trossen_arm_description/meshes/vxai/right_follower_finger.stl" />
         </geometry>
-        <material
-          name="">
-          <color
-            rgba="0.752941176470588 0.752941176470588 0.752941176470588 1" />
-        </material>
+        <material name="trossen_black"/>
       </visual>
       <collision>
@@ -587,9 +547,5 @@
             filename="package://trossen_arm_description/meshes/vxai/left_carriage.stl" />
         </geometry>
-        <material
-          name="">
-          <color
-            rgba="0.752941176470588 0.752941176470588 0.752941176470588 1" />
-        </material>
+        <material name="trossen_black"/>
       </visual>
       <collision>
@@ -644,9 +600,5 @@
             filename="package://trossen_arm_description/meshes/vxai/left_follower_finger.stl" />
         </geometry>
-        <material
-          name="">
-          <color
-            rgba="0.752941176470588 0.752941176470588 0.752941176470588 1" />
-        </material>
+        <material name="trossen_black"/>
       </visual>
       <collision>
