Commit message: standardize joint, link names. add placeholder for left

File: urdf/macros/_vxai.urdf.xacro (robot description, xacro)
@@ -9,88 +9,155 @@
   <xacro:macro name="vxai" params="variant arm_side:='' prefix:=''">
     <xacro:property name="mesh_directory" value="package://trossen_arm_description/meshes/${robot_model}"/>
-    <!-- base link right -->
     <link name="${prefix}base_link">
-      <inertial>
-        <origin
-          xyz="-2.199e-05 -0.03351643 6.205e-05"
-          rpy="0 0 0" />
-        <mass
-          value="1.8716501" />
-        <inertia
-          ixx="0.00209272"
-          ixy="-3.41e-06"
-          ixz="-1e-08"
-          iyy="0.00299206"
-          iyz="-6.8e-07"
-          izz="0.00207913" />
-      </inertial>
-      <visual>
-        <origin
-          xyz="0 0 0"
-          rpy="0 0 0" />
-        <geometry>
-          <mesh
-            filename="package://trossen_arm_description/meshes/vxai/base_link_right.stl" />
-        </geometry>
-        <material name="trossen_black"/>
-      </visual>
-      <collision>
-        <origin
-          xyz="0 0 0"
-          rpy="0 0 0" />
-        <geometry>
-          <mesh
-            filename="package://trossen_arm_description/meshes/vxai/base_link_right.stl" />
-        </geometry>
-      </collision>
-    </link>
-    <!-- link 1 right -->
+      <xacro:if value="${arm_side == 'right'}">
+        <inertial>
+          <origin
+            xyz="-2.199e-05 -0.03351643 6.205e-05"
+            rpy="0 0 0" />
+          <mass
+            value="1.8716501" />
+          <inertia
+            ixx="0.00209272"
+            ixy="-3.41e-06"
+            ixz="-1e-08"
+            iyy="0.00299206"
+            iyz="-6.8e-07"
+            izz="0.00207913" />
+        </inertial>
+        <visual>
+          <origin
+            xyz="0 0 0"
+            rpy="0 0 0" />
+          <geometry>
+            <mesh
+              filename="package://trossen_arm_description/meshes/vxai/base_link_right.stl" />
+          </geometry>
+          <material name="trossen_black"/>
+        </visual>
+        <collision>
+          <origin
+            xyz="0 0 0"
+            rpy="0 0 0" />
+          <geometry>
+            <mesh
+              filename="package://trossen_arm_description/meshes/vxai/base_link_right.stl" />
+          </geometry>
+        </collision>
+      </xacro:if>  <!-- arm_side == right -->
+      <xacro:if value="${arm_side == 'left'}">
+        <!-- <inertial>
+          <origin
+            xyz="-2.199e-05 -0.03351643 6.205e-05"
+            rpy="0 0 0" />
+          <mass
+            value="1.8716501" />
+          <inertia
+            ixx="0.00209272"
+            ixy="-3.41e-06"
+            ixz="-1e-08"
+            iyy="0.00299206"
+            iyz="-6.8e-07"
+            izz="0.00207913" />
+        </inertial>
+        <visual>
+          <origin
+            xyz="0 0 0"
+            rpy="0 0 0" />
+          <geometry>
+            <mesh
+              filename="package://trossen_arm_description/meshes/vxai/base_link_left.stl" />
+          </geometry>
+          <material name="trossen_black"/>
+        </visual>
+        <collision>
+          <origin
+            xyz="0 0 0"
+            rpy="0 0 0" />
+          <geometry>
+            <mesh
+              filename="package://trossen_arm_description/meshes/vxai/base_link_left.stl" />
+          </geometry>
+        </collision> -->
+      </xacro:if>  <!-- arm_side == left -->
+    </link>
     <link name="${prefix}link_1">
-      <inertial>
-        <origin
-          xyz="0.00275058 -0.0574464 -7.47e-05"
-          rpy="0 0 0" />
-        <mass
-          value="1.2811416" />
-        <inertia
-          ixx="0.00180008"
-          ixy="1.517e-05"
-          ixz="4.8e-07"
-          iyy="0.00124234"
-          iyz="-5.23e-06"
-          izz="0.00154695" />
-      </inertial>
-      <visual>
-        <origin
-          xyz="0 0 0"
-          rpy="0 0 0" />
-        <geometry>
-          <mesh
-            filename="package://trossen_arm_description/meshes/vxai/link_1_right.stl" />
-        </geometry>
-        <material name="trossen_black"/>
-      </visual>
-      <collision>
-        <origin
-          xyz="0 0 0"
-          rpy="0 0 0" />
-        <geometry>
-          <mesh
-            filename="package://trossen_arm_description/meshes/vxai/link_1_right.stl" />
-        </geometry>
-      </collision>
-    </link>
-    <joint
-      name="joint_0"
-      type="revolute">
+      <xacro:if value="${arm_side == 'right'}">
+        <inertial>
+          <origin
+            xyz="0.00275058 -0.0574464 -7.47e-05"
+            rpy="0 0 0" />
+          <mass
+            value="1.2811416" />
+          <inertia
+            ixx="0.00180008"
+            ixy="1.517e-05"
+            ixz="4.8e-07"
+            iyy="0.00124234"
+            iyz="-5.23e-06"
+            izz="0.00154695" />
+        </inertial>
+        <visual>
+          <origin
+            xyz="0 0 0"
+            rpy="0 0 0" />
+          <geometry>
+            <mesh
+              filename="package://trossen_arm_description/meshes/vxai/link_1_right.stl" />
+          </geometry>
+          <material name="trossen_black"/>
+        </visual>
+        <collision>
+          <origin
+            xyz="0 0 0"
+            rpy="0 0 0" />
+          <geometry>
+            <mesh
+              filename="package://trossen_arm_description/meshes/vxai/link_1_right.stl" />
+          </geometry>
+        </collision>
+      </xacro:if>  <!-- arm_side == right -->
+      <xacro:if value="${arm_side == 'left'}">
+        <inertial>
+          <origin
+            xyz="0.00275058 -0.0574464 -7.47e-05"
+            rpy="0 0 0" />
+          <mass
+            value="1.2811416" />
+          <inertia
+            ixx="0.00180008"
+            ixy="1.517e-05"
+            ixz="4.8e-07"
+            iyy="0.00124234"
+            iyz="-5.23e-06"
+            izz="0.00154695" />
+        </inertial>
+        <visual>
+          <origin
+            xyz="0 0 0"
+            rpy="0 0 0" />
+          <geometry>
+            <mesh
+              filename="package://trossen_arm_description/meshes/vxai/link_1_left.stl" />
+          </geometry>
+          <material name="trossen_black"/>
+        </visual>
+        <collision>
+          <origin
+            xyz="0 0 0"
+            rpy="0 0 0" />
+          <geometry>
+            <mesh
+              filename="package://trossen_arm_description/meshes/vxai/link_1_left.stl" />
+          </geometry>
+        </collision>
+      </xacro:if>  <!-- arm_side == left -->
+    </link>
+    <joint name="${prefix}joint_0" type="revolute">
       <origin
         xyz="0 -0.068 0"
         rpy="0 0 0" />
-      <parent
-        link="base_link" />
-      <child
-        link="link_1" />
-      <axis
-        xyz="0 -1 0" />
+      <parent link="${prefix}base_link" />
+      <child link="${prefix}link_1" />
+      <axis xyz="0 -1 0" />
       <limit
         effort="0"
@@ -105,6 +172,5 @@
           xyz="4.155e-05 4.77e-06 -0.09223936"
           rpy="0 0 0" />
-        <mass
-          value="1.5816851" />
+        <mass value="1.5816851" />
         <inertia
           ixx="0.0030354"
@@ -120,31 +186,24 @@
           rpy="0 0 0" />
         <geometry>
-          <mesh
-            filename="package://trossen_arm_description/meshes/vxai/link_2.stl" />
-        </geometry>
-        <material name="trossen_black"/>
-      </visual>
-      <collision>
-        <origin
-          xyz="0 0 0"
-          rpy="0 0 0" />
-        <geometry>
-          <mesh
-            filename="package://trossen_arm_description/meshes/vxai/link_2.stl" />
-        </geometry>
-      </collision>
-    </link>
-    <joint
-      name="joint_1"
-      type="revolute">
+          <mesh filename="package://trossen_arm_description/meshes/vxai/link_2.stl" />
+        </geometry>
+        <material name="trossen_black"/>
+      </visual>
+      <collision>
+        <origin
+          xyz="0 0 0"
+          rpy="0 0 0" />
+        <geometry>
+          <mesh filename="package://trossen_arm_description/meshes/vxai/link_2.stl" />
+        </geometry>
+      </collision>
+    </link>
+    <joint name="${prefix}joint_1" type="revolute">
       <origin
         xyz="0 -0.064 0"
         rpy="0 0 0" />
-      <parent
-        link="link_1" />
-      <child
-        link="link_2" />
-      <axis
-        xyz="-1 0 0" />
+      <parent link="${prefix}link_1" />
+      <child link="${prefix}link_2" />
+      <axis xyz="-1 0 0" />
       <limit
         effort="0"
@@ -155,50 +214,82 @@
     <!-- link 3 right -->
     <link name="${prefix}link_3">
-      <inertial>
-        <origin
-          xyz="0.01469489 -0.00233198 -0.13174594"
-          rpy="0 0 0" />
-        <mass
-          value="1.5152289" />
-        <inertia
-          ixx="0.00491722"
-          ixy="1.966e-05"
-          ixz="0.00061652"
-          iyy="0.00521379"
-          iyz="-8.813e-05"
-          izz="0.00131018" />
-      </inertial>
-      <visual>
-        <origin
-          xyz="0 0 0"
-          rpy="0 0 0" />
-        <geometry>
-          <mesh
-            filename="package://trossen_arm_description/meshes/vxai/link_3_right.stl" />
-        </geometry>
-        <material name="trossen_black"/>
-      </visual>
-      <collision>
-        <origin
-          xyz="0 0 0"
-          rpy="0 0 0" />
-        <geometry>
-          <mesh
-            filename="package://trossen_arm_description/meshes/vxai/link_3_right.stl" />
-        </geometry>
-      </collision>
-    </link>
-    <joint
-      name="joint_2"
-      type="revolute">
+      <xacro:if value="${arm_side == 'right'}">
+        <inertial>
+          <origin
+            xyz="0.01469489 -0.00233198 -0.13174594"
+            rpy="0 0 0" />
+          <mass
+            value="1.5152289" />
+          <inertia
+            ixx="0.00491722"
+            ixy="1.966e-05"
+            ixz="0.00061652"
+            iyy="0.00521379"
+            iyz="-8.813e-05"
+            izz="0.00131018" />
+        </inertial>
+        <visual>
+          <origin
+            xyz="0 0 0"
+            rpy="0 0 0" />
+          <geometry>
+            <mesh
+              filename="package://trossen_arm_description/meshes/vxai/link_3_right.stl" />
+          </geometry>
+          <material name="trossen_black"/>
+        </visual>
+        <collision>
+          <origin
+            xyz="0 0 0"
+            rpy="0 0 0" />
+          <geometry>
+            <mesh
+              filename="package://trossen_arm_description/meshes/vxai/link_3_right.stl" />
+          </geometry>
+        </collision>
+      </xacro:if>  <!-- arm_side == left -->
+      <xacro:if value="${arm_side == 'left'}">
+        <inertial>
+          <origin
+            xyz="0.01469489 -0.00233198 -0.13174594"
+            rpy="0 0 0" />
+          <mass
+            value="1.5152289" />
+          <inertia
+            ixx="0.00491722"
+            ixy="1.966e-05"
+            ixz="0.00061652"
+            iyy="0.00521379"
+            iyz="-8.813e-05"
+            izz="0.00131018" />
+        </inertial>
+        <visual>
+          <origin
+            xyz="0 0 0"
+            rpy="0 0 0" />
+          <geometry>
+            <mesh
+              filename="package://trossen_arm_description/meshes/vxai/link_3_left.stl" />
+          </geometry>
+          <material name="trossen_black"/>
+        </visual>
+        <collision>
+          <origin
+            xyz="0 0 0"
+            rpy="0 0 0" />
+          <geometry>
+            <mesh
+              filename="package://trossen_arm_description/meshes/vxai/link_3_left.stl" />
+          </geometry>
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
Commit message: fixed a flipped axis

File: urdf/macros/_vxai.urdf.xacro (robot description, xacro)
@@ -205,5 +205,5 @@
       <parent link="${prefix}link_1" />
       <child link="${prefix}link_2" />
-      <axis xyz="-1 0 0" />
+      <axis xyz="1 0 0" />
       <limit
         effort="0"
