Commit message: used raw values instead of scientific expression for left viper links

File: urdf/macros/_vxai.urdf.xacro (robot description, xacro)
@@ -13,4 +13,39 @@
         <inertial>
           <origin
+            xyz="-0.00002199 -0.03351643 0.00006205"
+            rpy="0 0 0" />
+          <mass
+            value="1.87165014" />
+          <inertia
+            ixx="0.00209272"
+            ixy="-0.00000341"
+            ixz="-0.00000001"
+            iyy="0.00299206"
+            iyz="-0.00000068"
+            izz="0.00207913" />
+        </inertial>
+        <visual>
+          <origin
+            xyz="0 0 0"
+            rpy="0 0 0" />
+          <geometry>
+            <mesh
+              filename="package://trossen_arm_description/meshes/vxai/base_link_right.stl" />
+          </geometry>
+          <material name="trossen_black"/>
+        </visual>
+        <collision>
+          <origin
+            xyz="0 0 0"
+            rpy="0 0 0" />
+          <geometry>
+            <mesh
+              filename="package://trossen_arm_description/meshes/vxai/base_link_right.stl" />
+          </geometry>
+        </collision>
+      </xacro:if>  <!-- arm_side == right -->
+      <xacro:if value="${arm_side == 'left'}">
+        <!-- <inertial>
+          <origin
             xyz="-2.199e-05 -0.03351643 6.205e-05"
             rpy="0 0 0" />
@@ -31,5 +66,5 @@
           <geometry>
             <mesh
-              filename="package://trossen_arm_description/meshes/vxai/base_link_right.stl" />
+              filename="package://trossen_arm_description/meshes/vxai/base_link_left.stl" />
           </geometry>
           <material name="trossen_black"/>
@@ -41,46 +76,46 @@
           <geometry>
             <mesh
-              filename="package://trossen_arm_description/meshes/vxai/base_link_right.stl" />
+              filename="package://trossen_arm_description/meshes/vxai/base_link_left.stl" />
+          </geometry>
+        </collision> -->
+      </xacro:if>  <!-- arm_side == left -->
+    </link>
+    <link name="${prefix}link_1">
+      <xacro:if value="${arm_side == 'right'}">
+        <inertial>
+          <origin
+            xyz="0.00275058 -0.05744640 -0.00007470"
+            rpy="0 0 0" />
+          <mass
+            value="1.28114157" />
+          <inertia
+            ixx="0.00180008"
+            ixy="0.00001517"
+            ixz="0.00000048"
+            iyy="0.00124234"
+            iyz="-0.00000523"
+            izz="0.00154695" />
+        </inertial>
+        <visual>
+          <origin
+            xyz="0 0 0"
+            rpy="0 0 0" />
+          <geometry>
+            <mesh
+              filename="package://trossen_arm_description/meshes/vxai/link_1_right.stl" />
+          </geometry>
+          <material name="trossen_black"/>
+        </visual>
+        <collision>
+          <origin
+            xyz="0 0 0"
+            rpy="0 0 0" />
+          <geometry>
+            <mesh
+              filename="package://trossen_arm_description/meshes/vxai/link_1_right.stl" />
           </geometry>
         </collision>
       </xacro:if>  <!-- arm_side == right -->
       <xacro:if value="${arm_side == 'left'}">
-        <!-- <inertial>
-          <origin
-            xyz="-2.199e-05 -0.03351643 6.205e-05"
-            rpy="0 0 0" />
-          <mass
-            value="1.8716501" />
-          <inertia
-            ixx="0.00209272"
-            ixy="-3.41e-06"
-            ixz="-1e-08"
-            iyy="0.00299206"
-            iyz="-6.8e-07"
-            izz="0.00207913" />
-        </inertial>
-        <visual>
-          <origin
-            xyz="0 0 0"
-            rpy="0 0 0" />
-          <geometry>
-            <mesh
-              filename="package://trossen_arm_description/meshes/vxai/base_link_left.stl" />
-          </geometry>
-          <material name="trossen_black"/>
-        </visual>
-        <collision>
-          <origin
-            xyz="0 0 0"
-            rpy="0 0 0" />
-          <geometry>
-            <mesh
-              filename="package://trossen_arm_description/meshes/vxai/base_link_left.stl" />
-          </geometry>
-        </collision> -->
-      </xacro:if>  <!-- arm_side == left -->
-    </link>
-    <link name="${prefix}link_1">
-      <xacro:if value="${arm_side == 'right'}">
         <inertial>
           <origin
@@ -103,5 +138,5 @@
           <geometry>
             <mesh
-              filename="package://trossen_arm_description/meshes/vxai/link_1_right.stl" />
+              filename="package://trossen_arm_description/meshes/vxai/link_1_left.stl" />
           </geometry>
           <material name="trossen_black"/>
@@ -113,22 +148,84 @@
           <geometry>
             <mesh
-              filename="package://trossen_arm_description/meshes/vxai/link_1_right.stl" />
+              filename="package://trossen_arm_description/meshes/vxai/link_1_left.stl" />
           </geometry>
         </collision>
-      </xacro:if>  <!-- arm_side == right -->
-      <xacro:if value="${arm_side == 'left'}">
+      </xacro:if>  <!-- arm_side == left -->
+    </link>
+    <joint name="${prefix}joint_0" type="revolute">
+      <origin
+        xyz="0 -0.068 0"
+        rpy="0 0 0" />
+      <parent link="${prefix}base_link" />
+      <child link="${prefix}link_1" />
+      <axis xyz="0 -1 0" />
+      <limit
+        effort="0"
+        lower="-3.14159265358979"
+        upper="3.14159265358979"
+        velocity="3.14" />
+    </joint>
+    <!-- link 2 universal -->
+    <link name="${prefix}link_2">
+      <inertial>
+        <origin
+            xyz="0.00004155 0.00000477 -0.09223936"
+          rpy="0 0 0" />
+        <mass value="1.58168513" />
+        <inertia
+          ixx="0.00303540"
+          ixy="0.00000094"
+          ixz="0.00000007"
+          iyy="0.00325708"
+          iyz="0.00000058"
+          izz="0.00202764" />
+      </inertial>
+      <visual>
+        <origin
+          xyz="0 0 0"
+          rpy="0 0 0" />
+        <geometry>
+          <mesh filename="package://trossen_arm_description/meshes/vxai/link_2.stl" />
+        </geometry>
+        <material name="trossen_black"/>
+      </visual>
+      <collision>
+        <origin
+          xyz="0 0 0"
+          rpy="0 0 0" />
+        <geometry>
+          <mesh filename="package://trossen_arm_description/meshes/vxai/link_2.stl" />
+        </geometry>
+      </collision>
+    </link>
+    <joint name="${prefix}joint_1" type="revolute">
+      <origin
+        xyz="0 -0.064 0"
+        rpy="0 0 0" />
+      <parent link="${prefix}link_1" />
+      <child link="${prefix}link_2" />
+      <axis xyz="1 0 0" />
+      <limit
+        effort="0"
+        lower="-3.14159265358979"
+        upper="3.14159265358979"
+        velocity="3.14" />
+    </joint>
+    <!-- link 3 right -->
+    <link name="${prefix}link_3">
+      <xacro:if value="${arm_side == 'right'}">
         <inertial>
           <origin
-            xyz="0.00275058 -0.0574464 -7.47e-05"
+            xyz="0.01469489 -0.00233198 -0.13174594"
             rpy="0 0 0" />
           <mass
-            value="1.2811416" />
+            value="1.51522891" />
           <inertia
-            ixx="0.00180008"
-            ixy="1.517e-05"
-            ixz="4.8e-07"
-            iyy="0.00124234"
-            iyz="-5.23e-06"
-            izz="0.00154695" />
+            ixx="0.00491722"
+            ixy="0.00001966"
+            ixz="0.00061652"
+            iyy="0.00521379"
+            iyz="-0.00008813"
+            izz="0.00131018" />
         </inertial>
         <visual>
@@ -138,5 +235,5 @@
           <geometry>
             <mesh
-              filename="package://trossen_arm_description/meshes/vxai/link_1_left.stl" />
+              filename="package://trossen_arm_description/meshes/vxai/link_3_right.stl" />
           </geometry>
           <material name="trossen_black"/>
@@ -148,71 +245,9 @@
           <geometry>
             <mesh
-              filename="package://trossen_arm_description/meshes/vxai/link_1_left.stl" />
+              filename="package://trossen_arm_description/meshes/vxai/link_3_right.stl" />
           </geometry>
         </collision>
       </xacro:if>  <!-- arm_side == left -->
-    </link>
-    <joint name="${prefix}joint_0" type="revolute">
-      <origin
-        xyz="0 -0.068 0"
-        rpy="0 0 0" />
-      <parent link="${prefix}base_link" />
-      <child link="${prefix}link_1" />
-      <axis xyz="0 -1 0" />
-      <limit
-        effort="0"
-        lower="-3.14159265358979"
-        upper="3.14159265358979"
-        velocity="3.14" />
-    </joint>
-    <!-- link 2 universal -->
-    <link name="${prefix}link_2">
-      <inertial>
-        <origin
-          xyz="4.155e-05 4.77e-06 -0.09223936"
-          rpy="0 0 0" />
-        <mass value="1.5816851" />
-        <inertia
-          ixx="0.0030354"
-          ixy="9.4e-07"
-          ixz="7e-08"
-          iyy="0.00325708"
-          iyz="5.8e-07"
-          izz="0.00202764" />
-      </inertial>
-      <visual>
-        <origin
-          xyz="0 0 0"
-          rpy="0 0 0" />
-        <geometry>
-          <mesh filename="package://trossen_arm_description/meshes/vxai/link_2.stl" />
-        </geometry>
-        <material name="trossen_black"/>
-      </visual>
-      <collision>
-        <origin
-          xyz="0 0 0"
-          rpy="0 0 0" />
-        <geometry>
-          <mesh filename="package://trossen_arm_description/meshes/vxai/link_2.stl" />
-        </geometry>
-      </collision>
-    </link>
-    <joint name="${prefix}joint_1" type="revolute">
-      <origin
-        xyz="0 -0.064 0"
-        rpy="0 0 0" />
-      <parent link="${prefix}link_1" />
-      <child link="${prefix}link_2" />
-      <axis xyz="1 0 0" />
-      <limit
-        effort="0"
-        lower="-3.14159265358979"
-        upper="3.14159265358979"
-        velocity="3.14" />
-    </joint>
-    <!-- link 3 right -->
-    <link name="${prefix}link_3">
-      <xacro:if value="${arm_side == 'right'}">
+      <xacro:if value="${arm_side == 'left'}">
         <inertial>
           <origin
@@ -235,5 +270,5 @@
           <geometry>
             <mesh
-              filename="package://trossen_arm_description/meshes/vxai/link_3_right.stl" />
+              filename="package://trossen_arm_description/meshes/vxai/link_3_left.stl" />
           </geometry>
           <material name="trossen_black"/>
@@ -245,39 +280,4 @@
           <geometry>
             <mesh
-              filename="package://trossen_arm_description/meshes/vxai/link_3_right.stl" />
-          </geometry>
-        </collision>
-      </xacro:if>  <!-- arm_side == left -->
-      <xacro:if value="${arm_side == 'left'}">
-        <inertial>
-          <origin
-            xyz="0.01469489 -0.00233198 -0.13174594"
-            rpy="0 0 0" />
-          <mass
-            value="1.5152289" />
-          <inertia
-            ixx="0.00491722"
-            ixy="1.966e-05"
-            ixz="0.00061652"
-            iyy="0.00521379"
-            iyz="-8.813e-05"
-            izz="0.00131018" />
-        </inertial>
-        <visual>
-          <origin
-            xyz="0 0 0"
-            rpy="0 0 0" />
-          <geometry>
-            <mesh
-              filename="package://trossen_arm_description/meshes/vxai/link_3_left.stl" />
-          </geometry>
-          <material name="trossen_black"/>
-        </visual>
-        <collision>
-          <origin
-            xyz="0 0 0"
-            rpy="0 0 0" />
-          <geometry>
-            <mesh
               filename="package://trossen_arm_description/meshes/vxai/link_3_left.stl" />
           </geometry>
@@ -301,13 +301,13 @@
       <inertial>
         <origin
-          xyz="-0.01788633 0.00011005 -0.0729305"
+          xyz="-0.01788633 0.00011005 -0.07293050"
           rpy="0 0 0" />
         <mass value="0.59839689" />
         <inertia
           ixx="0.00082356"
-          ixy="1.3e-07"
-          ixz="-8.634e-05"
+          ixy="0.00000013"
+          ixz="-0.00008634"
           iyy="0.00069719"
-          iyz="9.3e-07"
+          iyz="0.00000093"
           izz="0.00052102" />
       </inertial>
@@ -350,10 +350,10 @@
         <mass value="0.60644692" />
         <inertia
-          ixx="0.0009455"
-          ixy="3.75e-06"
-          ixz="-7.89e-06"
+          ixx="0.00094550"
+          ixy="0.00000375"
+          ixz="-0.00000789"
           iyy="0.00054664"
-          iyz="-2.14e-06"
-          izz="0.000661" />
+          iyz="-0.00000214"
+          izz="0.00066100" />
       </inertial>
       <visual>
@@ -391,13 +391,13 @@
       <inertial>
         <origin
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
Commit message: updated left viper inertia and meshes

File: urdf/macros/_vxai.urdf.xacro (robot description, xacro)
@@ -46,16 +46,16 @@
       </xacro:if>  <!-- arm_side == right -->
       <xacro:if value="${arm_side == 'left'}">
-        <!-- <inertial>
-          <origin
-            xyz="-2.199e-05 -0.03351643 6.205e-05"
+        <inertial>
+          <origin
+            xyz="-0.00002199 0.03351643 -0.00006205"
             rpy="0 0 0" />
           <mass
-            value="1.8716501" />
+            value="1.87165014" />
           <inertia
             ixx="0.00209272"
-            ixy="-3.41e-06"
-            ixz="-1e-08"
+            ixy="0.00000341"
+            ixz="0.00000001"
             iyy="0.00299206"
-            iyz="-6.8e-07"
+            iyz="-0.00000068"
             izz="0.00207913" />
         </inertial>
@@ -78,5 +78,5 @@
               filename="package://trossen_arm_description/meshes/vxai/base_link_left.stl" />
           </geometry>
-        </collision> -->
+        </collision>
       </xacro:if>  <!-- arm_side == left -->
     </link>
@@ -120,15 +120,15 @@
         <inertial>
           <origin
-            xyz="0.00275058 -0.0574464 -7.47e-05"
+            xyz="0.00275057 0.05743620 -0.00006878"
             rpy="0 0 0" />
           <mass
-            value="1.2811416" />
+            value="1.28114157" />
           <inertia
-            ixx="0.00180008"
-            ixy="1.517e-05"
-            ixz="4.8e-07"
-            iyy="0.00124234"
-            iyz="-5.23e-06"
-            izz="0.00154695" />
+            ixx="0.00179991"
+            ixy="-0.00001416"
+            ixz="-0.00000010"
+            iyy="0.00124087"
+            iyz="0.00000433"
+            izz="0.00154826" />
         </inertial>
         <visual>
@@ -252,15 +252,15 @@
         <inertial>
           <origin
-            xyz="0.01469489 -0.00233198 -0.13174594"
+            xyz="0.01468991 0.00233199 -0.13173731"
             rpy="0 0 0" />
           <mass
-            value="1.5152289" />
+            value="1.51522891" />
           <inertia
-            ixx="0.00491722"
-            ixy="1.966e-05"
-            ixz="0.00061652"
-            iyy="0.00521379"
-            iyz="-8.813e-05"
-            izz="0.00131018" />
+            ixx="0.00491799"
+            ixy="-0.00001908"
+            ixz="0.00061539"
+            iyy="0.00521300"
+            iyz="0.00008711"
+            izz="0.00130863" />
         </inertial>
         <visual>

Commit message: updated joints

File: urdf/macros/_vxai.urdf.xacro (robot description, xacro)
@@ -154,15 +154,28 @@
     </link>
     <joint name="${prefix}joint_0" type="revolute">
-      <origin
-        xyz="0 -0.068 0"
-        rpy="0 0 0" />
       <parent link="${prefix}base_link" />
       <child link="${prefix}link_1" />
-      <axis xyz="0 -1 0" />
-      <limit
-        effort="0"
-        lower="-3.14159265358979"
-        upper="3.14159265358979"
-        velocity="3.14" />
+      <xacro:if value="${arm_side == 'right'}">
+        <origin
+          xyz="0 -0.068 0"
+          rpy="0 0 0" />
+        <axis xyz="0 -1 0" />
+        <limit
+          effort="0"
+          lower="${-pi / 2}"
+          upper="${pi}"
+          velocity="${2 * pi}" />
+      </xacro:if>  <!-- arm_side == right -->
+      <xacro:if value="${arm_side == 'left'}">
+        <origin
+          xyz="0 0.068 0"
+          rpy="0 0 0" />
+        <axis xyz="0 1 0" />
+        <limit
+          effort="0"
+          lower="${-pi}"
+          upper="${pi / 2}"
+          velocity="${2 * pi}" />
+      </xacro:if>  <!-- arm_side == left -->
     </joint>
     <!-- link 2 universal -->
@@ -200,15 +213,27 @@
     </link>
     <joint name="${prefix}joint_1" type="revolute">
-      <origin
-        xyz="0 -0.064 0"
-        rpy="0 0 0" />
       <parent link="${prefix}link_1" />
       <child link="${prefix}link_2" />
       <axis xyz="1 0 0" />
-      <limit
-        effort="0"
-        lower="-3.14159265358979"
-        upper="3.14159265358979"
-        velocity="3.14" />
+      <xacro:if value="${arm_side == 'right'}">
+        <origin
+          xyz="0 -0.064 0"
+          rpy="0 0 0" />
+        <limit
+          effort="0"
+          lower="${-pi}"
+          upper="0.0"
+          velocity="${2 * pi}" />
+      </xacro:if>  <!-- arm_side == right -->
+      <xacro:if value="${arm_side == 'left'}">
+        <origin
+          xyz="0 0.064 0"
+          rpy="0 0 0" />
+        <limit
+          effort="0"
+          lower="0.0"
+          upper="${pi}"
+          velocity="${2 * pi}" />
+      </xacro:if>  <!-- arm_side == left -->
     </joint>
     <!-- link 3 right -->
@@ -294,7 +319,7 @@
       <limit
         effort="0"
-        lower="-3.14159265358979"
-        upper="3.14159265358979"
-        velocity="3.14" />
+        lower="${-pi / 2}"
+        upper="${pi / 2}"
+        velocity="${2 * pi}" />
     </joint>
     <link name="${prefix}link_4">
@@ -336,10 +361,20 @@
       <parent link="${prefix}link_3" />
       <child link="${prefix}link_4" />
-      <axis xyz="0 -1 0" />
-      <limit
-        effort="0"
-        lower="-3.14159265358979"
-        upper="3.14159265358979"
-        velocity="3.14" />
+      <xacro:if value="${arm_side == 'right'}">
+        <axis xyz="0 -1 0" />
+        <limit
+          effort="0"
+          lower="0.0"
+          upper="${3 * pi / 4}"
+          velocity="${2 * pi}" />
+      </xacro:if>  <!-- arm_side == right -->
+      <xacro:if value="${arm_side == 'left'}">
+        <axis xyz="0 1 0" />
+        <limit
+          effort="0"
+          lower="${-3 * pi / 4}"
+          upper="0.0"
+          velocity="${2 * pi}" />
+      </xacro:if>  <!-- arm_side == left -->
     </joint>
     <link name="${prefix}link_5">
@@ -384,7 +419,7 @@
       <limit
         effort="0"
-        lower="-3.14159265358979"
-        upper="3.14159265358979"
-        velocity="3.14" />
+        lower="${-pi / 2}"
+        upper="${pi / 2}"
+        velocity="${2 * pi}" />
     </joint>
     <link name="${prefix}link_6">
@@ -429,7 +464,7 @@
       <limit
         effort="0"
-        lower="-3.14159265358979"
-        upper="3.14159265358979"
-        velocity="3.14" />
+        lower="${-pi / 4}"
+        upper="${pi / 4}"
+        velocity="${2 * pi}" />
     </joint>
     <link name="${prefix}link_7">
@@ -474,7 +509,7 @@
       <limit
         effort="0"
-        lower="-3.14159265358979"
-        upper="3.14159265358979"
-        velocity="3.14" />
+        lower="${-pi / 2}"
+        upper="${pi / 2}"
+        velocity="${2 * pi}" />
     </joint>
     <link name="${prefix}carriage_right">
@@ -520,6 +555,6 @@
         effort="0"
         lower="0.0"
-        upper="0.44"
-        velocity="1.0" />
+        upper="0.04"
+        velocity="0.25" />
     </joint>
     <link name="${prefix}gripper_right">
@@ -605,6 +640,6 @@
         effort="0"
         lower="0.0"
-        upper="0.44"
-        velocity="1.0" />
+        upper="0.04"
+        velocity="0.25" />
     </joint>
     <link name="${prefix}gripper_left">

Commit message: Add mimic to carriage joint

File: urdf/macros/_vxai.urdf.xacro (robot description, xacro)
@@ -551,4 +551,5 @@
       <parent link="${prefix}link_7" />
       <child link="${prefix}carriage_right" />
+      <mimic joint="${prefix}left_carriage_joint" />
       <axis xyz="0 -1 0" />
       <limit

Commit message: Remove ee_gripper_link inertial properties

File: urdf/macros/_vxai.urdf.xacro (robot description, xacro)
@@ -692,16 +692,5 @@
       <axis xyz="1 0 0" />
     </joint>
-    <link name="${prefix}ee_gripper_link">
-      <inertial>
-        <mass value="0.001"/>
-        <inertia
-          ixx="0.0001"
-          iyy="0.0001"
-          izz="0.0001"
-          ixy="0"
-          ixz="0"
-          iyz="0"/>
-      </inertial>
-    </link>
+    <link name="${prefix}ee_gripper_link" />
   </xacro:macro>  <!-- vxai -->
 </robot>
