Commit message: updated first pass

File: urdf/macros/_leader.urdf.xacro (robot description, xacro)
@@ -13,15 +13,15 @@
         <inertial>
           <origin
-            xyz="-0.00002199 -0.03351643 0.00006205"
+            xyz="0.00005199 -0.03429087 0.00005295"
             rpy="0 0 0" />
           <mass
-            value="1.87165014" />
+            value="0.37290125" />
           <inertia
-            ixx="0.00209272"
-            ixy="-0.00000341"
-            ixz="-0.00000001"
-            iyy="0.00299206"
-            iyz="-0.00000068"
-            izz="0.00207913" />
+            ixx="0.00034804"
+            ixy="-0.00000039"
+            ixz="-0.00000003"
+            iyy="0.00014057"
+            iyz="-0.00000080"
+            izz="0.00034074" />
         </inertial>
         <visual>
@@ -85,15 +85,15 @@
         <inertial>
           <origin
-            xyz="0.00275058 -0.05744640 -0.00007470"
+            xyz="0.00331378 -0.03460068 -0.00004285"
             rpy="0 0 0" />
           <mass
-            value="1.28114157" />
+            value="0.45236030" />
           <inertia
-            ixx="0.00180008"
-            ixy="0.00001517"
-            ixz="0.00000048"
-            iyy="0.00124234"
-            iyz="-0.00000523"
-            izz="0.00154695" />
+            ixx="0.00018930"
+            ixy="0.00000360"
+            ixz="-0.00000033"
+            iyy="0.00043171"
+            iyz="0.00000000"
+            izz="0.00045089" />
         </inertial>
         <visual>
@@ -158,5 +158,5 @@
       <xacro:if value="${arm_side == 'right'}">
         <origin
-          xyz="0 -0.068 0"
+          xyz="0 -0.05825 0"
           rpy="0 0 0" />
         <axis xyz="0 -1 0" />
@@ -183,14 +183,14 @@
       <inertial>
         <origin
-          xyz="0.00004155 0.00000477 -0.09223936"
-          rpy="0 0 0" />
-        <mass value="1.58168513" />
+          xyz="-0.00000527 0.00001239 -0.08091014"
+          rpy="0 0 0" />
+        <mass value="0.33783172" />
         <inertia
-          ixx="0.00303540"
-          ixy="0.00000094"
-          ixz="0.00000007"
-          iyy="0.00325708"
-          iyz="0.00000058"
-          izz="0.00202764" />
+          ixx="0.00031788"
+          ixy="0.00000004"
+          ixz="-0.00000049"
+          iyy="0.00034942"
+          iyz="-0.00000045"
+          izz="0.00016037" />
       </inertial>
       <visual>
@@ -218,5 +218,5 @@
       <xacro:if value="${arm_side == 'right'}">
         <origin
-          xyz="0 -0.064 0"
+          xyz="0 -0.0365 0"
           rpy="0 0 0" />
         <limit
@@ -242,15 +242,15 @@
         <inertial>
           <origin
-            xyz="0.01469489 -0.00233198 -0.13174594"
+            xyz="0.01706827 0.00212153 -0.16679020"
             rpy="0 0 0" />
           <mass
-            value="1.51522891" />
+            value="0.46940642" />
           <inertia
-            ixx="0.00491722"
-            ixy="0.00001966"
-            ixz="0.00061652"
-            iyy="0.00521379"
-            iyz="-0.00008813"
-            izz="0.00131018" />
+            ixx="0.00182642"
+            ixy="-0.00000341"
+            ixz="0.00015666"
+            iyy="0.00165644"
+            iyz="0.00002673"
+            izz="0.00039819" />
         </inertial>
         <visual>
@@ -312,5 +312,5 @@
     <joint name="${prefix}joint_2" type="revolute">
       <origin
-        xyz="0 0 -0.1284"
+        xyz="0 0 -0.106"
         rpy="0 0 0" />
       <parent link="${prefix}link_2" />
@@ -326,14 +326,14 @@
       <inertial>
         <origin
-          xyz="-0.01788633 0.00011005 -0.07293050"
-          rpy="0 0 0" />
-        <mass value="0.59839689" />
+          xyz="-0.01912502 0.00002771 -0.08994190"
+          rpy="0 0 0" />
+        <mass value="0.19153172" />
         <inertia
-          ixx="0.00082356"
-          ixy="0.00000013"
-          ixz="-0.00008634"
-          iyy="0.00069719"
-          iyz="0.00000093"
-          izz="0.00052102" />
+          ixx="0.00019027"
+          ixy="-0.00000010"
+          ixz="-0.00001489"
+          iyy="0.00015938"
+          iyz="-0.00000047"
+          izz="0.00008565" />
       </inertial>
       <visual>
@@ -357,5 +357,5 @@
     <joint name="${prefix}joint_3" type="revolute">
       <origin
-        xyz="0.02 0 -0.159"
+        xyz="0.02 0 -0.1938"
         rpy="0 0 0" />
       <parent link="${prefix}link_3" />
@@ -381,14 +381,14 @@
       <inertial>
         <origin
-          xyz="-0.00011067 0.00225112 -0.04045079"
-          rpy="0 0 0" />
-        <mass value="0.60644692" />
+          xyz="-0.00025767 0.00302328 -0.03375968"
+          rpy="0 0 0" />
+        <mass value="0.24163171" />
         <inertia
-          ixx="0.00094550"
-          ixy="0.00000375"
-          ixz="-0.00000789"
-          iyy="0.00054664"
-          iyz="-0.00000214"
-          izz="0.00066100" />
+          ixx="0.00022638"
+          ixy="0.00000100"
+          ixz="-0.00000442"
+          iyy="0.00016124"
+          iyz="0.00000725"
+          izz="0.00013726" />
       </inertial>
       <visual>
@@ -412,5 +412,5 @@
     <joint name="${prefix}joint_4" type="revolute">
       <origin
-        xyz="-0.02 0 -0.1065"
+        xyz="-0.02 0 -0.1185"
         rpy="0 0 0" />
       <parent link="${prefix}link_4" />
@@ -426,14 +426,14 @@
       <inertial>
         <origin
-          xyz="-0.00058762 0.00058070 0.00001797"
-          rpy="0 0 0" />
-        <mass value="0.38858221" />
+          xyz="-0.01044529 0.00000910 0.00011242"
+          rpy="0 0 0" />
+        <mass value="0.18731697" />
         <inertia
-          ixx="0.00018958"
-          ixy="-0.00000050"
-          ixz="0.00000001"
-          iyy="0.00026787"
-          iyz="0.00000008"
-          izz="0.00031658" />
+          ixx="0.00006195"
+          ixy="-0.00000001"
+          ixz="-0.00000032"
+          iyy="0.00005051"
+          iyz="0.00000000"
+          izz="0.00006440" />
       </inertial>
       <visual>
@@ -457,5 +457,5 @@
     <joint name="${prefix}joint_5" type="revolute">
       <origin
-        xyz="0 0 -0.113"
+        xyz="0 0 -0.101"
         rpy="0 0 0" />
       <parent link="${prefix}link_5" />
@@ -471,14 +471,14 @@
       <inertial>
         <origin
-          xyz="-0.01847211 -0.00000697 -0.08476049"
-          rpy="0 0 0" />
-        <mass value="0.57903811" />
+          xyz="-0.04169427 0.00058029 -0.06323582"
+          rpy="0 0 0" />
+        <mass value="0.23686287" />
         <inertia
-          ixx="0.00135277"
-          ixy="-0.00000006"
-          ixz="-0.00009912"
-          iyy="0.00077371"
-          iyz="0.00000049"
-          izz="0.00085992" />
+          ixx="0.00019957"
+          ixy="-0.00000203"
+          ixz="0.00016948"
+          iyy="0.00053905"
+          iyz="0.00000192"
+          izz="0.00038760" />
       </inertial>
       <visual>
@@ -502,5 +502,5 @@
     <joint name="${prefix}joint_6" type="revolute">
       <origin
-        xyz="0.021 0 0"
+        xyz="-0.034 0 0"
         rpy="0 0 0" />
       <parent link="${prefix}link_6" />
@@ -513,17 +513,17 @@
         velocity="${2 * pi}" />
     </joint>
-    <link name="${prefix}carriage_right">
+    <link name="link_8">
       <inertial>
         <origin
-          xyz="0.00457901 0.00403514 0.00889602"
-          rpy="0 0 0" />
-        <mass value="0.05036313" />
+          xyz="-0.01502064 0.00191435 0.00656522"
+          rpy="0 0 0" />
+        <mass value="0.00915397" />
         <inertia
-          ixx="0.00001378"
-          ixy="-0.00000172"
-          ixz="-0.00000104"
-          iyy="0.00000591"
-          iyz="-0.00000165"
-          izz="0.00001736" />
+          ixx="0.00000120"
+          ixy="-0.00000021"
+          ixz="0.00000102"
+          iyy="0.00000385"
+          iyz="0.00000011"
+          izz="0.00000284" />
       </inertial>
       <visual>
@@ -532,5 +532,5 @@
           rpy="0 0 0" />
         <geometry>
-          <mesh filename="package://trossen_arm_description/meshes/leader/carriage_right.stl" />
+          <mesh filename="package://trossen_arm_description/meshes/leader/link_8.stl" />
         </geometry>
         <material name="trossen_black"/>
@@ -541,144 +541,20 @@
           rpy="0 0 0" />
         <geometry>
-          <mesh filename="package://trossen_arm_description/meshes/leader/carriage_right.stl" />
+          <mesh filename="package://trossen_arm_description/meshes/leader/link_8.stl" />
         </geometry>
       </collision>
     </link>
-    <joint name="${prefix}right_carriage_joint" type="prismatic">
-      <origin
-        xyz="-0.021 -0.022974 -0.1305"
-        rpy="0 0 0" />
-      <parent link="${prefix}link_7" />
-      <child link="${prefix}carriage_right" />
-      <mimic joint="${prefix}left_carriage_joint" />
-      <axis xyz="0 -1 0" />
-      <limit
-        effort="0"
-        lower="0"
-        upper="0.04"
-        velocity="0.25" />
-    </joint>
-    <link name="${prefix}gripper_right">
-      <inertial>
-        <origin
-          xyz="-0.00215452 0.00901223 -0.01893989"
-          rpy="0 0 0" />
-        <mass value="0.03090786" />
-        <inertia
-          ixx="0.00001184"
-          ixy="0.00000020"
-          ixz="-0.00000029"
-          iyy="0.00001487"
-          iyz="0.00000321"
-          izz="0.00000769" />
-      </inertial>
-      <visual>
-        <origin
-          xyz="0 0 0"
-          rpy="0 0 0" />
-        <geometry>
-          <mesh filename="package://trossen_arm_description/meshes/leader/gripper_right.stl" />
-        </geometry>
-        <material name="trossen_black"/>
-      </visual>
-      <collision>
-        <origin
-          xyz="0 0 0"
-          rpy="0 0 0" />
-        <geometry>
-          <mesh filename="package://trossen_arm_description/meshes/leader/gripper_right.stl" />
-        </geometry>
-      </collision>
-    </link>
-    <joint name="${prefix}right_gripper_joint" type="fixed">
-      <origin
-        xyz="0 0 0"
-        rpy="0 0 0" />
-      <parent link="${prefix}carriage_right" />
-      <child link="${prefix}gripper_right" />
-    </joint>
-    <link name="${prefix}carriage_left">
-      <inertial>
-        <origin
-          xyz="-0.00457908 -0.00403515 0.00889602"
-          rpy="0 0 0" />
-        <mass value="0.05036313" />
-        <inertia
-          ixx="0.00001378"
-          ixy="-0.00000172"
-          ixz="0.00000104"
-          iyy="0.00000591"
-          iyz="0.00000165"
-          izz="0.00001736" />
-      </inertial>
-      <visual>
-        <origin
-          xyz="0 0 0"
-          rpy="0 0 0" />
-        <geometry>
-          <mesh filename="package://trossen_arm_description/meshes/leader/carriage_left.stl" />
-        </geometry>
-        <material name="trossen_black"/>
-      </visual>
-      <collision>
-        <origin
-          xyz="0 0 0"
-          rpy="0 0 0" />
-        <geometry>
-          <mesh filename="package://trossen_arm_description/meshes/leader/carriage_left.stl" />
-        </geometry>
-      </collision>
-    </link>
-    <joint name="${prefix}left_carriage_joint" type="prismatic">
-      <origin
-        xyz="-0.021 0.022974 -0.1305"
-        rpy="0 0 0" />
-      <parent link="${prefix}link_7" />
-      <child link="${prefix}carriage_left" />
+    <joint name="joint_7" type="revolute">
+      <origin
+        xyz="-0.02847106 0.01930000 -0.07900135"
+        rpy="0 0 0" />
+      <parent link="link_7" />
+      <child link="link_8" />
       <axis xyz="0 1 0" />
       <limit
+        lower="-1.5707963267948966"
+        upper="1.5707963267948966"
         effort="0"
-        lower="0"
-        upper="0.04"
-        velocity="0.25" />
-    </joint>
-    <link name="${prefix}gripper_left">
-      <inertial>
-        <origin
-          xyz="-0.00215462 -0.00901217 -0.01893993"
-          rpy="0 0 0" />
-        <mass value="0.03090787" />
-        <inertia
-          ixx="0.00001184"
-          ixy="-0.00000020"
-          ixz="-0.00000029"
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
Commit message: updated leader xacro second pass

File: urdf/macros/_leader.urdf.xacro (robot description, xacro)
@@ -31,5 +31,5 @@
           <geometry>
             <mesh
-              filename="package://trossen_arm_description/meshes/leader/base_link_right.stl" />
+              filename="${mesh_directory}/base_link_right.stl" />
           </geometry>
           <material name="trossen_black"/>
@@ -41,5 +41,5 @@
           <geometry>
             <mesh
-              filename="package://trossen_arm_description/meshes/leader/base_link_right.stl" />
+              filename="${mesh_directory}/base_link_right.stl" />
           </geometry>
         </collision>
@@ -66,5 +66,5 @@
           <geometry>
             <mesh
-              filename="package://trossen_arm_description/meshes/leader/base_link_left.stl" />
+              filename="${mesh_directory}/base_link_left.stl" />
           </geometry>
           <material name="trossen_black"/>
@@ -76,5 +76,5 @@
           <geometry>
             <mesh
-              filename="package://trossen_arm_description/meshes/leader/base_link_left.stl" />
+              filename="${mesh_directory}/base_link_left.stl" />
           </geometry>
         </collision>
@@ -103,5 +103,5 @@
           <geometry>
             <mesh
-              filename="package://trossen_arm_description/meshes/leader/link_1_right.stl" />
+              filename="${mesh_directory}/link_1_right.stl" />
           </geometry>
           <material name="trossen_black"/>
@@ -113,5 +113,5 @@
           <geometry>
             <mesh
-              filename="package://trossen_arm_description/meshes/leader/link_1_right.stl" />
+              filename="${mesh_directory}/link_1_right.stl" />
           </geometry>
         </collision>
@@ -138,5 +138,5 @@
           <geometry>
             <mesh
-              filename="package://trossen_arm_description/meshes/leader/link_1_left.stl" />
+              filename="${mesh_directory}/link_1_left.stl" />
           </geometry>
           <material name="trossen_black"/>
@@ -148,5 +148,5 @@
           <geometry>
             <mesh
-              filename="package://trossen_arm_description/meshes/leader/link_1_left.stl" />
+              filename="${mesh_directory}/link_1_left.stl" />
           </geometry>
         </collision>
@@ -199,5 +199,5 @@
           rpy="0 0 0" />
         <geometry>
-          <mesh filename="package://trossen_arm_description/meshes/leader/link_2.stl" />
+          <mesh filename="${mesh_directory}/link_2.stl" />
         </geometry>
         <material name="trossen_black"/>
@@ -208,5 +208,5 @@
           rpy="0 0 0" />
         <geometry>
-          <mesh filename="package://trossen_arm_description/meshes/leader/link_2.stl" />
+          <mesh filename="${mesh_directory}/link_2.stl" />
         </geometry>
       </collision>
@@ -260,5 +260,5 @@
           <geometry>
             <mesh
-              filename="package://trossen_arm_description/meshes/leader/link_3_right.stl" />
+              filename="${mesh_directory}/link_3_right.stl" />
           </geometry>
           <material name="trossen_black"/>
@@ -270,5 +270,5 @@
           <geometry>
             <mesh
-              filename="package://trossen_arm_description/meshes/leader/link_3_right.stl" />
+              filename="${mesh_directory}/link_3_right.stl" />
           </geometry>
         </collision>
@@ -295,5 +295,5 @@
           <geometry>
             <mesh
-              filename="package://trossen_arm_description/meshes/leader/link_3_left.stl" />
+              filename="${mesh_directory}/link_3_left.stl" />
           </geometry>
           <material name="trossen_black"/>
@@ -305,5 +305,5 @@
           <geometry>
             <mesh
-              filename="package://trossen_arm_description/meshes/leader/link_3_left.stl" />
+              filename="${mesh_directory}/link_3_left.stl" />
           </geometry>
         </collision>
@@ -342,5 +342,5 @@
           rpy="0 0 0" />
         <geometry>
-          <mesh filename="package://trossen_arm_description/meshes/leader/link_4.stl" />
+          <mesh filename="${mesh_directory}/link_4.stl" />
         </geometry>
         <material name="trossen_black"/>
@@ -351,5 +351,5 @@
           rpy="0 0 0" />
         <geometry>
-          <mesh filename="package://trossen_arm_description/meshes/leader/link_4.stl" />
+          <mesh filename="${mesh_directory}/link_4.stl" />
         </geometry>
       </collision>
@@ -397,5 +397,5 @@
           rpy="0 0 0" />
         <geometry>
-          <mesh filename="package://trossen_arm_description/meshes/leader/link_5.stl" />
+          <mesh filename="${mesh_directory}/link_5.stl" />
         </geometry>
         <material name="trossen_black"/>
@@ -406,5 +406,5 @@
           rpy="0 0 0" />
         <geometry>
-          <mesh filename="package://trossen_arm_description/meshes/leader/link_5.stl" />
+          <mesh filename="${mesh_directory}/link_5.stl" />
         </geometry>
       </collision>
@@ -442,5 +442,5 @@
           rpy="0 0 0" />
         <geometry>
-          <mesh filename="package://trossen_arm_description/meshes/leader/link_6.stl" />
+          <mesh filename="${mesh_directory}/link_6.stl" />
         </geometry>
         <material name="trossen_black"/>
@@ -451,5 +451,5 @@
           rpy="0 0 0" />
         <geometry>
-          <mesh filename="package://trossen_arm_description/meshes/leader/link_6.stl" />
+          <mesh filename="${mesh_directory}/link_6.stl" />
         </geometry>
       </collision>
@@ -487,5 +487,5 @@
           rpy="0 0 0" />
         <geometry>
-          <mesh filename="package://trossen_arm_description/meshes/leader/link_7.stl" />
+          <mesh filename="${mesh_directory}/link_7.stl" />
         </geometry>
         <material name="trossen_black"/>
@@ -496,5 +496,5 @@
           rpy="0 0 0" />
         <geometry>
-          <mesh filename="package://trossen_arm_description/meshes/leader/link_7.stl" />
+          <mesh filename="${mesh_directory}/link_7.stl" />
         </geometry>
       </collision>
@@ -532,5 +532,5 @@
           rpy="0 0 0" />
         <geometry>
-          <mesh filename="package://trossen_arm_description/meshes/leader/link_8.stl" />
+          <mesh filename="${mesh_directory}/link_8.stl" />
         </geometry>
         <material name="trossen_black"/>
@@ -541,5 +541,5 @@
           rpy="0 0 0" />
         <geometry>
-          <mesh filename="package://trossen_arm_description/meshes/leader/link_8.stl" />
+          <mesh filename="${mesh_directory}/link_8.stl" />
         </geometry>
       </collision>

Commit message: flipped all y in left

File: urdf/macros/_leader.urdf.xacro (robot description, xacro)
@@ -48,5 +48,5 @@
         <inertial>
           <origin
-            xyz="0.00005199 -0.03429087 0.00005295"
+            xyz="0.00005199 0.03429087 0.00005295"
             rpy="0 0 0" />
           <mass
@@ -54,8 +54,8 @@
           <inertia
             ixx="0.00034804"
-            ixy="-0.00000039"
+            ixy="0.00000039"
             ixz="-0.00000003"
             iyy="0.00014057"
-            iyz="-0.00000080"
+            iyz="0.00000080"
             izz="0.00034074" />
         </inertial>
@@ -120,5 +120,5 @@
         <inertial>
           <origin
-            xyz="0.00331378 -0.03460068 -0.00004285"
+            xyz="0.00331378 0.03460068 -0.00004285"
             rpy="0 0 0" />
           <mass
@@ -126,8 +126,8 @@
           <inertia
             ixx="0.00018930"
-            ixy="0.00000360"
+            ixy="-0.00000360"
             ixz="-0.00000033"
             iyy="0.00043171"
-            iyz="0.00000000"
+            iyz="-0.00000000"
             izz="0.00045089" />
         </inertial>
@@ -169,5 +169,5 @@
       <xacro:if value="${arm_side == 'left'}">
         <origin
-          xyz="0 -0.05825 0"
+          xyz="0 0.05825 0"
           rpy="0 0 0" />
         <axis xyz="0 1 0" />
@@ -228,5 +228,5 @@
       <xacro:if value="${arm_side == 'left'}">
         <origin
-          xyz="0 -0.0365 0"
+          xyz="0 0.0365 0"
           rpy="0 0 0" />
         <limit
@@ -277,5 +277,5 @@
         <inertial>
           <origin
-            xyz="0.01706827 0.00212153 -0.16679020"
+            xyz="0.01706827 -0.00212153 -0.16679020"
             rpy="0 0 0" />
           <mass
@@ -283,8 +283,8 @@
           <inertia
             ixx="0.00182642"
-            ixy="-0.00000341"
+            ixy="0.00000341"
             ixz="0.00015666"
             iyy="0.00165644"
-            iyz="0.00002673"
+            iyz="-0.00002673"
             izz="0.00039819" />
         </inertial>
@@ -546,15 +546,28 @@
     </link>
     <joint name="joint_7" type="revolute">
-      <origin
-        xyz="-0.02847106 0.01930000 -0.07900135"
-        rpy="0 0 0" />
       <parent link="link_7" />
       <child link="link_8" />
-      <axis xyz="0 1 0" />
-      <limit
-        lower="-1.5707963267948966"
-        upper="1.5707963267948966"
-        effort="0"
-        velocity="0" />
+      <xacro:if value="${arm_side == 'right'}">
+        <origin
+          xyz="-0.02847106 0.01930000 -0.07900135"
+          rpy="0 0 0" />
+        <axis xyz="0 1 0" />
+        <limit
+          lower="${-pi / 6}"
+          upper="0"
+          effort="0"
+          velocity="0" />
+      </xacro:if>  <!-- arm_side == right -->
+      <xacro:if value="${arm_side == 'left'}">
+        <origin
+          xyz="-0.02847106 -0.01930000 -0.07900135"
+          rpy="0 0 0" />
+        <axis xyz="0 -1 0" />
+        <limit
+          lower="0"
+          upper="${pi / 6}"
+          effort="0"
+          velocity="0" />
+      </xacro:if>  <!-- arm_side == left -->
     </joint>
     <joint name="${prefix}ee_gripper" type="fixed">
