Commit message: Allow for link prefixes

File: urdf/macros/_wxai.urdf.xacro (robot description, xacro)
@@ -7,5 +7,5 @@
     value="6"
     scope="global"/>
-  <xacro:macro name="wxai" params="variant arm_side use_world_frame base_link_frame">
+  <xacro:macro name="wxai" params="variant arm_side use_world_frame base_link_frame prefix:=''">
     <material name="trossen_black">
       <texture filename="package://trossen_arm_description/meshes/trossen_black.png"/>
@@ -14,5 +14,5 @@
     <xacro:property name="variant"                    value="$(arg variant)"/>
     <xacro:property name="arm_side"                   value="$(arg arm_side)"/>
-    <link name="base_link">
+    <link name="${prefix}base_link">
       <inertial>
         <origin
@@ -46,5 +46,5 @@
       </collision>
     </link>
-    <link name="link_1">
+    <link name="${prefix}link_1">
       <inertial>
         <origin
@@ -91,5 +91,5 @@
         velocity="3.375" />
     </joint>
-    <link name="link_2">
+    <link name="${prefix}link_2">
       <inertial>
         <origin
@@ -136,5 +136,5 @@
         velocity="3.375" />
     </joint>
-    <link name="link_3">
+    <link name="${prefix}link_3">
       <inertial>
         <origin
@@ -181,5 +181,5 @@
         velocity="3.375" />
     </joint>
-    <link name="link_4">
+    <link name="${prefix}link_4">
       <inertial>
         <origin
@@ -226,5 +226,5 @@
         velocity="7.0" />
     </joint>
-    <link name="link_5">
+    <link name="${prefix}link_5">
       <inertial>
         <origin
@@ -271,5 +271,5 @@
         velocity="7.0" />
     </joint>
-    <link name="link_6">
+    <link name="${prefix}link_6">
       <inertial>
         <origin
@@ -316,5 +316,5 @@
         velocity="7.0" />
     </joint>
-    <link name="carriage_right">
+    <link name="${prefix}carriage_right">
       <inertial>
         <origin
@@ -361,5 +361,5 @@
         velocity="0.0875" />
     </joint>
-    <link name="carriage_left">
+    <link name="${prefix}carriage_left">
       <inertial>
         <origin
@@ -407,5 +407,5 @@
     </joint>
     <xacro:if value="${variant == 'follower'}">
-      <link name="camera_mount_d405">
+      <link name="${prefix}camera_mount_d405">
         <inertial>
           <origin
@@ -456,5 +456,5 @@
     <xacro:if value="${variant == 'leader'}">
       <xacro:if value="${arm_side == 'left'}">
-        <link name="handle">
+        <link name="${prefix}handle">
           <inertial>
             <origin
@@ -496,5 +496,5 @@
           <axis xyz="0 0 0" />
         </joint>
-        <link name="leader_finger_left_index">
+        <link name="${prefix}leader_finger_left_index">
           <inertial>
             <origin
@@ -536,5 +536,5 @@
           <axis xyz="0 0 0" />
         </joint>
-        <link name="leader_finger_left_thumb">
+        <link name="${prefix}leader_finger_left_thumb">
           <inertial>
             <origin
@@ -578,5 +578,5 @@
       </xacro:if> <!-- arm_side == 'left' -->
       <xacro:if value="${arm_side == 'right'}">
-        <link name="handle">
+        <link name="${prefix}handle">
           <inertial>
             <origin
@@ -618,5 +618,5 @@
           <axis xyz="0 0 0" />
         </joint>
-        <link name="leader_finger_right_thumb">
+        <link name="${prefix}leader_finger_right_thumb">
           <inertial>
             <origin
@@ -658,5 +658,5 @@
           <axis xyz="0 0 0" />
         </joint>
-        <link name="leader_finger_right_index">
+        <link name="${prefix}leader_finger_right_index">
           <inertial>
             <origin
@@ -701,5 +701,5 @@
     </xacro:if> <!-- variant == 'leader' -->
     <xacro:if value="${variant in ('base', 'follower')}">
-      <link name="gripper_left">
+      <link name="${prefix}gripper_left">
         <inertial>
           <origin
@@ -741,5 +741,5 @@
         <axis xyz="0 0 0" />
       </joint>
-      <link name="gripper_right">
+      <link name="${prefix}gripper_right">
         <inertial>
           <origin
@@ -789,5 +789,5 @@
         <axis xyz="1 0 0" />
       </joint>
-      <link name="ee_gripper_link">
+      <link name="${prefix}ee_gripper_link">
         <inertial>
           <mass value="0.001"/>

Commit message: fix link prefix, material

File: urdf/macros/_wxai.urdf.xacro (robot description, xacro)
@@ -8,7 +8,4 @@
     scope="global"/>
   <xacro:macro name="wxai" params="variant arm_side use_world_frame base_link_frame prefix:=''">
-    <material name="trossen_black">
-      <texture filename="package://trossen_arm_description/meshes/trossen_black.png"/>
-    </material>
     <xacro:property name="mesh_directory"             value="package://trossen_arm_description/meshes/${robot_model}"/>
     <xacro:property name="variant"                    value="$(arg variant)"/>
@@ -78,10 +75,10 @@
       </collision>
     </link>
-    <joint name="joint_0" type="revolute">
+    <joint name="${prefix}joint_0" type="revolute">
       <origin
         xyz="0 0 0.05725"
         rpy="0 0 0" />
-      <parent link="base_link" />
-      <child link="link_1" />
+      <parent link="${prefix}base_link" />
+      <child link="${prefix}link_1" />
       <axis xyz="0 0 1" />
       <limit
@@ -123,10 +120,10 @@
       </collision>
     </link>
-    <joint name="joint_1" type="revolute">
+    <joint name="${prefix}joint_1" type="revolute">
       <origin
         xyz="0.02 0 0.04625"
         rpy="0 0 0" />
-      <parent link="link_1" />
-      <child link="link_2" />
+      <parent link="${prefix}link_1" />
+      <child link="${prefix}link_2" />
       <axis xyz="0 1 0" />
       <limit
@@ -168,10 +165,10 @@
       </collision>
     </link>
-    <joint name="joint_2" type="revolute">
+    <joint name="${prefix}joint_2" type="revolute">
       <origin
         xyz="-0.264 0 0"
         rpy="0 0 0" />
-      <parent link="link_2" />
-      <child link="link_3" />
+      <parent link="${prefix}link_2" />
+      <child link="${prefix}link_3" />
       <axis xyz="0 -1 0" />
       <limit
@@ -213,10 +210,10 @@
       </collision>
     </link>
-    <joint name="joint_3" type="revolute">
+    <joint name="${prefix}joint_3" type="revolute">
       <origin
         xyz="0.245 0 0.06"
         rpy="0 0 0" />
-      <parent link="link_3" />
-      <child link="link_4" />
+      <parent link="${prefix}link_3" />
+      <child link="${prefix}link_4" />
       <axis xyz="0 -1 0" />
       <limit
@@ -258,10 +255,10 @@
       </collision>
     </link>
-    <joint name="joint_4" type="revolute">
+    <joint name="${prefix}joint_4" type="revolute">
       <origin
         xyz="0.06775 0 0.0455"
         rpy="0 0 0" />
-      <parent link="link_4" />
-      <child link="link_5" />
+      <parent link="${prefix}link_4" />
+      <child link="${prefix}link_5" />
       <axis xyz="0 0 -1" />
       <limit
@@ -303,10 +300,10 @@
       </collision>
     </link>
-    <joint name="joint_5" type="revolute">
+    <joint name="${prefix}joint_5" type="revolute">
       <origin
         xyz="0.02895 0 -0.0455"
         rpy="0 0 0" />
-      <parent link="link_5" />
-      <child link="link_6" />
+      <parent link="${prefix}link_5" />
+      <child link="${prefix}link_6" />
       <axis xyz="1 0 0" />
       <limit
@@ -348,10 +345,10 @@
       </collision>
     </link>
-    <joint name="right_carriage_joint" type="prismatic">
+    <joint name="${prefix}right_carriage_joint" type="prismatic">
       <origin
         xyz="0.0865 -0.023 0"
         rpy="0 0 0" />
-      <parent link="link_6" />
-      <child link="carriage_right" />
+      <parent link="${prefix}link_6" />
+      <child link="${prefix}carriage_right" />
       <axis xyz="0 -1 0" />
       <limit
@@ -393,10 +390,10 @@
       </collision>
     </link>
-    <joint name="left_carriage_joint" type="prismatic">
+    <joint name="${prefix}left_carriage_joint" type="prismatic">
       <origin
         xyz="0.0865 0.023 0"
         rpy="0 0 0" />
-      <parent link="link_6" />
-      <child link="carriage_left" />
+      <parent link="${prefix}link_6" />
+      <child link="${prefix}carriage_left" />
       <axis xyz="0 1 0" />
       <limit
@@ -439,10 +436,10 @@
         </collision>
       </link>
-      <joint name="camera_mount_joint" type="fixed">
+      <joint name="${prefix}camera_mount_joint" type="fixed">
         <origin
           xyz="0.012 0 0"
           rpy="0 0 0" />
-        <parent link="link_6" />
-        <child link="camera_mount_d405" />
+        <parent link="${prefix}link_6" />
+        <child link="${prefix}camera_mount_d405" />
         <axis xyz="0 0 0" />
       </joint>
@@ -488,10 +485,10 @@
           </collision>
         </link>
-        <joint name="handle_joint" type="fixed">
+        <joint name="${prefix}handle_joint" type="fixed">
           <origin
             xyz="0.012 0 0"
             rpy="0 0 0" />
-          <parent link="link_6" />
-          <child link="handle" />
+          <parent link="${prefix}link_6" />
+          <child link="${prefix}handle" />
           <axis xyz="0 0 0" />
         </joint>
@@ -528,10 +525,10 @@
           </collision>
         </link>
-        <joint name="left_index_joint" type="fixed">
-          <origin
-            xyz="0 0 0"
-            rpy="0 0 0" />
-          <parent link="carriage_left" />
-          <child link="leader_finger_left_index" />
+        <joint name="${prefix}left_index_joint" type="fixed">
+          <origin
+            xyz="0 0 0"
+            rpy="0 0 0" />
+          <parent link="${prefix}carriage_left" />
+          <child link="${prefix}leader_finger_left_index" />
           <axis xyz="0 0 0" />
         </joint>
@@ -568,10 +565,10 @@
           </collision>
         </link>
-        <joint name="left_thumb_joint" type="fixed">
-          <origin
-            xyz="0 0 0"
-            rpy="0 0 0" />
-          <parent link="carriage_right" />
-          <child link="leader_finger_left_thumb" />
+        <joint name="${prefix}left_thumb_joint" type="fixed">
+          <origin
+            xyz="0 0 0"
+            rpy="0 0 0" />
+          <parent link="${prefix}carriage_right" />
+          <child link="${prefix}leader_finger_left_thumb" />
           <axis xyz="0 0 0" />
         </joint>
@@ -610,10 +607,10 @@
           </collision>
         </link>
-        <joint name="handle_joint" type="fixed">
+        <joint name="${prefix}handle_joint" type="fixed">
           <origin
             xyz="0.012 0 0"
             rpy="0 0 0" />
-          <parent link="link_6" />
-          <child link="handle" />
+          <parent link="${prefix}link_6" />
+          <child link="${prefix}handle" />
           <axis xyz="0 0 0" />
         </joint>
@@ -650,10 +647,10 @@
           </collision>
         </link>
-        <joint name="right_thumb_joint" type="fixed">
-          <origin
-            xyz="0 0 0"
-            rpy="0 0 0" />
-          <parent link="carriage_left" />
-          <child link="leader_finger_right_thumb" />
+        <joint name="${prefix}right_thumb_joint" type="fixed">
+          <origin
+            xyz="0 0 0"
+            rpy="0 0 0" />
+          <parent link="${prefix}carriage_left" />
+          <child link="${prefix}leader_finger_right_thumb" />
           <axis xyz="0 0 0" />
         </joint>
@@ -690,10 +687,10 @@
           </collision>
         </link>
-        <joint name="right_index_joint" type="fixed">
-          <origin
-            xyz="0 0 0"
-            rpy="0 0 0" />
-          <parent link="carriage_right" />
-          <child link="leader_finger_right_index" />
+        <joint name="${prefix}right_index_joint" type="fixed">
+          <origin
+            xyz="0 0 0"
+            rpy="0 0 0" />
+          <parent link="${prefix}carriage_right" />
+          <child link="${prefix}leader_finger_right_index" />
           <axis xyz="0 0 0" />
         </joint>
@@ -733,10 +730,10 @@
         </collision>
       </link>
-      <joint name="left_gripper_joint" type="fixed">
-        <origin
-          xyz="0 0 0"
-          rpy="0 0 0" />
-        <parent link="carriage_left" />
-        <child link="gripper_left" />
+      <joint name="${prefix}left_gripper_joint" type="fixed">
+        <origin
+          xyz="0 0 0"
+          rpy="0 0 0" />
+        <parent link="${prefix}carriage_left" />
+        <child link="${prefix}gripper_left" />
         <axis xyz="0 0 0" />
       </joint>
@@ -773,18 +770,18 @@
         </collision>
       </link>
-      <joint name="right_gripper_joint" type="fixed">
-        <origin
-          xyz="0 0 0"
-          rpy="0 0 0" />
-        <parent link="carriage_right" />
-        <child link="gripper_right" />
+      <joint name="${prefix}right_gripper_joint" type="fixed">
+        <origin
+          xyz="0 0 0"
+          rpy="0 0 0" />
+        <parent link="${prefix}carriage_right" />
+        <child link="${prefix}gripper_right" />
         <axis xyz="0 0 0" />
       </joint>
-      <joint name="ee_gripper" type="fixed">
+      <joint name="${prefix}ee_gripper" type="fixed">
         <origin
           xyz="0.154 0 0"
           rpy="0 0 0" />
-        <parent link="link_6" />
-        <child link="ee_gripper_link" />
+        <parent link="${prefix}link_6" />
+        <child link="${prefix}ee_gripper_link" />
         <axis xyz="1 0 0" />
       </joint>

File: urdf/wxai.urdf.xacro (robot description, xacro)
@@ -15,4 +15,6 @@
   </xacro:if> <!-- use_world_frame -->
   <xacro:include filename="$(find trossen_arm_description)/urdf/macros/_wxai.urdf.xacro" />
+  <xacro:include filename="$(find trossen_arm_description)/urdf/macros/_common.urdf.xacro" />
+  <xacro:trossen_black/>
   <xacro:wxai
     arm_side="$(arg arm_side)"

Commit message: fixes

File: urdf/macros/_wxai.urdf.xacro (robot description, xacro)
@@ -3,12 +3,10 @@
   <xacro:property name="robot_model"
     value="wxai"
-    scope="global"/>
+    scope="local"/>
   <xacro:property name="dof"
     value="6"
-    scope="global"/>
-  <xacro:macro name="wxai" params="variant arm_side use_world_frame base_link_frame prefix:=''">
+    scope="local"/>
+  <xacro:macro name="wxai" params="variant arm_side base_link_frame prefix:=''">
     <xacro:property name="mesh_directory"             value="package://trossen_arm_description/meshes/${robot_model}"/>
-    <xacro:property name="variant"                    value="$(arg variant)"/>
-    <xacro:property name="arm_side"                   value="$(arg arm_side)"/>
     <link name="${prefix}base_link">
       <inertial>

File: urdf/wxai.urdf.xacro (robot description, xacro)
@@ -19,5 +19,4 @@
   <xacro:wxai
     arm_side="$(arg arm_side)"
-    use_world_frame="$(arg use_world_frame)"
     base_link_frame="$(arg base_link_frame)"
     variant="$(arg variant)"/>

Commit message: fixes

File: urdf/macros/_wxai.urdf.xacro (robot description, xacro)
@@ -7,5 +7,5 @@
     value="6"
     scope="local"/>
-  <xacro:macro name="wxai" params="variant arm_side base_link_frame prefix:=''">
+  <xacro:macro name="wxai" params="variant arm_side:='' prefix:=''">
     <xacro:property name="mesh_directory"             value="package://trossen_arm_description/meshes/${robot_model}"/>
     <link name="${prefix}base_link">

File: urdf/wxai.urdf.xacro (robot description, xacro)
@@ -19,5 +19,4 @@
   <xacro:wxai
     arm_side="$(arg arm_side)"
-    base_link_frame="$(arg base_link_frame)"
     variant="$(arg variant)"/>
 </robot>

Commit message: Add mobile_ai

File: urdf/macros/_wxai.urdf.xacro (robot description, xacro)
@@ -8,5 +8,5 @@
     scope="local"/>
   <xacro:macro name="wxai" params="variant arm_side:='' prefix:=''">
-    <xacro:property name="mesh_directory"             value="package://trossen_arm_description/meshes/${robot_model}"/>
+    <xacro:property name="mesh_directory" value="package://trossen_arm_description/meshes/${robot_model}"/>
     <link name="${prefix}base_link">
       <inertial>
@@ -443,5 +443,8 @@
       </joint>
       <xacro:include filename="$(find trossen_arm_description)/urdf/peripherals/rs_d405.urdf.xacro" />
-      <xacro:sensor_d405 parent="camera_mount_d405" use_nominal_extrinsics="true">
+      <xacro:sensor_d405
+        name="${prefix}camera"
+        parent="${prefix}camera_mount_d405"
+        use_nominal_extrinsics="true">
         <origin
           xyz="0.02927207801 0 0.03824951197"
@@ -784,16 +787,5 @@
         <axis xyz="1 0 0" />
       </joint>
-      <link name="${prefix}ee_gripper_link">
-        <inertial>
-          <mass value="0.001"/>
-          <inertia
-            ixx="0.0001"
-            iyy="0.0001"
-            izz="0.0001"
-            ixy="0"
-            ixz="0"
-            iyz="0"/>
-        </inertial>
-      </link>
+      <link name="${prefix}ee_gripper_link" />
     </xacro:if> <!-- variant in ('base', 'follower') -->
   </xacro:macro>  <!-- wxai -->

Commit message: Add ros2_control

File: urdf/macros/_wxai.urdf.xacro (robot description, xacro)
@@ -7,6 +7,11 @@
     value="6"
     scope="local"/>
-  <xacro:macro name="wxai" params="variant arm_side:='' prefix:=''">
+  <xacro:macro name="wxai" params="variant arm_side:='' prefix:='' use_fake_hardware:=false">
     <xacro:property name="mesh_directory"             value="package://trossen_arm_description/meshes/${robot_model}"/>
+    <xacro:include filename="$(find trossen_arm_description)/urdf/macros/_wxai.ros2_control.xacro"/>
+    <xacro:wxai_ros2_control
+      use_fake_hardware="${use_fake_hardware}"
+      prefix="${prefix}"
+      ip_address="192.168.1.2"/>  <!-- TODO(lukeschmitt-tr): pass this -->
     <link name="${prefix}base_link">
       <inertial>

Commit message: Add ros2_control

File: urdf/macros/_wxai.urdf.xacro (robot description, xacro)
@@ -7,6 +7,11 @@
     value="6"
     scope="local"/>
-  <xacro:macro name="wxai" params="variant arm_side:='' prefix:=''">
+  <xacro:macro name="wxai" params="variant arm_side:='' prefix:='' use_fake_hardware:=false">
     <xacro:property name="mesh_directory" value="package://trossen_arm_description/meshes/${robot_model}"/>
+    <xacro:include filename="$(find trossen_arm_description)/urdf/macros/_wxai.ros2_control.xacro"/>
+    <xacro:wxai_ros2_control
+      use_fake_hardware="${use_fake_hardware}"
+      prefix="${prefix}"
+      ip_address="192.168.1.2"/>  <!-- TODO(lukeschmitt-tr): pass this -->
     <link name="${prefix}base_link">
       <inertial>

File: urdf/wxai.urdf.xacro (robot description, xacro)
@@ -4,4 +4,5 @@
   <xacro:arg name="arm_side"                        default=""/>          <!-- '', 'left', 'right' -->
   <xacro:arg name="use_world_frame"                 default="false"/>     <!-- 'true', 'false' -->
+  <xacro:arg name="use_fake_hardware"               default="false"/>     <!-- 'true', 'false' -->
   <xacro:arg name="base_link_frame"                 default="base_link"/>
   <xacro:if value="$(arg use_world_frame)">
@@ -19,4 +20,5 @@
   <xacro:wxai
     arm_side="$(arg arm_side)"
-    variant="$(arg variant)"/>
+    variant="$(arg variant)"
+    use_fake_hardware="$(arg use_fake_hardware)"/>
 </robot>

Commit message: add mimic tag to carriage joint

File: urdf/macros/_wxai.urdf.xacro (robot description, xacro)
@@ -349,4 +349,5 @@
       <parent link="${prefix}link_6" />
       <child link="${prefix}carriage_right" />
+      <mimic joint="${prefix}left_carriage_joint" />
       <axis xyz="0 -1 0" />
       <limit

Commit message: Add ros2_control macros to wxai (#16)
* Add ros2_control

* revise ros2_control macro

* moveit works

* use_fake_hardware -> ros2_control_hardware_type

* explicitly define gripper joints

* add initial states for mock hardware

* Fix real hardware condition

* use carriage instead of gripper joint

* right carriage doesn't have cmd interface

* Remove unused right carriage joint

* Pass IP address to wxai ros2_control macro

* remove unused update_period param

* Cleanup

* format

* standard ordering of macro args

* Remove defaults from macro args

https://github.com/TrossenRobotics/trossen_arm_description/pull/16#discussion_r2172889273

File: urdf/macros/_wxai.urdf.xacro (robot description, xacro)
@@ -7,6 +7,11 @@
     value="6"
     scope="local"/>
-  <xacro:macro name="wxai" params="variant arm_side:='' prefix:=''">
+  <xacro:macro name="wxai" params="variant arm_side:='' prefix:='' ros2_control_hardware_type ip_address">
     <xacro:property name="mesh_directory" value="package://trossen_arm_description/meshes/${robot_model}"/>
+    <xacro:include filename="$(find trossen_arm_description)/urdf/macros/_wxai.ros2_control.xacro"/>
+    <xacro:wxai_ros2_control
+      prefix="${prefix}"
+      ip_address="${ip_address}"
+      ros2_control_hardware_type="${ros2_control_hardware_type}"/>
     <link name="${prefix}base_link">
       <inertial>

File: urdf/wxai.urdf.xacro (robot description, xacro)
@@ -1,7 +1,9 @@
 <?xml version="1.0" encoding="utf-8"?>
 <robot name="wxai" xmlns:xacro="http://ros.org/wiki/xacro">
-  <xacro:arg name="variant"                         default="base"/>      <!-- 'base', 'leader', 'follower' -->
-  <xacro:arg name="arm_side"                        default=""/>          <!-- '', 'left', 'right' -->
-  <xacro:arg name="use_world_frame"                 default="false"/>     <!-- 'true', 'false' -->
+  <xacro:arg name="variant"                         default="base"/>        <!-- 'base', 'leader', 'follower' -->
+  <xacro:arg name="arm_side"                        default=""/>            <!-- '', 'left', 'right' -->
+  <xacro:arg name="use_world_frame"                 default="false"/>       <!-- 'true', 'false' -->
+  <xacro:arg name="ros2_control_hardware_type"      default="real"/>        <!-- 'real', 'mock_components' -->
+  <xacro:arg name="ip_address"                      default="192.168.1.2"/>
   <xacro:arg name="base_link_frame"                 default="base_link"/>
   <xacro:if value="$(arg use_world_frame)">
@@ -18,5 +20,7 @@
   <xacro:trossen_black/>
   <xacro:wxai
+    variant="$(arg variant)"
     arm_side="$(arg arm_side)"
-    variant="$(arg variant)"/>
+    ros2_control_hardware_type="$(arg ros2_control_hardware_type)"
+    ip_address="$(arg ip_address)"/>
 </robot>
