Commit message: use_fake_hardware -> ros2_control_hardware_type

File: urdf/macros/_wxai.ros2_control.xacro (robot description, xacro)
@@ -15,16 +15,17 @@
     </joint>
   </xacro:macro>
-  <xacro:macro name="wxai_ros2_control" params="prefix ip_address use_fake_hardware">
+  <xacro:macro name="wxai_ros2_control" params="prefix ip_address ros2_control_hardware_type">
     <ros2_control name="TrossenArmHardwareInterface" type="system">
       <hardware>
-        <xacro:if value="${use_fake_hardware}">
+        <xacro:if value="${ros2_control_hardware_type == 'mock_components'}">
           <plugin>fake_components/GenericSystem</plugin>
-        </xacro:if>  <!-- use_fake_hardware -->
-        <xacro:unless value="${use_fake_hardware}">
+          <!-- <plugin>mock_components/GenericSystem</plugin> -->
+        </xacro:if>  <!-- ros2_control_hardware_type == 'mock_components' -->
+        <xacro:unless value="${ros2_control_hardware_type == 'real'}">
           <plugin>trossen_arm_hardware/TrossenArmHardwareInterface</plugin>
           <param name="robot_model">0</param>        <!-- 0: wxai_v0 -->
           <param name="ip_address">${ip_address}</param>
           <param name="update_period">0.1</param>
-        </xacro:unless>  <!-- use_fake_hardware -->
+        </xacro:unless>  <!-- ros2_control_hardware_type == 'real' -->
       </hardware>
       <xacro:ros2_control_joint name="${prefix}joint_0"/>

File: urdf/macros/_wxai.urdf.xacro (robot description, xacro)
@@ -7,9 +7,9 @@
     value="6"
     scope="local"/>
-  <xacro:macro name="wxai" params="variant arm_side:='' prefix:='' use_fake_hardware:=false">
+  <xacro:macro name="wxai" params="variant arm_side:='' prefix:='' ros2_control_hardware_type:='real'">
     <xacro:property name="mesh_directory" value="package://trossen_arm_description/meshes/${robot_model}"/>
     <xacro:include filename="$(find trossen_arm_description)/urdf/macros/_wxai.ros2_control.xacro"/>
     <xacro:wxai_ros2_control
-      use_fake_hardware="${use_fake_hardware}"
+      ros2_control_hardware_type="${ros2_control_hardware_type}"
       prefix="${prefix}"
       ip_address="192.168.1.2"/>  <!-- TODO(lukeschmitt-tr): pass this -->

File: urdf/wxai.urdf.xacro (robot description, xacro)
@@ -4,5 +4,5 @@
   <xacro:arg name="arm_side"                        default=""/>          <!-- '', 'left', 'right' -->
   <xacro:arg name="use_world_frame"                 default="false"/>     <!-- 'true', 'false' -->
-  <xacro:arg name="use_fake_hardware"               default="false"/>     <!-- 'true', 'false' -->
+  <xacro:arg name="ros2_control_hardware_type"      default="real"/>      <!-- 'real', 'mock_components' -->
   <xacro:arg name="base_link_frame"                 default="base_link"/>
   <xacro:if value="$(arg use_world_frame)">
@@ -21,4 +21,4 @@
     arm_side="$(arg arm_side)"
     variant="$(arg variant)"
-    use_fake_hardware="$(arg use_fake_hardware)"/>
+    ros2_control_hardware_type="$(arg ros2_control_hardware_type)"/>
 </robot>

Commit message: explicitly define gripper joints

File: urdf/macros/_wxai.ros2_control.xacro (robot description, xacro)
@@ -35,6 +35,20 @@
       <xacro:ros2_control_joint name="${prefix}joint_4"/>
       <xacro:ros2_control_joint name="${prefix}joint_5"/>
-      <xacro:ros2_control_joint name="${prefix}left_gripper_joint"/>
-      <xacro:ros2_control_joint name="${prefix}right_gripper_joint"/>
+      <joint name="${prefix}left_gripper_joint">
+          <command_interface name="position" />
+          <state_interface name="position">
+            <param name="initial_value">0.0</param>
+          </state_interface>
+          <state_interface name="velocity"/>
+      </joint>
+      <joint name="${prefix}right_gripper_joint">
+          <param name="mimic">${prefix}left_gripper_joint</param>
+          <param name="multiplier">1</param>
+          <command_interface name="position" />
+          <state_interface name="position">
+            <param name="initial_value">0.0</param>
+          </state_interface>
+          <state_interface name="velocity"/>
+      </joint>
     </ros2_control>
   </xacro:macro>

Commit message: joint name changes

File: urdf/macros/_wxai.ros2_control.xacro (robot description, xacro)
@@ -35,5 +35,5 @@
       <xacro:ros2_control_joint name="${prefix}joint_4"/>
       <xacro:ros2_control_joint name="${prefix}joint_5"/>
-      <joint name="${prefix}left_gripper_joint">
+      <joint name="${prefix}left_carriage_joint">
           <command_interface name="position" />
           <state_interface name="position">
@@ -47,6 +47,6 @@
           </state_interface>
       </joint>
-      <joint name="${prefix}right_gripper_joint">
-          <param name="mimic">${prefix}left_gripper_joint</param>
+      <!-- <joint name="${prefix}right_carriage_joint">
+          <param name="mimic">${prefix}left_carriage_joint</param>
           <param name="multiplier">1</param>
           <command_interface name="position" />
@@ -60,5 +60,5 @@
             <param name="initial_value">0.0</param>
           </state_interface>
-      </joint>
+      </joint> -->
     </ros2_control>
   </xacro:macro>

Commit message: use carriage instead of gripper joint

File: urdf/macros/_wxai.ros2_control.xacro (robot description, xacro)
@@ -35,5 +35,5 @@
       <xacro:ros2_control_joint name="${prefix}joint_4"/>
       <xacro:ros2_control_joint name="${prefix}joint_5"/>
-      <joint name="${prefix}left_gripper_joint">
+      <joint name="${prefix}left_carriage_joint">
           <command_interface name="position" />
           <state_interface name="position">
@@ -47,6 +47,6 @@
           </state_interface>
       </joint>
-      <joint name="${prefix}right_gripper_joint">
-          <param name="mimic">${prefix}left_gripper_joint</param>
+      <joint name="${prefix}right_carriage_joint">
+          <param name="mimic">${prefix}left_carriage_joint</param>
           <param name="multiplier">1</param>
           <command_interface name="position" />

Commit message: Remove unused right carriage joint

File: urdf/macros/_wxai.ros2_control.xacro (robot description, xacro)
@@ -47,19 +47,4 @@
           </state_interface>
       </joint>
-      <!-- right_carriage_joint is a mimic of the left_carriage_joint and does not get a command interface -->
-      <joint name="${prefix}right_carriage_joint">
-          <param name="mimic">${prefix}left_carriage_joint</param>
-          <param name="multiplier">1</param>
-          <!-- <command_interface name="position" /> -->
-          <state_interface name="position">
-            <param name="initial_value">0.0</param>
-          </state_interface>
-          <state_interface name="velocity">
-            <param name="initial_value">0.0</param>
-          </state_interface>
-          <state_interface name="effort">
-            <param name="initial_value">0.0</param>
-          </state_interface>
-      </joint>
     </ros2_control>
   </xacro:macro>

Commit message: Pass IP address to wxai ros2_control macro

File: urdf/macros/_wxai.ros2_control.xacro (robot description, xacro)
@@ -15,5 +15,5 @@
     </joint>
   </xacro:macro>
-  <xacro:macro name="wxai_ros2_control" params="prefix ip_address ros2_control_hardware_type">
+  <xacro:macro name="wxai_ros2_control" params="prefix ros2_control_hardware_type:='real' ip_address:='192.168.1.2'">
     <ros2_control name="TrossenArmHardwareInterface" type="system">
       <hardware>

File: urdf/macros/_wxai.urdf.xacro (robot description, xacro)
@@ -7,5 +7,5 @@
     value="6"
     scope="local"/>
-  <xacro:macro name="wxai" params="variant arm_side:='' prefix:='' ros2_control_hardware_type:='real'">
+  <xacro:macro name="wxai" params="variant arm_side:='' prefix:='' ros2_control_hardware_type:='real' ip_address:='192.168.1.2'">
     <xacro:property name="mesh_directory" value="package://trossen_arm_description/meshes/${robot_model}"/>
     <xacro:include filename="$(find trossen_arm_description)/urdf/macros/_wxai.ros2_control.xacro"/>
@@ -13,5 +13,5 @@
       ros2_control_hardware_type="${ros2_control_hardware_type}"
       prefix="${prefix}"
-      ip_address="192.168.1.2"/>  <!-- TODO(lukeschmitt-tr): pass this -->
+      ip_address="${ip_address}"/>
     <link name="${prefix}base_link">
       <inertial>

File: urdf/wxai.urdf.xacro (robot description, xacro)
@@ -1,8 +1,9 @@
 <?xml version="1.0" encoding="utf-8"?>
 <robot name="wxai" xmlns:xacro="http://ros.org/wiki/xacro">
-  <xacro:arg name="variant"                         default="base"/>      <!-- 'base', 'leader', 'follower' -->
-  <xacro:arg name="arm_side"                        default=""/>          <!-- '', 'left', 'right' -->
-  <xacro:arg name="use_world_frame"                 default="false"/>     <!-- 'true', 'false' -->
-  <xacro:arg name="ros2_control_hardware_type"      default="real"/>      <!-- 'real', 'mock_components' -->
+  <xacro:arg name="variant"                         default="base"/>        <!-- 'base', 'leader', 'follower' -->
+  <xacro:arg name="arm_side"                        default=""/>            <!-- '', 'left', 'right' -->
+  <xacro:arg name="use_world_frame"                 default="false"/>       <!-- 'true', 'false' -->
+  <xacro:arg name="ros2_control_hardware_type"      default="real"/>        <!-- 'real', 'mock_components' -->
+  <xacro:arg name="ip_address"                      default="192.168.1.2"/>
   <xacro:arg name="base_link_frame"                 default="base_link"/>
   <xacro:if value="$(arg use_world_frame)">
@@ -21,4 +22,5 @@
     arm_side="$(arg arm_side)"
     variant="$(arg variant)"
+    ip_address="$(arg ip_address)"
     ros2_control_hardware_type="$(arg ros2_control_hardware_type)"/>
 </robot>

Commit message: Remove defaults from macro args
https://github.com/TrossenRobotics/trossen_arm_description/pull/16#discussion_r2172889273

File: urdf/macros/_wxai.ros2_control.xacro (robot description, xacro)
@@ -15,5 +15,5 @@
     </joint>
   </xacro:macro>
-  <xacro:macro name="wxai_ros2_control" params="prefix ros2_control_hardware_type:='real' ip_address:='192.168.1.2'">
+  <xacro:macro name="wxai_ros2_control" params="prefix ros2_control_hardware_type ip_address">
     <ros2_control name="TrossenArmHardwareInterface" type="system">
       <hardware>

File: urdf/macros/_wxai.urdf.xacro (robot description, xacro)
@@ -7,5 +7,5 @@
     value="6"
     scope="local"/>
-  <xacro:macro name="wxai" params="variant arm_side:='' prefix:='' ros2_control_hardware_type:='real' ip_address:='192.168.1.2'">
+  <xacro:macro name="wxai" params="variant arm_side:='' prefix:='' ros2_control_hardware_type ip_address">
     <xacro:property name="mesh_directory" value="package://trossen_arm_description/meshes/${robot_model}"/>
     <xacro:include filename="$(find trossen_arm_description)/urdf/macros/_wxai.ros2_control.xacro"/>

Commit message: Pass variant to ros2_control

File: urdf/macros/_wxai.ros2_control.xacro (robot description, xacro)
@@ -15,5 +15,5 @@
     </joint>
   </xacro:macro>
-  <xacro:macro name="wxai_ros2_control" params="prefix ros2_control_hardware_type ip_address">
+  <xacro:macro name="wxai_ros2_control" params="prefix ros2_control_hardware_type ip_address variant">
     <ros2_control name="TrossenArmHardwareInterface" type="system">
       <hardware>
@@ -23,5 +23,6 @@
         <xacro:if value="${ros2_control_hardware_type == 'real'}">
           <plugin>trossen_arm_hardware/TrossenArmHardwareInterface</plugin>
-          <param name="robot_model">0</param>        <!-- 0: wxai_v0 -->
+          <param name="robot_model">0</param>             <!-- 0: wxai_v0 -->
+          <param name="end_effector">${variant}</param>   <!-- 'base', 'follower' -->
           <param name="ip_address">${ip_address}</param>
         </xacro:if>  <!-- ros2_control_hardware_type == 'real' -->

File: urdf/macros/_wxai.urdf.xacro (robot description, xacro)
@@ -13,5 +13,6 @@
       prefix="${prefix}"
       ip_address="${ip_address}"
-      ros2_control_hardware_type="${ros2_control_hardware_type}"/>
+      ros2_control_hardware_type="${ros2_control_hardware_type}"
+      end_effector="${variant}"/>
     <link name="${prefix}base_link">
       <inertial>

Commit message: Pass arm variant to ros2_control hardware interface macro (#24)
* Pass variant to ros2_control

* lint

* Fix macro arg

File: urdf/macros/_wxai.ros2_control.xacro (robot description, xacro)
@@ -15,5 +15,5 @@
     </joint>
   </xacro:macro>
-  <xacro:macro name="wxai_ros2_control" params="prefix ros2_control_hardware_type ip_address">
+  <xacro:macro name="wxai_ros2_control" params="prefix ros2_control_hardware_type ip_address variant">
     <ros2_control name="TrossenArmHardwareInterface" type="system">
       <hardware>
@@ -23,5 +23,6 @@
         <xacro:if value="${ros2_control_hardware_type == 'real'}">
           <plugin>trossen_arm_hardware/TrossenArmHardwareInterface</plugin>
-          <param name="robot_model">0</param>        <!-- 0: wxai_v0 -->
+          <param name="robot_model">0</param>             <!-- 0: wxai_v0 -->
+          <param name="end_effector">${variant}</param>   <!-- 'base', 'follower' -->
           <param name="ip_address">${ip_address}</param>
         </xacro:if>  <!-- ros2_control_hardware_type == 'real' -->

Commit message: feat: added external torque control mode to the hw interface

File: urdf/macros/_wxai.ros2_control.xacro (robot description, xacro)
@@ -1,7 +1,7 @@
 <?xml version="1.0"?>
 <robot xmlns:xacro="http://www.ros.org/wiki/xacro">
-  <xacro:macro name="ros2_control_joint" params="name">
+  <xacro:macro name="ros2_control_joint" params="name command_interface:='position'">
     <joint name="${name}">
-      <command_interface name="position"/>
+      <command_interface name="${command_interface}"/>
       <state_interface name="position">
         <param name="initial_value">0.0</param>
@@ -15,5 +15,5 @@
     </joint>
   </xacro:macro>
-  <xacro:macro name="wxai_ros2_control" params="prefix ros2_control_hardware_type ip_address variant">
+  <xacro:macro name="wxai_ros2_control" params="prefix ros2_control_hardware_type ip_address variant command_interface:='position'">
     <ros2_control name="TrossenArmHardwareInterface" type="system">
       <hardware>
@@ -28,12 +28,12 @@
         </xacro:if>  <!-- ros2_control_hardware_type == 'real' -->
       </hardware>
-      <xacro:ros2_control_joint name="${prefix}joint_0"/>
-      <xacro:ros2_control_joint name="${prefix}joint_1"/>
-      <xacro:ros2_control_joint name="${prefix}joint_2"/>
-      <xacro:ros2_control_joint name="${prefix}joint_3"/>
-      <xacro:ros2_control_joint name="${prefix}joint_4"/>
-      <xacro:ros2_control_joint name="${prefix}joint_5"/>
+      <xacro:ros2_control_joint name="${prefix}joint_0" command_interface="${command_interface}"/>
+      <xacro:ros2_control_joint name="${prefix}joint_1" command_interface="${command_interface}"/>
+      <xacro:ros2_control_joint name="${prefix}joint_2" command_interface="${command_interface}"/>
+      <xacro:ros2_control_joint name="${prefix}joint_3" command_interface="${command_interface}"/>
+      <xacro:ros2_control_joint name="${prefix}joint_4" command_interface="${command_interface}"/>
+      <xacro:ros2_control_joint name="${prefix}joint_5" command_interface="${command_interface}"/>
       <joint name="${prefix}left_carriage_joint">
-        <command_interface name="position" />
+        <command_interface name="${command_interface}"/>
         <state_interface name="position">
           <param name="initial_value">0.0</param>

File: urdf/macros/_wxai.urdf.xacro (robot description, xacro)
@@ -7,5 +7,5 @@
     value="6"
     scope="local"/>
-  <xacro:macro name="wxai" params="variant arm_side:='' prefix:='' ros2_control_hardware_type ip_address">
+  <xacro:macro name="wxai" params="variant arm_side:='' prefix:='' ros2_control_hardware_type ip_address command_interface:='position'">
     <xacro:property name="mesh_directory" value="package://trossen_arm_description/meshes/${robot_model}"/>
     <xacro:include filename="$(find trossen_arm_description)/urdf/macros/_wxai.ros2_control.xacro"/>
@@ -14,5 +14,6 @@
       ip_address="${ip_address}"
       ros2_control_hardware_type="${ros2_control_hardware_type}"
-      variant="${variant}"/>
+      variant="${variant}"
+      command_interface="${command_interface}"/>
     <link name="${prefix}base_link">
       <inertial>

File: urdf/wxai.urdf.xacro (robot description, xacro)
@@ -8,4 +8,5 @@
   <xacro:arg name="ip_address"                      default="192.168.1.2"/>
   <xacro:arg name="base_link_frame"                 default="base_link"/>
+  <xacro:arg name="command_interface"               default="position"/>    <!-- 'position', 'effort' -->
   <xacro:if value="$(arg use_world_frame)">
     <link name="world"/>
@@ -25,4 +26,5 @@
     prefix="$(arg prefix)"
     ros2_control_hardware_type="$(arg ros2_control_hardware_type)"
-    ip_address="$(arg ip_address)"/>
+    ip_address="$(arg ip_address)"
+    command_interface="$(arg command_interface)"/>
 </robot>
