Commit message: add maple_tabletop texture update _common.urdf.xacro

File: urdf/macros/_common.urdf.xacro (robot description, xacro)
@@ -6,3 +6,8 @@
     </material>
   </xacro:macro>  <!-- trossen_black -->
+  <xacro:macro name="maple_tabletop">
+    <material name="maple_tabletop">
+      <texture filename="package://trossen_arm_description/meshes/maple_tabletop.png"/>
+    </material>
+  </xacro:macro>  <!-- maple_tabletop -->
 </robot>
