Commit message: generated urdf

File: urdf/generated/leader/leader_left.urdf (robot description, URDF)
Before this commit: robot leader, 10 links, 9 joints
Joints:
- joint joint_0: limit lower=-3.141592653589793 upper=1.5707963267948966 effort=0 velocity=6.283185307179586 -> lower=-3.141592653589793 upper=1.5707963267948966 effort=27.0 velocity=6.283185307179586
- joint joint_1: limit lower=0 upper=3.141592653589793 effort=0 velocity=6.283185307179586 -> lower=0 upper=3.141592653589793 effort=27.0 velocity=6.283185307179586
- joint joint_2: limit lower=-1.5707963267948966 upper=1.5707963267948966 effort=0 velocity=6.283185307179586 -> lower=-1.5707963267948966 upper=1.5707963267948966 effort=7.0 velocity=6.283185307179586
- joint joint_3: limit lower=-2.356194490192345 upper=0 effort=0 velocity=6.283185307179586 -> lower=-2.356194490192345 upper=0 effort=7.0 velocity=6.283185307179586
- joint joint_4: limit lower=-1.5707963267948966 upper=1.5707963267948966 effort=0 velocity=6.283185307179586 -> lower=-1.5707963267948966 upper=1.5707963267948966 effort=3.0 velocity=6.283185307179586
- joint joint_5: limit lower=-0.7853981633974483 upper=0.7853981633974483 effort=0 velocity=6.283185307179586 -> lower=-0.7853981633974483 upper=0.7853981633974483 effort=3.0 velocity=6.283185307179586
- joint joint_6: limit lower=-1.5707963267948966 upper=1.5707963267948966 effort=0 velocity=6.283185307179586 -> lower=-1.5707963267948966 upper=1.5707963267948966 effort=3.0 velocity=6.283185307179586
- joint joint_7: limit lower=0 upper=0.5235987755982988 effort=0 velocity=0 -> lower=0 upper=0.5235987755982988 effort=3.0 velocity=6.283185307179586

File: urdf/generated/leader/leader_right.urdf (robot description, URDF)
Before this commit: robot leader, 10 links, 9 joints
Joints:
- joint joint_0: limit lower=-1.5707963267948966 upper=3.141592653589793 effort=0 velocity=6.283185307179586 -> lower=-1.5707963267948966 upper=3.141592653589793 effort=27.0 velocity=6.283185307179586
- joint joint_1: limit lower=-3.141592653589793 upper=0 effort=0 velocity=6.283185307179586 -> lower=-3.141592653589793 upper=0 effort=27.0 velocity=6.283185307179586
- joint joint_2: limit lower=-1.5707963267948966 upper=1.5707963267948966 effort=0 velocity=6.283185307179586 -> lower=-1.5707963267948966 upper=1.5707963267948966 effort=7.0 velocity=6.283185307179586
- joint joint_3: limit lower=0 upper=2.356194490192345 effort=0 velocity=6.283185307179586 -> lower=0 upper=2.356194490192345 effort=7.0 velocity=6.283185307179586
- joint joint_4: limit lower=-1.5707963267948966 upper=1.5707963267948966 effort=0 velocity=6.283185307179586 -> lower=-1.5707963267948966 upper=1.5707963267948966 effort=3.0 velocity=6.283185307179586
- joint joint_5: limit lower=-0.7853981633974483 upper=0.7853981633974483 effort=0 velocity=6.283185307179586 -> lower=-0.7853981633974483 upper=0.7853981633974483 effort=3.0 velocity=6.283185307179586
- joint joint_6: limit lower=-1.5707963267948966 upper=1.5707963267948966 effort=0 velocity=6.283185307179586 -> lower=-1.5707963267948966 upper=1.5707963267948966 effort=3.0 velocity=6.283185307179586
- joint joint_7: limit lower=-1.5707963267948966 upper=1.5707963267948966 effort=0 velocity=0 -> lower=-0.5235987755982988 upper=0 effort=3.0 velocity=6.283185307179586

Commit message: fixed axes and ee gripper

File: urdf/generated/leader/leader_left.urdf (robot description, URDF)
Before this commit: robot leader, 10 links, 9 joints
Joints:
- joint ee_gripper: origin xyz=-0.021 0 -0.200062 rpy=0 0 0 -> xyz=0 0 0 rpy=0 0 0
- joint joint_3: axis 0 1 0 -> 0 -1 0; limit lower=-2.356194490192345 upper=0 effort=7.0 velocity=6.283185307179586 -> lower=0 upper=2.356194490192345 effort=7.0 velocity=6.283185307179586
- joint joint_6: axis 1 0 0 -> -1 0 0

File: urdf/generated/leader/leader_right.urdf (robot description, URDF)
Before this commit: robot leader, 10 links, 9 joints
Joints:
- joint ee_gripper: origin xyz=-0.021 0 -0.200062 rpy=0 0 0 -> xyz=0 0 0 rpy=0 0 0
- joint joint_3: axis 0 -1 0 -> 0 1 0; limit lower=0 upper=2.356194490192345 effort=7.0 velocity=6.283185307179586 -> lower=-2.356194490192345 upper=0 effort=7.0 velocity=6.283185307179586
- joint joint_6: axis 1 0 0 -> -1 0 0

File: urdf/macros/_leader.urdf.xacro (robot description, xacro)
@@ -362,4 +362,12 @@
       <child link="${prefix}link_4" />
       <xacro:if value="${arm_side == 'right'}">
+        <axis xyz="0 1 0" />
+        <limit
+          effort="7.0"
+          lower="${-3 * pi / 4}"
+          upper="0"
+          velocity="${2 * pi}" />
+      </xacro:if>  <!-- arm_side == right -->
+      <xacro:if value="${arm_side == 'left'}">
         <axis xyz="0 -1 0" />
         <limit
@@ -367,12 +375,4 @@
           lower="0"
           upper="${3 * pi / 4}"
-          velocity="${2 * pi}" />
-      </xacro:if>  <!-- arm_side == right -->
-      <xacro:if value="${arm_side == 'left'}">
-        <axis xyz="0 1 0" />
-        <limit
-          effort="7.0"
-          lower="${-3 * pi / 4}"
-          upper="0"
           velocity="${2 * pi}" />
       </xacro:if>  <!-- arm_side == left -->
@@ -506,5 +506,5 @@
       <parent link="${prefix}link_6" />
       <child link="${prefix}link_7" />
-      <axis xyz="1 0 0" />
+      <axis xyz="-1 0 0" />
       <limit
         effort="3.0"
@@ -573,5 +573,5 @@
     <joint name="${prefix}ee_gripper" type="fixed">
       <origin
-        xyz="-0.021 0 -0.200062"
+        xyz="0 0 0"
         rpy="0 0 0" />
       <parent link="${prefix}link_8" />
