Commit message: update stationary_ai.urdf.xacro and generated urdf file

File: urdf/generated/stationary_ai.urdf (robot description, URDF)
Before this commit: robot stationary_ai, 71 links, 70 joints
Links:
- removed link base_footprint
- removed link base_link
- removed link cam_overhead_bottom_screw_frame
- removed link cam_overhead_color_frame
- removed link cam_overhead_color_optical_frame
- removed link cam_overhead_depth_frame
- removed link cam_overhead_depth_optical_frame
- removed link cam_overhead_infra1_frame
- removed link cam_overhead_infra1_optical_frame
- removed link cam_overhead_infra2_frame
- removed link cam_overhead_infra2_optical_frame
- removed link cam_overhead_link
- removed link cam_worms_eye_bottom_screw_frame
- removed link cam_worms_eye_color_frame
- removed link cam_worms_eye_color_optical_frame
- removed link cam_worms_eye_depth_frame
- removed link cam_worms_eye_depth_optical_frame
- removed link cam_worms_eye_infra1_frame
- removed link cam_worms_eye_infra1_optical_frame
- removed link cam_worms_eye_infra2_frame
- removed link cam_worms_eye_infra2_optical_frame
- removed link cam_worms_eye_link
- removed link overhead_cam_mount_link
- removed link worms_eye_cam_mount_link
- added link cam_high_bottom_screw_frame
- added link cam_high_color_frame
- added link cam_high_color_optical_frame
- added link cam_high_depth_frame
- added link cam_high_depth_optical_frame
- added link cam_high_infra1_frame
- added link cam_high_infra1_optical_frame
- added link cam_high_infra2_frame
- added link cam_high_infra2_optical_frame
- added link cam_high_link, mass 0.072; collision box size=0.023 0.042 0.042; visual mesh filename=package://trossen_arm_description/meshes/peripherals/d405.s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 scale=0.001 0.001 0.001
- added link cam_high_mount_link, mass 0.1; collision mesh filename=package://trossen_arm_description/meshes/stationary_ai/cam_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; visual mesh filename=package://trossen_arm_description/meshes/stationary_ai/cam_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
- added link cam_low_bottom_screw_frame
- added link cam_low_color_frame
- added link cam_low_color_optical_frame
- added link cam_low_depth_frame
- added link cam_low_depth_optical_frame
- added link cam_low_infra1_frame
- added link cam_low_infra1_optical_frame
- added link cam_low_infra2_frame
- added link cam_low_infra2_optical_frame
- added link cam_low_link, mass 0.072; collision box size=0.023 0.042 0.042; visual mesh filename=package://trossen_arm_description/meshes/peripherals/d405.s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 scale=0.001 0.001 0.001
- added link cam_low_mount_link, mass 0.1; collision mesh filename=package://trossen_arm_description/meshes/stationary_ai/cam_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; visual mesh filename=package://trossen_arm_description/meshes/stationary_ai/cam_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
- added link tabletop_link, mass 10.0; collision mesh filename=package://trossen_arm_description/meshes/stationary_ai/tabl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; visual mesh filename=package://trossen_arm_description/meshes/stationary_ai/tabl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
Joints:
- removed joint base_footprint_joint
- removed joint cam_overhead_color_joint
- removed joint cam_overhead_color_optical_joint
- removed joint cam_overhead_depth_joint
- removed joint cam_overhead_depth_optical_joint
- removed joint cam_overhead_infra1_joint
- removed joint cam_overhead_infra1_optical_joint
- removed joint cam_overhead_infra2_joint
- removed joint cam_overhead_infra2_optical_joint
- removed joint cam_overhead_joint
- removed joint cam_overhead_link_joint
- removed joint cam_worms_eye_color_joint
- removed joint cam_worms_eye_color_optical_joint
- removed joint cam_worms_eye_depth_joint
- removed joint cam_worms_eye_depth_optical_joint
- removed joint cam_worms_eye_infra1_joint
- removed joint cam_worms_eye_infra1_optical_joint
- removed joint cam_worms_eye_infra2_joint
- removed joint cam_worms_eye_infra2_optical_joint
- removed joint cam_worms_eye_joint
- removed joint cam_worms_eye_link_joint
- removed joint overhead_cam_mount_joint
- removed joint worms_eye_cam_mount_joint
- added joint cam_high_color_joint: type fixed, parent cam_high_link, child cam_high_color_frame, origin xyz=0 0.0 0 rpy=0 0 0
- added joint cam_high_color_optical_joint: type fixed, parent cam_high_color_frame, child cam_high_color_optical_frame, origin xyz=0 0 0 rpy=-1.5707963267948966 0 -1.5707963267948966
- added joint cam_high_depth_joint: type fixed, parent cam_high_link, child cam_high_depth_frame, origin xyz=0 0 0 rpy=0 0 0
- added joint cam_high_depth_optical_joint: type fixed, parent cam_high_depth_frame, child cam_high_depth_optical_frame, origin xyz=0 0 0 rpy=-1.5707963267948966 0 -1.5707963267948966
- added joint cam_high_infra1_joint: type fixed, parent cam_high_link, child cam_high_infra1_frame, origin xyz=0 0.0 0 rpy=0 0 0
- added joint cam_high_infra1_optical_joint: type fixed, parent cam_high_infra1_frame, child cam_high_infra1_optical_frame, origin xyz=0 0 0 rpy=-1.5707963267948966 0 -1.5707963267948966
- added joint cam_high_infra2_joint: type fixed, parent cam_high_link, child cam_high_infra2_frame, origin xyz=0 -0.018 0 rpy=0 0 0
- added joint cam_high_infra2_optical_joint: type fixed, parent cam_high_infra2_frame, child cam_high_infra2_optical_frame, origin xyz=0 0 0 rpy=-1.5707963267948966 0 -1.5707963267948966
- added joint cam_high_joint: type fixed, parent cam_high_mount_link, child cam_high_bottom_screw_frame, origin xyz=0.040000 0.056352 0.036829 rpy=-3.141592653589793 -1.1344640137963142 1.5707963267948966
- added joint cam_high_link_joint: type fixed, parent cam_high_bottom_screw_frame, child cam_high_link, origin xyz=0.01085 0.009 0.021 rpy=0 0 0
- added joint cam_high_mount_joint: type fixed, parent frame_link, child cam_high_mount_link, origin xyz=-0.401982 -0.040000 1.059852 rpy=-3.141592653589793 0 1.5707963267948966
- added joint cam_low_color_joint: type fixed, parent cam_low_link, child cam_low_color_frame, origin xyz=0 0.0 0 rpy=0 0 0
- added joint cam_low_color_optical_joint: type fixed, parent cam_low_color_frame, child cam_low_color_optical_frame, origin xyz=0 0 0 rpy=-1.5707963267948966 0 -1.5707963267948966
- added joint cam_low_depth_joint: type fixed, parent cam_low_link, child cam_low_depth_frame, origin xyz=0 0 0 rpy=0 0 0
- added joint cam_low_depth_optical_joint: type fixed, parent cam_low_depth_frame, child cam_low_depth_optical_frame, origin xyz=0 0 0 rpy=-1.5707963267948966 0 -1.5707963267948966
- added joint cam_low_infra1_joint: type fixed, parent cam_low_link, child cam_low_infra1_frame, origin xyz=0 0.0 0 rpy=0 0 0
- added joint cam_low_infra1_optical_joint: type fixed, parent cam_low_infra1_frame, child cam_low_infra1_optical_frame, origin xyz=0 0 0 rpy=-1.5707963267948966 0 -1.5707963267948966
- added joint cam_low_infra2_joint: type fixed, parent cam_low_link, child cam_low_infra2_frame, origin xyz=0 -0.018 0 rpy=0 0 0
- added joint cam_low_infra2_optical_joint: type fixed, parent cam_low_infra2_frame, child cam_low_infra2_optical_frame, origin xyz=0 0 0 rpy=-1.5707963267948966 0 -1.5707963267948966
- added joint cam_low_joint: type fixed, parent cam_low_mount_link, child cam_low_bottom_screw_frame, origin xyz=0.024884 0.031947 0.033325 rpy=-3.141592653589793 0.09599310885968812 1.5707963267948966
- added joint cam_low_link_joint: type fixed, parent cam_low_bottom_screw_frame, child cam_low_link, origin xyz=0.01085 0.009 0.021 rpy=0 0 0
- added joint cam_low_mount_joint: type fixed, parent frame_link, child cam_low_mount_link, origin xyz=-0.415000 -0.024884 0.044061 rpy=-3.141592653589793 0 1.5707963267948966
- joint frame_joint: parent base_link -> tabletop_link

File: urdf/stationary_ai.urdf.xacro (robot description, xacro)
@@ -1,6 +1,6 @@
 <?xml version="1.0" encoding="utf-8"?>
 <robot name="stationary_ai" xmlns:xacro="http://ros.org/wiki/xacro">
-  <xacro:arg name="ip_address_left" default="192.168.1.10"/>
-  <xacro:arg name="ip_address_right" default="192.168.1.11"/>
+  <xacro:arg name="ip_address_left" default="192.168.1.5"/>
+  <xacro:arg name="ip_address_right" default="192.168.1.4"/>
   <xacro:arg name="ros2_control_hardware_type" default="mock_components"/>
   <xacro:property name="robot_model"
@@ -12,5 +12,6 @@
   <xacro:property name="mesh_directory" value="package://trossen_arm_description/meshes/stationary_ai"/>
   <xacro:trossen_black/>
-  <link name="base_link">
+  <xacro:maple_tabletop/>
+  <link name="tabletop_link">
     <inertial>
       <origin
@@ -31,25 +32,17 @@
         rpy="0 0 0" />
       <geometry>
-        <mesh filename="${mesh_directory}/base_link.stl" />
-      </geometry>
-      <material name="trossen_black"/>
-    </visual>
-    <collision>
-      <origin
-        xyz="0 0 0"
-        rpy="0 0 0" />
-      <geometry>
-        <mesh filename="${mesh_directory}/base_link.stl" />
-      </geometry>
-    </collision>
-  </link>
-  <link name="base_footprint"/>
-  <joint
-    name="base_footprint_joint"
-    type="fixed">
-    <origin xyz="0 0 0.020" rpy="0 0 0"/>
-    <parent link="base_footprint"/>
-    <child link="base_link"/>
-  </joint>
+        <mesh filename="${mesh_directory}/tabletop_link.stl" />
+      </geometry>
+      <material name="maple_tabletop"/>
+    </visual>
+    <collision>
+      <origin
+        xyz="0 0 0"
+        rpy="0 0 0" />
+      <geometry>
+        <mesh filename="${mesh_directory}/tabletop_link.stl" />
+      </geometry>
+    </collision>
+  </link>
   <link name="frame_link">
     <inertial>
@@ -90,8 +83,8 @@
       xyz="0.0 0.0 0.0"
       rpy="0 0 0" />
-    <parent link="base_link" />
+    <parent link="tabletop_link" />
     <child link="frame_link" />
   </joint>
-  <link name="overhead_cam_mount_link">
+  <link name="cam_high_mount_link">
     <inertial>
       <origin
@@ -112,5 +105,5 @@
         rpy="0 0 0" />
       <geometry>
-        <mesh filename="${mesh_directory}/overhead_cam_mount_link.stl" />
+        <mesh filename="${mesh_directory}/cam_high_mount_link.stl" />
       </geometry>
       <material name="trossen_black"/>
@@ -121,10 +114,10 @@
         rpy="0 0 0" />
       <geometry>
-        <mesh filename="${mesh_directory}/overhead_cam_mount_link.stl" />
-      </geometry>
-    </collision>
-  </link>
-  <joint
-    name="overhead_cam_mount_joint"
+        <mesh filename="${mesh_directory}/cam_high_mount_link.stl" />
+      </geometry>
+    </collision>
+  </link>
+  <joint
+    name="cam_high_mount_joint"
     type="fixed">
     <origin
@@ -132,9 +125,9 @@
       rpy="${radians(-180)} 0 ${radians(90)}" />
     <parent link="frame_link" />
-    <child link="overhead_cam_mount_link" />
+    <child link="cam_high_mount_link" />
   </joint>
   <xacro:sensor_d405
-    name="cam_overhead"
-    parent="overhead_cam_mount_link"
+    name="cam_high"
+    parent="cam_high_mount_link"
     use_nominal_extrinsics="true">
     <origin
@@ -142,5 +135,5 @@
       rpy="${radians(-180)} ${radians(-65)} ${radians(90)}" />
   </xacro:sensor_d405>
-  <link name="worms_eye_cam_mount_link">
+  <link name="cam_low_mount_link">
     <inertial>
       <origin
@@ -161,5 +154,5 @@
         rpy="0 0 0" />
       <geometry>
-        <mesh filename="${mesh_directory}/worms_eye_cam_mount_link.stl" />
+        <mesh filename="${mesh_directory}/cam_low_mount_link.stl" />
       </geometry>
       <material name="trossen_black"/>
@@ -170,10 +163,10 @@
         rpy="0 0 0" />
       <geometry>
-        <mesh filename="${mesh_directory}/worms_eye_cam_mount_link.stl" />
-      </geometry>
-    </collision>
-  </link>
-  <joint
-    name="worms_eye_cam_mount_joint"
+        <mesh filename="${mesh_directory}/cam_low_mount_link.stl" />
+      </geometry>
+    </collision>
+  </link>
+  <joint
+    name="cam_low_mount_joint"
     type="fixed">
     <origin
@@ -181,9 +174,9 @@
       rpy="${radians(-180)} 0 ${radians(90)}" />
     <parent link="frame_link" />
-    <child link="worms_eye_cam_mount_link" />
+    <child link="cam_low_mount_link" />
   </joint>
   <xacro:sensor_d405
-    name="cam_worms_eye"
-    parent="worms_eye_cam_mount_link"
+    name="cam_low"
+    parent="cam_low_mount_link"
     use_nominal_extrinsics="true">
     <origin

Commit message: update cam pos xacro and generated urdf

File: urdf/generated/stationary_ai.urdf (robot description, URDF)
Before this commit: robot stationary_ai, 70 links, 69 joints
Joints:
- joint cam_high_joint: origin xyz=0.040000 0.056352 0.036829 rpy=-3.141592653589793 -1.1344640137963142 1.5707963267948966 -> xyz=0.040000 0.056252 0.030 rpy=-3.141592653589793 -1.1344640137963142 1.5707963267948966
- joint cam_low_joint: origin xyz=0.024884 0.031947 0.033325 rpy=-3.141592653589793 0.09599310885968812 1.5707963267948966 -> xyz=0.024884 0.0253 0.033325 rpy=-3.141592653589793 0.09599310885968812 1.5707963267948966

File: urdf/stationary_ai.urdf.xacro (robot description, xacro)
@@ -132,5 +132,5 @@
     use_nominal_extrinsics="true">
     <origin
-      xyz="0.040000 0.056352 0.036829"
+      xyz="0.040000 0.056252 0.030"
       rpy="${radians(-180)} ${radians(-65)} ${radians(90)}" />
   </xacro:sensor_d405>
@@ -181,5 +181,5 @@
     use_nominal_extrinsics="true">
     <origin
-      xyz="0.024884 0.031947 0.033325"
+      xyz="0.024884 0.0253 0.033325"
       rpy="${radians(-180)} ${radians(5.5)} ${radians(90)}" />
   </xacro:sensor_d405>

Commit message: generated urdf and updated xacro

File: urdf/generated/stationary_ai.urdf (robot description, URDF)
Before this commit: robot stationary_ai, 70 links, 69 joints
Joints:
- joint cam_high_joint: origin xyz=0.040000 0.056252 0.030 rpy=-3.141592653589793 -1.1344640137963142 1.5707963267948966 -> xyz=-0.348293 -0.000000 1.028733 rpy=0 1.1344640137963142 0; parent cam_high_mount_link -> frame_link
- joint cam_high_mount_joint: origin xyz=-0.401982 -0.040000 1.059852 rpy=-3.141592653589793 0 1.5707963267948966 -> xyz=-0.401982 -0.040000 1.059852 rpy=-3.141592653589793 0.0 1.5707963267948966
- joint cam_low_joint: origin xyz=0.024884 0.0253 0.033325 rpy=-3.141592653589793 0.09599310885968812 1.5707963267948966 -> xyz=-0.389324 0.000000 0.010132 rpy=0 -0.09599310885968812 0; parent cam_low_mount_link -> frame_link
- joint cam_low_mount_joint: origin xyz=-0.415000 -0.024884 0.044061 rpy=-3.141592653589793 0 1.5707963267948966 -> xyz=-0.415000 -0.024884 0.044061 rpy=-3.141592653589793 0.0 1.5707963267948966
- joint frame_joint: origin xyz=0.0 0.0 0.0 rpy=0 0 0 -> xyz=0.0 0.0 0.02 rpy=0 0 0

File: urdf/stationary_ai.urdf.xacro (robot description, xacro)
@@ -81,5 +81,5 @@
     type="fixed">
     <origin
-      xyz="0.0 0.0 0.0"
+      xyz="0.0 0.0 0.02"
       rpy="0 0 0" />
     <parent link="tabletop_link" />
@@ -123,5 +123,5 @@
     <origin
       xyz="-0.401982 -0.040000 1.059852"
-      rpy="${radians(-180)} 0 ${radians(90)}" />
+      rpy="${radians(-180)} ${radians(-0)} ${radians(90)}" />
     <parent link="frame_link" />
     <child link="cam_high_mount_link" />
@@ -129,9 +129,9 @@
   <xacro:sensor_d405
     name="cam_high"
-    parent="cam_high_mount_link"
+    parent="frame_link"
     use_nominal_extrinsics="true">
     <origin
-      xyz="0.040000 0.056252 0.030"
-      rpy="${radians(-180)} ${radians(-65)} ${radians(90)}" />
+      xyz="-0.348293 -0.000000 1.028733"
+      rpy="0 ${radians(65)} 0" />
   </xacro:sensor_d405>
   <link name="cam_low_mount_link">
@@ -172,5 +172,5 @@
     <origin
       xyz="-0.415000 -0.024884 0.044061"
-      rpy="${radians(-180)} 0 ${radians(90)}" />
+      rpy="${radians(-180)} ${radians(-0)} ${radians(90)}" />
     <parent link="frame_link" />
     <child link="cam_low_mount_link" />
@@ -178,9 +178,9 @@
   <xacro:sensor_d405
     name="cam_low"
-    parent="cam_low_mount_link"
+    parent="frame_link"
     use_nominal_extrinsics="true">
     <origin
-      xyz="0.024884 0.0253 0.033325"
-      rpy="${radians(-180)} ${radians(5.5)} ${radians(90)}" />
+      xyz="-0.389324 0.000000 0.010132"
+      rpy="0 ${radians(-5.5)} 0" />
   </xacro:sensor_d405>
   <joint
