Commit message: Update generated URDF

File: urdf/generated/mobile_ai.urdf (robot description, URDF)
Before this commit: robot mobile_ai, 58 links, 57 joints
Links:
- added link camera_low_bottom_screw_frame
- added link camera_low_color_frame
- added link camera_low_color_optical_frame
- added link camera_low_depth_frame
- added link camera_low_depth_optical_frame
- added link camera_low_infra1_frame
- added link camera_low_infra1_optical_frame
- added link camera_low_infra2_frame
- added link camera_low_infra2_optical_frame
- added link camera_low_link, mass 0.072; collision box size=0.023 0.042 0.042; visual mesh filename=package://trossen_arm_description/meshes/peripherals/d405.s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 scale=0.001 0.001 0.001
- link base_link: mass 45.1929991042861 -> 80
- link caster_swivel_front_left: mass 0.0318006084570262 -> 0.10000000
- link caster_swivel_front_right: mass 0.0318006084570262 -> 0.10000000
- link caster_swivel_rear_left: mass 0.0318006084570262 -> 0.10000000
- link caster_swivel_rear_right: mass 0.0318006084570262 -> 0.10000000
- link caster_wheel_front_left: mass 0.0898231658107286 -> 0.53500000
- link caster_wheel_front_right: mass 0.0898231658107286 -> 0.53500000
- link caster_wheel_rear_left: mass 0.0898231658107286 -> 0.53500000
- link caster_wheel_rear_right: mass 0.0898231658107286 -> 0.53500000
- link left_wheel_link: mass 0.981755254019503 -> 3.00000000
Joints:
- added joint camera_low_color_joint: type fixed, parent camera_low_link, child camera_low_color_frame, origin xyz=0 0.0 0 rpy=0 0 0
- added joint camera_low_color_optical_joint: type fixed, parent camera_low_color_frame, child camera_low_color_optical_frame, origin xyz=0 0 0 rpy=-1.5707963267948966 0 -1.5707963267948966
- added joint camera_low_depth_joint: type fixed, parent camera_low_link, child camera_low_depth_frame, origin xyz=0 0 0 rpy=0 0 0
- added joint camera_low_depth_optical_joint: type fixed, parent camera_low_depth_frame, child camera_low_depth_optical_frame, origin xyz=0 0 0 rpy=-1.5707963267948966 0 -1.5707963267948966
- added joint camera_low_infra1_joint: type fixed, parent camera_low_link, child camera_low_infra1_frame, origin xyz=0 0.0 0 rpy=0 0 0
- added joint camera_low_infra1_optical_joint: type fixed, parent camera_low_infra1_frame, child camera_low_infra1_optical_frame, origin xyz=0 0 0 rpy=-1.5707963267948966 0 -1.5707963267948966
- added joint camera_low_infra2_joint: type fixed, parent camera_low_link, child camera_low_infra2_frame, origin xyz=0 -0.018 0 rpy=0 0 0
- added joint camera_low_infra2_optical_joint: type fixed, parent camera_low_infra2_frame, child camera_low_infra2_optical_frame, origin xyz=0 0 0 rpy=-1.5707963267948966 0 -1.5707963267948966
- added joint camera_low_joint: type fixed, parent base_link, child camera_low_bottom_screw_frame, origin xyz=0.209805 0 1.031778 rpy=0 0.6457718232379019 0
- added joint camera_low_link_joint: type fixed, parent camera_low_bottom_screw_frame, child camera_low_link, origin xyz=0.01085 0.009 0.021 rpy=0 0 0

Commit message: camera naming

File: urdf/generated/mobile_ai.urdf (robot description, URDF)
Before this commit: robot mobile_ai, 68 links, 67 joints
Links:
- removed link camera_low_bottom_screw_frame
- removed link camera_low_color_frame
- removed link camera_low_color_optical_frame
- removed link camera_low_depth_frame
- removed link camera_low_depth_optical_frame
- removed link camera_low_infra1_frame
- removed link camera_low_infra1_optical_frame
- removed link camera_low_infra2_frame
- removed link camera_low_infra2_optical_frame
- removed link camera_low_link
- added link cam_high_bottom_screw_frame
- added link cam_high_color_frame
- added link cam_high_color_optical_frame
- added link cam_high_depth_frame
- added link cam_high_depth_optical_frame
- added link cam_high_infra1_frame
- added link cam_high_infra1_optical_frame
- added link cam_high_infra2_frame
- added link cam_high_infra2_optical_frame
- added link cam_high_link, mass 0.072; collision box size=0.023 0.042 0.042; visual mesh filename=package://trossen_arm_description/meshes/peripherals/d405.s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 scale=0.001 0.001 0.001
Joints:
- removed joint camera_low_color_joint
- removed joint camera_low_color_optical_joint
- removed joint camera_low_depth_joint
- removed joint camera_low_depth_optical_joint
- removed joint camera_low_infra1_joint
- removed joint camera_low_infra1_optical_joint
- removed joint camera_low_infra2_joint
- removed joint camera_low_infra2_optical_joint
- removed joint camera_low_joint
- removed joint camera_low_link_joint
- added joint cam_high_color_joint: type fixed, parent cam_high_link, child cam_high_color_frame, origin xyz=0 0.0 0 rpy=0 0 0
- added joint cam_high_color_optical_joint: type fixed, parent cam_high_color_frame, child cam_high_color_optical_frame, origin xyz=0 0 0 rpy=-1.5707963267948966 0 -1.5707963267948966
- added joint cam_high_depth_joint: type fixed, parent cam_high_link, child cam_high_depth_frame, origin xyz=0 0 0 rpy=0 0 0
- added joint cam_high_depth_optical_joint: type fixed, parent cam_high_depth_frame, child cam_high_depth_optical_frame, origin xyz=0 0 0 rpy=-1.5707963267948966 0 -1.5707963267948966
- added joint cam_high_infra1_joint: type fixed, parent cam_high_link, child cam_high_infra1_frame, origin xyz=0 0.0 0 rpy=0 0 0
- added joint cam_high_infra1_optical_joint: type fixed, parent cam_high_infra1_frame, child cam_high_infra1_optical_frame, origin xyz=0 0 0 rpy=-1.5707963267948966 0 -1.5707963267948966
- added joint cam_high_infra2_joint: type fixed, parent cam_high_link, child cam_high_infra2_frame, origin xyz=0 -0.018 0 rpy=0 0 0
- added joint cam_high_infra2_optical_joint: type fixed, parent cam_high_infra2_frame, child cam_high_infra2_optical_frame, origin xyz=0 0 0 rpy=-1.5707963267948966 0 -1.5707963267948966
- added joint cam_high_joint: type fixed, parent base_link, child cam_high_bottom_screw_frame, origin xyz=0.209805 0 1.031778 rpy=0 0.6457718232379019 0
- added joint cam_high_link_joint: type fixed, parent cam_high_bottom_screw_frame, child cam_high_link, origin xyz=0.01085 0.009 0.021 rpy=0 0 0

File: urdf/mobile_ai.urdf.xacro (robot description, xacro)
@@ -157,5 +157,5 @@
   <xacro:include filename="$(find trossen_arm_description)/urdf/peripherals/rs_d405.urdf.xacro" />
   <xacro:sensor_d405
-    name="camera_low"
+    name="cam_high"
     parent="base_link"
     use_nominal_extrinsics="true">

Commit message: update generated mobile-ai urdf

File: urdf/generated/mobile_ai.urdf (robot description, URDF)
Before this commit: robot mobile_ai, 68 links, 67 joints
Joints:
- joint caster_swivel_joint_front_left: limit (none) -> effort=0 velocity=3.141592653589793
- joint caster_swivel_joint_front_right: limit (none) -> effort=0 velocity=3.141592653589793
- joint caster_swivel_joint_rear_left: limit (none) -> effort=0 velocity=3.141592653589793
- joint caster_swivel_joint_rear_right: limit (none) -> effort=0 velocity=3.141592653589793
- joint caster_wheel_joint_front_left: limit (none) -> effort=0 velocity=3.141592653589793
- joint caster_wheel_joint_front_right: limit (none) -> effort=0 velocity=3.141592653589793
- joint caster_wheel_joint_rear_left: limit (none) -> effort=0 velocity=3.141592653589793
- joint caster_wheel_joint_rear_right: limit (none) -> effort=0 velocity=3.141592653589793
- joint left_wheel: limit effort=0 velocity=0 -> effort=4 velocity=12.566370614359172
- joint right_wheel: limit effort=0 velocity=0 -> effort=4 velocity=12.566370614359172

Commit message: put the default ee gripper to the tip of the fingers

File: urdf/generated/mobile_ai.urdf (robot description, URDF)
Before this commit: robot mobile_ai, 68 links, 67 joints
Joints:
- joint follower_left/ee_gripper: origin xyz=0.154 0 0 rpy=0 0 0 -> xyz=0.156062 0 0 rpy=0 0 0
- joint follower_right/ee_gripper: origin xyz=0.154 0 0 rpy=0 0 0 -> xyz=0.156062 0 0 rpy=0 0 0

File: urdf/generated/wxai/wxai_base.urdf (robot description, URDF)
Before this commit: robot wxai, 12 links, 11 joints
Joints:
- joint ee_gripper: origin xyz=0.154 0 0 rpy=0 0 0 -> xyz=0.156062 0 0 rpy=0 0 0

File: urdf/generated/wxai/wxai_follower.urdf (robot description, URDF)
Before this commit: robot wxai, 23 links, 22 joints
Joints:
- joint ee_gripper: origin xyz=0.154 0 0 rpy=0 0 0 -> xyz=0.156062 0 0 rpy=0 0 0

File: urdf/macros/_wxai.urdf.xacro (robot description, xacro)
@@ -781,5 +781,5 @@
       <joint name="${prefix}ee_gripper" type="fixed">
         <origin
-          xyz="0.154 0 0"
+          xyz="0.156062 0 0"
           rpy="0 0 0" />
         <parent link="${prefix}link_6" />

Commit message: removed axis of the fixed joints

File: urdf/generated/mobile_ai.urdf (robot description, URDF)
Before this commit: robot mobile_ai, 68 links, 67 joints
Joints:
- joint follower_left/camera_mount_joint: axis 0 0 0 -> (none)
- joint follower_left/ee_gripper: axis 1 0 0 -> (none)
- joint follower_left/left_gripper_joint: axis 0 0 0 -> (none)
- joint follower_left/right_carriage_joint: mimic (none) -> joint=follower_left/left_carriage_joint
- joint follower_left/right_gripper_joint: axis 0 0 0 -> (none)
- joint follower_right/camera_mount_joint: axis 0 0 0 -> (none)
- joint follower_right/ee_gripper: axis 1 0 0 -> (none)
- joint follower_right/left_gripper_joint: axis 0 0 0 -> (none)
- joint follower_right/right_carriage_joint: mimic (none) -> joint=follower_right/left_carriage_joint
- joint follower_right/right_gripper_joint: axis 0 0 0 -> (none)

File: urdf/generated/wxai/wxai_base.urdf (robot description, URDF)
Before this commit: robot wxai, 12 links, 11 joints
Joints:
- joint ee_gripper: axis 1 0 0 -> (none)
- joint left_gripper_joint: axis 0 0 0 -> (none)
- joint right_gripper_joint: axis 0 0 0 -> (none)

File: urdf/generated/wxai/wxai_follower.urdf (robot description, URDF)
Before this commit: robot wxai, 23 links, 22 joints
Joints:
- joint camera_mount_joint: axis 0 0 0 -> (none)
- joint ee_gripper: axis 1 0 0 -> (none)
- joint left_gripper_joint: axis 0 0 0 -> (none)
- joint right_gripper_joint: axis 0 0 0 -> (none)

File: urdf/generated/wxai/wxai_leader_left.urdf (robot description, URDF)
Before this commit: robot wxai, 12 links, 11 joints
Joints:
- joint handle_joint: axis 0 0 0 -> (none)
- joint left_index_joint: axis 0 0 0 -> (none)
- joint left_thumb_joint: axis 0 0 0 -> (none)

File: urdf/generated/wxai/wxai_leader_right.urdf (robot description, URDF)
Before this commit: robot wxai, 12 links, 11 joints
Joints:
- joint handle_joint: axis 0 0 0 -> (none)
- joint right_index_joint: axis 0 0 0 -> (none)
- joint right_thumb_joint: axis 0 0 0 -> (none)

File: urdf/macros/_wxai.urdf.xacro (robot description, xacro)
@@ -441,5 +441,4 @@
         <parent link="${prefix}link_6" />
         <child link="${prefix}camera_mount_d405" />
-        <axis xyz="0 0 0" />
       </joint>
       <xacro:include filename="$(find trossen_arm_description)/urdf/peripherals/rs_d405.urdf.xacro" />
@@ -493,5 +492,4 @@
           <parent link="${prefix}link_6" />
           <child link="${prefix}handle" />
-          <axis xyz="0 0 0" />
         </joint>
         <link name="${prefix}leader_finger_left_index">
@@ -533,5 +531,4 @@
           <parent link="${prefix}carriage_left" />
           <child link="${prefix}leader_finger_left_index" />
-          <axis xyz="0 0 0" />
         </joint>
         <link name="${prefix}leader_finger_left_thumb">
@@ -573,5 +570,4 @@
           <parent link="${prefix}carriage_right" />
           <child link="${prefix}leader_finger_left_thumb" />
-          <axis xyz="0 0 0" />
         </joint>
       </xacro:if> <!-- arm_side == 'left' -->
@@ -615,5 +611,4 @@
           <parent link="${prefix}link_6" />
           <child link="${prefix}handle" />
-          <axis xyz="0 0 0" />
         </joint>
         <link name="${prefix}leader_finger_right_thumb">
@@ -655,5 +650,4 @@
           <parent link="${prefix}carriage_left" />
           <child link="${prefix}leader_finger_right_thumb" />
-          <axis xyz="0 0 0" />
         </joint>
         <link name="${prefix}leader_finger_right_index">
@@ -695,5 +689,4 @@
           <parent link="${prefix}carriage_right" />
           <child link="${prefix}leader_finger_right_index" />
-          <axis xyz="0 0 0" />
         </joint>
       </xacro:if> <!-- leader_polarity == 'right' -->
@@ -738,5 +731,4 @@
         <parent link="${prefix}carriage_left" />
         <child link="${prefix}gripper_left" />
-        <axis xyz="0 0 0" />
       </joint>
       <link name="${prefix}gripper_right">
@@ -778,5 +770,4 @@
         <parent link="${prefix}carriage_right" />
         <child link="${prefix}gripper_right" />
-        <axis xyz="0 0 0" />
       </joint>
       <joint name="${prefix}ee_gripper" type="fixed">
@@ -786,5 +777,4 @@
         <parent link="${prefix}link_6" />
         <child link="${prefix}ee_gripper_link" />
-        <axis xyz="1 0 0" />
       </joint>
       <link name="${prefix}ee_gripper_link" />
