Commit message: matched widow joint limits with defaults

File: urdf/generated/mobile_ai.urdf (robot description, URDF)
Before this commit: robot mobile_ai, 68 links, 67 joints
Joints:
- joint follower_left/joint_0: limit lower=-3.0543261909900767 upper=3.0543261909900767 effort=27.0 velocity=3.375 -> lower=-3.141592653589793 upper=3.141592653589793 effort=27.0 velocity=6.283185307179586
- joint follower_left/joint_1: limit lower=0.0 upper=3.141592653589793 effort=27.0 velocity=3.375 -> lower=0.0 upper=3.141592653589793 effort=27.0 velocity=6.283185307179586
- joint follower_left/joint_2: limit lower=0.0 upper=2.356194490192345 effort=27.0 velocity=3.375 -> lower=0.0 upper=2.356194490192345 effort=27.0 velocity=6.283185307179586
- joint follower_left/joint_3: limit lower=-1.5707963267948966 upper=1.5707963267948966 effort=7.0 velocity=7.0 -> lower=-1.5707963267948966 upper=1.5707963267948966 effort=7.0 velocity=9.42477796076938
- joint follower_left/joint_4: limit lower=-1.5707963267948966 upper=1.5707963267948966 effort=7.0 velocity=7.0 -> lower=-1.5707963267948966 upper=1.5707963267948966 effort=7.0 velocity=9.42477796076938
- joint follower_left/joint_5: limit lower=-3.141592653589793 upper=3.141592653589793 effort=7.0 velocity=7.0 -> lower=-3.141592653589793 upper=3.141592653589793 effort=7.0 velocity=9.42477796076938
- joint follower_left/left_carriage_joint: limit lower=0.0 upper=0.044 effort=400.0 velocity=0.0875 -> lower=0.0 upper=0.04 effort=100.0 velocity=0.25
- joint follower_left/right_carriage_joint: limit lower=0.0 upper=0.044 effort=400.0 velocity=0.0875 -> lower=0.0 upper=0.04 effort=100.0 velocity=0.25
- joint follower_right/joint_0: limit lower=-3.0543261909900767 upper=3.0543261909900767 effort=27.0 velocity=3.375 -> lower=-3.141592653589793 upper=3.141592653589793 effort=27.0 velocity=6.283185307179586
- joint follower_right/joint_1: limit lower=0.0 upper=3.141592653589793 effort=27.0 velocity=3.375 -> lower=0.0 upper=3.141592653589793 effort=27.0 velocity=6.283185307179586
- joint follower_right/joint_2: limit lower=0.0 upper=2.356194490192345 effort=27.0 velocity=3.375 -> lower=0.0 upper=2.356194490192345 effort=27.0 velocity=6.283185307179586
- joint follower_right/joint_3: limit lower=-1.5707963267948966 upper=1.5707963267948966 effort=7.0 velocity=7.0 -> lower=-1.5707963267948966 upper=1.5707963267948966 effort=7.0 velocity=9.42477796076938
- joint follower_right/joint_4: limit lower=-1.5707963267948966 upper=1.5707963267948966 effort=7.0 velocity=7.0 -> lower=-1.5707963267948966 upper=1.5707963267948966 effort=7.0 velocity=9.42477796076938
- joint follower_right/joint_5: limit lower=-3.141592653589793 upper=3.141592653589793 effort=7.0 velocity=7.0 -> lower=-3.141592653589793 upper=3.141592653589793 effort=7.0 velocity=9.42477796076938
- joint follower_right/left_carriage_joint: limit lower=0.0 upper=0.044 effort=400.0 velocity=0.0875 -> lower=0.0 upper=0.04 effort=100.0 velocity=0.25
- joint follower_right/right_carriage_joint: limit lower=0.0 upper=0.044 effort=400.0 velocity=0.0875 -> lower=0.0 upper=0.04 effort=100.0 velocity=0.25

File: urdf/generated/wxai/wxai_base.urdf (robot description, URDF)
Before this commit: robot wxai, 12 links, 11 joints
Joints:
- joint joint_0: limit lower=-3.0543261909900767 upper=3.0543261909900767 effort=27.0 velocity=3.375 -> lower=-3.141592653589793 upper=3.141592653589793 effort=27.0 velocity=6.283185307179586
- joint joint_1: limit lower=0.0 upper=3.141592653589793 effort=27.0 velocity=3.375 -> lower=0.0 upper=3.141592653589793 effort=27.0 velocity=6.283185307179586
- joint joint_2: limit lower=0.0 upper=2.356194490192345 effort=27.0 velocity=3.375 -> lower=0.0 upper=2.356194490192345 effort=27.0 velocity=6.283185307179586
- joint joint_3: limit lower=-1.5707963267948966 upper=1.5707963267948966 effort=7.0 velocity=7.0 -> lower=-1.5707963267948966 upper=1.5707963267948966 effort=7.0 velocity=9.42477796076938
- joint joint_4: limit lower=-1.5707963267948966 upper=1.5707963267948966 effort=7.0 velocity=7.0 -> lower=-1.5707963267948966 upper=1.5707963267948966 effort=7.0 velocity=9.42477796076938
- joint joint_5: limit lower=-3.141592653589793 upper=3.141592653589793 effort=7.0 velocity=7.0 -> lower=-3.141592653589793 upper=3.141592653589793 effort=7.0 velocity=9.42477796076938
- joint left_carriage_joint: limit lower=0.0 upper=0.044 effort=400.0 velocity=0.0875 -> lower=0.0 upper=0.04 effort=100.0 velocity=0.25
- joint right_carriage_joint: limit lower=0.0 upper=0.044 effort=400.0 velocity=0.0875 -> lower=0.0 upper=0.04 effort=100.0 velocity=0.25

File: urdf/generated/wxai/wxai_follower.urdf (robot description, URDF)
Before this commit: robot wxai, 23 links, 22 joints
Joints:
- joint joint_0: limit lower=-3.0543261909900767 upper=3.0543261909900767 effort=27.0 velocity=3.375 -> lower=-3.141592653589793 upper=3.141592653589793 effort=27.0 velocity=6.283185307179586
- joint joint_1: limit lower=0.0 upper=3.141592653589793 effort=27.0 velocity=3.375 -> lower=0.0 upper=3.141592653589793 effort=27.0 velocity=6.283185307179586
- joint joint_2: limit lower=0.0 upper=2.356194490192345 effort=27.0 velocity=3.375 -> lower=0.0 upper=2.356194490192345 effort=27.0 velocity=6.283185307179586
- joint joint_3: limit lower=-1.5707963267948966 upper=1.5707963267948966 effort=7.0 velocity=7.0 -> lower=-1.5707963267948966 upper=1.5707963267948966 effort=7.0 velocity=9.42477796076938
- joint joint_4: limit lower=-1.5707963267948966 upper=1.5707963267948966 effort=7.0 velocity=7.0 -> lower=-1.5707963267948966 upper=1.5707963267948966 effort=7.0 velocity=9.42477796076938
- joint joint_5: limit lower=-3.141592653589793 upper=3.141592653589793 effort=7.0 velocity=7.0 -> lower=-3.141592653589793 upper=3.141592653589793 effort=7.0 velocity=9.42477796076938
- joint left_carriage_joint: limit lower=0.0 upper=0.044 effort=400.0 velocity=0.0875 -> lower=0.0 upper=0.04 effort=100.0 velocity=0.25
- joint right_carriage_joint: limit lower=0.0 upper=0.044 effort=400.0 velocity=0.0875 -> lower=0.0 upper=0.04 effort=100.0 velocity=0.25

File: urdf/generated/wxai/wxai_leader_left.urdf (robot description, URDF)
Before this commit: robot wxai, 12 links, 11 joints
Joints:
- joint joint_0: limit lower=-3.0543261909900767 upper=3.0543261909900767 effort=27.0 velocity=3.375 -> lower=-3.141592653589793 upper=3.141592653589793 effort=27.0 velocity=6.283185307179586
- joint joint_1: limit lower=0.0 upper=3.141592653589793 effort=27.0 velocity=3.375 -> lower=0.0 upper=3.141592653589793 effort=27.0 velocity=6.283185307179586
- joint joint_2: limit lower=0.0 upper=2.356194490192345 effort=27.0 velocity=3.375 -> lower=0.0 upper=2.356194490192345 effort=27.0 velocity=6.283185307179586
- joint joint_3: limit lower=-1.5707963267948966 upper=1.5707963267948966 effort=7.0 velocity=7.0 -> lower=-1.5707963267948966 upper=1.5707963267948966 effort=7.0 velocity=9.42477796076938
- joint joint_4: limit lower=-1.5707963267948966 upper=1.5707963267948966 effort=7.0 velocity=7.0 -> lower=-1.5707963267948966 upper=1.5707963267948966 effort=7.0 velocity=9.42477796076938
- joint joint_5: limit lower=-3.141592653589793 upper=3.141592653589793 effort=7.0 velocity=7.0 -> lower=-3.141592653589793 upper=3.141592653589793 effort=7.0 velocity=9.42477796076938
- joint left_carriage_joint: limit lower=0.0 upper=0.044 effort=400.0 velocity=0.0875 -> lower=0.0 upper=0.04 effort=100.0 velocity=0.25
- joint right_carriage_joint: limit lower=0.0 upper=0.044 effort=400.0 velocity=0.0875 -> lower=0.0 upper=0.04 effort=100.0 velocity=0.25

File: urdf/generated/wxai/wxai_leader_right.urdf (robot description, URDF)
Before this commit: robot wxai, 12 links, 11 joints
Joints:
- joint joint_0: limit lower=-3.0543261909900767 upper=3.0543261909900767 effort=27.0 velocity=3.375 -> lower=-3.141592653589793 upper=3.141592653589793 effort=27.0 velocity=6.283185307179586
- joint joint_1: limit lower=0.0 upper=3.141592653589793 effort=27.0 velocity=3.375 -> lower=0.0 upper=3.141592653589793 effort=27.0 velocity=6.283185307179586
- joint joint_2: limit lower=0.0 upper=2.356194490192345 effort=27.0 velocity=3.375 -> lower=0.0 upper=2.356194490192345 effort=27.0 velocity=6.283185307179586
- joint joint_3: limit lower=-1.5707963267948966 upper=1.5707963267948966 effort=7.0 velocity=7.0 -> lower=-1.5707963267948966 upper=1.5707963267948966 effort=7.0 velocity=9.42477796076938
- joint joint_4: limit lower=-1.5707963267948966 upper=1.5707963267948966 effort=7.0 velocity=7.0 -> lower=-1.5707963267948966 upper=1.5707963267948966 effort=7.0 velocity=9.42477796076938
- joint joint_5: limit lower=-3.141592653589793 upper=3.141592653589793 effort=7.0 velocity=7.0 -> lower=-3.141592653589793 upper=3.141592653589793 effort=7.0 velocity=9.42477796076938
- joint left_carriage_joint: limit lower=0.0 upper=0.044 effort=400.0 velocity=0.0875 -> lower=0.0 upper=0.04 effort=100.0 velocity=0.25
- joint right_carriage_joint: limit lower=0.0 upper=0.044 effort=400.0 velocity=0.0875 -> lower=0.0 upper=0.04 effort=100.0 velocity=0.25

File: urdf/macros/_wxai.urdf.xacro (robot description, xacro)
@@ -81,8 +81,8 @@
       <axis xyz="0 0 1" />
       <limit
-        lower="${-radians(180 - 5)}"
-        upper="${radians(180 - 5)}"
+        lower="-${pi}"
+        upper="${pi}"
         effort="27.0"
-        velocity="3.375" />
+        velocity="${2 * pi}" />
     </joint>
     <link name="${prefix}link_2">
@@ -129,5 +129,5 @@
         upper="${pi}"
         effort="27.0"
-        velocity="3.375" />
+        velocity="${2 * pi}" />
     </joint>
     <link name="${prefix}link_3">
@@ -174,5 +174,5 @@
         upper="${3 * pi / 4}"
         effort="27.0"
-        velocity="3.375" />
+        velocity="${2 * pi}" />
     </joint>
     <link name="${prefix}link_4">
@@ -219,5 +219,5 @@
         upper="${pi / 2.0}"
         effort="7.0"
-        velocity="7.0" />
+        velocity="${3 * pi}" />
     </joint>
     <link name="${prefix}link_5">
@@ -264,5 +264,5 @@
         upper="${pi / 2.0}"
         effort="7.0"
-        velocity="7.0" />
+        velocity="${3 * pi}" />
     </joint>
     <link name="${prefix}link_6">
@@ -309,5 +309,5 @@
         upper="${pi}"
         effort="7.0"
-        velocity="7.0" />
+        velocity="${3 * pi}" />
     </joint>
     <link name="${prefix}carriage_right">
@@ -353,7 +353,7 @@
       <limit
         lower="0.0"
-        upper="0.044"
-        effort="400.0"
-        velocity="0.0875" />
+        upper="0.04"
+        effort="100.0"
+        velocity="0.25" />
     </joint>
     <link name="${prefix}carriage_left">
@@ -398,7 +398,7 @@
       <limit
         lower="0.0"
-        upper="0.044"
-        effort="400.0"
-        velocity="0.0875" />
+        upper="0.04"
+        effort="100.0"
+        velocity="0.25" />
     </joint>
     <xacro:if value="${variant == 'follower'}">
