Commit message: update wheel mass, add ip address and ros control to both the arms

File: urdf/generated/mobile_ai.urdf (robot description, URDF)
Before this commit: robot mobile_ai, 68 links, 67 joints
Links:
- removed link follower_left/base_link
- removed link follower_left/camera_bottom_screw_frame
- removed link follower_left/camera_color_frame
- removed link follower_left/camera_color_optical_frame
- removed link follower_left/camera_depth_frame
- removed link follower_left/camera_depth_optical_frame
- removed link follower_left/camera_infra1_frame
- removed link follower_left/camera_infra1_optical_frame
- removed link follower_left/camera_infra2_frame
- removed link follower_left/camera_infra2_optical_frame
- removed link follower_left/camera_link
- removed link follower_left/camera_mount_d405
- removed link follower_left/carriage_left
- removed link follower_left/carriage_right
- removed link follower_left/ee_gripper_link
- removed link follower_left/gripper_left
- removed link follower_left/gripper_right
- removed link follower_left/link_1
- removed link follower_left/link_2
- removed link follower_left/link_3
- removed link follower_left/link_4
- removed link follower_left/link_5
- removed link follower_left/link_6
- removed link follower_right/base_link
- removed link follower_right/camera_bottom_screw_frame
- removed link follower_right/camera_color_frame
- removed link follower_right/camera_color_optical_frame
- removed link follower_right/camera_depth_frame
- removed link follower_right/camera_depth_optical_frame
- removed link follower_right/camera_infra1_frame
- removed link follower_right/camera_infra1_optical_frame
- removed link follower_right/camera_infra2_frame
- removed link follower_right/camera_infra2_optical_frame
- removed link follower_right/camera_link
- removed link follower_right/camera_mount_d405
- removed link follower_right/carriage_left
- removed link follower_right/carriage_right
- removed link follower_right/ee_gripper_link
- removed link follower_right/gripper_left
- removed link follower_right/gripper_right
- removed link follower_right/link_1
- removed link follower_right/link_2
- removed link follower_right/link_3
- removed link follower_right/link_4
- removed link follower_right/link_5
- removed link follower_right/link_6
- added link follower_left_base_link, mass 0.45969858; collision mesh filename=package://trossen_arm_description/meshes/wxai/base_link.stl; visual mesh filename=package://trossen_arm_description/meshes/wxai/base_link.stl
- added link follower_left_camera_bottom_screw_frame
- added link follower_left_camera_color_frame
- added link follower_left_camera_color_optical_frame
- added link follower_left_camera_depth_frame
- added link follower_left_camera_depth_optical_frame
- added link follower_left_camera_infra1_frame
- added link follower_left_camera_infra1_optical_frame
- added link follower_left_camera_infra2_frame
- added link follower_left_camera_infra2_optical_frame
- added link follower_left_camera_link, mass 0.072; collision box size=0.023 0.042 0.042; visual mesh filename=package://trossen_arm_description/meshes/peripherals/d405.s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 scale=0.001 0.001 0.001
- added link follower_left_camera_mount_d405, mass 0.04518012; collision mesh filename=package://trossen_arm_description/meshes/wxai/camera_mount_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; visual mesh filename=package://trossen_arm_description/meshes/wxai/camera_mount_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
- added link follower_left_carriage_left, mass 0.05036313; collision mesh filename=package://trossen_arm_description/meshes/wxai/carriage_left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; visual mesh filename=package://trossen_arm_description/meshes/wxai/carriage_left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
- added link follower_left_carriage_right, mass 0.05036313; collision mesh filename=package://trossen_arm_description/meshes/wxai/carriage_righ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; visual mesh filename=package://trossen_arm_description/meshes/wxai/carriage_righ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
- added link follower_left_ee_gripper_link
- added link follower_left_gripper_left, mass 0.03090787; collision mesh filename=package://trossen_arm_description/meshes/wxai/gripper_left.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; visual mesh filename=package://trossen_arm_description/meshes/wxai/gripper_left.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
- added link follower_left_gripper_right, mass 0.03090786; collision mesh filename=package://trossen_arm_description/meshes/wxai/gripper_right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; visual mesh filename=package://trossen_arm_description/meshes/wxai/gripper_right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
- added link follower_left_link_1, mass 0.15270428; collision mesh filename=package://trossen_arm_description/meshes/wxai/link_1.stl; visual mesh filename=package://trossen_arm_description/meshes/wxai/link_1.stl
- added link follower_left_link_2, mass 1.15316319; collision mesh filename=package://trossen_arm_description/meshes/wxai/link_2.stl; visual mesh filename=package://trossen_arm_description/meshes/wxai/link_2.stl
- added link follower_left_link_3, mass 0.68666638; collision mesh filename=package://trossen_arm_description/meshes/wxai/link_3.stl; visual mesh filename=package://trossen_arm_description/meshes/wxai/link_3.stl
- added link follower_left_link_4, mass 0.45789905; collision mesh filename=package://trossen_arm_description/meshes/wxai/link_4.stl; visual mesh filename=package://trossen_arm_description/meshes/wxai/link_4.stl
- added link follower_left_link_5, mass 0.36693910; collision mesh filename=package://trossen_arm_description/meshes/wxai/link_5.stl; visual mesh filename=package://trossen_arm_description/meshes/wxai/link_5.stl
- added link follower_left_link_6, mass 0.55469347; collision mesh filename=package://trossen_arm_description/meshes/wxai/link_6.stl; visual mesh filename=package://trossen_arm_description/meshes/wxai/link_6.stl
- added link follower_right_base_link, mass 0.45969858; collision mesh filename=package://trossen_arm_description/meshes/wxai/base_link.stl; visual mesh filename=package://trossen_arm_description/meshes/wxai/base_link.stl
- added link follower_right_camera_bottom_screw_frame
- added link follower_right_camera_color_frame
- added link follower_right_camera_color_optical_frame
- added link follower_right_camera_depth_frame
- added link follower_right_camera_depth_optical_frame
- added link follower_right_camera_infra1_frame
- added link follower_right_camera_infra1_optical_frame
- added link follower_right_camera_infra2_frame
- added link follower_right_camera_infra2_optical_frame
- added link follower_right_camera_link, mass 0.072; collision box size=0.023 0.042 0.042; visual mesh filename=package://trossen_arm_description/meshes/peripherals/d405.s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 scale=0.001 0.001 0.001
- added link follower_right_camera_mount_d405, mass 0.04518012; collision mesh filename=package://trossen_arm_description/meshes/wxai/camera_mount_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; visual mesh filename=package://trossen_arm_description/meshes/wxai/camera_mount_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
- added link follower_right_carriage_left, mass 0.05036313; collision mesh filename=package://trossen_arm_description/meshes/wxai/carriage_left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; visual mesh filename=package://trossen_arm_description/meshes/wxai/carriage_left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
- added link follower_right_carriage_right, mass 0.05036313; collision mesh filename=package://trossen_arm_description/meshes/wxai/carriage_righ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; visual mesh filename=package://trossen_arm_description/meshes/wxai/carriage_righ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
- added link follower_right_ee_gripper_link
- added link follower_right_gripper_left, mass 0.03090787; collision mesh filename=package://trossen_arm_description/meshes/wxai/gripper_left.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; visual mesh filename=package://trossen_arm_description/meshes/wxai/gripper_left.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
- added link follower_right_gripper_right, mass 0.03090786; collision mesh filename=package://trossen_arm_description/meshes/wxai/gripper_right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; visual mesh filename=package://trossen_arm_description/meshes/wxai/gripper_right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
- added link follower_right_link_1, mass 0.15270428; collision mesh filename=package://trossen_arm_description/meshes/wxai/link_1.stl; visual mesh filename=package://trossen_arm_description/meshes/wxai/link_1.stl
- added link follower_right_link_2, mass 1.15316319; collision mesh filename=package://trossen_arm_description/meshes/wxai/link_2.stl; visual mesh filename=package://trossen_arm_description/meshes/wxai/link_2.stl
- added link follower_right_link_3, mass 0.68666638; collision mesh filename=package://trossen_arm_description/meshes/wxai/link_3.stl; visual mesh filename=package://trossen_arm_description/meshes/wxai/link_3.stl
- added link follower_right_link_4, mass 0.45789905; collision mesh filename=package://trossen_arm_description/meshes/wxai/link_4.stl; visual mesh filename=package://trossen_arm_description/meshes/wxai/link_4.stl
- added link follower_right_link_5, mass 0.36693910; collision mesh filename=package://trossen_arm_description/meshes/wxai/link_5.stl; visual mesh filename=package://trossen_arm_description/meshes/wxai/link_5.stl
- added link follower_right_link_6, mass 0.55469347; collision mesh filename=package://trossen_arm_description/meshes/wxai/link_6.stl; visual mesh filename=package://trossen_arm_description/meshes/wxai/link_6.stl
- link right_wheel_link: mass 0.981755254019503 -> 3.00000000
Joints:
- removed joint follower_left/camera_color_joint
- removed joint follower_left/camera_color_optical_joint
- removed joint follower_left/camera_depth_joint
- removed joint follower_left/camera_depth_optical_joint
- removed joint follower_left/camera_infra1_joint
- removed joint follower_left/camera_infra1_optical_joint
- removed joint follower_left/camera_infra2_joint
- removed joint follower_left/camera_infra2_optical_joint
- removed joint follower_left/camera_joint
- removed joint follower_left/camera_link_joint
- removed joint follower_left/camera_mount_joint
- removed joint follower_left/ee_gripper
- removed joint follower_left/joint_0
- removed joint follower_left/joint_1
- removed joint follower_left/joint_2
- removed joint follower_left/joint_3
- removed joint follower_left/joint_4
- removed joint follower_left/joint_5
- removed joint follower_left/left_carriage_joint
- removed joint follower_left/left_gripper_joint
- removed joint follower_left/right_carriage_joint
- removed joint follower_left/right_gripper_joint
- removed joint follower_right/camera_color_joint
- removed joint follower_right/camera_color_optical_joint
- removed joint follower_right/camera_depth_joint
- removed joint follower_right/camera_depth_optical_joint
- removed joint follower_right/camera_infra1_joint
- removed joint follower_right/camera_infra1_optical_joint
- removed joint follower_right/camera_infra2_joint
- removed joint follower_right/camera_infra2_optical_joint
- removed joint follower_right/camera_joint
- removed joint follower_right/camera_link_joint
- removed joint follower_right/camera_mount_joint
- removed joint follower_right/ee_gripper
- removed joint follower_right/joint_0
- removed joint follower_right/joint_1
- removed joint follower_right/joint_2
- removed joint follower_right/joint_3
- removed joint follower_right/joint_4
- removed joint follower_right/joint_5
- removed joint follower_right/left_carriage_joint
- removed joint follower_right/left_gripper_joint
- removed joint follower_right/right_carriage_joint
- removed joint follower_right/right_gripper_joint
- added joint follower_left_camera_color_joint: type fixed, parent follower_left_camera_link, child follower_left_camera_color_frame, origin xyz=0 0.0 0 rpy=0 0 0
- added joint follower_left_camera_color_optical_joint: type fixed, parent follower_left_camera_color_frame, child follower_left_camera_color_optical_frame, origin xyz=0 0 0 rpy=-1.5707963267948966 0 -1.5707963267948966
- added joint follower_left_camera_depth_joint: type fixed, parent follower_left_camera_link, child follower_left_camera_depth_frame, origin xyz=0 0 0 rpy=0 0 0
- added joint follower_left_camera_depth_optical_joint: type fixed, parent follower_left_camera_depth_frame, child follower_left_camera_depth_optical_frame, origin xyz=0 0 0 rpy=-1.5707963267948966 0 -1.5707963267948966
- added joint follower_left_camera_infra1_joint: type fixed, parent follower_left_camera_link, child follower_left_camera_infra1_frame, origin xyz=0 0.0 0 rpy=0 0 0
- added joint follower_left_camera_infra1_optical_joint: type fixed, parent follower_left_camera_infra1_frame, child follower_left_camera_infra1_optical_frame, origin xyz=0 0 0 rpy=-1.5707963267948966 0 -1.5707963267948966
- added joint follower_left_camera_infra2_joint: type fixed, parent follower_left_camera_link, child follower_left_camera_infra2_frame, origin xyz=0 -0.018 0 rpy=0 0 0
- added joint follower_left_camera_infra2_optical_joint: type fixed, parent follower_left_camera_infra2_frame, child follower_left_camera_infra2_optical_frame, origin xyz=0 0 0 rpy=-1.5707963267948966 0 -1.5707963267948966
- added joint follower_left_camera_joint: type fixed, parent follower_left_camera_mount_d405, child follower_left_camera_bottom_screw_frame, origin xyz=0.02927207801 0 0.03824951197 rpy=0 0.3490658503988659 0
- added joint follower_left_camera_link_joint: type fixed, parent follower_left_camera_bottom_screw_frame, child follower_left_camera_link, origin xyz=0.01085 0.009 0.021 rpy=0 0 0
- added joint follower_left_camera_mount_joint: type fixed, parent follower_left_link_6, child follower_left_camera_mount_d405, origin xyz=0.012 0 0 rpy=0 0 0
- added joint follower_left_ee_gripper: type fixed, parent follower_left_link_6, child follower_left_ee_gripper_link, origin xyz=0.156062 0 0 rpy=0 0 0
- added joint follower_left_joint_0: type revolute, parent follower_left_base_link, child follower_left_link_1, origin xyz=0 0 0.05725 rpy=0 0 0, axis 0 0 1, limit lower=-3.0543261909900767 upper=3.0543261909900767 effort=27.0 velocity=3.375
- added joint follower_left_joint_1: type revolute, parent follower_left_link_1, child follower_left_link_2, origin xyz=0.02 0 0.04625 rpy=0 0 0, axis 0 1 0, limit lower=0.0 upper=3.141592653589793 effort=27.0 velocity=3.375
- added joint follower_left_joint_2: type revolute, parent follower_left_link_2, child follower_left_link_3, origin xyz=-0.264 0 0 rpy=0 0 0, axis 0 -1 0, limit lower=0.0 upper=2.356194490192345 effort=27.0 velocity=3.375
- added joint follower_left_joint_3: type revolute, parent follower_left_link_3, child follower_left_link_4, origin xyz=0.245 0 0.06 rpy=0 0 0, axis 0 -1 0, limit lower=-1.5707963267948966 upper=1.5707963267948966 effort=7.0 velocity=7.0
- added joint follower_left_joint_4: type revolute, parent follower_left_link_4, child follower_left_link_5, origin xyz=0.06775 0 0.0455 rpy=0 0 0, axis 0 0 -1, limit lower=-1.5707963267948966 upper=1.5707963267948966 effort=7.0 velocity=7.0
- added joint follower_left_joint_5: type revolute, parent follower_left_link_5, child follower_left_link_6, origin xyz=0.02895 0 -0.0455 rpy=0 0 0, axis 1 0 0, limit lower=-3.141592653589793 upper=3.141592653589793 effort=7.0 velocity=7.0
- added joint follower_left_left_carriage_joint: type prismatic, parent follower_left_link_6, child follower_left_carriage_left, origin xyz=0.0865 0.023 0 rpy=0 0 0, axis 0 1 0, limit lower=0.0 upper=0.044 effort=400.0 velocity=0.0875
- added joint follower_left_left_gripper_joint: type fixed, parent follower_left_carriage_left, child follower_left_gripper_left, origin xyz=0 0 0 rpy=0 0 0
- added joint follower_left_right_carriage_joint: type prismatic, parent follower_left_link_6, child follower_left_carriage_right, origin xyz=0.0865 -0.023 0 rpy=0 0 0, axis 0 -1 0, limit lower=0.0 upper=0.044 effort=400.0 velocity=0.0875, mimic joint=follower_left_left_carriage_joint
- added joint follower_left_right_gripper_joint: type fixed, parent follower_left_carriage_right, child follower_left_gripper_right, origin xyz=0 0 0 rpy=0 0 0
- added joint follower_right_camera_color_joint: type fixed, parent follower_right_camera_link, child follower_right_camera_color_frame, origin xyz=0 0.0 0 rpy=0 0 0
- added joint follower_right_camera_color_optical_joint: type fixed, parent follower_right_camera_color_frame, child follower_right_camera_color_optical_frame, origin xyz=0 0 0 rpy=-1.5707963267948966 0 -1.5707963267948966
- added joint follower_right_camera_depth_joint: type fixed, parent follower_right_camera_link, child follower_right_camera_depth_frame, origin xyz=0 0 0 rpy=0 0 0
- added joint follower_right_camera_depth_optical_joint: type fixed, parent follower_right_camera_depth_frame, child follower_right_camera_depth_optical_frame, origin xyz=0 0 0 rpy=-1.5707963267948966 0 -1.5707963267948966
- added joint follower_right_camera_infra1_joint: type fixed, parent follower_right_camera_link, child follower_right_camera_infra1_frame, origin xyz=0 0.0 0 rpy=0 0 0
- added joint follower_right_camera_infra1_optical_joint: type fixed, parent follower_right_camera_infra1_frame, child follower_right_camera_infra1_optical_frame, origin xyz=0 0 0 rpy=-1.5707963267948966 0 -1.5707963267948966
- added joint follower_right_camera_infra2_joint: type fixed, parent follower_right_camera_link, child follower_right_camera_infra2_frame, origin xyz=0 -0.018 0 rpy=0 0 0
- added joint follower_right_camera_infra2_optical_joint: type fixed, parent follower_right_camera_infra2_frame, child follower_right_camera_infra2_optical_frame, origin xyz=0 0 0 rpy=-1.5707963267948966 0 -1.5707963267948966
- added joint follower_right_camera_joint: type fixed, parent follower_right_camera_mount_d405, child follower_right_camera_bottom_screw_frame, origin xyz=0.02927207801 0 0.03824951197 rpy=0 0.3490658503988659 0
- added joint follower_right_camera_link_joint: type fixed, parent follower_right_camera_bottom_screw_frame, child follower_right_camera_link, origin xyz=0.01085 0.009 0.021 rpy=0 0 0
- added joint follower_right_camera_mount_joint: type fixed, parent follower_right_link_6, child follower_right_camera_mount_d405, origin xyz=0.012 0 0 rpy=0 0 0
- added joint follower_right_ee_gripper: type fixed, parent follower_right_link_6, child follower_right_ee_gripper_link, origin xyz=0.156062 0 0 rpy=0 0 0
- added joint follower_right_joint_0: type revolute, parent follower_right_base_link, child follower_right_link_1, origin xyz=0 0 0.05725 rpy=0 0 0, axis 0 0 1, limit lower=-3.0543261909900767 upper=3.0543261909900767 effort=27.0 velocity=3.375
- added joint follower_right_joint_1: type revolute, parent follower_right_link_1, child follower_right_link_2, origin xyz=0.02 0 0.04625 rpy=0 0 0, axis 0 1 0, limit lower=0.0 upper=3.141592653589793 effort=27.0 velocity=3.375
- added joint follower_right_joint_2: type revolute, parent follower_right_link_2, child follower_right_link_3, origin xyz=-0.264 0 0 rpy=0 0 0, axis 0 -1 0, limit lower=0.0 upper=2.356194490192345 effort=27.0 velocity=3.375
- added joint follower_right_joint_3: type revolute, parent follower_right_link_3, child follower_right_link_4, origin xyz=0.245 0 0.06 rpy=0 0 0, axis 0 -1 0, limit lower=-1.5707963267948966 upper=1.5707963267948966 effort=7.0 velocity=7.0
- added joint follower_right_joint_4: type revolute, parent follower_right_link_4, child follower_right_link_5, origin xyz=0.06775 0 0.0455 rpy=0 0 0, axis 0 0 -1, limit lower=-1.5707963267948966 upper=1.5707963267948966 effort=7.0 velocity=7.0
- added joint follower_right_joint_5: type revolute, parent follower_right_link_5, child follower_right_link_6, origin xyz=0.02895 0 -0.0455 rpy=0 0 0, axis 1 0 0, limit lower=-3.141592653589793 upper=3.141592653589793 effort=7.0 velocity=7.0
- added joint follower_right_left_carriage_joint: type prismatic, parent follower_right_link_6, child follower_right_carriage_left, origin xyz=0.0865 0.023 0 rpy=0 0 0, axis 0 1 0, limit lower=0.0 upper=0.044 effort=400.0 velocity=0.0875
- added joint follower_right_left_gripper_joint: type fixed, parent follower_right_carriage_left, child follower_right_gripper_left, origin xyz=0 0 0 rpy=0 0 0
- added joint follower_right_right_carriage_joint: type prismatic, parent follower_right_link_6, child follower_right_carriage_right, origin xyz=0.0865 -0.023 0 rpy=0 0 0, axis 0 -1 0, limit lower=0.0 upper=0.044 effort=400.0 velocity=0.0875, mimic joint=follower_right_left_carriage_joint
- added joint follower_right_right_gripper_joint: type fixed, parent follower_right_carriage_right, child follower_right_gripper_right, origin xyz=0 0 0 rpy=0 0 0

File: urdf/mobile_ai.urdf.xacro (robot description, xacro)
@@ -1,4 +1,7 @@
 <?xml version="1.0" encoding="utf-8"?>
 <robot name="mobile_ai" xmlns:xacro="http://ros.org/wiki/xacro">
+  <xacro:arg name="ip_address_left" default="192.168.1.5"/>
+  <xacro:arg name="ip_address_right" default="192.168.1.4"/>
+  <xacro:arg name="ros2_control_hardware_type" default="mock_components"/>
   <xacro:property name="robot_model"
     value="mobile_ai"
@@ -218,5 +221,5 @@
         xyz="0 0 0"
         rpy="0 0 0" />
-      <mass value="0.981755254019503" />
+      <mass value="3.00000000" />
       <inertia
         ixx="0.00165792997375718"
@@ -280,5 +283,7 @@
   <xacro:wxai
     variant="follower"
-    prefix="follower_left/"/>
+    prefix="follower_left_"
+    ip_address="$(arg ip_address_left)"
+    ros2_control_hardware_type="$(arg ros2_control_hardware_type)"/>
   <joint
     name="follower_right/mount_joint"
@@ -292,4 +297,6 @@
   <xacro:wxai
     variant="follower"
-    prefix="follower_right/"/>
+    prefix="follower_right_"
+    ip_address="$(arg ip_address_right)"
+    ros2_control_hardware_type="$(arg ros2_control_hardware_type)"/>
 </robot>

Commit message: replace / with _ for the link and joint name

File: urdf/generated/mobile_ai.urdf (robot description, URDF)
Before this commit: robot mobile_ai, 68 links, 67 joints
Joints:
- removed joint follower_left/mount_joint
- removed joint follower_right/mount_joint
- added joint follower_left_mount_joint: type fixed, parent base_link, child follower_left_base_link, origin xyz=0.331 0.3 0.831 rpy=0 0 0
- added joint follower_right_mount_joint: type fixed, parent base_link, child follower_right_base_link, origin xyz=0.331 -0.3 0.831 rpy=0 0 0

File: urdf/mobile_ai.urdf.xacro (robot description, xacro)
@@ -273,5 +273,5 @@
   </xacro:caster_wheel>
   <joint
-    name="follower_left/mount_joint"
+    name="follower_left_mount_joint"
     type="fixed">
     <origin
@@ -279,5 +279,5 @@
       rpy="0 0 0" />
     <parent link="base_link" />
-    <child link="follower_left/base_link" />
+    <child link="follower_left_base_link" />
   </joint>
   <xacro:wxai
@@ -287,5 +287,5 @@
     ros2_control_hardware_type="$(arg ros2_control_hardware_type)"/>
   <joint
-    name="follower_right/mount_joint"
+    name="follower_right_mount_joint"
     type="fixed">
     <origin
@@ -293,5 +293,5 @@
       rpy="0 0 0" />
     <parent link="base_link" />
-    <child link="follower_right/base_link" />
+    <child link="follower_right_base_link" />
   </joint>
   <xacro:wxai
