Commit message: set trigger joint limits

File: urdf/generated/glide_left.urdf (robot description, URDF)
Before this commit: robot glide_left, 8 links, 7 joints
Joints:
- joint joint_6: limit lower=0.0 upper=4.571428571428571 effort=0.8750000000000001 velocity=28.57142857142857 -> lower=0.0 upper=0.7853981633974483 effort=1.8 velocity=5.0

File: urdf/generated/glide_right.urdf (robot description, URDF)
Before this commit: robot glide_right, 8 links, 7 joints
Joints:
- joint joint_6: limit lower=0.0 upper=4.571428571428571 effort=0.8750000000000001 velocity=28.57142857142857 -> lower=0.0 upper=0.7853981633974483 effort=1.8 velocity=5.0

File: urdf/macros/_glide_left.urdf.xacro (robot description, xacro)
@@ -7,5 +7,4 @@
     <xacro:property name="mesh_directory" value="package://trossen_arm_description/meshes/${robot_model}"/>
     <!-- TODO(abhismirai42): inertial properties are placeholders -->
-    <!-- TODO(abhismirai42): joint limits not yet known for joint_6 (trigger) -->
     <link name="${prefix}base_link">
       <inertial>
@@ -343,7 +342,7 @@
       <limit
         lower="0.0"
-        upper="${0.04 / 0.00875}"
-        effort="${100.0 * 0.00875}"
-        velocity="${0.25 / 0.00875}" />
+        upper="${pi / 4}"
+        effort="1.8"
+        velocity="5.0" />
     </joint>
   </xacro:macro> <!-- glide_left -->

File: urdf/macros/_glide_right.urdf.xacro (robot description, xacro)
@@ -7,5 +7,4 @@
     <xacro:property name="mesh_directory" value="package://trossen_arm_description/meshes/${robot_model}"/>
     <!-- TODO(abhismirai42): inertial properties are placeholders -->
-    <!-- TODO(abhismirai42): joint limits not yet known for joint_6 (trigger) -->
     <link name="${prefix}base_link">
       <inertial>
@@ -343,7 +342,7 @@
       <limit
         lower="0.0"
-        upper="${0.04 / 0.00875}"
-        effort="${100.0 * 0.00875}"
-        velocity="${0.25 / 0.00875}" />
+        upper="${pi / 4}"
+        effort="1.8"
+        velocity="5.0" />
     </joint>
   </xacro:macro> <!-- glide_right -->
