Commit message: update workbench mesh and urdf files

File: urdf/generated/workbench.urdf (robot description, URDF)
Before this commit: robot workbench, 30 links, 29 joints
Joints:
- joint follower_left_mount_joint: origin xyz=0.274 0.062 0.006 rpy=0 0 1.5707963267948966 -> xyz=-0.274 0.062 0.006 rpy=0 0 1.5707963267948966
- joint follower_right_mount_joint: origin xyz=-0.274 0.062 0.006 rpy=0 0 1.5707963267948966 -> xyz=0.274 0.062 0.006 rpy=0 0 1.5707963267948966

File: urdf/workbench.urdf.xacro (robot description, xacro)
@@ -78,5 +78,5 @@
   <joint name="follower_left_mount_joint" type="fixed">
     <origin
-      xyz="0.274 0.062 0.006"
+      xyz="-0.274 0.062 0.006"
       rpy="0 0 ${pi / 2}" />
     <parent link="workbench_base_link"/>
@@ -86,5 +86,5 @@
   <joint name="follower_right_mount_joint" type="fixed">
     <origin
-      xyz="-0.274 0.062 0.006"
+      xyz="0.274 0.062 0.006"
       rpy="0 0 ${pi / 2}" />
     <parent link="workbench_base_link"/>

Commit message: update workbench links oriantation

File: urdf/generated/workbench.urdf (robot description, URDF)
Before this commit: robot workbench, 30 links, 29 joints
Joints:
- joint follower_left_mount_joint: origin xyz=-0.274 0.062 0.006 rpy=0 0 1.5707963267948966 -> xyz=0.062 0.274 0.006 rpy=0 0 0
- joint follower_right_mount_joint: origin xyz=0.274 0.062 0.006 rpy=0 0 1.5707963267948966 -> xyz=0.062 -0.274 0.006 rpy=0 0 0

File: urdf/workbench.urdf.xacro (robot description, xacro)
@@ -76,19 +76,19 @@
     <child link="cam_high"/>
   </joint>
+  <joint name="follower_right_mount_joint" type="fixed">
+    <origin
+      xyz="0.062 -0.274 0.006"
+      rpy="0 0 0" />
+    <parent link="workbench_base_link"/>
+    <child link="follower_right_base_link"/>
+  </joint>
+  <xacro:wxpro prefix="follower_right_"/>
   <joint name="follower_left_mount_joint" type="fixed">
     <origin
-      xyz="-0.274 0.062 0.006"
-      rpy="0 0 ${pi / 2}" />
+      xyz="0.062 0.274 0.006"
+      rpy="0 0 0" />
     <parent link="workbench_base_link"/>
     <child link="follower_left_base_link"/>
   </joint>
   <xacro:wxpro prefix="follower_left_"/>
-  <joint name="follower_right_mount_joint" type="fixed">
-    <origin
-      xyz="0.274 0.062 0.006"
-      rpy="0 0 ${pi / 2}" />
-    <parent link="workbench_base_link"/>
-    <child link="follower_right_base_link"/>
-  </joint>
-  <xacro:wxpro prefix="follower_right_"/>
 </robot>

Commit message: update cam and base mesh (lite version)

File: urdf/generated/workbench.urdf (robot description, URDF)
Before this commit: robot workbench, 30 links, 29 joints
Joints:
- joint cam_high_joint: origin xyz=0 0 0 rpy=0 0 0 -> xyz=0.049994 0 0.856358 rpy=0 0.872665 0
- joint follower_left_mount_joint: origin xyz=0.062 0.274 0.006 rpy=0 0 0 -> xyz=0 0.274 0.0064 rpy=0 0 0
- joint follower_right_mount_joint: origin xyz=0.062 -0.274 0.006 rpy=0 0 0 -> xyz=0 -0.274 0.0064 rpy=0 0 0

File: urdf/workbench.urdf.xacro (robot description, xacro)
@@ -71,6 +71,6 @@
   <joint name="cam_high_joint" type="fixed">
     <origin
-      xyz="0 0 0"
-      rpy="0 0 0" />
+      xyz="0.049994 0 0.856358"
+      rpy="0 0.872665 0" />
     <parent link="workbench_base_link"/>
     <child link="cam_high"/>
@@ -78,5 +78,5 @@
   <joint name="follower_right_mount_joint" type="fixed">
     <origin
-      xyz="0.062 -0.274 0.006"
+      xyz="0 -0.274 0.0064"
       rpy="0 0 0" />
     <parent link="workbench_base_link"/>
@@ -86,5 +86,5 @@
   <joint name="follower_left_mount_joint" type="fixed">
     <origin
-      xyz="0.062 0.274 0.006"
+      xyz="0 0.274 0.0064"
       rpy="0 0 0" />
     <parent link="workbench_base_link"/>

Commit message: update camera mount joint, use offical xacro for zed x cameras

File: urdf/generated/workbench.urdf (robot description, URDF)
Before this commit: robot workbench, 30 links, 29 joints
Links:
- removed link cam_high
- removed link follower_left_camera
- removed link follower_right_camera
- added link cam_high_camera_center, mass 0.15; collision mesh filename=package://trossen_arm_description/meshes/peripherals/zedxm.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; visual mesh filename=package://trossen_arm_description/meshes/peripherals/zedxm.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
- added link cam_high_camera_link
- added link cam_high_left_camera_frame
- added link cam_high_left_camera_frame_optical
- added link cam_high_right_camera_frame
- added link cam_high_right_camera_frame_optical
- added link follower_left_wrist_camera_center, mass 0.075; collision mesh filename=package://trossen_arm_description/meshes/peripherals/zedxna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; visual mesh filename=package://trossen_arm_description/meshes/peripherals/zedxna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
- added link follower_left_wrist_camera_link
- added link follower_left_wrist_left_camera_frame
- added link follower_left_wrist_left_camera_frame_optical
- added link follower_left_wrist_right_camera_frame
- added link follower_left_wrist_right_camera_frame_optical
- added link follower_right_wrist_camera_center, mass 0.075; collision mesh filename=package://trossen_arm_description/meshes/peripherals/zedxna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; visual mesh filename=package://trossen_arm_description/meshes/peripherals/zedxna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
- added link follower_right_wrist_camera_link
- added link follower_right_wrist_left_camera_frame
- added link follower_right_wrist_left_camera_frame_optical
- added link follower_right_wrist_right_camera_frame
- added link follower_right_wrist_right_camera_frame_optical
Joints:
- removed joint cam_high_joint
- removed joint follower_left_camera_joint
- removed joint follower_right_camera_joint
- added joint cam_high_camera_center_joint: type fixed, parent cam_high_camera_link, child cam_high_camera_center, origin xyz=0 0 0.016 rpy=0 0 0
- added joint cam_high_left_camera_joint: type fixed, parent cam_high_camera_center, child cam_high_left_camera_frame, origin xyz=-0.01 0.025 0 rpy=0 0 0
- added joint cam_high_left_camera_optical_joint: type fixed, parent cam_high_left_camera_frame, child cam_high_left_camera_frame_optical, origin xyz=0 0 0 rpy=-1.5707963267948966 0 -1.5707963267948966
- added joint cam_high_mount_joint: type fixed, parent workbench_base_link, child cam_high_camera_link, origin xyz=0.028173 0 0.857613 rpy=0 0.872665 0
- added joint cam_high_right_camera_joint: type fixed, parent cam_high_camera_center, child cam_high_right_camera_frame, origin xyz=-0.01 -0.025 0 rpy=0 0 0
- added joint cam_high_right_camera_optical_joint: type fixed, parent cam_high_right_camera_frame, child cam_high_right_camera_frame_optical, origin xyz=0 0 0 rpy=-1.5707963267948966 0 -1.5707963267948966
- added joint follower_left_wrist_camera_center_joint: type fixed, parent follower_left_wrist_camera_link, child follower_left_wrist_camera_center, origin xyz=0 0 0.01525 rpy=0 0 0
- added joint follower_left_wrist_left_camera_joint: type fixed, parent follower_left_wrist_camera_center, child follower_left_wrist_left_camera_frame, origin xyz=-0.01 0.009 0 rpy=0 0 0
- added joint follower_left_wrist_left_camera_optical_joint: type fixed, parent follower_left_wrist_left_camera_frame, child follower_left_wrist_left_camera_frame_optical, origin xyz=0 0 0 rpy=-1.5707963267948966 0 -1.5707963267948966
- added joint follower_left_wrist_mount_joint: type fixed, parent follower_left_link_6, child follower_left_wrist_camera_link, origin xyz=0.086133 0 0.057843 rpy=0 0.436 0
- added joint follower_left_wrist_right_camera_joint: type fixed, parent follower_left_wrist_camera_center, child follower_left_wrist_right_camera_frame, origin xyz=-0.01 -0.009 0 rpy=0 0 0
- added joint follower_left_wrist_right_camera_optical_joint: type fixed, parent follower_left_wrist_right_camera_frame, child follower_left_wrist_right_camera_frame_optical, origin xyz=0 0 0 rpy=-1.5707963267948966 0 -1.5707963267948966
- added joint follower_right_wrist_camera_center_joint: type fixed, parent follower_right_wrist_camera_link, child follower_right_wrist_camera_center, origin xyz=0 0 0.01525 rpy=0 0 0
- added joint follower_right_wrist_left_camera_joint: type fixed, parent follower_right_wrist_camera_center, child follower_right_wrist_left_camera_frame, origin xyz=-0.01 0.009 0 rpy=0 0 0
- added joint follower_right_wrist_left_camera_optical_joint: type fixed, parent follower_right_wrist_left_camera_frame, child follower_right_wrist_left_camera_frame_optical, origin xyz=0 0 0 rpy=-1.5707963267948966 0 -1.5707963267948966
- added joint follower_right_wrist_mount_joint: type fixed, parent follower_right_link_6, child follower_right_wrist_camera_link, origin xyz=0.086133 0 0.057843 rpy=0 0.436 0
- added joint follower_right_wrist_right_camera_joint: type fixed, parent follower_right_wrist_camera_center, child follower_right_wrist_right_camera_frame, origin xyz=-0.01 -0.009 0 rpy=0 0 0
- added joint follower_right_wrist_right_camera_optical_joint: type fixed, parent follower_right_wrist_right_camera_frame, child follower_right_wrist_right_camera_frame_optical, origin xyz=0 0 0 rpy=-1.5707963267948966 0 -1.5707963267948966
- joint follower_left_camera_mount_joint: origin xyz=0.104 0 0 rpy=0 0 0 -> xyz=0.102 0 0 rpy=0 0 0
- joint follower_right_camera_mount_joint: origin xyz=0.104 0 0 rpy=0 0 0 -> xyz=0.102 0 0 rpy=0 0 0

File: urdf/workbench.urdf.xacro (robot description, xacro)
@@ -5,6 +5,7 @@
     scope="global"/>
   <xacro:include filename="$(find trossen_arm_description)/urdf/macros/_wxpro.urdf.xacro" />
+  <xacro:include filename="$(find trossen_arm_description)/urdf/peripherals/zed_camera.urdf.xacro" />
   <xacro:property name="mesh_directory" value="package://trossen_arm_description/meshes/workbench"/>
-  <!-- TODO(abhismirai42): update inertial property for workbench_base and cam_high -->
+  <!-- TODO(abhismirai42): update inertial property for workbench_base -->
   <link name="workbench_base_link">
     <inertial>
@@ -38,42 +39,9 @@
     </collision>
   </link>
-  <link name="cam_high">
-    <inertial>
-      <origin
-        xyz="0 0 0"
-        rpy="0 0 0" />
-      <mass value="0.1"/>
-      <inertia
-        ixx="0.001"
-        ixy="0.0"
-        ixz="0.0"
-        iyy="0.001"
-        iyz="0.0"
-        izz="0.001"/>
-    </inertial>
-    <visual>
-      <origin
-        xyz="0 0 0"
-        rpy="0 0 0" />
-      <geometry>
-        <mesh filename="${mesh_directory}/cam_high.obj"/>
-      </geometry>
-    </visual>
-    <collision>
-      <origin
-        xyz="0 0 0"
-        rpy="0 0 0" />
-      <geometry>
-        <mesh filename="${mesh_directory}/cam_high.obj"/>
-      </geometry>
-    </collision>
-  </link>
-  <joint name="cam_high_joint" type="fixed">
+  <xacro:zed_camera name="cam_high" model="zedxm" parent="workbench_base_link">
     <origin
-      xyz="0.049994 0 0.856358"
+      xyz="0.028173 0 0.857613"
       rpy="0 0.872665 0" />
-    <parent link="workbench_base_link"/>
-    <child link="cam_high"/>
-  </joint>
+  </xacro:zed_camera>
   <joint name="follower_right_mount_joint" type="fixed">
     <origin

Commit message: rename workbench_base_link to base_link

File: urdf/generated/workbench.urdf (robot description, URDF)
Before this commit: robot workbench, 45 links, 44 joints
Links:
- removed link workbench_base_link
- added link base_link, mass 10.0; collision mesh filename=package://trossen_arm_description/meshes/workbench/workbenc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; visual mesh filename=package://trossen_arm_description/meshes/workbench/workbenc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
Joints:
- joint cam_high_mount_joint: parent workbench_base_link -> base_link
- joint follower_left_mount_joint: parent workbench_base_link -> base_link
- joint follower_right_mount_joint: parent workbench_base_link -> base_link

File: urdf/workbench.urdf.xacro (robot description, xacro)
@@ -8,5 +8,5 @@
   <xacro:property name="mesh_directory" value="package://trossen_arm_description/meshes/workbench"/>
   <!-- TODO(abhismirai42): update inertial property for workbench_base -->
-  <link name="workbench_base_link">
+  <link name="base_link">
     <inertial>
       <origin
@@ -39,5 +39,5 @@
     </collision>
   </link>
-  <xacro:zed_camera name="cam_high" model="zedxm" parent="workbench_base_link">
+  <xacro:zed_camera name="cam_high" model="zedxm" parent="base_link">
     <origin
       xyz="0.028173 0 0.857613"
@@ -48,5 +48,5 @@
       xyz="0 -0.274 0.0064"
       rpy="0 0 0" />
-    <parent link="workbench_base_link"/>
+    <parent link="base_link"/>
     <child link="follower_right_base_link"/>
   </joint>
@@ -56,5 +56,5 @@
       xyz="0 0.274 0.0064"
       rpy="0 0 0" />
-    <parent link="workbench_base_link"/>
+    <parent link="base_link"/>
     <child link="follower_left_base_link"/>
   </joint>
