Commit message: update joints limit
Co-Authored-By: Claude Opus 5.5 <noreply@anthropic.com>

File: urdf/generated/workbench.urdf (robot description, URDF)
Before this commit: robot workbench, 45 links, 44 joints
Joints:
- joint follower_left_joint_0: limit lower=-3.0543261909900767 upper=3.0543261909900767 effort=27.0 velocity=3.375 -> lower=-2.8797932657906435 upper=2.8797932657906435 effort=27.0 velocity=3.375
- joint follower_left_joint_1: limit lower=0.0 upper=3.141592653589793 effort=27.0 velocity=3.375 -> lower=0.0 upper=3.5779249665883754 effort=97.0 velocity=3.375
- joint follower_left_joint_2: limit lower=0.0 upper=2.356194490192345 effort=27.0 velocity=3.375 -> lower=0.0 upper=3.141592653589793 effort=27.0 velocity=3.375
- joint follower_left_joint_5: limit lower=-3.141592653589793 upper=3.141592653589793 effort=7.0 velocity=7.0 -> lower=-2.007128639793479 upper=2.007128639793479 effort=7.0 velocity=7.0
- joint follower_left_left_carriage_joint: limit lower=0.0 upper=0.044 effort=400.0 velocity=0.0875 -> lower=0.0 upper=0.045 effort=400.0 velocity=0.0875
- joint follower_left_right_carriage_joint: limit lower=0.0 upper=0.044 effort=400.0 velocity=0.0875 -> lower=0.0 upper=0.045 effort=400.0 velocity=0.0875
- joint follower_right_joint_0: limit lower=-3.0543261909900767 upper=3.0543261909900767 effort=27.0 velocity=3.375 -> lower=-2.8797932657906435 upper=2.8797932657906435 effort=27.0 velocity=3.375
- joint follower_right_joint_1: limit lower=0.0 upper=3.141592653589793 effort=27.0 velocity=3.375 -> lower=0.0 upper=3.5779249665883754 effort=97.0 velocity=3.375
- joint follower_right_joint_2: limit lower=0.0 upper=2.356194490192345 effort=27.0 velocity=3.375 -> lower=0.0 upper=3.141592653589793 effort=27.0 velocity=3.375
- joint follower_right_joint_5: limit lower=-3.141592653589793 upper=3.141592653589793 effort=7.0 velocity=7.0 -> lower=-2.007128639793479 upper=2.007128639793479 effort=7.0 velocity=7.0
- joint follower_right_left_carriage_joint: limit lower=0.0 upper=0.044 effort=400.0 velocity=0.0875 -> lower=0.0 upper=0.045 effort=400.0 velocity=0.0875
- joint follower_right_right_carriage_joint: limit lower=0.0 upper=0.044 effort=400.0 velocity=0.0875 -> lower=0.0 upper=0.045 effort=400.0 velocity=0.0875
