Commit message: joint_6 glide_right axis flip

File: urdf/generated/glide_right.urdf (robot description, URDF)
Before this commit: robot glide_right, 8 links, 7 joints
Joints:
- joint joint_6: axis 0 1 0 -> 0 -1 0

File: urdf/macros/_glide_right.urdf.xacro (robot description, xacro)
@@ -339,5 +339,5 @@
       <parent link="${prefix}link_6"/>
       <child link="${prefix}trigger"/>
-      <axis xyz="0 1 0"/>
+      <axis xyz="0 -1 0"/>
       <limit
         lower="0.0"
