Commit message: update joints limit
Co-Authored-By: Claude Opus 5.5 <noreply@anthropic.com>

File: urdf/generated/wxpro.urdf (robot description, URDF)
Before this commit: robot wxpro, 19 links, 18 joints
Joints:
- joint joint_0: limit lower=-3.0543261909900767 upper=3.0543261909900767 effort=27.0 velocity=3.375 -> lower=-2.8797932657906435 upper=2.8797932657906435 effort=27.0 velocity=3.375
- joint joint_1: limit lower=0.0 upper=3.141592653589793 effort=27.0 velocity=3.375 -> lower=0.0 upper=3.5779249665883754 effort=97.0 velocity=3.375
- joint joint_2: limit lower=0.0 upper=2.356194490192345 effort=27.0 velocity=3.375 -> lower=0.0 upper=3.141592653589793 effort=27.0 velocity=3.375
- joint joint_5: limit lower=-3.141592653589793 upper=3.141592653589793 effort=7.0 velocity=7.0 -> lower=-2.007128639793479 upper=2.007128639793479 effort=7.0 velocity=7.0
- joint left_carriage_joint: limit lower=0.0 upper=0.044 effort=400.0 velocity=0.0875 -> lower=0.0 upper=0.045 effort=400.0 velocity=0.0875
- joint right_carriage_joint: limit lower=0.0 upper=0.044 effort=400.0 velocity=0.0875 -> lower=0.0 upper=0.045 effort=400.0 velocity=0.0875

File: urdf/macros/_wxpro.urdf.xacro (robot description, xacro)
@@ -78,6 +78,6 @@
       <axis xyz="0 0 1"/>
       <limit
-        lower="${-radians(180 - 5)}"
-        upper="${radians(180 - 5)}"
+        lower="${-radians(165)}"
+        upper="${radians(165)}"
         effort="27.0"
         velocity="3.375" />
@@ -123,6 +123,6 @@
       <limit
         lower="0.0"
-        upper="${pi}"
-        effort="27.0"
+        upper="${radians(205)}"
+        effort="97.0"
         velocity="3.375" />
     </joint>
@@ -167,5 +167,5 @@
       <limit
         lower="0.0"
-        upper="${3 * pi / 4}"
+        upper="${pi}"
         effort="27.0"
         velocity="3.375" />
@@ -298,6 +298,6 @@
       <axis xyz="1 0 0"/>
       <limit
-        lower="-${pi}"
-        upper="${pi}"
+        lower="${-radians(115)}"
+        upper="${radians(115)}"
         effort="7.0"
         velocity="7.0" />
@@ -345,5 +345,5 @@
       <limit
         lower="0.0"
-        upper="0.044"
+        upper="0.045"
         effort="400.0"
         velocity="0.0875" />
@@ -389,5 +389,5 @@
       <limit
         lower="0.0"
-        upper="0.044"
+        upper="0.045"
         effort="400.0"
         velocity="0.0875" />
