Commit message: Updates, rename to wxpro

File: urdf/generated/wxpro.urdf (robot description, URDF)
Before this commit: robot widowx_pro, 14 links, 13 joints
Links:
- link base_link: geometry collision mesh filename=package://trossen_arm_description/meshes/wxpro/base_link.obj; visual mesh filename=package://trossen_arm_description/meshes/wxpro/base_link.obj
- link camera: geometry collision mesh filename=package://trossen_arm_description/meshes/wxpro/camera.obj; visual mesh filename=package://trossen_arm_description/meshes/wxpro/camera.obj
- link camera_mount: geometry collision mesh filename=package://trossen_arm_description/meshes/wxpro/camera_mount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; visual mesh filename=package://trossen_arm_description/meshes/wxpro/camera_mount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
- link carriage_left: geometry collision mesh filename=package://trossen_arm_description/meshes/wxpro/carriage_lef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; visual mesh filename=package://trossen_arm_description/meshes/wxpro/carriage_lef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
- link carriage_right: geometry collision mesh filename=package://trossen_arm_description/meshes/wxpro/carriage_rig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; visual mesh filename=package://trossen_arm_description/meshes/wxpro/carriage_rig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
- link ee_gripper_link: geometry 
- link gripper_left: geometry collision mesh filename=package://trossen_arm_description/meshes/wxpro/gripper_left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; visual mesh filename=package://trossen_arm_description/meshes/wxpro/gripper_left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
- link gripper_right: geometry collision mesh filename=package://trossen_arm_description/meshes/wxpro/gripper_righ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; visual mesh filename=package://trossen_arm_description/meshes/wxpro/gripper_righ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
- link link_1: geometry collision mesh filename=package://trossen_arm_description/meshes/wxpro/link_1.obj; visual mesh filename=package://trossen_arm_description/meshes/wxpro/link_1.obj
- link link_2: geometry collision mesh filename=package://trossen_arm_description/meshes/wxpro/link_2.obj; visual mesh filename=package://trossen_arm_description/meshes/wxpro/link_2.obj
- link link_3: geometry collision mesh filename=package://trossen_arm_description/meshes/wxpro/link_3.obj; visual mesh filename=package://trossen_arm_description/meshes/wxpro/link_3.obj
- link link_4: geometry collision mesh filename=package://trossen_arm_description/meshes/wxpro/link_4.obj; visual mesh filename=package://trossen_arm_description/meshes/wxpro/link_4.obj
- link link_5: geometry collision mesh filename=package://trossen_arm_description/meshes/wxpro/link_5.obj; visual mesh filename=package://trossen_arm_description/meshes/wxpro/link_5.obj
- link link_6: geometry collision mesh filename=package://trossen_arm_description/meshes/wxpro/link_6.obj; visual mesh filename=package://trossen_arm_description/meshes/wxpro/link_6.obj

File: urdf/macros/_wxpro.urdf.xacro (robot description, xacro)
@@ -1,9 +1,10 @@
 <?xml version="1.0" encoding="utf-8"?>
-<robot name="widowx_pro" xmlns:xacro="http://ros.org/wiki/xacro">
+<robot name="wxpro" xmlns:xacro="http://ros.org/wiki/xacro">
   <xacro:property name="robot_model"
-    value="widowx_pro"/>
-  <xacro:macro name="widowx_pro" params="prefix:=''">
+    value="wxpro"
+    scope="local"/>
+  <xacro:macro name="wxpro" params="prefix:=''">
     <xacro:property name="mesh_directory" value="package://trossen_arm_description/meshes/${robot_model}"/>
-    <!-- TODO(abhismirai42): ros2_control  -->
+    <!-- TODO(abhismirai42): ros2_control -->
     <link name="${prefix}base_link">
       <inertial>
@@ -24,11 +25,15 @@
           xyz="0 0 0"
           rpy="0 0 0" />
-        <geometry><mesh filename="${mesh_directory}/base_link.obj"/></geometry>
-      </visual>
-      <collision>
-        <origin
-          xyz="0 0 0"
-          rpy="0 0 0" />
-        <geometry><mesh filename="${mesh_directory}/base_link.obj"/></geometry>
+        <geometry>
+          <mesh filename="${mesh_directory}/base_link.obj"/>
+        </geometry>
+      </visual>
+      <collision>
+        <origin
+          xyz="0 0 0"
+          rpy="0 0 0" />
+        <geometry>
+          <mesh filename="${mesh_directory}/base_link.obj"/>
+        </geometry>
       </collision>
     </link>
@@ -51,11 +56,15 @@
           xyz="0 0 0"
           rpy="0 0 0" />
-        <geometry><mesh filename="${mesh_directory}/link_1.obj"/></geometry>
-      </visual>
-      <collision>
-        <origin
-          xyz="0 0 0"
-          rpy="0 0 0" />
-        <geometry><mesh filename="${mesh_directory}/link_1.obj"/></geometry>
+        <geometry>
+          <mesh filename="${mesh_directory}/link_1.obj"/>
+        </geometry>
+      </visual>
+      <collision>
+        <origin
+          xyz="0 0 0"
+          rpy="0 0 0" />
+        <geometry>
+          <mesh filename="${mesh_directory}/link_1.obj"/>
+        </geometry>
       </collision>
     </link>
@@ -70,6 +79,6 @@
         lower="${-radians(180 - 5)}"
         upper="${radians(180 - 5)}"
-        velocity="3.375"
-        effort="27.0" />
+        effort="27.0"
+        velocity="3.375" />
     </joint>
     <link name="${prefix}link_2">
@@ -91,11 +100,15 @@
           xyz="0 0 0"
           rpy="0 0 0" />
-        <geometry><mesh filename="${mesh_directory}/link_2.obj"/></geometry>
-      </visual>
-      <collision>
-        <origin
-          xyz="0 0 0"
-          rpy="0 0 0" />
-        <geometry><mesh filename="${mesh_directory}/link_2.obj"/></geometry>
+        <geometry>
+          <mesh filename="${mesh_directory}/link_2.obj"/>
+        </geometry>
+      </visual>
+      <collision>
+        <origin
+          xyz="0 0 0"
+          rpy="0 0 0" />
+        <geometry>
+          <mesh filename="${mesh_directory}/link_2.obj"/>
+        </geometry>
       </collision>
     </link>
@@ -110,6 +123,6 @@
         lower="0.0"
         upper="${pi}"
-        velocity="3.375"
-        effort="27.0" />
+        effort="27.0"
+        velocity="3.375" />
     </joint>
     <link name="${prefix}link_3">
@@ -131,11 +144,15 @@
           xyz="0 0 0"
           rpy="0 0 0" />
-        <geometry><mesh filename="${mesh_directory}/link_3.obj"/></geometry>
-      </visual>
-      <collision>
-        <origin
-          xyz="0 0 0"
-          rpy="0 0 0" />
-        <geometry><mesh filename="${mesh_directory}/link_3.obj"/></geometry>
+        <geometry>
+          <mesh filename="${mesh_directory}/link_3.obj"/>
+        </geometry>
+      </visual>
+      <collision>
+        <origin
+          xyz="0 0 0"
+          rpy="0 0 0" />
+        <geometry>
+          <mesh filename="${mesh_directory}/link_3.obj"/>
+        </geometry>
       </collision>
     </link>
@@ -150,6 +167,6 @@
         lower="0.0"
         upper="${3 * pi / 4}"
-        velocity="3.375"
-        effort="27.0" />
+        effort="27.0"
+        velocity="3.375" />
     </joint>
     <link name="${prefix}link_4">
@@ -171,11 +188,15 @@
           xyz="0 0 0"
           rpy="0 0 0" />
-        <geometry><mesh filename="${mesh_directory}/link_4.obj"/></geometry>
-      </visual>
-      <collision>
-        <origin
-          xyz="0 0 0"
-          rpy="0 0 0" />
-        <geometry><mesh filename="${mesh_directory}/link_4.obj"/></geometry>
+        <geometry>
+          <mesh filename="${mesh_directory}/link_4.obj"/>
+        </geometry>
+      </visual>
+      <collision>
+        <origin
+          xyz="0 0 0"
+          rpy="0 0 0" />
+        <geometry>
+          <mesh filename="${mesh_directory}/link_4.obj"/>
+        </geometry>
       </collision>
     </link>
@@ -188,8 +209,8 @@
       <axis xyz="0 -1 0"/>
       <limit
-        lower="${-pi / 2}"
+        lower="-${pi / 2}"
         upper="${pi / 2}"
-        velocity="7.0"
-        effort="7.0" />
+        effort="7.0"
+        velocity="7.0" />
     </joint>
     <link name="${prefix}link_5">
@@ -211,11 +232,15 @@
           xyz="0 0 0"
           rpy="0 0 0" />
-        <geometry><mesh filename="${mesh_directory}/link_5.obj"/></geometry>
-      </visual>
-      <collision>
-        <origin
-          xyz="0 0 0"
-          rpy="0 0 0" />
-        <geometry><mesh filename="${mesh_directory}/link_5.obj"/></geometry>
+        <geometry>
+          <mesh filename="${mesh_directory}/link_5.obj"/>
+        </geometry>
+      </visual>
+      <collision>
+        <origin
+          xyz="0 0 0"
+          rpy="0 0 0" />
+        <geometry>
+          <mesh filename="${mesh_directory}/link_5.obj"/>
+        </geometry>
       </collision>
     </link>
@@ -228,8 +253,8 @@
       <axis xyz="0 0 -1"/>
       <limit
-        lower="${-pi / 2}"
+        lower="-${pi / 2}"
         upper="${pi / 2}"
-        velocity="7.0"
-        effort="7.0" />
+        effort="7.0"
+        velocity="7.0" />
     </joint>
     <link name="${prefix}link_6">
@@ -251,11 +276,15 @@
           xyz="0 0 0"
           rpy="0 0 0" />
-        <geometry><mesh filename="${mesh_directory}/link_6.obj"/></geometry>
-      </visual>
-      <collision>
-        <origin
-          xyz="0 0 0"
-          rpy="0 0 0" />
-        <geometry><mesh filename="${mesh_directory}/link_6.obj"/></geometry>
+        <geometry>
+          <mesh filename="${mesh_directory}/link_6.obj"/>
+        </geometry>
+      </visual>
+      <collision>
+        <origin
+          xyz="0 0 0"
+          rpy="0 0 0" />
+        <geometry>
+          <mesh filename="${mesh_directory}/link_6.obj"/>
+        </geometry>
       </collision>
     </link>
@@ -268,10 +297,10 @@
       <axis xyz="1 0 0"/>
       <limit
-        lower="${-pi}"
+        lower="-${pi}"
         upper="${pi}"
-        velocity="7.0"
-        effort="7.0" />
-    </joint>
-    <!-- TODO(abhismirai42): verify intertial properties carrige_links, gripper_links and camera_link -->
+        effort="7.0"
+        velocity="7.0" />
+    </joint>
+    <!-- TODO(abhismirai42): verify inertial properties carriage_links, gripper_links and camera_link -->
     <link name="${prefix}carriage_right">
       <inertial>
@@ -292,11 +321,15 @@
           xyz="0 0 0"
           rpy="0 0 0" />
-        <geometry><mesh filename="${mesh_directory}/carriage_right.obj"/></geometry>
-      </visual>
-      <collision>
-        <origin
-          xyz="0 0 0"
-          rpy="0 0 0" />
-        <geometry><mesh filename="${mesh_directory}/carriage_right.obj"/></geometry>
+        <geometry>
+          <mesh filename="${mesh_directory}/carriage_right.obj"/>
+        </geometry>
+      </visual>
+      <collision>
+        <origin
+          xyz="0 0 0"
+          rpy="0 0 0" />
+        <geometry>
+          <mesh filename="${mesh_directory}/carriage_right.obj"/>
+        </geometry>
       </collision>
     </link>
@@ -312,6 +345,6 @@
         lower="0.0"
         upper="0.044"
-        velocity="0.0875"
-        effort="400.0" />
+        effort="400.0"
+        velocity="0.0875" />
     </joint>
     <link name="${prefix}carriage_left">
@@ -333,11 +366,15 @@
           xyz="0 0 0"
           rpy="0 0 0" />
-        <geometry><mesh filename="${mesh_directory}/carriage_left.obj"/></geometry>
-      </visual>
-      <collision>
-        <origin
-          xyz="0 0 0"
-          rpy="0 0 0" />
-        <geometry><mesh filename="${mesh_directory}/carriage_left.obj"/></geometry>
+        <geometry>
+          <mesh filename="${mesh_directory}/carriage_left.obj"/>
+        </geometry>
+      </visual>
+      <collision>
+        <origin
+          xyz="0 0 0"
+          rpy="0 0 0" />
+        <geometry>
+          <mesh filename="${mesh_directory}/carriage_left.obj"/>
+        </geometry>
       </collision>
     </link>
@@ -345,5 +382,5 @@
       <origin
         xyz="0.1285 0.0225 0"
-        rpy="${pi} 0 ${-pi / 2}" />
+        rpy="${pi} 0 -${pi / 2}" />
       <parent link="${prefix}link_6"/>
       <child link="${prefix}carriage_left"/>
@@ -352,6 +389,6 @@
         lower="0.0"
         upper="0.044"
-        velocity="0.0875"
-        effort="400.0" />
+        effort="400.0"
+        velocity="0.0875" />
     </joint>
     <link name="${prefix}gripper_left">
@@ -373,11 +410,15 @@
           xyz="0 0 0"
           rpy="0 0 0" />
-        <geometry><mesh filename="${mesh_directory}/gripper_left.obj"/></geometry>
-      </visual>
-      <collision>
-        <origin
-          xyz="0 0 0"
-          rpy="0 0 0" />
-        <geometry><mesh filename="${mesh_directory}/gripper_left.obj"/></geometry>
+        <geometry>
+          <mesh filename="${mesh_directory}/gripper_left.obj"/>
+        </geometry>
+      </visual>
+      <collision>
+        <origin
+          xyz="0 0 0"
+          rpy="0 0 0" />
+        <geometry>
+          <mesh filename="${mesh_directory}/gripper_left.obj"/>
+        </geometry>
       </collision>
     </link>
@@ -407,11 +448,15 @@
           xyz="0 0 0"
           rpy="0 0 0" />
-        <geometry><mesh filename="${mesh_directory}/gripper_right.obj"/></geometry>
-      </visual>
-      <collision>
-        <origin
-          xyz="0 0 0"
-          rpy="0 0 0" />
-        <geometry><mesh filename="${mesh_directory}/gripper_right.obj"/></geometry>
+        <geometry>
+          <mesh filename="${mesh_directory}/gripper_right.obj"/>
+        </geometry>
+      </visual>
+      <collision>
+        <origin
+          xyz="0 0 0"
+          rpy="0 0 0" />
+        <geometry>
+          <mesh filename="${mesh_directory}/gripper_right.obj"/>
+        </geometry>
       </collision>
     </link>
@@ -423,12 +468,5 @@
       <child link="${prefix}gripper_right"/>
     </joint>
-    <link name="${prefix}ee_gripper_link">
-      <visual>
-        <origin
-          xyz="0 0 0"
-          rpy="0 0 0" />
-        <geometry><sphere radius="0.003"/></geometry>
-      </visual>
-    </link>
+    <link name="${prefix}ee_gripper_link" />
     <joint name="${prefix}ee_gripper" type="fixed">
       <origin
@@ -456,11 +494,15 @@
           xyz="0 0 0"
           rpy="0 0 0" />
-        <geometry><mesh filename="${mesh_directory}/camera_mount.obj"/></geometry>
-      </visual>
-      <collision>
-        <origin
-          xyz="0 0 0"
-          rpy="0 0 0" />
-        <geometry><mesh filename="${mesh_directory}/camera_mount.obj"/></geometry>
+        <geometry>
+          <mesh filename="${mesh_directory}/camera_mount.obj"/>
+        </geometry>
+      </visual>
+      <collision>
+        <origin
+          xyz="0 0 0"
+          rpy="0 0 0" />
+        <geometry>
+          <mesh filename="${mesh_directory}/camera_mount.obj"/>
+        </geometry>
       </collision>
     </link>
@@ -472,5 +514,5 @@
       <child link="${prefix}camera_mount"/>
     </joint>
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
File: urdf/wxpro.urdf.xacro (robot description, xacro)
@@ -1,4 +1,4 @@
 <?xml version="1.0" encoding="utf-8"?>
-<robot name="widowx_pro" xmlns:xacro="http://ros.org/wiki/xacro">
+<robot name="wxpro" xmlns:xacro="http://ros.org/wiki/xacro">
   <xacro:arg name="prefix"                          default=""/>
   <xacro:arg name="use_world_frame"                 default="false"/>       <!-- 'true', 'false' -->
@@ -14,6 +14,6 @@
     </joint>
   </xacro:if> <!-- use_world_frame -->
-  <xacro:include filename="$(find trossen_arm_description)/urdf/macros/_widowx_pro.urdf.xacro" />
-  <xacro:widowx_pro
+  <xacro:include filename="$(find trossen_arm_description)/urdf/macros/_wxpro.urdf.xacro" />
+  <xacro:wxpro
     prefix="$(arg prefix)"/>
 </robot>

Commit message: update camera mount joint, use offical xacro for zed x camera

File: urdf/generated/wxpro.urdf (robot description, URDF)
Before this commit: robot wxpro, 14 links, 13 joints
Links:
- removed link camera
- added link wrist_camera_center, mass 0.075; collision mesh filename=package://trossen_arm_description/meshes/peripherals/zedxna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; visual mesh filename=package://trossen_arm_description/meshes/peripherals/zedxna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
- added link wrist_camera_link
- added link wrist_left_camera_frame
- added link wrist_left_camera_frame_optical
- added link wrist_right_camera_frame
- added link wrist_right_camera_frame_optical
Joints:
- removed joint camera_joint
- added joint wrist_camera_center_joint: type fixed, parent wrist_camera_link, child wrist_camera_center, origin xyz=0 0 0.01525 rpy=0 0 0
- added joint wrist_left_camera_joint: type fixed, parent wrist_camera_center, child wrist_left_camera_frame, origin xyz=-0.01 0.009 0 rpy=0 0 0
- added joint wrist_left_camera_optical_joint: type fixed, parent wrist_left_camera_frame, child wrist_left_camera_frame_optical, origin xyz=0 0 0 rpy=-1.5707963267948966 0 -1.5707963267948966
- added joint wrist_mount_joint: type fixed, parent link_6, child wrist_camera_link, origin xyz=0.086133 0 0.057843 rpy=0 0.436 0
- added joint wrist_right_camera_joint: type fixed, parent wrist_camera_center, child wrist_right_camera_frame, origin xyz=-0.01 -0.009 0 rpy=0 0 0
- added joint wrist_right_camera_optical_joint: type fixed, parent wrist_right_camera_frame, child wrist_right_camera_frame_optical, origin xyz=0 0 0 rpy=-1.5707963267948966 0 -1.5707963267948966
- joint camera_mount_joint: origin xyz=0.104 0 0 rpy=0 0 0 -> xyz=0.102 0 0 rpy=0 0 0

File: urdf/macros/_wxpro.urdf.xacro (robot description, xacro)
@@ -4,4 +4,5 @@
     value="wxpro"
     scope="local"/>
+  <xacro:include filename="$(find trossen_arm_description)/urdf/peripherals/zed_camera.urdf.xacro" />
   <xacro:macro name="wxpro" params="prefix:=''">
     <xacro:property name="mesh_directory" value="package://trossen_arm_description/meshes/${robot_model}"/>
@@ -509,48 +510,14 @@
     <joint name="${prefix}camera_mount_joint" type="fixed">
       <origin
-        xyz="0.104 0 0"
+        xyz="0.102 0 0"
         rpy="0 0 0" />
       <parent link="${prefix}link_6"/>
       <child link="${prefix}camera_mount"/>
     </joint>
-    <!-- TODO(abhismirai42): use official zed camera xacro model -->
-    <link name="${prefix}camera">
-      <inertial>
-        <origin
-          xyz="-0.00555 0 0.07215"
-          rpy="0 0 0" />
-        <mass value="0.0695"/>
-        <inertia
-          ixx="0.0000195"
-          ixy="0.0"
-          ixz="0.0"
-          iyy="0.0000192"
-          iyz="0.0"
-          izz="0.0000202"/>
-      </inertial>
-      <visual>
-        <origin
-          xyz="0 0 0"
-          rpy="0 0 0" />
-        <geometry>
-          <mesh filename="${mesh_directory}/camera.obj"/>
-        </geometry>
-      </visual>
-      <collision>
-        <origin
-          xyz="0 0 0"
-          rpy="0 0 0" />
-        <geometry>
-          <mesh filename="${mesh_directory}/camera.obj"/>
-        </geometry>
-      </collision>
-    </link>
-    <joint name="${prefix}camera_joint" type="fixed">
-      <origin
-        xyz="-0.002173 0 0.001068"
-        rpy="0 0 0" />
-      <parent link="${prefix}camera_mount"/>
-      <child link="${prefix}camera"/>
-    </joint>
+    <xacro:zed_camera name="${prefix}wrist" model="zedxnano" parent="${prefix}link_6">
+      <origin
+        xyz="0.086133 0 0.057843"
+        rpy="0 0.436 0" />
+    </xacro:zed_camera>
   </xacro:macro> <!-- wxpro -->
 </robot>

Commit message: fix joint_5, carriage, ee_gripper and wrist camera positions from cad

File: urdf/generated/wxpro.urdf (robot description, URDF)
Before this commit: robot wxpro, 19 links, 18 joints
Joints:
- joint ee_gripper: origin xyz=0.22 0 0 rpy=0 0 0 -> xyz=0.218 0 0 rpy=0 0 0
- joint joint_5: origin xyz=-0.012 0.0 -0.048 rpy=0 0 0 -> xyz=-0.009 0.0 -0.048 rpy=0 0 0
- joint left_carriage_joint: origin xyz=0.1285 0.0225 0 rpy=3.141592653589793 0 -1.5707963267948966 -> xyz=0.1265 0.0225 0 rpy=3.141592653589793 0 -1.5707963267948966
- joint right_carriage_joint: origin xyz=0.1285 -0.0225 0 rpy=0 0 1.5707963267948966 -> xyz=0.1265 -0.0225 0 rpy=0 0 1.5707963267948966
- joint wrist_mount_joint: origin xyz=0.086133 0 0.057843 rpy=0 0.436 0 -> xyz=0.091112 0 0.057797 rpy=0 0.436332 0

File: urdf/macros/_wxpro.urdf.xacro (robot description, xacro)
@@ -292,5 +292,5 @@
     <joint name="${prefix}joint_5" type="revolute">
       <origin
-        xyz="-0.012 0.0 -0.048"
+        xyz="-0.009 0.0 -0.048"
         rpy="0 0 0" />
       <parent link="${prefix}link_5"/>
@@ -337,5 +337,5 @@
     <joint name="${prefix}right_carriage_joint" type="prismatic">
       <origin
-        xyz="0.1285 -0.0225 0"
+        xyz="0.1265 -0.0225 0"
         rpy="0 0 ${pi / 2}" />
       <parent link="${prefix}link_6"/>
@@ -382,5 +382,5 @@
     <joint name="${prefix}left_carriage_joint" type="prismatic">
       <origin
-        xyz="0.1285 0.0225 0"
+        xyz="0.1265 0.0225 0"
         rpy="${pi} 0 -${pi / 2}" />
       <parent link="${prefix}link_6"/>
@@ -472,5 +472,5 @@
     <joint name="${prefix}ee_gripper" type="fixed">
       <origin
-        xyz="0.22 0 0"
+        xyz="0.218 0 0"
         rpy="0 0 0" />
       <parent link="${prefix}link_6"/>
@@ -517,6 +517,6 @@
     <xacro:zed_camera name="${prefix}wrist" model="zedxnano" parent="${prefix}link_6">
       <origin
-        xyz="0.086133 0 0.057843"
-        rpy="0 0.436 0" />
+        xyz="0.091112 0 0.057797"
+        rpy="0 0.436332 0" />
     </xacro:zed_camera>
   </xacro:macro> <!-- wxpro -->
