Commit message: update inertials from cad

File: urdf/generated/wxpro.urdf (robot description, URDF)
Before this commit: robot wxpro, 19 links, 18 joints
Links:
- link base_link: mass 1.01890997 -> 1.05999025
- link camera_mount: mass 0.0496 -> 0.02632005
- link carriage_left: mass 0.06140653 -> 0.05823866
- link carriage_right: mass 0.06140653 -> 0.05823866
- link gripper_left: mass 0.03751074 -> 0.04941995
- link gripper_right: mass 0.03751074 -> 0.04941995
- link link_1: mass 0.25186508 -> 0.24812120
- link link_2: mass 1.73323784 -> 1.77730310
- link link_3: mass 0.95073232 -> 0.94523715
- link link_4: mass 0.44927258 -> 0.45161249
- link link_5: mass 0.07121851 -> 0.04891458
- link link_6: mass 0.84380465 -> 0.79969124

File: urdf/macros/_wxpro.urdf.xacro (robot description, xacro)
@@ -11,14 +11,14 @@
       <inertial>
         <origin
-          xyz="-0.00615208 0.00004245 0.05031879"
-          rpy="0 0 0" />
-        <mass value="1.01890997"/>
-        <inertia
-          ixx="0.00159523"
-          ixy="0.00000435"
-          ixz="0.00001353"
-          iyy="0.00194612"
-          iyz="-0.00000116"
-          izz="0.00171486"/>
+          xyz="-0.00671439 0.00015929 0.04936050"
+          rpy="0 0 0" />
+        <mass value="1.05999025"/>
+        <inertia
+          ixx="0.00169813"
+          ixy="0.00000821"
+          ixz="-0.00007146"
+          iyy="0.00208830"
+          iyz="-0.00000414"
+          izz="0.00185425"/>
       </inertial>
       <visual>
@@ -42,14 +42,14 @@
       <inertial>
         <origin
-          xyz="0.00269514 -0.00016097 0.01933509"
-          rpy="0 0 0"/>
-        <mass value="0.25186508"/>
-        <inertia
-          ixx="0.00035496"
-          ixy="0.00000196"
-          ixz="-0.00004191"
-          iyy="0.00019037"
-          iyz="-0.00000057"
-          izz="0.00033701"/>
+          xyz="0.00268577 -0.00033976 0.01932318"
+          rpy="0 0 0" />
+        <mass value="0.24812120"/>
+        <inertia
+          ixx="0.00034951"
+          ixy="0.00000169"
+          ixz="-0.00004116"
+          iyy="0.00018796"
+          iyz="-0.00000106"
+          izz="0.00033238"/>
       </inertial>
       <visual>
@@ -86,14 +86,14 @@
       <inertial>
         <origin
-          xyz="-0.10122360 -0.00183082 0.00500847"
-          rpy="0 0 0" />
-        <mass value="1.73323784"/>
-        <inertia
-          ixx="0.00124418"
-          ixy="0.00018835"
-          ixz="0.00080780"
-          iyy="0.02572488"
-          iyz="-0.00001351"
-          izz="0.02574169"/>
+          xyz="-0.09993640 -0.00179613 0.00495252"
+          rpy="0 0 0" />
+        <mass value="1.77730310"/>
+        <inertia
+          ixx="0.00126288"
+          ixy="0.00020880"
+          ixz="0.00082567"
+          iyy="0.02634184"
+          iyz="-0.00001394"
+          izz="0.02635834"/>
       </inertial>
       <visual>
@@ -130,14 +130,14 @@
       <inertial>
         <origin
-          xyz="0.15078963 -0.00011014 0.05540400"
-          rpy="0 0 0" />
-        <mass value="0.95073232"/>
-        <inertia
-          ixx="0.00082328"
-          ixy="0.00000511"
-          ixz="-0.00066824"
-          iyy="0.01003685"
-          iyz="-0.00000307"
-          izz="0.01001162"/>
+          xyz="0.14856512 -0.00093837 0.05470195"
+          rpy="0 0 0" />
+        <mass value="0.94523715"/>
+        <inertia
+          ixx="0.00084253"
+          ixy="-0.00003556"
+          ixz="-0.00075363"
+          iyy="0.01013070"
+          iyz="-0.00002509"
+          izz="0.01007403"/>
       </inertial>
       <visual>
@@ -174,14 +174,14 @@
       <inertial>
         <origin
-          xyz="0.05224276 -0.00099433 0.05517984"
-          rpy="0 0 0" />
-        <mass value="0.44927258"/>
-        <inertia
-          ixx="0.00053844"
-          ixy="-0.00002118"
-          ixz="-0.00024825"
-          iyy="0.00066140"
-          iyz="-0.00002265"
-          izz="0.00055157"/>
+          xyz="0.05026711 -0.00029826 0.05475366"
+          rpy="0 0 0" />
+        <mass value="0.45161249"/>
+        <inertia
+          ixx="0.00058366"
+          ixy="-0.00000429"
+          ixz="-0.00027871"
+          iyy="0.00071884"
+          iyz="-0.00000537"
+          izz="0.00057217"/>
       </inertial>
       <visual>
@@ -218,14 +218,14 @@
       <inertial>
         <origin
-          xyz="-0.00579062 0.00000000 -0.02720844"
-          rpy="0 0 0" />
-        <mass value="0.07121851"/>
-        <inertia
-          ixx="0.00004021"
-          ixy="0.00000000"
-          ixz="-0.00000666"
-          iyy="0.00003792"
-          iyz="0.00000000"
-          izz="0.00001254"/>
+          xyz="-0.00539755 -0.00000007 -0.02459526"
+          rpy="0 0 0" />
+        <mass value="0.04891458"/>
+        <inertia
+          ixx="0.0000265430"
+          ixy="0.0000000000"
+          ixz="-0.0000044943"
+          iyy="0.0000248750"
+          iyz="0.0000000000"
+          izz="0.0000101230"/>
       </inertial>
       <visual>
@@ -262,14 +262,14 @@
       <inertial>
         <origin
-          xyz="0.06129266 -0.00002029 -0.00026366"
-          rpy="0 0 0" />
-        <mass value="0.84380465"/>
-        <inertia
-          ixx="0.00046982"
-          ixy="-0.00000111"
-          ixz="-0.00001431"
-          iyy="0.00127174"
-          iyz="-0.00000064"
-          izz="0.00130342"/>
+          xyz="0.06477211 -0.00005660 -0.00026172"
+          rpy="0 0 0" />
+        <mass value="0.79969124"/>
+        <inertia
+          ixx="0.00045275"
+          ixy="-0.00000048"
+          ixz="-0.00000703"
+          iyy="0.00122431"
+          iyz="-0.00000034"
+          izz="0.00124214"/>
       </inertial>
       <visual>
@@ -303,18 +303,17 @@
         velocity="7.0" />
     </joint>
-    <!-- TODO(abhismirai42): verify inertial properties carriage_links, gripper_links and camera_link -->
     <link name="${prefix}carriage_right">
       <inertial>
         <origin
-          xyz="0.01255019 0.00449652 0.00963255"
-          rpy="0 0 0" />
-        <mass value="0.06140653"/>
-        <inertia
-          ixx="0.0000091193"
-          ixy="-0.0000005807"
-          ixz="-0.0000082661"
-          iyy="0.0000310840"
-          iyz="-0.0000004457"
-          izz="0.0000224261"/>
+          xyz="0.03198817 0.01024525 0.01710190"
+          rpy="0 0 0" />
+        <mass value="0.05823866"/>
+        <inertia
+          ixx="0.0000076862"
+          ixy="-0.0000040815"
+          ixz="-0.0000070993"
+          iyy="0.0000307237"
+          iyz="-0.0000014148"
+          izz="0.0000263411"/>
       </inertial>
       <visual>
@@ -352,14 +351,14 @@
       <inertial>
         <origin
-          xyz="0.01255019 0.00449652 0.00963255"
-          rpy="0 0 0" />
-        <mass value="0.06140653"/>
-        <inertia
-          ixx="0.0000091193"
-          ixy="-0.0000005807"
-          ixz="-0.0000082661"
-          iyy="0.0000310840"
-          iyz="-0.0000004457"
-          izz="0.0000224261"/>
+          xyz="0.03198817 0.01024525 0.01710190"
+          rpy="0 0 0" />
+        <mass value="0.05823866"/>
+        <inertia
+          ixx="0.0000076862"
+          ixy="-0.0000040815"
+          ixz="-0.0000070993"
+          iyy="0.0000307237"
+          iyz="-0.0000014148"
+          izz="0.0000263411"/>
       </inertial>
       <visual>
@@ -396,14 +395,14 @@
       <inertial>
         <origin
-          xyz="0.00275423 0.00000726 0.02059910"
-          rpy="0 0 0" />
-        <mass value="0.03751074"/>
-        <inertia
-          ixx="0.00002087"
-          ixy="0.00000000"
-          ixz="-0.00000338"
-          iyy="0.00002044"
-          iyz="0.00000000"
-          izz="0.00000456"/>
+          xyz="0.00101084 -0.00003183 0.02641115"
+          rpy="0 0 0" />
+        <mass value="0.04941995"/>
+        <inertia
+          ixx="0.0000309841"
+          ixy="-0.0000000016"
+          ixz="-0.0000056184"
+          iyy="0.0000323622"
+          iyz="-0.0000000687"
+          izz="0.0000056007"/>
       </inertial>
       <visual>
@@ -434,14 +433,14 @@
       <inertial>
         <origin
-          xyz="0.00275423 0.00000726 0.02059910"
-          rpy="0 0 0" />
-        <mass value="0.03751074"/>
-        <inertia
-          ixx="0.00002087"
-          ixy="0.00000000"
-          ixz="-0.00000338"
-          iyy="0.00002044"
-          iyz="0.00000000"
-          izz="0.00000456"/>
+          xyz="0.00101084 -0.00003183 0.02641115"
+          rpy="0 0 0" />
+        <mass value="0.04941995"/>
+        <inertia
+          ixx="0.0000309841"
+          ixy="-0.0000000016"
+          ixz="-0.0000056184"
+          iyy="0.0000323622"
+          iyz="-0.0000000687"
+          izz="0.0000056007"/>
       </inertial>
       <visual>
@@ -480,14 +479,14 @@
       <inertial>
         <origin
-          xyz="-0.01095 0 0.03905"
-          rpy="0 0 0" />
-        <mass value="0.0496"/>
-        <inertia
-          ixx="0.0000188"
-          ixy="0.0"
-          ixz="0.0"
-          iyy="0.0000105"
-          iyz="0.0"
-          izz="0.0000123"/>
+          xyz="-0.00817605 -0.00042266 0.04038287"
+          rpy="0 0 0" />
+        <mass value="0.02632005"/>
+        <inertia
+          ixx="0.0000101629"
+          ixy="0.0000000518"
+          ixz="0.0000002760"
+          iyy="0.0000067858"
+          iyz="0.0000003826"
+          izz="0.0000067649"/>
       </inertial>
       <visual>
