Commit message: fix joint_5, carriage and ee_gripper positions from cad

File: urdf/generated/wxheavy.urdf (robot description, URDF)
Before this commit: robot wxheavy, 19 links, 18 joints
Joints:
- joint ee_gripper: origin xyz=0.22 0 0 rpy=0 0 0 -> xyz=0.218 0 0 rpy=0 0 0
- joint joint_5: origin xyz=-0.012 0.0 -0.048 rpy=0 0 0 -> xyz=-0.009 0.0 -0.048 rpy=0 0 0
- joint left_carriage_joint: origin xyz=0.1285 0.0225 0 rpy=3.141592653589793 0 -1.5707963267948966 -> xyz=0.1265 0.0225 0 rpy=3.141592653589793 0 -1.5707963267948966
- joint right_carriage_joint: origin xyz=0.1285 -0.0225 0 rpy=0 0 1.5707963267948966 -> xyz=0.1265 -0.0225 0 rpy=0 0 1.5707963267948966

File: urdf/macros/_wxheavy.urdf.xacro (robot description, xacro)
@@ -292,5 +292,5 @@
     <joint name="${prefix}joint_5" type="revolute">
       <origin
-        xyz="-0.012 0.0 -0.048"
+        xyz="-0.009 0.0 -0.048"
         rpy="0 0 0" />
       <parent link="${prefix}link_5"/>
@@ -337,5 +337,5 @@
     <joint name="${prefix}right_carriage_joint" type="prismatic">
       <origin
-        xyz="0.1285 -0.0225 0"
+        xyz="0.1265 -0.0225 0"
         rpy="0 0 ${pi / 2}" />
       <parent link="${prefix}link_6"/>
@@ -382,5 +382,5 @@
     <joint name="${prefix}left_carriage_joint" type="prismatic">
       <origin
-        xyz="0.1285 0.0225 0"
+        xyz="0.1265 0.0225 0"
         rpy="${pi} 0 -${pi / 2}" />
       <parent link="${prefix}link_6"/>
@@ -472,5 +472,5 @@
     <joint name="${prefix}ee_gripper" type="fixed">
       <origin
-        xyz="0.22 0 0"
+        xyz="0.218 0 0"
         rpy="0 0 0" />
       <parent link="${prefix}link_6"/>
