Commit message: update camera mount joint pos and use zed x xacro for cameras

File: urdf/generated/wxcore.urdf (robot description, URDF)
Before this commit: robot wxcore, 14 links, 13 joints
Links:
- removed link camera
- added link wrist_camera_center, mass 0.075; collision mesh filename=package://trossen_arm_description/meshes/peripherals/zedxna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; visual mesh filename=package://trossen_arm_description/meshes/peripherals/zedxna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
- added link wrist_camera_link
- added link wrist_left_camera_frame
- added link wrist_left_camera_frame_optical
- added link wrist_right_camera_frame
- added link wrist_right_camera_frame_optical
Joints:
- removed joint camera_joint
- added joint wrist_camera_center_joint: type fixed, parent wrist_camera_link, child wrist_camera_center, origin xyz=0 0 0.01525 rpy=0 0 0
- added joint wrist_left_camera_joint: type fixed, parent wrist_camera_center, child wrist_left_camera_frame, origin xyz=-0.01 0.009 0 rpy=0 0 0
- added joint wrist_left_camera_optical_joint: type fixed, parent wrist_left_camera_frame, child wrist_left_camera_frame_optical, origin xyz=0 0 0 rpy=-1.5707963267948966 0 -1.5707963267948966
- added joint wrist_mount_joint: type fixed, parent link_6, child wrist_camera_link, origin xyz=0.086133 0 0.057843 rpy=0 0.436 0
- added joint wrist_right_camera_joint: type fixed, parent wrist_camera_center, child wrist_right_camera_frame, origin xyz=-0.01 -0.009 0 rpy=0 0 0
- added joint wrist_right_camera_optical_joint: type fixed, parent wrist_right_camera_frame, child wrist_right_camera_frame_optical, origin xyz=0 0 0 rpy=-1.5707963267948966 0 -1.5707963267948966
- joint camera_mount_joint: origin xyz=0.104 0 0 rpy=0 0 0 -> xyz=0.102 0 0 rpy=0 0 0

File: urdf/macros/_wxcore.urdf.xacro (robot description, xacro)
@@ -4,4 +4,5 @@
     value="wxcore"
     scope="local"/>
+  <xacro:include filename="$(find trossen_arm_description)/urdf/peripherals/zed_camera.urdf.xacro" />
   <xacro:macro name="wxcore" params="prefix:=''">
     <xacro:property name="mesh_directory" value="package://trossen_arm_description/meshes/${robot_model}"/>
@@ -509,48 +510,14 @@
     <joint name="${prefix}camera_mount_joint" type="fixed">
       <origin
-        xyz="0.104 0 0"
+        xyz="0.102 0 0"
         rpy="0 0 0" />
       <parent link="${prefix}link_6"/>
       <child link="${prefix}camera_mount"/>
     </joint>
-    <!-- TODO(abhismirai42): use official zed camera xacro model -->
-    <link name="${prefix}camera">
-      <inertial>
-        <origin
-          xyz="-0.00555 0 0.07215"
-          rpy="0 0 0" />
-        <mass value="0.0695"/>
-        <inertia
-          ixx="0.0000195"
-          ixy="0.0"
-          ixz="0.0"
-          iyy="0.0000192"
-          iyz="0.0"
-          izz="0.0000202"/>
-      </inertial>
-      <visual>
-        <origin
-          xyz="0 0 0"
-          rpy="0 0 0" />
-        <geometry>
-          <mesh filename="${mesh_directory}/camera.obj"/>
-        </geometry>
-      </visual>
-      <collision>
-        <origin
-          xyz="0 0 0"
-          rpy="0 0 0" />
-        <geometry>
-          <mesh filename="${mesh_directory}/camera.obj"/>
-        </geometry>
-      </collision>
-    </link>
-    <joint name="${prefix}camera_joint" type="fixed">
-      <origin
-        xyz="-0.002173 0 0.001068"
-        rpy="0 0 0" />
-      <parent link="${prefix}camera_mount"/>
-      <child link="${prefix}camera"/>
-    </joint>
+    <xacro:zed_camera name="${prefix}wrist" model="zedxnano" parent="${prefix}link_6">
+      <origin
+        xyz="0.086133 0 0.057843"
+        rpy="0 0.436 0" />
+    </xacro:zed_camera>
   </xacro:macro> <!-- wxcore -->
 </robot>

Commit message: fix joint_5, carriage, ee_gripper and wrist camera positions from cad

File: urdf/generated/wxcore.urdf (robot description, URDF)
Before this commit: robot wxcore, 19 links, 18 joints
Joints:
- joint ee_gripper: origin xyz=0.22 0 0 rpy=0 0 0 -> xyz=0.218 0 0 rpy=0 0 0
- joint joint_5: origin xyz=-0.012 0.0 -0.048 rpy=0 0 0 -> xyz=-0.009 0.0 -0.048 rpy=0 0 0
- joint left_carriage_joint: origin xyz=0.1285 0.0225 0 rpy=3.141592653589793 0 -1.5707963267948966 -> xyz=0.1265 0.0225 0 rpy=3.141592653589793 0 -1.5707963267948966
- joint right_carriage_joint: origin xyz=0.1285 -0.0225 0 rpy=0 0 1.5707963267948966 -> xyz=0.1265 -0.0225 0 rpy=0 0 1.5707963267948966
- joint wrist_mount_joint: origin xyz=0.086133 0 0.057843 rpy=0 0.436 0 -> xyz=0.091112 0 0.057797 rpy=0 0.436332 0

File: urdf/macros/_wxcore.urdf.xacro (robot description, xacro)
@@ -292,5 +292,5 @@
     <joint name="${prefix}joint_5" type="revolute">
       <origin
-        xyz="-0.012 0.0 -0.048"
+        xyz="-0.009 0.0 -0.048"
         rpy="0 0 0" />
       <parent link="${prefix}link_5"/>
@@ -337,5 +337,5 @@
     <joint name="${prefix}right_carriage_joint" type="prismatic">
       <origin
-        xyz="0.1285 -0.0225 0"
+        xyz="0.1265 -0.0225 0"
         rpy="0 0 ${pi / 2}" />
       <parent link="${prefix}link_6"/>
@@ -382,5 +382,5 @@
     <joint name="${prefix}left_carriage_joint" type="prismatic">
       <origin
-        xyz="0.1285 0.0225 0"
+        xyz="0.1265 0.0225 0"
         rpy="${pi} 0 -${pi / 2}" />
       <parent link="${prefix}link_6"/>
@@ -472,5 +472,5 @@
     <joint name="${prefix}ee_gripper" type="fixed">
       <origin
-        xyz="0.22 0 0"
+        xyz="0.218 0 0"
         rpy="0 0 0" />
       <parent link="${prefix}link_6"/>
@@ -517,6 +517,6 @@
     <xacro:zed_camera name="${prefix}wrist" model="zedxnano" parent="${prefix}link_6">
       <origin
-        xyz="0.086133 0 0.057843"
-        rpy="0 0.436 0" />
+        xyz="0.091112 0 0.057797"
+        rpy="0 0.436332 0" />
     </xacro:zed_camera>
   </xacro:macro> <!-- wxcore -->

Commit message: update inertials from cad

File: urdf/generated/wxcore.urdf (robot description, URDF)
Before this commit: robot wxcore, 19 links, 18 joints
Links:
- link base_link: mass 1.01890997 -> 1.05999025
- link camera_mount: mass 0.0496 -> 0.02632005
- link carriage_left: mass 0.06140653 -> 0.05823866
- link carriage_right: mass 0.06140653 -> 0.05823866
- link gripper_left: mass 0.03751074 -> 0.04941995
- link gripper_right: mass 0.03751074 -> 0.04941995
- link link_1: mass 0.137839 -> 0.24434760
- link link_2: mass 0.899971 -> 1.28563686
- link link_3: mass 0.95073232 -> 0.94523715
- link link_4: mass 0.44927258 -> 0.45161249
- link link_5: mass 0.07121851 -> 0.04891458
- link link_6: mass 0.84380465 -> 0.79969124

File: urdf/macros/_wxcore.urdf.xacro (robot description, xacro)
@@ -11,14 +11,14 @@
       <inertial>
         <origin
-          xyz="-0.00615208 0.00004245 0.05031879"
-          rpy="0 0 0" />
-        <mass value="1.01890997"/>
-        <inertia
-          ixx="0.00159523"
-          ixy="0.00000435"
-          ixz="0.00001353"
-          iyy="0.00194612"
-          iyz="-0.00000116"
-          izz="0.00171486"/>
+          xyz="-0.00671439 0.00015929 0.04936050"
+          rpy="0 0 0" />
+        <mass value="1.05999025"/>
+        <inertia
+          ixx="0.00169813"
+          ixy="0.00000821"
+          ixz="-0.00007146"
+          iyy="0.00208830"
+          iyz="-0.00000414"
+          izz="0.00185425"/>
       </inertial>
       <visual>
@@ -42,14 +42,14 @@
       <inertial>
         <origin
-          xyz="0.00380039 0 0.0172804"
-          rpy="0 0 0"/>
-        <mass value="0.137839"/>
-        <inertia
-          ixx="0.000183111"
-          ixy="0.0"
-          ixz="-0.0000132383"
-          iyy="0.000077663"
-          iyz="0.0"
-          izz="0.000195525"/>
+          xyz="0.00265807 -0.00223121 0.01713183"
+          rpy="0 0 0" />
+        <mass value="0.24434760"/>
+        <inertia
+          ixx="0.00030654"
+          ixy="0.00001055"
+          ixz="-0.00003439"
+          iyy="0.00015923"
+          iyz="0.00001202"
+          izz="0.00031679"/>
       </inertial>
       <visual>
@@ -86,14 +86,14 @@
       <inertial>
         <origin
-          xyz="-0.131697 0 0.0000805119"
-          rpy="0 0 0" />
-        <mass value="0.899971"/>
-        <inertia
-          ixx="0.000450486"
-          ixy="0.0"
-          ixz="-0.00000807059"
-          iyy="0.00911893"
-          iyz="0.0"
-          izz="0.00918148"/>
+          xyz="-0.13201452 -0.00047895 0.00007208"
+          rpy="0 0 0" />
+        <mass value="1.28563686"/>
+        <inertia
+          ixx="0.00076836"
+          ixy="0.00000135"
+          ixz="-0.00000528"
+          iyy="0.01793702"
+          iyz="-0.00000123"
+          izz="0.01805880"/>
       </inertial>
       <visual>
@@ -130,14 +130,14 @@
       <inertial>
         <origin
-          xyz="0.15078963 -0.00011014 0.05540400"
-          rpy="0 0 0" />
-        <mass value="0.95073232"/>
-        <inertia
-          ixx="0.00082328"
-          ixy="0.00000511"
-          ixz="-0.00066824"
-          iyy="0.01003685"
-          iyz="-0.00000307"
-          izz="0.01001162"/>
+          xyz="0.14856512 -0.00093837 0.05470195"
+          rpy="0 0 0" />
+        <mass value="0.94523715"/>
+        <inertia
+          ixx="0.00084253"
+          ixy="-0.00003556"
+          ixz="-0.00075363"
+          iyy="0.01013070"
+          iyz="-0.00002509"
+          izz="0.01007403"/>
       </inertial>
       <visual>
@@ -174,14 +174,14 @@
       <inertial>
         <origin
-          xyz="0.05224276 -0.00099433 0.05517984"
-          rpy="0 0 0" />
-        <mass value="0.44927258"/>
-        <inertia
-          ixx="0.00053844"
-          ixy="-0.00002118"
-          ixz="-0.00024825"
-          iyy="0.00066140"
-          iyz="-0.00002265"
-          izz="0.00055157"/>
+          xyz="0.05026711 -0.00029826 0.05475366"
+          rpy="0 0 0" />
+        <mass value="0.45161249"/>
+        <inertia
+          ixx="0.00058366"
+          ixy="-0.00000429"
+          ixz="-0.00027871"
+          iyy="0.00071884"
+          iyz="-0.00000537"
+          izz="0.00057217"/>
       </inertial>
       <visual>
@@ -218,14 +218,14 @@
       <inertial>
         <origin
-          xyz="-0.00579062 0.00000000 -0.02720844"
-          rpy="0 0 0" />
-        <mass value="0.07121851"/>
-        <inertia
-          ixx="0.00004021"
-          ixy="0.00000000"
-          ixz="-0.00000666"
-          iyy="0.00003792"
-          iyz="0.00000000"
-          izz="0.00001254"/>
+          xyz="-0.00539755 -0.00000007 -0.02459526"
+          rpy="0 0 0" />
+        <mass value="0.04891458"/>
+        <inertia
+          ixx="0.0000265430"
+          ixy="0.0000000000"
+          ixz="-0.0000044943"
+          iyy="0.0000248750"
+          iyz="0.0000000000"
+          izz="0.0000101230"/>
       </inertial>
       <visual>
@@ -262,14 +262,14 @@
       <inertial>
         <origin
-          xyz="0.06129266 -0.00002029 -0.00026366"
-          rpy="0 0 0" />
-        <mass value="0.84380465"/>
-        <inertia
-          ixx="0.00046982"
-          ixy="-0.00000111"
-          ixz="-0.00001431"
-          iyy="0.00127174"
-          iyz="-0.00000064"
-          izz="0.00130342"/>
+          xyz="0.06477211 -0.00005660 -0.00026172"
+          rpy="0 0 0" />
+        <mass value="0.79969124"/>
+        <inertia
+          ixx="0.00045275"
+          ixy="-0.00000048"
+          ixz="-0.00000703"
+          iyy="0.00122431"
+          iyz="-0.00000034"
+          izz="0.00124214"/>
       </inertial>
       <visual>
@@ -303,18 +303,17 @@
         velocity="7.0" />
     </joint>
-    <!-- TODO(abhismirai42): verify inertial properties carriage_links, gripper_links and camera_link -->
     <link name="${prefix}carriage_right">
       <inertial>
         <origin
-          xyz="0.01255019 0.00449652 0.00963255"
-          rpy="0 0 0" />
-        <mass value="0.06140653"/>
-        <inertia
-          ixx="0.0000091193"
-          ixy="-0.0000005807"
-          ixz="-0.0000082661"
-          iyy="0.0000310840"
-          iyz="-0.0000004457"
-          izz="0.0000224261"/>
+          xyz="0.03198817 0.01024525 0.01710190"
+          rpy="0 0 0" />
+        <mass value="0.05823866"/>
+        <inertia
+          ixx="0.0000076862"
+          ixy="-0.0000040815"
+          ixz="-0.0000070993"
+          iyy="0.0000307237"
+          iyz="-0.0000014148"
+          izz="0.0000263411"/>
       </inertial>
       <visual>
@@ -352,14 +351,14 @@
       <inertial>
         <origin
-          xyz="0.01255019 0.00449652 0.00963255"
-          rpy="0 0 0" />
-        <mass value="0.06140653"/>
-        <inertia
-          ixx="0.0000091193"
-          ixy="-0.0000005807"
-          ixz="-0.0000082661"
-          iyy="0.0000310840"
-          iyz="-0.0000004457"
-          izz="0.0000224261"/>
+          xyz="0.03198817 0.01024525 0.01710190"
+          rpy="0 0 0" />
+        <mass value="0.05823866"/>
+        <inertia
+          ixx="0.0000076862"
+          ixy="-0.0000040815"
+          ixz="-0.0000070993"
+          iyy="0.0000307237"
+          iyz="-0.0000014148"
+          izz="0.0000263411"/>
       </inertial>
       <visual>
@@ -396,14 +395,14 @@
       <inertial>
         <origin
-          xyz="0.00275423 0.00000726 0.02059910"
-          rpy="0 0 0" />
-        <mass value="0.03751074"/>
-        <inertia
-          ixx="0.00002087"
-          ixy="0.00000000"
-          ixz="-0.00000338"
-          iyy="0.00002044"
-          iyz="0.00000000"
-          izz="0.00000456"/>
+          xyz="0.00101084 -0.00003183 0.02641115"
+          rpy="0 0 0" />
+        <mass value="0.04941995"/>
+        <inertia
+          ixx="0.0000309841"
+          ixy="-0.0000000016"
+          ixz="-0.0000056184"
+          iyy="0.0000323622"
+          iyz="-0.0000000687"
+          izz="0.0000056007"/>
       </inertial>
       <visual>
@@ -434,14 +433,14 @@
       <inertial>
         <origin
-          xyz="0.00275423 0.00000726 0.02059910"
-          rpy="0 0 0" />
-        <mass value="0.03751074"/>
-        <inertia
-          ixx="0.00002087"
-          ixy="0.00000000"
-          ixz="-0.00000338"
-          iyy="0.00002044"
-          iyz="0.00000000"
-          izz="0.00000456"/>
+          xyz="0.00101084 -0.00003183 0.02641115"
+          rpy="0 0 0" />
+        <mass value="0.04941995"/>
+        <inertia
+          ixx="0.0000309841"
+          ixy="-0.0000000016"
+          ixz="-0.0000056184"
+          iyy="0.0000323622"
+          iyz="-0.0000000687"
+          izz="0.0000056007"/>
       </inertial>
       <visual>
@@ -480,14 +479,14 @@
       <inertial>
         <origin
-          xyz="-0.01095 0 0.03905"
-          rpy="0 0 0" />
-        <mass value="0.0496"/>
-        <inertia
-          ixx="0.0000188"
-          ixy="0.0"
-          ixz="0.0"
-          iyy="0.0000105"
-          iyz="0.0"
-          izz="0.0000123"/>
+          xyz="-0.00817605 -0.00042266 0.04038287"
+          rpy="0 0 0" />
+        <mass value="0.02632005"/>
+        <inertia
+          ixx="0.0000101629"
+          ixy="0.0000000518"
+          ixz="0.0000002760"
+          iyy="0.0000067858"
+          iyz="0.0000003826"
+          izz="0.0000067649"/>
       </inertial>
       <visual>
