Commit message: update rivet mesh and urdf files

File: urdf/generated/rivet.urdf (robot description, URDF)
Before this commit: robot rivet, 38 links, 37 joints
Joints:
- joint swivel_drive_1: limit (none) -> effort=4 velocity=18.691589
- joint swivel_drive_2: limit (none) -> effort=4 velocity=18.691589
- joint swivel_drive_3: limit (none) -> effort=4 velocity=18.691589
- joint swivel_steer_1: limit (none) -> lower=-3.141592653589793 upper=3.141592653589793 effort=10 velocity=6.283185; type continuous -> revolute
- joint swivel_steer_2: limit (none) -> lower=-3.141592653589793 upper=3.141592653589793 effort=10 velocity=6.283185; type continuous -> revolute
- joint swivel_steer_3: limit (none) -> lower=-3.141592653589793 upper=3.141592653589793 effort=10 velocity=6.283185; type continuous -> revolute

File: urdf/rivet.urdf.xacro (robot description, xacro)
@@ -161,5 +161,5 @@
       </collision>
     </link>
-    <joint name="swivel_steer_${suffix}" type="continuous">
+    <joint name="swivel_steer_${suffix}" type="revolute">
       <origin
         xyz="${steer_joint_xyz}"
@@ -168,4 +168,9 @@
       <child link="swivel_${suffix}"/>
       <axis xyz="0 0 1"/>
+      <limit
+        lower="${-pi}"
+        upper="${pi}"
+        effort="10"
+        velocity="6.283185" />
     </joint>
     <link name="wheel_${suffix}">
@@ -207,4 +212,7 @@
       <child link="wheel_${suffix}"/>
       <axis xyz="-1 0 0"/>
+      <limit
+        effort="4"
+        velocity="18.691589" />
     </joint>
   </xacro:macro> <!-- swivel_module -->

Commit message: update all link origin frame orientation, carriage link upper and lower limits, make swivel joint  continuous

File: urdf/generated/rivet.urdf (robot description, URDF)
Before this commit: robot rivet, 38 links, 37 joints
Joints:
- removed joint swivel_drive_1
- removed joint swivel_drive_2
- removed joint swivel_drive_3
- removed joint swivel_steer_1
- removed joint swivel_steer_2
- removed joint swivel_steer_3
- added joint swivel_joint_1: type continuous, parent base_link, child swivel_1, origin xyz=-0.24 0.0 0.003 rpy=0 0 0, axis 0 0 1, limit effort=10 velocity=6.283185
- added joint swivel_joint_2: type continuous, parent base_link, child swivel_2, origin xyz=0.24 -0.190 0.003 rpy=0 0 0, axis 0 0 1, limit effort=10 velocity=6.283185
- added joint swivel_joint_3: type continuous, parent base_link, child swivel_3, origin xyz=0.24 0.190 0.003 rpy=0 0 0, axis 0 0 1, limit effort=10 velocity=6.283185
- added joint wheel_joint_1: type continuous, parent swivel_1, child wheel_1, origin xyz=0 0 -0.078 rpy=0 0 0, axis 0 -1 0, limit effort=4 velocity=18.691589
- added joint wheel_joint_2: type continuous, parent swivel_2, child wheel_2, origin xyz=0 0 -0.078 rpy=0 0 0, axis 0 -1 0, limit effort=4 velocity=18.691589
- added joint wheel_joint_3: type continuous, parent swivel_3, child wheel_3, origin xyz=0 0 -0.078 rpy=0 0 0, axis 0 -1 0, limit effort=4 velocity=18.691589
- joint camera_mount_joint: origin xyz=0 0.0786917 0.351299 rpy=-0.436332 0 0 -> xyz=0.0786917 0 0.351299 rpy=0 0.436332 0
- joint carriage_lift_joint: limit lower=-0.32 upper=0.42 effort=1 velocity=1 -> lower=0.0 upper=0.858 effort=1 velocity=1; origin xyz=-0.000125 0.165 0.595105 rpy=0 0 0 -> xyz=0.165 0.0 0.181 rpy=0 0 0
- joint follower_left_mount_joint: origin xyz=-0.275 0.0615 0.031 rpy=0 0 1.5707963267948966 -> xyz=0.0615 0.275 0.031 rpy=0 0 0
- joint follower_right_mount_joint: origin xyz=0.275 0.0615 0.031 rpy=0 0 1.5707963267948966 -> xyz=0.0615 -0.275 0.031 rpy=0 0 0

File: urdf/rivet.urdf.xacro (robot description, xacro)
@@ -10,13 +10,13 @@
     <inertial>
       <origin
-        xyz="-0.00387668 -0.0332838 0.198466"
+        xyz="-0.0332838 0.00387668 0.198466"
         rpy="0 0 0" />
       <mass value="73.7606"/>
       <inertia
-        ixx="6.32878"
-        ixy="-0.0384037"
-        ixz="-0.00555349"
-        iyy="5.76624"
-        iyz="-0.51839"
+        ixx="5.76624"
+        ixy="0.0"
+        ixz="-0.51839"
+        iyy="6.32878"
+        iyz="0.00555349"
         izz="2.94862"/>
     </inertial>
@@ -46,8 +46,7 @@
     <child link="base_link"/>
   </joint>
-  <!--TODO(abhismirai42): lower/upper are placeholders.-->
   <joint name="carriage_lift_joint" type="prismatic">
     <origin
-      xyz="-0.000125 0.165 0.595105"
+      xyz="0.165 0.0 0.181"
       rpy="0 0 0" />
     <parent link="base_link"/>
@@ -55,6 +54,6 @@
     <axis xyz="0 0 1"/>
     <limit
-      lower="-0.32"
-      upper="0.42"
+      lower="0.0"
+      upper="0.858"
       effort="1"
       velocity="1" />
@@ -63,13 +62,13 @@
     <inertial>
       <origin
-        xyz="0 0.0543177 0.0192157"
+        xyz="0.0543177 0 0.0192157"
         rpy="0 0 0" />
       <mass value="2.69782"/>
       <inertia
-        ixx="0.0103103"
+        ixx="0.102184"
         ixy="0.0"
-        ixz="0.0"
-        iyy="0.102184"
-        iyz="-0.000235492"
+        ixz="-0.000235492"
+        iyy="0.0103103"
+        iyz="0.0"
         izz="0.0952441"/>
     </inertial>
@@ -94,12 +93,12 @@
     <inertial>
       <origin
-        xyz="0 0.0181899 0"
+        xyz="0.0181899 0 0"
         rpy="0 0 0" />
       <mass value="0.0982026"/>
       <inertia
-        ixx="0.0000174033"
+        ixx="0.0000756992"
         ixy="0.0"
         ixz="0.0"
-        iyy="0.0000756992"
+        iyy="0.0000174033"
         iyz="0.0"
         izz="0.0000778027"/>
@@ -124,6 +123,6 @@
   <joint name="camera_mount_joint" type="fixed">
     <origin
-      xyz="0 0.0786917 0.351299"
-      rpy="-0.436332 0 0" />
+      xyz="0.0786917 0 0.351299"
+      rpy="0 0.436332 0" />
     <parent link="carriage_lift_link"/>
     <child link="camera"/>
@@ -137,8 +136,8 @@
         <mass value="0.619024"/>
         <inertia
-          ixx="0.000923685"
+          ixx="0.00137238"
           ixy="0.0"
           ixz="0.0"
-          iyy="0.00137238"
+          iyy="0.000923685"
           iyz="0.0"
           izz="0.00117765"/>
@@ -161,5 +160,5 @@
       </collision>
     </link>
-    <joint name="swivel_steer_${suffix}" type="revolute">
+    <joint name="swivel_joint_${suffix}" type="continuous">
       <origin
         xyz="${steer_joint_xyz}"
@@ -169,6 +168,4 @@
       <axis xyz="0 0 1"/>
       <limit
-        lower="${-pi}"
-        upper="${pi}"
         effort="10"
         velocity="6.283185" />
@@ -181,8 +178,8 @@
         <mass value="0.330766"/>
         <inertia
-          ixx="0.000500429"
+          ixx="0.000294662"
           ixy="0.0"
           ixz="0.0"
-          iyy="0.000294662"
+          iyy="0.000500429"
           iyz="0.0"
           izz="0.000294662"/>
@@ -205,5 +202,5 @@
       </collision>
     </link>
-    <joint name="swivel_drive_${suffix}" type="continuous">
+    <joint name="wheel_joint_${suffix}" type="continuous">
       <origin
         xyz="0 0 -0.078"
@@ -211,5 +208,5 @@
       <parent link="swivel_${suffix}"/>
       <child link="wheel_${suffix}"/>
-      <axis xyz="-1 0 0"/>
+      <axis xyz="0 -1 0"/>
       <limit
         effort="4"
@@ -218,27 +215,27 @@
   </xacro:macro> <!-- swivel_module -->
   <xacro:swivel_module suffix="1"
-    steer_joint_xyz="0.000125 -0.24 0.003"
+    steer_joint_xyz="-0.24 0.0 0.003"
     steer_joint_rpy="0 0 0"/>
   <xacro:swivel_module suffix="2"
-    steer_joint_xyz="-0.189875 0.24 0.003"
+    steer_joint_xyz="0.24 -0.190 0.003"
     steer_joint_rpy="0 0 0"/>
   <xacro:swivel_module suffix="3"
-    steer_joint_xyz="0.190125 0.24 0.003"
+    steer_joint_xyz="0.24 0.190 0.003"
     steer_joint_rpy="0 0 0"/>
+  <joint name="follower_right_mount_joint" type="fixed">
+    <origin
+      xyz="0.0615 -0.275 0.031"
+      rpy="0 0 0" />
+    <parent link="carriage_lift_link"/>
+    <child link="follower_right_base_link"/>
+  </joint>
+  <xacro:wxpro prefix="follower_right_"/>
   <joint name="follower_left_mount_joint" type="fixed">
     <origin
-      xyz="-0.275 0.0615 0.031"
-      rpy="0 0 ${pi / 2}" />
+      xyz="0.0615 0.275 0.031"
+      rpy="0 0 0" />
     <parent link="carriage_lift_link"/>
     <child link="follower_left_base_link"/>
   </joint>
   <xacro:wxpro prefix="follower_left_"/>
-  <joint name="follower_right_mount_joint" type="fixed">
-    <origin
-      xyz="0.275 0.0615 0.031"
-      rpy="0 0 ${pi / 2}" />
-    <parent link="carriage_lift_link"/>
-    <child link="follower_right_base_link"/>
-  </joint>
-  <xacro:wxpro prefix="follower_right_"/>
 </robot>

Commit message: update wheels rotation direction

File: urdf/generated/rivet.urdf (robot description, URDF)
Before this commit: robot rivet, 38 links, 37 joints
Joints:
- joint wheel_joint_1: axis 0 -1 0 -> 0 1 0
- joint wheel_joint_2: axis 0 -1 0 -> 0 1 0
- joint wheel_joint_3: axis 0 -1 0 -> 0 1 0

File: urdf/rivet.urdf.xacro (robot description, xacro)
@@ -208,5 +208,5 @@
       <parent link="swivel_${suffix}"/>
       <child link="wheel_${suffix}"/>
-      <axis xyz="0 -1 0"/>
+      <axis xyz="0 1 0"/>
       <limit
         effort="4"

Commit message: Rename links and joints

File: urdf/generated/rivet.urdf (robot description, URDF)
Before this commit: robot rivet, 38 links, 37 joints
Links:
- removed link carriage_lift_link
- removed link swivel_1
- removed link swivel_2
- removed link swivel_3
- removed link wheel_1
- removed link wheel_2
- removed link wheel_3
- added link b_drive_link, mass 0.330766; collision mesh filename=package://trossen_arm_description/meshes/rivet/wheel.obj; visual mesh filename=package://trossen_arm_description/meshes/rivet/wheel.obj
- added link b_pivot_link, mass 0.619024; collision mesh filename=package://trossen_arm_description/meshes/rivet/pivot_link.o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; visual mesh filename=package://trossen_arm_description/meshes/rivet/pivot_link.o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
- added link fl_drive_link, mass 0.330766; collision mesh filename=package://trossen_arm_description/meshes/rivet/wheel.obj; visual mesh filename=package://trossen_arm_description/meshes/rivet/wheel.obj
- added link fl_pivot_link, mass 0.619024; collision mesh filename=package://trossen_arm_description/meshes/rivet/pivot_link.o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; visual mesh filename=package://trossen_arm_description/meshes/rivet/pivot_link.o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
- added link fr_drive_link, mass 0.330766; collision mesh filename=package://trossen_arm_description/meshes/rivet/wheel.obj; visual mesh filename=package://trossen_arm_description/meshes/rivet/wheel.obj
- added link fr_pivot_link, mass 0.619024; collision mesh filename=package://trossen_arm_description/meshes/rivet/pivot_link.o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; visual mesh filename=package://trossen_arm_description/meshes/rivet/pivot_link.o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
- added link lift_link, mass 2.69782; collision mesh filename=package://trossen_arm_description/meshes/rivet/lift_link.obj; visual mesh filename=package://trossen_arm_description/meshes/rivet/lift_link.obj
Joints:
- removed joint carriage_lift_joint
- removed joint swivel_joint_1
- removed joint swivel_joint_2
- removed joint swivel_joint_3
- removed joint wheel_joint_1
- removed joint wheel_joint_2
- removed joint wheel_joint_3
- added joint b_drive: type continuous, parent b_pivot_link, child b_drive_link, origin xyz=0 0 -0.078 rpy=0 0 0, axis 0 1 0, limit effort=4 velocity=18.691589
- added joint b_pivot: type continuous, parent base_link, child b_pivot_link, origin xyz=-0.24 0.0 0.003 rpy=0 0 0, axis 0 0 1, limit effort=10 velocity=6.283185
- added joint fl_drive: type continuous, parent fl_pivot_link, child fl_drive_link, origin xyz=0 0 -0.078 rpy=0 0 0, axis 0 1 0, limit effort=4 velocity=18.691589
- added joint fl_pivot: type continuous, parent base_link, child fl_pivot_link, origin xyz=0.24 0.190 0.003 rpy=0 0 0, axis 0 0 1, limit effort=10 velocity=6.283185
- added joint fr_drive: type continuous, parent fr_pivot_link, child fr_drive_link, origin xyz=0 0 -0.078 rpy=0 0 0, axis 0 1 0, limit effort=4 velocity=18.691589
- added joint fr_pivot: type continuous, parent base_link, child fr_pivot_link, origin xyz=0.24 -0.190 0.003 rpy=0 0 0, axis 0 0 1, limit effort=10 velocity=6.283185
- added joint lift: type prismatic, parent base_link, child lift_link, origin xyz=0.165 0.0 0.181 rpy=0 0 0, axis 0 0 1, limit lower=0.0 upper=0.858 effort=1 velocity=1
- joint camera_mount_joint: parent carriage_lift_link -> lift_link
- joint follower_left_mount_joint: parent carriage_lift_link -> lift_link
- joint follower_right_mount_joint: parent carriage_lift_link -> lift_link

File: urdf/rivet.urdf.xacro (robot description, xacro)
@@ -46,10 +46,10 @@
     <child link="base_link"/>
   </joint>
-  <joint name="carriage_lift_joint" type="prismatic">
+  <joint name="lift" type="prismatic">
     <origin
       xyz="0.165 0.0 0.181"
       rpy="0 0 0" />
     <parent link="base_link"/>
-    <child link="carriage_lift_link"/>
+    <child link="lift_link"/>
     <axis xyz="0 0 1"/>
     <limit
@@ -59,5 +59,5 @@
       velocity="1" />
   </joint>
-  <link name="carriage_lift_link">
+  <link name="lift_link">
     <inertial>
       <origin
@@ -78,5 +78,5 @@
         rpy="0 0 0" />
       <geometry>
-        <mesh filename="${mesh_directory}/carriage_lift_link.obj"/>
+        <mesh filename="${mesh_directory}/lift_link.obj"/>
       </geometry>
     </visual>
@@ -86,5 +86,5 @@
         rpy="0 0 0" />
       <geometry>
-        <mesh filename="${mesh_directory}/carriage_lift_link.obj"/>
+        <mesh filename="${mesh_directory}/lift_link.obj"/>
       </geometry>
     </collision>
@@ -125,9 +125,9 @@
       xyz="0.0786917 0 0.351299"
       rpy="0 0.436332 0" />
-    <parent link="carriage_lift_link"/>
+    <parent link="lift_link"/>
     <child link="camera"/>
   </joint>
-  <xacro:macro name="swivel_module" params="suffix steer_joint_xyz steer_joint_rpy">
-    <link name="swivel_${suffix}">
+  <xacro:macro name="swerve_module" params="prefix pivot_xyz pivot_rpy">
+    <link name="${prefix}_pivot_link">
       <inertial>
         <origin
@@ -148,5 +148,5 @@
           rpy="0 0 0" />
         <geometry>
-          <mesh filename="${mesh_directory}/swivel.obj"/>
+          <mesh filename="${mesh_directory}/pivot_link.obj"/>
         </geometry>
       </visual>
@@ -156,14 +156,14 @@
           rpy="0 0 0" />
         <geometry>
-          <mesh filename="${mesh_directory}/swivel.obj"/>
+          <mesh filename="${mesh_directory}/pivot_link.obj"/>
         </geometry>
       </collision>
     </link>
-    <joint name="swivel_joint_${suffix}" type="continuous">
-      <origin
-        xyz="${steer_joint_xyz}"
-        rpy="${steer_joint_rpy}" />
+    <joint name="${prefix}_pivot" type="continuous">
+      <origin
+        xyz="${pivot_xyz}"
+        rpy="${pivot_rpy}" />
       <parent link="base_link"/>
-      <child link="swivel_${suffix}"/>
+      <child link="${prefix}_pivot_link"/>
       <axis xyz="0 0 1"/>
       <limit
@@ -171,5 +171,5 @@
         velocity="6.283185" />
     </joint>
-    <link name="wheel_${suffix}">
+    <link name="${prefix}_drive_link">
       <inertial>
         <origin
@@ -202,10 +202,10 @@
       </collision>
     </link>
-    <joint name="wheel_joint_${suffix}" type="continuous">
+    <joint name="${prefix}_drive" type="continuous">
       <origin
         xyz="0 0 -0.078"
         rpy="0 0 0" />
-      <parent link="swivel_${suffix}"/>
-      <child link="wheel_${suffix}"/>
+      <parent link="${prefix}_pivot_link"/>
+      <child link="${prefix}_drive_link"/>
       <axis xyz="0 1 0"/>
       <limit
@@ -213,19 +213,19 @@
         velocity="18.691589" />
     </joint>
-  </xacro:macro> <!-- swivel_module -->
-  <xacro:swivel_module suffix="1"
-    steer_joint_xyz="-0.24 0.0 0.003"
-    steer_joint_rpy="0 0 0"/>
-  <xacro:swivel_module suffix="2"
-    steer_joint_xyz="0.24 -0.190 0.003"
-    steer_joint_rpy="0 0 0"/>
-  <xacro:swivel_module suffix="3"
-    steer_joint_xyz="0.24 0.190 0.003"
-    steer_joint_rpy="0 0 0"/>
+  </xacro:macro> <!-- swerve_module -->
+  <xacro:swerve_module prefix="fl"
+    pivot_xyz="0.24 0.190 0.003"
+    pivot_rpy="0 0 0"/>
+  <xacro:swerve_module prefix="fr"
+    pivot_xyz="0.24 -0.190 0.003"
+    pivot_rpy="0 0 0"/>
+  <xacro:swerve_module prefix="b"
+    pivot_xyz="-0.24 0.0 0.003"
+    pivot_rpy="0 0 0"/>
   <joint name="follower_right_mount_joint" type="fixed">
     <origin
       xyz="0.0615 -0.275 0.031"
       rpy="0 0 0" />
-    <parent link="carriage_lift_link"/>
+    <parent link="lift_link"/>
     <child link="follower_right_base_link"/>
   </joint>
@@ -235,5 +235,5 @@
       xyz="0.0615 0.275 0.031"
       rpy="0 0 0" />
-    <parent link="carriage_lift_link"/>
+    <parent link="lift_link"/>
     <child link="follower_left_base_link"/>
   </joint>
