Commit message: update main camera to use zed x camera xacro file

File: urdf/generated/rivet.urdf (robot description, URDF)
Before this commit: robot rivet, 38 links, 37 joints
Links:
- removed link camera
- removed link follower_left_camera
- removed link follower_right_camera
- added link cam_high_camera_center, mass 0.15; collision mesh filename=package://trossen_arm_description/meshes/peripherals/zedxm.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; visual mesh filename=package://trossen_arm_description/meshes/peripherals/zedxm.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
- added link cam_high_camera_link
- added link cam_high_left_camera_frame
- added link cam_high_left_camera_frame_optical
- added link cam_high_right_camera_frame
- added link cam_high_right_camera_frame_optical
- added link follower_left_wrist_camera_center, mass 0.075; collision mesh filename=package://trossen_arm_description/meshes/peripherals/zedxna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; visual mesh filename=package://trossen_arm_description/meshes/peripherals/zedxna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
- added link follower_left_wrist_camera_link
- added link follower_left_wrist_left_camera_frame
- added link follower_left_wrist_left_camera_frame_optical
- added link follower_left_wrist_right_camera_frame
- added link follower_left_wrist_right_camera_frame_optical
- added link follower_right_wrist_camera_center, mass 0.075; collision mesh filename=package://trossen_arm_description/meshes/peripherals/zedxna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; visual mesh filename=package://trossen_arm_description/meshes/peripherals/zedxna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
- added link follower_right_wrist_camera_link
- added link follower_right_wrist_left_camera_frame
- added link follower_right_wrist_left_camera_frame_optical
- added link follower_right_wrist_right_camera_frame
- added link follower_right_wrist_right_camera_frame_optical
Joints:
- removed joint camera_mount_joint
- removed joint follower_left_camera_joint
- removed joint follower_right_camera_joint
- added joint cam_high_camera_center_joint: type fixed, parent cam_high_camera_link, child cam_high_camera_center, origin xyz=0 0 0.016 rpy=0 0 0
- added joint cam_high_left_camera_joint: type fixed, parent cam_high_camera_center, child cam_high_left_camera_frame, origin xyz=-0.01 0.025 0 rpy=0 0 0
- added joint cam_high_left_camera_optical_joint: type fixed, parent cam_high_left_camera_frame, child cam_high_left_camera_frame_optical, origin xyz=0 0 0 rpy=-1.5707963267948966 0 -1.5707963267948966
- added joint cam_high_mount_joint: type fixed, parent lift_link, child cam_high_camera_link, origin xyz=0.0906 0 0.3267 rpy=0 0.436332 0
- added joint cam_high_right_camera_joint: type fixed, parent cam_high_camera_center, child cam_high_right_camera_frame, origin xyz=-0.01 -0.025 0 rpy=0 0 0
- added joint cam_high_right_camera_optical_joint: type fixed, parent cam_high_right_camera_frame, child cam_high_right_camera_frame_optical, origin xyz=0 0 0 rpy=-1.5707963267948966 0 -1.5707963267948966
- added joint follower_left_wrist_camera_center_joint: type fixed, parent follower_left_wrist_camera_link, child follower_left_wrist_camera_center, origin xyz=0 0 0.01525 rpy=0 0 0
- added joint follower_left_wrist_left_camera_joint: type fixed, parent follower_left_wrist_camera_center, child follower_left_wrist_left_camera_frame, origin xyz=-0.01 0.009 0 rpy=0 0 0
- added joint follower_left_wrist_left_camera_optical_joint: type fixed, parent follower_left_wrist_left_camera_frame, child follower_left_wrist_left_camera_frame_optical, origin xyz=0 0 0 rpy=-1.5707963267948966 0 -1.5707963267948966
- added joint follower_left_wrist_mount_joint: type fixed, parent follower_left_link_6, child follower_left_wrist_camera_link, origin xyz=0.086133 0 0.057843 rpy=0 0.436 0
- added joint follower_left_wrist_right_camera_joint: type fixed, parent follower_left_wrist_camera_center, child follower_left_wrist_right_camera_frame, origin xyz=-0.01 -0.009 0 rpy=0 0 0
- added joint follower_left_wrist_right_camera_optical_joint: type fixed, parent follower_left_wrist_right_camera_frame, child follower_left_wrist_right_camera_frame_optical, origin xyz=0 0 0 rpy=-1.5707963267948966 0 -1.5707963267948966
- added joint follower_right_wrist_camera_center_joint: type fixed, parent follower_right_wrist_camera_link, child follower_right_wrist_camera_center, origin xyz=0 0 0.01525 rpy=0 0 0
- added joint follower_right_wrist_left_camera_joint: type fixed, parent follower_right_wrist_camera_center, child follower_right_wrist_left_camera_frame, origin xyz=-0.01 0.009 0 rpy=0 0 0
- added joint follower_right_wrist_left_camera_optical_joint: type fixed, parent follower_right_wrist_left_camera_frame, child follower_right_wrist_left_camera_frame_optical, origin xyz=0 0 0 rpy=-1.5707963267948966 0 -1.5707963267948966
- added joint follower_right_wrist_mount_joint: type fixed, parent follower_right_link_6, child follower_right_wrist_camera_link, origin xyz=0.086133 0 0.057843 rpy=0 0.436 0
- added joint follower_right_wrist_right_camera_joint: type fixed, parent follower_right_wrist_camera_center, child follower_right_wrist_right_camera_frame, origin xyz=-0.01 -0.009 0 rpy=0 0 0
- added joint follower_right_wrist_right_camera_optical_joint: type fixed, parent follower_right_wrist_right_camera_frame, child follower_right_wrist_right_camera_frame_optical, origin xyz=0 0 0 rpy=-1.5707963267948966 0 -1.5707963267948966
- joint follower_left_camera_mount_joint: origin xyz=0.104 0 0 rpy=0 0 0 -> xyz=0.102 0 0 rpy=0 0 0
- joint follower_right_camera_mount_joint: origin xyz=0.104 0 0 rpy=0 0 0 -> xyz=0.102 0 0 rpy=0 0 0

File: urdf/rivet.urdf.xacro (robot description, xacro)
@@ -5,4 +5,5 @@
     scope="global"/>
   <xacro:include filename="$(find trossen_arm_description)/urdf/macros/_wxpro.urdf.xacro" />
+  <xacro:include filename="$(find trossen_arm_description)/urdf/peripherals/zed_camera.urdf.xacro" />
   <xacro:property name="mesh_directory" value="package://trossen_arm_description/meshes/rivet"/>
   <!-- TODO(abhismirai42): update inertial property for rivet links -->
@@ -90,42 +91,9 @@
     </collision>
   </link>
-  <link name="camera">
-    <inertial>
-      <origin
-        xyz="0.0181899 0 0"
-        rpy="0 0 0" />
-      <mass value="0.0982026"/>
-      <inertia
-        ixx="0.0000756992"
-        ixy="0.0"
-        ixz="0.0"
-        iyy="0.0000174033"
-        iyz="0.0"
-        izz="0.0000778027"/>
-    </inertial>
-    <visual>
-      <origin
-        xyz="0 0 0"
-        rpy="0 0 0" />
-      <geometry>
-        <mesh filename="${mesh_directory}/camera.obj"/>
-      </geometry>
-    </visual>
-    <collision>
-      <origin
-        xyz="0 0 0"
-        rpy="0 0 0" />
-      <geometry>
-        <mesh filename="${mesh_directory}/camera.obj"/>
-      </geometry>
-    </collision>
-  </link>
-  <joint name="camera_mount_joint" type="fixed">
-    <origin
-      xyz="0.0786917 0 0.351299"
+  <xacro:zed_camera name="cam_high" model="zedxm" parent="lift_link">
+    <origin
+      xyz="0.0906 0 0.3267"
       rpy="0 0.436332 0" />
-    <parent link="lift_link"/>
-    <child link="camera"/>
-  </joint>
+  </xacro:zed_camera>
   <xacro:macro name="swerve_module" params="prefix pivot_xyz pivot_rpy">
     <link name="${prefix}_pivot_link">

Commit message: update generated urdf for pro wrist fix

File: urdf/generated/rivet.urdf (robot description, URDF)
Before this commit: robot rivet, 53 links, 52 joints
Joints:
- joint follower_left_ee_gripper: origin xyz=0.22 0 0 rpy=0 0 0 -> xyz=0.218 0 0 rpy=0 0 0
- joint follower_left_joint_5: origin xyz=-0.012 0.0 -0.048 rpy=0 0 0 -> xyz=-0.009 0.0 -0.048 rpy=0 0 0
- joint follower_left_left_carriage_joint: origin xyz=0.1285 0.0225 0 rpy=3.141592653589793 0 -1.5707963267948966 -> xyz=0.1265 0.0225 0 rpy=3.141592653589793 0 -1.5707963267948966
- joint follower_left_right_carriage_joint: origin xyz=0.1285 -0.0225 0 rpy=0 0 1.5707963267948966 -> xyz=0.1265 -0.0225 0 rpy=0 0 1.5707963267948966
- joint follower_left_wrist_mount_joint: origin xyz=0.086133 0 0.057843 rpy=0 0.436 0 -> xyz=0.091112 0 0.057797 rpy=0 0.436332 0
- joint follower_right_ee_gripper: origin xyz=0.22 0 0 rpy=0 0 0 -> xyz=0.218 0 0 rpy=0 0 0
- joint follower_right_joint_5: origin xyz=-0.012 0.0 -0.048 rpy=0 0 0 -> xyz=-0.009 0.0 -0.048 rpy=0 0 0
- joint follower_right_left_carriage_joint: origin xyz=0.1285 0.0225 0 rpy=3.141592653589793 0 -1.5707963267948966 -> xyz=0.1265 0.0225 0 rpy=3.141592653589793 0 -1.5707963267948966
- joint follower_right_right_carriage_joint: origin xyz=0.1285 -0.0225 0 rpy=0 0 1.5707963267948966 -> xyz=0.1265 -0.0225 0 rpy=0 0 1.5707963267948966
- joint follower_right_wrist_mount_joint: origin xyz=0.086133 0 0.057843 rpy=0 0.436 0 -> xyz=0.091112 0 0.057797 rpy=0 0.436332 0

Commit message: update inertials from cad

File: urdf/generated/rivet.urdf (robot description, URDF)
Before this commit: robot rivet, 53 links, 52 joints
Links:
- link follower_left_base_link: mass 1.01890997 -> 1.05999025
- link follower_left_camera_mount: mass 0.0496 -> 0.02632005
- link follower_left_carriage_left: mass 0.06140653 -> 0.05823866
- link follower_left_carriage_right: mass 0.06140653 -> 0.05823866
- link follower_left_gripper_left: mass 0.03751074 -> 0.04941995
- link follower_left_gripper_right: mass 0.03751074 -> 0.04941995
- link follower_left_link_1: mass 0.25186508 -> 0.24812120
- link follower_left_link_2: mass 1.73323784 -> 1.77730310
- link follower_left_link_3: mass 0.95073232 -> 0.94523715
- link follower_left_link_4: mass 0.44927258 -> 0.45161249
- link follower_left_link_5: mass 0.07121851 -> 0.04891458
- link follower_left_link_6: mass 0.84380465 -> 0.79969124
- link follower_right_base_link: mass 1.01890997 -> 1.05999025
- link follower_right_camera_mount: mass 0.0496 -> 0.02632005
- link follower_right_carriage_left: mass 0.06140653 -> 0.05823866
- link follower_right_carriage_right: mass 0.06140653 -> 0.05823866
- link follower_right_gripper_left: mass 0.03751074 -> 0.04941995
- link follower_right_gripper_right: mass 0.03751074 -> 0.04941995
- link follower_right_link_1: mass 0.25186508 -> 0.24812120
- link follower_right_link_2: mass 1.73323784 -> 1.77730310
- link follower_right_link_3: mass 0.95073232 -> 0.94523715
- link follower_right_link_4: mass 0.44927258 -> 0.45161249
- link follower_right_link_5: mass 0.07121851 -> 0.04891458
- link follower_right_link_6: mass 0.84380465 -> 0.79969124

Commit message: update lift, pivot and drive limits from firmware

File: urdf/generated/rivet.urdf (robot description, URDF)
Before this commit: robot rivet, 53 links, 52 joints
Joints:
- joint b_drive: limit effort=4 velocity=18.691589 -> effort=6 velocity=41
- joint b_pivot: limit effort=10 velocity=6.283185 -> effort=10 velocity=45
- joint fl_drive: limit effort=4 velocity=18.691589 -> effort=6 velocity=41
- joint fl_pivot: limit effort=10 velocity=6.283185 -> effort=10 velocity=45
- joint fr_drive: limit effort=4 velocity=18.691589 -> effort=6 velocity=41
- joint fr_pivot: limit effort=10 velocity=6.283185 -> effort=10 velocity=45
- joint lift: limit lower=0.0 upper=0.858 effort=1 velocity=1 -> lower=0.0 upper=0.858 effort=2845 velocity=0.3

File: urdf/rivet.urdf.xacro (robot description, xacro)
@@ -57,6 +57,6 @@
       lower="0.0"
       upper="0.858"
-      effort="1"
-      velocity="1" />
+      effort="2845"
+      velocity="0.3" />
   </joint>
   <link name="lift_link">
@@ -137,5 +137,5 @@
       <limit
         effort="10"
-        velocity="6.283185" />
+        velocity="45" />
     </joint>
     <link name="${prefix}_drive_link">
@@ -178,6 +178,6 @@
       <axis xyz="0 1 0"/>
       <limit
-        effort="4"
-        velocity="18.691589" />
+        effort="6"
+        velocity="41" />
     </joint>
   </xacro:macro> <!-- swerve_module -->
